Commit message: Update robotiq-cri

File: aist_description/devices/urdf/robotiq_hande_gripper_with_tip_link.urdf.xacro (robot description, xacro)
@@ -2,13 +2,12 @@
 <!-- This macro adds a convenient TF frame at the tip of the closed gripper. -->
 <!-- The position of the TF frame has not been measured at all and needs to be calibrated. -->
-<robot name="robotiq_hande_with_tip_link"
+<robot name="robotiq_hande_gripper_with_tip_link"
        xmlns:xacro="http://wiki.ros.org/xacro">
-  <xacro:macro name="robotiq_hande_with_tip_link"
+  <xacro:macro name="robotiq_hande_gripper_with_tip_link"
 	       params="prefix parent *origin">
-    <xacro:include filename="$(find robotiq_description)/urdf/robotiq_hande.urdf.xacro"/>
-    <xacro:robotiq_hande prefix="${prefix}" parent="${parent}"
-			 MAC="_000000000004">
+    <xacro:include filename="$(find robotiq_description)/urdf/robotiq_hande_gripper.urdf.xacro"/>
+    <xacro:robotiq_hande_gripper prefix="${prefix}" parent="${parent}">
       <xacro:insert_block name="origin"/>
-    </xacro:robotiq_hande>
+    </xacro:robotiq_hande_gripper>
     <!-- Add additional links for us to plan with. Oriented like the UR frame. -->
     <link name="${prefix}robotiq_hande_tip_link"/>

File: aist_description/scenes/urdf/fvision_base_scene.urdf.xacro (robot description, xacro)
@@ -44,8 +44,9 @@
   </joint>
   <!-- Spawn and attach gripper -->
-  <xacro:include filename="$(find aist_description)/devices/urdf/robotiq_hande_with_tip_link.urdf.xacro"/>
-  <xacro:robotiq_hande_with_tip_link prefix="d_bot_" parent="d_bot_ee_link">
+  <xacro:include filename="$(find aist_description)/devices/urdf/robotiq_hande_gripper_with_tip_link.urdf.xacro"/>
+  <xacro:robotiq_hande_gripper_with_tip_link prefix="d_bot_"
+					     parent="d_bot_ee_link">
     <origin xyz="0 0 0" rpy="0 0 0"/>
-  </xacro:robotiq_hande_with_tip_link>
+  </xacro:robotiq_hande_gripper_with_tip_link>
   <!-- Add PhoXi 3D scanner -->
   <xacro:include filename="$(find aist_phoxi_camera)/urdf/phoxi_m_camera.urdf.xacro"/>

File: aist_description/scenes/urdf/ur5e_base_scene.urdf.xacro (robot description, xacro)
@@ -78,8 +78,9 @@
   <!--   <origin xyz="0 0 0" rpy="0 0 0"/> -->
   <!-- </xacro:robotiq_85_gripper_with_tip_link> -->
-  <xacro:include filename="$(find aist_description)/devices/urdf/robotiq_hande_with_tip_link.urdf.xacro"/>
-  <xacro:robotiq_hande_with_tip_link prefix="d_bot_" parent="d_bot_ee_link">
+  <xacro:include filename="$(find aist_description)/devices/urdf/robotiq_hande_gripper_with_tip_link.urdf.xacro"/>
+  <xacro:robotiq_hande_gripper_with_tip_link prefix="d_bot_"
+					     parent="d_bot_ee_link">
     <origin xyz="0 0 0" rpy="0 0 0"/>
-  </xacro:robotiq_hande_with_tip_link>
+  </xacro:robotiq_hande_gripper_with_tip_link>
   <!-- Add PhoXi 3D scanner -->
   <xacro:include filename="$(find aist_phoxi_camera)/urdf/phoxi_m_camera.urdf.xacro"/>
