Commit message: Rename links and joints of robotiq grippers

File: aist_description/devices/urdf/robotiq_140_gripper_with_tip_link.urdf.xacro (robot description, xacro)
@@ -11,8 +11,8 @@
     </xacro:robotiq_140_gripper>
     <!-- Add additional links for us to plan with. Oriented like the UR frame. -->
-    <link name="${prefix}robotiq_140_tip_link"/>
-    <joint name="${prefix}robotiq_140_tip_link_joint" type="fixed">
-      <parent link="${prefix}robotiq_140_base_link"/>
-      <child link="${prefix}robotiq_140_tip_link"/>
+    <link name="${prefix}tip_link"/>
+    <joint name="${prefix}tip_link_joint" type="fixed">
+      <parent link="${prefix}base_link"/>
+      <child link="${prefix}tip_link"/>
       <origin rpy="0.0 0.0 0.0" xyz=".233 0.0 0.0"/>
     </joint>

File: aist_description/devices/urdf/robotiq_85_gripper_with_tip_link.urdf.xacro (robot description, xacro)
@@ -11,8 +11,8 @@
     </xacro:robotiq_85_gripper>
     <!-- Add additional links for us to plan with. Oriented like the UR frame. -->
-    <link name="${prefix}robotiq_85_tip_link"/>
-    <joint name="${prefix}robotiq_85_tip_link_joint" type="fixed">
-      <parent link="${prefix}robotiq_85_base_link"/>
-      <child link="${prefix}robotiq_85_tip_link"/>
+    <link name="${prefix}tip_link"/>
+    <joint name="${prefix}tip_link_joint" type="fixed">
+      <parent link="${prefix}base_link"/>
+      <child link="${prefix}tip_link"/>
       <origin rpy="0.0 0.0 0.0" xyz=".163 0.0 0.0"/>
     </joint>

File: aist_description/devices/urdf/robotiq_hande_gripper_with_tip_link.urdf.xacro (robot description, xacro)
@@ -11,8 +11,8 @@
     </xacro:robotiq_hande_gripper>
     <!-- Add additional links for us to plan with. Oriented like the UR frame. -->
-    <link name="${prefix}robotiq_hande_tip_link"/>
-    <joint name="${prefix}robotiq_hande_tip_link_joint" type="fixed">
-      <parent link="${prefix}robotiq_hande_base_link"/>
-      <child link="${prefix}robotiq_hande_tip_link"/>
+    <link name="${prefix}tip_link"/>
+    <joint name="${prefix}tip_link_joint" type="fixed">
+      <parent link="${prefix}base_link"/>
+      <child link="${prefix}tip_link"/>
       <origin rpy="0.0 0.0 0.0" xyz=".146 0.0 0.0"/>
     </joint>

File: aist_description/scenes/urdf/aist_base_scene.urdf.xacro (robot description, xacro)
@@ -71,11 +71,11 @@
   <xacro:include filename="$(find robotiq_description
 			   )/urdf/robotiq_arg2f_coupling.urdf.xacro"/>
-  <xacro:robotiq_arg2f_coupling prefix="a_bot_"
+  <xacro:robotiq_arg2f_coupling prefix="a_bot_gripper_coupling_"
 				parent="a_bot_ft300_flange_link">
     <origin xyz="0 0 0" rpy="0 0 0"/>
   </xacro:robotiq_arg2f_coupling>
   <xacro:include filename="$(find aist_description)/devices/urdf/robotiq_85_gripper_with_tip_link.urdf.xacro"/>
-  <xacro:robotiq_85_gripper_with_tip_link prefix="a_bot_"
-					  parent="a_bot_robotiq_arg2f_coupling_flange_link">
+  <xacro:robotiq_85_gripper_with_tip_link prefix="a_bot_gripper_"
+					  parent="a_bot_gripper_coupling_flange_link">
     <origin xyz="0 0 0" rpy="0 0 0"/>
   </xacro:robotiq_85_gripper_with_tip_link>
@@ -106,5 +106,5 @@
 			   )/devices/urdf/wrist_cameras.urdf.xacro" />
   <xacro:wrist_cameras prefix="a_bot_"
-		       parent="a_bot_robotiq_85_base_link"/>
+		       parent="a_bot_gripper_base_link"/>
   <!-- I would like to remove the "world" link definition, but apparently it is necessary for Gazebo -->
   <link name="world"/>

File: aist_description/scenes/urdf/fvision_base_scene.urdf.xacro (robot description, xacro)
@@ -46,11 +46,11 @@
   <xacro:include filename="$(find robotiq_description
 			   )/urdf/robotiq_arg2f_coupling.urdf.xacro"/>
-  <xacro:robotiq_arg2f_coupling prefix="d_bot_"
+  <xacro:robotiq_arg2f_coupling prefix="d_bot_gripper_coupling_"
 				parent="d_bot_ee_link">
     <origin xyz="0 0 0" rpy="0 0 0"/>
   </xacro:robotiq_arg2f_coupling>
   <xacro:include filename="$(find aist_description)/devices/urdf/robotiq_hande_gripper_with_tip_link.urdf.xacro"/>
-  <xacro:robotiq_hande_gripper_with_tip_link prefix="d_bot_"
-					     parent="d_bot_robotiq_arg2f_coupling_flange_link">
+  <xacro:robotiq_hande_gripper_with_tip_link prefix="d_bot_gripper_"
+					     parent="d_bot_gripper_coupling_flange_link">
     <origin xyz="0 0 0" rpy="0 0 0"/>
   </xacro:robotiq_hande_gripper_with_tip_link>

File: aist_description/scenes/urdf/mocap_base_scene.urdf.xacro (robot description, xacro)
@@ -43,5 +43,5 @@
   <xacro:include filename="$(find robotiq_description
 			   )/urdf/robotiq_arg2f_coupling.urdf.xacro"/>
-  <xacro:robotiq_arg2f_coupling prefix="c_bot_"
+  <xacro:robotiq_arg2f_coupling prefix="c_bot_gripper_coupling_"
 				parent="c_bot_ee_link">
     <origin xyz="0 0 0" rpy="0 0 0"/>
@@ -49,6 +49,6 @@
   <xacro:include filename="$(find aist_description
 			   )/devices/urdf/robotiq_85_gripper_with_tip_link.urdf.xacro"/>
-  <xacro:robotiq_85_gripper_with_tip_link prefix="c_bot_"
-					  parent="c_bot_robotiq_arg2f_coupling_flange_link">
+  <xacro:robotiq_85_gripper_with_tip_link prefix="c_bot_gripper_"
+					  parent="c_bot_gripper_coupling_flange_link">
     <origin xyz="0 0 0" rpy="0 0 0"/>
   </xacro:robotiq_85_gripper_with_tip_link>

File: aist_description/scenes/urdf/ur10e_base_scene.urdf.xacro (robot description, xacro)
@@ -45,11 +45,11 @@
   <xacro:include filename="$(find robotiq_description
 			   )/urdf/robotiq_arg2f_coupling.urdf.xacro"/>
-  <xacro:robotiq_arg2f_coupling prefix="a_bot_"
+  <xacro:robotiq_arg2f_coupling prefix="a_bot_gripper_coupling_"
 				parent="a_bot_ee_link">
     <origin xyz="0 0 0" rpy="0 0 0"/>
   </xacro:robotiq_arg2f_coupling>
   <xacro:include filename="$(find aist_description)/devices/urdf/robotiq_140_gripper_with_tip_link.urdf.xacro"/>
-  <xacro:robotiq_140_gripper_with_tip_link prefix="a_bot_"
-					   parent="a_bot_robotiq_arg2f_coupling_flange_link">
+  <xacro:robotiq_140_gripper_with_tip_link prefix="a_bot_gripper_"
+					   parent="a_bot_gripper_coupling_flange_link">
     <origin xyz="0 0 0" rpy="0 0 0"/>
   </xacro:robotiq_140_gripper_with_tip_link>

File: aist_description/scenes/urdf/ur5e_base_scene.urdf.xacro (robot description, xacro)
@@ -62,11 +62,11 @@
   <xacro:include filename="$(find robotiq_description
 			   )/urdf/robotiq_arg2f_coupling.urdf.xacro"/>
-  <xacro:robotiq_arg2f_coupling prefix="c_bot_"
+  <xacro:robotiq_arg2f_coupling prefix="c_bot_gripper_coupling_"
 				parent="c_bot_ee_link">
     <origin xyz="0 0 0" rpy="0 0 0"/>
   </xacro:robotiq_arg2f_coupling>
   <xacro:include filename="$(find aist_description)/devices/urdf/robotiq_85_gripper_with_tip_link.urdf.xacro"/>
-  <xacro:robotiq_85_gripper_with_tip_link prefix="c_bot_"
-					  parent="c_bot_robotiq_arg2f_coupling_flange_link">
+  <xacro:robotiq_85_gripper_with_tip_link prefix="c_bot_gripper_"
+					  parent="c_bot_gripper_coupling_flange_link">
     <origin xyz="0 0 0" rpy="0 0 0"/>
   </xacro:robotiq_85_gripper_with_tip_link>
@@ -84,11 +84,11 @@
   <!--   <origin xyz="0 0 0" rpy="0 0 0"/> -->
   <!-- </xacro:robotiq_85_gripper_with_tip_link> -->
-  <xacro:robotiq_arg2f_coupling prefix="d_bot_"
+  <xacro:robotiq_arg2f_coupling prefix="d_bot_gripper_coupling_"
 				parent="d_bot_ee_link">
     <origin xyz="0 0 0" rpy="0 0 0"/>
   </xacro:robotiq_arg2f_coupling>
   <xacro:include filename="$(find aist_description)/devices/urdf/robotiq_hande_gripper_with_tip_link.urdf.xacro"/>
-  <xacro:robotiq_hande_gripper_with_tip_link prefix="d_bot_"
-					     parent="d_bot_robotiq_arg2f_coupling_flange_link">
+  <xacro:robotiq_hande_gripper_with_tip_link prefix="d_bot_gripper_"
+					     parent="d_bot_gripper_coupling_flange_link">
     <origin xyz="0 0 0" rpy="0 0 0"/>
   </xacro:robotiq_hande_gripper_with_tip_link>

File: aist_description/scenes/urdf/ur_trial_a_base_scene.urdf.xacro (robot description, xacro)
@@ -51,11 +51,11 @@
   <xacro:include filename="$(find robotiq_description
 			   )/urdf/robotiq_arg2f_coupling.urdf.xacro"/>
-  <xacro:robotiq_arg2f_coupling prefix="a_bot_"
+  <xacro:robotiq_arg2f_coupling prefix="a_bot_gripper_coupling_"
 				parent="a_bot_ft300_flange_link">
     <origin xyz="0 0 0" rpy="0 0 0"/>
   </xacro:robotiq_arg2f_coupling>
   <xacro:include filename="$(find aist_description)/devices/urdf/robotiq_85_gripper_with_tip_link.urdf.xacro"/>
-  <xacro:robotiq_85_gripper_with_tip_link prefix="a_bot_"
-  					  parent="a_bot_robotiq_arg2f_coupling_flange_link">
+  <xacro:robotiq_85_gripper_with_tip_link prefix="a_bot_gripper_"
+  					  parent="a_bot_gripper_coupling_flange_link">
     <origin xyz="0 0 0" rpy="0 0 0"/>
   </xacro:robotiq_85_gripper_with_tip_link>
