Commit message: Rename links and joints of suction gripper and ft-sensor

File: aist_description/devices/urdf/dual_suction_gripper.urdf (robot description, URDF)
Before this commit: robot aaa, 1 links, 0 joints
Links:
- removed link base_link
- added link world

File: aist_description/devices/urdf/dual_suction_gripper.urdf.xacro (robot description, xacro)
@@ -5,5 +5,5 @@
 	       params="prefix parent *origin">
     <!-- A link representing the gripper and a joint attaching it to parnet -->
-    <link name="${prefix}dual_suction_gripper_base_link">
+    <link name="${prefix}base_link">
       <visual>
         <origin xyz="0.1855 -0.035 -0.035" rpy="0 0 ${pi/2}"/>
@@ -29,19 +29,19 @@
       </inertial>
     </link>
-    <joint name="${prefix}dual_suction_gripper_joint" type="fixed">
+    <joint name="${prefix}base_joint" type="fixed">
       <parent link="${parent}"/>
-      <child  link="${prefix}dual_suction_gripper_base_link"/>
+      <child  link="${prefix}base_link"/>
        <xacro:insert_block name="origin"/>
     </joint>
     <!-- A link representing the tip of the pad and a joint attaching
 	 it to the gripper -->
-    <link name="${prefix}dual_suction_gripper_pad_link"/>
-    <joint name="${prefix}dual_suction_gripper_pad_joint" type="fixed">
-      <parent link="${prefix}dual_suction_gripper_base_link"/>
-      <child  link="${prefix}dual_suction_gripper_pad_link"/>
+    <link name="${prefix}pad_link"/>
+    <joint name="${prefix}pad_joint" type="fixed">
+      <parent link="${prefix}base_link"/>
+      <child  link="${prefix}pad_link"/>
       <origin xyz="0.1855 0 0" rpy="0 0 0"/>
     </joint>
     <joint name="${prefix}robotiq_85_suction_tool_tip_joint" type="fixed">
-      <parent link="${prefix}dual_suction_gripper_pad_link"/>
+      <parent link="${prefix}pad_link"/>
       <child link="${prefix}suction_tool_tip_link"/>
       <origin rpy="0.0 0.0 0.0" xyz="0.0 0.0 0.0 "/>
@@ -50,8 +50,8 @@
     <!-- A link representing the tip of the coander gripper
 	 and a joint attaching it to the gripper -->
-    <link name="${prefix}dual_suction_gripper_coanda_link"/>
-    <joint name="${prefix}dual_suction_gripper_coanda_joint" type="fixed">
-      <parent link="${prefix}dual_suction_gripper_base_link"/>
-      <child  link="${prefix}dual_suction_gripper_coanda_link"/>
+    <link name="${prefix}coanda_link"/>
+    <joint name="${prefix}coanda_joint" type="fixed">
+      <parent link="${prefix}base_link"/>
+      <child  link="${prefix}coanda_link"/>
       <origin xyz="0.0505 0.145 0" rpy="0 0 ${pi/2}"/>
     </joint>

File: aist_description/devices/urdf/single_suction_gripper.urdf (robot description, URDF)
Before this commit: robot aaa, 1 links, 0 joints
Links:
- removed link base_link
- added link world

File: aist_description/devices/urdf/single_suction_gripper.urdf.xacro (robot description, xacro)
@@ -5,5 +5,5 @@
 	       params="prefix parent *origin">
     <!-- A link representing the gripper and a joint attaching it to parnet -->
-    <link name="${prefix}single_suction_gripper_base_link">
+    <link name="${prefix}base_link">
       <visual>
         <origin xyz="0.1855 -0.035 -0.035" rpy="0 0 ${pi/2}"/>
@@ -29,15 +29,15 @@
       </inertial>
     </link>
-    <joint name="${prefix}single_suction_gripper_joint" type="fixed">
+    <joint name="${prefix}base_joint" type="fixed">
       <parent link="${parent}"/>
-      <child  link="${prefix}single_suction_gripper_base_link"/>
+      <child  link="${prefix}base_link"/>
       <xacro:insert_block name="origin"/>
     </joint>
     <!-- A link representing the tip of the pad and a joint attaching
 	 it to the gripper -->
-    <link name="${prefix}single_suction_gripper_pad_link"/>
-    <joint name="${prefix}single_suction_gripper_pad_joint" type="fixed">
-      <parent link="${prefix}single_suction_gripper_base_link"/>
-      <child  link="${prefix}single_suction_gripper_pad_link"/>
+    <link name="${prefix}pad_link"/>
+    <joint name="${prefix}pad_joint" type="fixed">
+      <parent link="${prefix}base_link"/>
+      <child  link="${prefix}pad_link"/>
       <origin xyz="0.1855 0 0" rpy="0 0 0"/>
     </joint>

File: aist_description/scenes/urdf/aist_base_scene.urdf.xacro (robot description, xacro)
@@ -62,8 +62,8 @@
   <!-- Spawn and attach force sensor -->
   <xacro:include filename="$(find aist_ftsensor)/urdf/ft300.urdf.xacro"/>
-  <xacro:ft300 prefix="a_bot_" parent="a_bot_ee_link">
+  <xacro:ft300 prefix="a_bot_ftsensor_" parent="a_bot_ee_link">
     <origin xyz="0 0 0" rpy="0 0 0"/>
   </xacro:ft300>
-  <xacro:ft300 prefix="b_bot_" parent="b_bot_ee_link">
+  <xacro:ft300 prefix="b_bot_ftsensor_" parent="b_bot_ee_link">
     <origin xyz="0 0 0" rpy="0 0 0"/>
   </xacro:ft300>
@@ -72,5 +72,5 @@
 			   )/urdf/robotiq_arg2f_coupling.urdf.xacro"/>
   <xacro:robotiq_arg2f_coupling prefix="a_bot_gripper_coupling_"
-				parent="a_bot_ft300_flange_link">
+				parent="a_bot_ftsensor_flange_link">
     <origin xyz="0 0 0" rpy="0 0 0"/>
   </xacro:robotiq_arg2f_coupling>
@@ -81,6 +81,6 @@
   </xacro:robotiq_85_gripper_with_tip_link>
   <xacro:include filename="$(find aist_description)/devices/urdf/single_suction_gripper.urdf.xacro"/>
-  <xacro:single_suction_gripper prefix="b_bot_"
-  				parent="b_bot_ft300_flange_link">
+  <xacro:single_suction_gripper prefix="b_bot_gripper_"
+  				parent="b_bot_ftsensor_flange_link">
     <!-- <origin xyz="0 0 0" rpy="0 ${0.2*pi/180} ${-1.2*pi/180}"/> -->
     <origin xyz="0 0 0" rpy="0 ${-0.1*pi/180} ${0.45*pi/180}"/>

File: aist_description/scenes/urdf/diiwa_base_scene.urdf.xacro (robot description, xacro)
@@ -42,5 +42,5 @@
   <xacro:include filename="$(find robotiq_description
 			   )/urdf/robotiq_arg2f_coupling.urdf.xacro"/>
-  <xacro:robotiq_arg2f_coupling prefix="a_iiwa_"
+  <xacro:robotiq_arg2f_coupling prefix="a_iiwa_gripper_coupling_"
 				parent="a_iiwa_ee_link">
     <origin xyz="0 0 0" rpy="0 0 0"/>
@@ -48,11 +48,12 @@
   <xacro:include filename="$(find aist_description
   			   )/devices/urdf/robotiq_85_gripper_with_tip_link.urdf.xacro"/>
-  <xacro:robotiq_85_gripper_with_tip_link prefix="a_iiwa_"
-  					  parent="a_iiwa_robotiq_arg2f_coupling_flange_link">
+  <xacro:robotiq_85_gripper_with_tip_link prefix="a_iiwa_gripper_"
+  					  parent="a_iiwa_gripper_coupling_flange_link">
     <origin xyz="0 0 0" rpy="0 0 0"/>
   </xacro:robotiq_85_gripper_with_tip_link>
   <xacro:include filename="$(find aist_description
 			   )/devices/urdf/single_suction_gripper.urdf.xacro"/>
-  <xacro:single_suction_gripper prefix="b_iiwa_" parent="b_iiwa_ee_link">
+  <xacro:single_suction_gripper prefix="b_iiwa_gripper_"
+				parent="b_iiwa_ee_link">
     <origin xyz="0 0 0" rpy="0 0 0"/>
   </xacro:single_suction_gripper>

File: aist_ftsensor/urdf/ft300.urdf (robot description, URDF)
Before this commit: robot aaa, 1 links, 0 joints
Links:
- removed link base_link
- added link world

File: aist_ftsensor/urdf/ft300.urdf.xacro (robot description, xacro)
@@ -4,5 +4,5 @@
   <xacro:property name="ft300_length" value="0.0360"/>
   <xacro:macro name="ft300" params="prefix parent *origin">
-    <link name="${prefix}ft300_link">
+    <link name="${prefix}base_link">
       <visual>
         <origin xyz="${ft300_length} 0 0" rpy="${pi} ${pi/2} 0"/>
@@ -33,17 +33,17 @@
     <joint name="${prefix}ft300_joint" type="fixed">
       <parent link="${parent}"/>
-      <child  link="${prefix}ft300_link"/>
+      <child  link="${prefix}base_link"/>
       <xacro:insert_block name="origin"/>
     </joint>
-    <link name="${prefix}ft300_flange_link"/>
-    <joint name="${prefix}ft300_flange_joint" type="fixed">
-      <parent link="${prefix}ft300_link"/>
-      <child  link="${prefix}ft300_flange_link"/>
+    <link name="${prefix}flange_link"/>
+    <joint name="${prefix}flange_joint" type="fixed">
+      <parent link="${prefix}base_link"/>
+      <child  link="${prefix}flange_link"/>
       <origin xyz="${ft300_length} 0 0" rpy="0 0 0"/>
     </joint>
-    <link name="${prefix}ft300_wrench_link"/>
-    <joint name="${prefix}ft300_wrench_joint" type="fixed">
-      <parent link="${prefix}ft300_flange_link"/>
-      <child  link="${prefix}ft300_wrench_link"/>
+    <link name="${prefix}wrench_link"/>
+    <joint name="${prefix}wrench_joint" type="fixed">
+      <parent link="${prefix}flange_link"/>
+      <child  link="${prefix}wrench_link"/>
       <origin xyz="0 0 0" rpy="${-pi/2} 0 ${-pi/2}"/>
     </joint>
