Commit message: Make gazebo's topic names identical with real

File: aist_description/devices/urdf/_d435.urdf.xacro (robot description, xacro)
@@ -44,5 +44,5 @@
           <depthImageTopicName>aligned_depth_to_color/image_raw</depthImageTopicName>
           <depthImageCameraInfoTopicName>depth/camera_info</depthImageCameraInfoTopicName>
-          <pointCloudTopicName>depth/points</pointCloudTopicName>
+          <pointCloudTopicName>depth/color/points</pointCloudTopicName>
           <pointCloudCutoff>0.1</pointCloudCutoff>
           <!-- <hackBaseline>0.07</hackBaseline> -->

File: aist_description/devices/urdf/_r410.urdf.xacro (robot description, xacro)
@@ -44,5 +44,5 @@
           <depthImageTopicName>aligned_depth_to_color/image_raw</depthImageTopicName>
           <depthImageCameraInfoTopicName>depth/camera_info</depthImageCameraInfoTopicName>
-          <pointCloudTopicName>depth/points</pointCloudTopicName>
+          <pointCloudTopicName>depth/color/points</pointCloudTopicName>
           <pointCloudCutoff>0.1</pointCloudCutoff>
           <!-- <hackBaseline>0.07</hackBaseline> -->

File: aist_description/devices/urdf/_r430.urdf.xacro (robot description, xacro)
@@ -44,5 +44,5 @@
           <depthImageTopicName>aligned_depth_to_color/image_raw</depthImageTopicName>
           <depthImageCameraInfoTopicName>depth/camera_info</depthImageCameraInfoTopicName>
-          <pointCloudTopicName>depth/points</pointCloudTopicName>
+          <pointCloudTopicName>depth/color/points</pointCloudTopicName>
           <pointCloudCutoff>0.1</pointCloudCutoff>
           <!-- <hackBaseline>0.07</hackBaseline> -->

File: aist_description/devices/urdf/_sr305.urdf.xacro (robot description, xacro)
@@ -5,5 +5,5 @@
 -->
 <robot name="sensor_sr305" xmlns:xacro="http://ros.org/wiki/xacro">
-  <xacro:macro name="sensor_sr305" params="prefix parent use_bottom_mount:=false *origin">
+  <xacro:macro name="sensor_sr305" params="parent *origin name:=camera use_bottom_mount:=false">
     <!-- TODO: Allow placing the camera using bottom mount or back mount -->
     <xacro:property name="M_PI" value="3.1415926535897931" />
@@ -31,31 +31,31 @@
     <!-- camera body, with origin at bottom screw mount -->
     <xacro:if value="${use_bottom_mount}">
-      <joint name="${prefix}camera_joint" type="fixed">
+      <joint name="${name}_joint" type="fixed">
         <xacro:insert_block name="origin" />
         <parent link="${parent}"/>
-        <child link="${prefix}camera_bottom_screw_frame" />
+        <child link="${name}_bottom_screw_frame" />
       </joint>
-      <link name="${prefix}camera_bottom_screw_frame"/>
-      <joint name="${prefix}camera_link_joint" type="fixed">
+      <link name="${name}_bottom_screw_frame"/>
+      <joint name="${name}_link_joint" type="fixed">
         <origin xyz="${sr305_cam_depth_px} ${sr305_cam_depth_py} ${sr305_cam_depth_pz}" rpy="0 0 0"/>
-        <parent link="${prefix}camera_bottom_screw_frame"/>
-        <child link="${prefix}camera_link" />
+        <parent link="${name}_bottom_screw_frame"/>
+        <child link="${name}_link" />
       </joint>
     </xacro:if>
     <xacro:if value="${not use_bottom_mount}">
       <!-- I forgot which conventions exist for "camera_joint" and "camera_link_joint" so I hesitate to delete one. -->
-      <joint name="${prefix}camera_joint" type="fixed">
+      <joint name="${name}_joint" type="fixed">
         <xacro:insert_block name="origin" />
         <parent link="${parent}"/>
-        <child link="${prefix}camera_connector_link" />
+        <child link="${name}_connector_link" />
       </joint>
-      <link name="${prefix}camera_connector_link"/>
-      <joint name="${prefix}camera_link_joint" type="fixed">
+      <link name="${name}_connector_link"/>
+      <joint name="${name}_link_joint" type="fixed">
         <origin xyz="0 0 0" rpy="0 0 0"/>
-        <parent link="${prefix}camera_connector_link"/>
-        <child link="${prefix}camera_link" />
+        <parent link="${name}_connector_link"/>
+        <child link="${name}_link" />
       </joint>
     </xacro:if>
-    <link name="${prefix}camera_link">
+    <link name="${name}_link">
       <visual>
       <origin xyz="${0} ${-sr305_cam_depth_py} 0" rpy="${M_PI/2} 0 ${M_PI/2}"/>
@@ -86,57 +86,57 @@
     </link>
     <!-- camera depth joints and links -->
-    <joint name="${prefix}camera_depth_joint" type="fixed">
+    <joint name="${name}_depth_joint" type="fixed">
       <origin xyz=".003721 0 0" rpy="0 0 0"/>
-      <parent link="${prefix}camera_link"/>
-      <child link="${prefix}camera_depth_frame" />
+      <parent link="${name}_link"/>
+      <child link="${name}_depth_frame" />
     </joint>
-    <link name="${prefix}camera_depth_frame"/>
-    <joint name="${prefix}camera_depth_optical_joint" type="fixed">
+    <link name="${name}_depth_frame"/>
+    <joint name="${name}_depth_optical_joint" type="fixed">
       <origin xyz="0 0 0" rpy="${-M_PI/2} 0 ${-M_PI/2}" />
-      <parent link="${prefix}camera_depth_frame" />
-      <child link="${prefix}camera_depth_optical_frame" />
+      <parent link="${name}_depth_frame" />
+      <child link="${name}_depth_optical_frame" />
     </joint>
-    <link name="${prefix}camera_depth_optical_frame"/>
+    <link name="${name}_depth_optical_frame"/>
     <!-- camera left IR joints and links -->
-    <joint name="${prefix}camera_left_ir_joint" type="fixed">
+    <joint name="${name}_left_ir_joint" type="fixed">
       <origin xyz="0 ${sr305_cam_depth_to_left_ir_offset} 0" rpy="0 0 0" />
-      <parent link="${prefix}camera_depth_frame" />
-      <child link="${prefix}camera_left_ir_frame" />
+      <parent link="${name}_depth_frame" />
+      <child link="${name}_left_ir_frame" />
     </joint>
-    <link name="${prefix}camera_left_ir_frame"/>
-    <joint name="${prefix}camera_left_ir_optical_joint" type="fixed">
+    <link name="${name}_left_ir_frame"/>
+    <joint name="${name}_left_ir_optical_joint" type="fixed">
       <origin xyz="0 0 0" rpy="${-M_PI/2} 0 ${-M_PI/2}" />
-      <parent link="${prefix}camera_left_ir_frame" />
-      <child link="${prefix}camera_left_ir_optical_frame" />
+      <parent link="${name}_left_ir_frame" />
+      <child link="${name}_left_ir_optical_frame" />
     </joint>
-    <link name="${prefix}camera_left_ir_optical_frame"/>
+    <link name="${name}_left_ir_optical_frame"/>
     <!-- camera right IR joints and links -->
-    <joint name="${prefix}camera_right_ir_joint" type="fixed">
+    <joint name="${name}_right_ir_joint" type="fixed">
       <origin xyz="0 ${sr305_cam_depth_to_right_ir_offset} 0" rpy="0 0 0" />
-      <parent link="${prefix}camera_depth_frame" />
-      <child link="${prefix}camera_right_ir_frame" />
+      <parent link="${name}_depth_frame" />
+      <child link="${name}_right_ir_frame" />
     </joint>
-    <link name="${prefix}camera_right_ir_frame"/>
-    <joint name="${prefix}camera_right_ir_optical_joint" type="fixed">
+    <link name="${name}_right_ir_frame"/>
+    <joint name="${name}_right_ir_optical_joint" type="fixed">
       <origin xyz="0 0 0" rpy="${-M_PI/2} 0 ${-M_PI/2}" />
-      <parent link="${prefix}camera_right_ir_frame" />
-      <child link="${prefix}camera_right_ir_optical_frame" />
+      <parent link="${name}_right_ir_frame" />
+      <child link="${name}_right_ir_optical_frame" />
     </joint>
-    <link name="${prefix}camera_right_ir_optical_frame"/>
+    <link name="${name}_right_ir_optical_frame"/>
     <!-- camera color joints and links -->
-    <joint name="${prefix}camera_color_joint" type="fixed">
+    <joint name="${name}_color_joint" type="fixed">
       <origin xyz="0 ${sr305_cam_depth_to_color_offset} 0" rpy="0 0 0" />
-      <parent link="${prefix}camera_depth_frame" />
-      <child link="${prefix}camera_color_frame" />
+      <parent link="${name}_depth_frame" />
+      <child link="${name}_color_frame" />
     </joint>
-    <link name="${prefix}camera_color_frame"/>
-    <joint name="${prefix}camera_color_optical_joint" type="fixed">
+    <link name="${name}_color_frame"/>
+    <joint name="${name}_color_optical_joint" type="fixed">
       <origin xyz="0 0 0" rpy="${-M_PI/2} 0 ${-M_PI/2}" />
-      <parent link="${prefix}camera_color_frame" />
-      <child link="${prefix}camera_color_optical_frame" />
+      <parent link="${name}_color_frame" />
+      <child link="${name}_color_optical_frame" />
     </joint>
-    <link name="${prefix}camera_color_optical_frame"/>
-    <gazebo reference="${prefix}camera_depth_frame">
-      <sensor type="depth" name="${prefix}camera">
+    <link name="${name}_color_optical_frame"/>
+    <gazebo reference="${name}_depth_frame">
+      <sensor type="depth" name="${name}">
 	<always_on>true</always_on>
 	<visualize>true</visualize>
@@ -155,16 +155,16 @@
           </clip>
 	</camera>
-	<plugin name="${prefix}cam_controller"
+	<plugin name="${name}_controller"
 		filename="libgazebo_ros_openni_kinect.so">
           <baseline>0.2</baseline>
           <alwaysOn>true</alwaysOn>
           <updateRate>10.0</updateRate>
-          <cameraName>${prefix}camera</cameraName>
-          <frameName>${prefix}camera_color_optical_frame</frameName>
+          <cameraName>${name}</cameraName>
+          <frameName>${name}_color_optical_frame</frameName>
           <imageTopicName>color/image_raw</imageTopicName>
           <cameraInfoTopicName>color/camera_info</cameraInfoTopicName>
           <depthImageTopicName>aligned_depth_to_color/image_raw</depthImageTopicName>
           <depthImageCameraInfoTopicName>aligned_depth_to_color/camera_info</depthImageCameraInfoTopicName>
-          <pointCloudTopicName>depth/points</pointCloudTopicName>
+          <pointCloudTopicName>depth/color/points</pointCloudTopicName>
           <pointCloudCutoff>0.1</pointCloudCutoff>
           <!-- <hackBaseline>0.07</hackBaseline> -->

File: aist_description/devices/urdf/wrist_cameras.urdf.xacro (robot description, xacro)
@@ -36,8 +36,8 @@
       <origin xyz="0.035 0.0 0.025" rpy="0 0 0"/>
     </joint>
-    <xacro:sensor_sr305 prefix="${prefix}inside_" parent="${parent}">
+    <xacro:sensor_sr305 name="${prefix}inside_camera" parent="${parent}">
       <origin xyz="0.026 0 0.0595" rpy="0 ${20.0*pi/180.0} 0" />
     </xacro:sensor_sr305>
-    <xacro:sensor_sr305 prefix="${prefix}outside_" parent="${parent}">
+    <xacro:sensor_sr305 name="${prefix}outside_camera" parent="${parent}">
       <origin xyz="0.026 0 ${0.0595+.024}" rpy="0 ${-15.0*pi/180.0} 0" />
     </xacro:sensor_sr305>
