Commit message: Confirmed that loading camera calibration into URDF successful

File: aist_description/devices/urdf/wrist_cameras.urdf.xacro (robot description, xacro)
@@ -2,5 +2,5 @@
 <!-- This macro adds a convenient TF frame at the tip of the closed gripper. -->
 <!-- The position of the TF frame has not been measured at all and needs to be calibrated. -->
-<robot name="robotiq_85_gripper_o2ac" xmlns:xacro="http://www.ros.org/wiki/xacro">
+<robot name="wrist_cameras" xmlns:xacro="http://www.ros.org/wiki/xacro">
   <xacro:macro name="wrist_cameras" params="prefix parent">
     <xacro:include filename="$(find aist_description
@@ -36,9 +36,27 @@
       <origin xyz="0.035 0.0 0.025" rpy="0 0 0"/>
     </joint>
+    <xacro:include filename="$(find aist_description
+			     )/scenes/urdf/load_calibration.urdf.xacro"/>
+    <xacro:load_calibration directory="$(find aist_handeye_calibration)/calib"
+			    name="${prefix}inside_camera"
+			    property_name="inside_camera_origin"/>
     <xacro:sensor_sr305 name="${prefix}inside_camera" parent="${parent}">
-      <origin xyz="0.026 0 0.0595" rpy="0 ${20.0*pi/180.0} 0" />
+      <origin xyz="${inside_camera_origin[0]}
+		   ${inside_camera_origin[1]}
+		   ${inside_camera_origin[2]}"
+    	      rpy="${inside_camera_origin[3]}
+		   ${inside_camera_origin[4]}
+		   ${inside_camera_origin[5]}"/>
     </xacro:sensor_sr305>
+    <xacro:load_calibration directory="$(find aist_handeye_calibration)/calib"
+			    name="${prefix}outside_camera"
+			    property_name="outside_camera_origin"/>
     <xacro:sensor_sr305 name="${prefix}outside_camera" parent="${parent}">
-      <origin xyz="0.026 0 ${0.0595+.024}" rpy="0 ${-15.0*pi/180.0} 0" />
+      <origin xyz="${outside_camera_origin[0]}
+		   ${outside_camera_origin[1]}
+		   ${outside_camera_origin[2]}"
+    	      rpy="${outside_camera_origin[3]}
+		   ${outside_camera_origin[4]}
+		   ${outside_camera_origin[5]}"/>
     </xacro:sensor_sr305>
   </xacro:macro>

File: aist_description/scenes/urdf/aist_base_scene.urdf.xacro (robot description, xacro)
@@ -2,5 +2,4 @@
 <robot xmlns:xacro="http://wiki.ros.org/xacro" name="aist_base_scene" >
   <xacro:arg name="scene" default=""/>
-  <!-- Calibration help: If the robot is not moving far enough to the calibration point, increase these distances -->
   <xacro:property name="a_bot_x" value="0"/>
   <xacro:property name="a_bot_y" value="-0.4875"/>
@@ -10,12 +9,11 @@
   <xacro:property name="b_bot_theta" value="${pi}"/>
   <xacro:property name="bots_z" value="0.77"/>
-  <!-- This is the main file defining our robot arrangement and physical environment. -->
-  <!-- Main workspace -->
-  <!-- The surface is 0.01 m below the robot bases and the "workspace_center" frame. -->
+  <!-- ground and workspace -->
   <link name="ground"/>
-  <xacro:include filename="$(find aist_description)/objects/urdf/aist_box.urdf.xacro"/>
   <xacro:property name="table_w" value="0.9"/>
   <xacro:property name="table_l" value="1.8"/>
   <xacro:property name="table_h" value="0.01"/>
+  <xacro:include filename="$(find aist_description
+			   )/objects/urdf/aist_box.urdf.xacro"/>
   <xacro:aist_box name="workbox"
 		  width="${table_w}" length="${table_l}" height="${table_h}"
@@ -30,5 +28,4 @@
   </joint>
   <!-- robot arms -->
-  <!-- <xacro:include filename="$(find ur_description)/urdf/common.gazebo.xacro"/> -->
   <xacro:include filename="$(find ur_gazebo)/urdf/ur_macro.xacro"/>
   <xacro:ur_robot_gazebo
@@ -43,5 +40,4 @@
 				  )/config/a_bot_calibration.yaml"
       transmission_hw_interface="hardware_interface/PositionJointInterface"/>
-  <!-- <xacro:gazebo_ros_control ns="/b_bot"/> -->
   <xacro:ur_robot_gazebo
       prefix="b_bot_"
@@ -91,5 +87,5 @@
   				parent="b_bot_ftsensor_flange_link">
     <!-- <origin xyz="0 0 0" rpy="0 ${0.2*pi/180} ${-1.2*pi/180}"/> -->
-    <origin xyz="0 0 0" rpy="0 ${-0.1*pi/180} ${0.15*pi/180}"/>
+    <origin xyz="0 0 0" rpy="0 ${0.7*pi/180} ${-0.1*pi/180}"/>
   </xacro:single_suction_gripper>
   <!-- Add virtual wall to avoid collisions-->
@@ -99,19 +95,19 @@
   </xacro:aist_box>
   <!-- Add PhoXi 3D scanner -->
+  <xacro:include filename="$(find aist_description
+			   )/scenes/urdf/load_calibration.urdf.xacro"/>
+  <xacro:load_calibration directory="$(find aist_handeye_calibration)/calib"
+			  name="a_phoxi_m_camera"/>
   <xacro:include filename="$(find aist_phoxi_camera
 			   )/urdf/phoxi_m_camera.urdf.xacro"/>
   <xacro:phoxi_m_camera name="a_phoxi_m_camera" parent="workspace_center">
-    <origin xyz="0.483543436025
-		 -0.0149511700982
-		 0.633792706454"
-	    rpy="${-152.286950706*pi/180}
-		 ${-2.00315281361*pi/180}
-		 ${86.7522427304*pi/180}"/>
+    <origin xyz="${origin[0]} ${origin[1]} ${origin[2]}"
+    	    rpy="${origin[3]} ${origin[4]} ${origin[5]}"/>
   </xacro:phoxi_m_camera>
   <!-- Add RealSense camera -->
   <xacro:include filename="$(find aist_description
-			   )/devices/urdf/wrist_cameras.urdf.xacro" />
+  			   )/devices/urdf/wrist_cameras.urdf.xacro" />
   <xacro:wrist_cameras prefix="a_bot_"
-		       parent="a_bot_gripper_base_link"/>
+  		       parent="a_bot_gripper_base_link"/>
   <!-- I would like to remove the "world" link definition, but apparently it is necessary for Gazebo -->
   <link name="world"/>

File: aist_description/scenes/urdf/load_calibration.urdf.xacro (robot description, xacro)
@@ -1,7 +1,8 @@
 <robot xmlns:xacro="http://wiki.ros.org/xacro" name="load_calibration">
-  <xacro:macro name="load_calibration" params="directory name">
+  <xacro:macro name="load_calibration"
+	       params="directory name property_name:=origin">
     <xacro:property name="calibration_parameters"
 		    value="${xacro.load_yaml(directory + '/' + name + '.yaml')}"/>
-    <xacro:property name="${name + '_origin'}"
+    <xacro:property name="${property_name}"
 		    value="${calibration_parameters['origin']}"
 		    scope="parent"/>

File: aist_description/scenes/urdf/mocap_base_scene.urdf.xacro (robot description, xacro)
@@ -63,10 +63,6 @@
   <xacro:sensor_d435 name="realsenseD435" parent="workspace_center"
 		     use_nominal_extrinsics="true">
-    <origin xyz="${realsenseD435_origin[0]}
-		 ${realsenseD435_origin[1]}
-		 ${realsenseD435_origin[2]}"
-    	    rpy="${realsenseD435_origin[3]}
-		 ${realsenseD435_origin[4]}
-		 ${realsenseD435_origin[5]}"/>
+    <origin xyz="${origin[0]} ${origin[1]} ${origin[2]}"
+    	    rpy="${origin[3]} ${origin[4]} ${origin[5]}"/>
   </xacro:sensor_d435>
   <!-- I would like to remove the "world" link definition, but apparently it is necessary for Gazebo -->

Commit message: Simplify API of xacro for importing calibration

File: aist_description/devices/urdf/wrist_cameras.urdf.xacro (robot description, xacro)
@@ -38,7 +38,7 @@
     <xacro:include filename="$(find aist_description
 			     )/scenes/urdf/load_calibration.urdf.xacro"/>
-    <xacro:load_calibration directory="$(find aist_handeye_calibration)/calib"
-			    name="${prefix}inside_camera"
-			    property_name="inside_camera_origin"/>
+    <xacro:load_calibration filename="$(find aist_handeye_calibration
+				      )/calib/${prefix}inside_camera.yaml"
+			    propname="inside_camera_origin"/>
     <xacro:sensor_sr305 name="${prefix}inside_camera" parent="${parent}">
       <origin xyz="${inside_camera_origin[0]}
@@ -49,7 +49,7 @@
 		   ${inside_camera_origin[5]}"/>
     </xacro:sensor_sr305>
-    <xacro:load_calibration directory="$(find aist_handeye_calibration)/calib"
-			    name="${prefix}outside_camera"
-			    property_name="outside_camera_origin"/>
+    <xacro:load_calibration filename="$(find aist_handeye_calibration
+				      )/calib/${prefix}outside_camera.yaml"
+			    propname="outside_camera_origin"/>
     <xacro:sensor_sr305 name="${prefix}outside_camera" parent="${parent}">
       <origin xyz="${outside_camera_origin[0]}

File: aist_description/scenes/urdf/aist_base_scene.urdf.xacro (robot description, xacro)
@@ -97,6 +97,6 @@
   <xacro:include filename="$(find aist_description
 			   )/scenes/urdf/load_calibration.urdf.xacro"/>
-  <xacro:load_calibration directory="$(find aist_handeye_calibration)/calib"
-			  name="a_phoxi_m_camera"/>
+  <xacro:load_calibration filename="$(find aist_handeye_calibration
+				    )/calib/a_phoxi_m_camera.yaml"/>
   <xacro:include filename="$(find aist_phoxi_camera
 			   )/urdf/phoxi_m_camera.urdf.xacro"/>

File: aist_description/scenes/urdf/load_calibration.urdf.xacro (robot description, xacro)
@@ -1,8 +1,9 @@
+<?xml version="1.0"?>
 <robot xmlns:xacro="http://wiki.ros.org/xacro" name="load_calibration">
   <xacro:macro name="load_calibration"
-	       params="directory name property_name:=origin">
+	       params="filename propname:=origin">
     <xacro:property name="calibration_parameters"
-		    value="${xacro.load_yaml(directory + '/' + name + '.yaml')}"/>
-    <xacro:property name="${property_name}"
+		    value="${xacro.load_yaml(filename)}"/>
+    <xacro:property name="${propname}"
 		    value="${calibration_parameters['origin']}"
 		    scope="parent"/>

File: aist_description/scenes/urdf/mocap_base_scene.urdf.xacro (robot description, xacro)
@@ -57,6 +57,6 @@
   <xacro:include filename="$(find aist_description
 			   )/scenes/urdf/load_calibration.urdf.xacro"/>
-  <xacro:load_calibration directory="$(find aist_handeye_calibration)/calib"
-			  name="realsenseD435"/>
+  <xacro:load_calibration filename="$(find aist_handeye_calibration
+				    )/calib/realsenseD435.yaml"/>
   <xacro:include filename="$(find aist_description
 			   )/devices/urdf/_d435.urdf.xacro"/>
