Commit message: Cleanup handeye calibration

File: aist_description/devices/urdf/_d405.urdf.xacro (robot description, xacro)
@@ -7,135 +7,15 @@
 -->
 <robot name="sensor_d405" xmlns:xacro="http://ros.org/wiki/xacro">
-  <!-- Includes -->
-  <xacro:include filename="$(find realsense2_description)/urdf/_materials.urdf.xacro" />
-  <xacro:include filename="$(find realsense2_description)/urdf/_usb_plug.urdf.xacro" />
-  <xacro:macro name="sensor_d405" params="parent *origin name:=camera use_nominal_extrinsics:=false add_plug:=false use_mesh:=true">
-    <xacro:property name="M_PI" value="3.1415926535897931" />
-    <!-- The following values are approximate, and the camera node
-     publishing TF values with actual calibrated camera extrinsic values -->
-    <xacro:property name="d405_cam_depth_to_infra1_offset" value="0.0"/>
-    <xacro:property name="d405_cam_depth_to_infra2_offset" value="-0.018"/>
-    <xacro:property name="d405_cam_depth_to_color_offset" value="0.000"/>
-    <!-- The following values model the aluminum peripherial case for the
-  	D405 camera, with the camera joint represented by the actual
-  	peripherial camera tripod mount -->
-    <xacro:property name="d405_cam_width" value="0.042"/>
-    <xacro:property name="d405_cam_height" value="0.042"/>
-    <xacro:property name="d405_cam_depth" value="0.023"/>
-    <xacro:property name="d405_cam_mount_from_center_offset" value="0.0149"/>
-    <!-- glass cover is 0.1 mm inwards from front aluminium plate -->
-    <xacro:property name="d405_glass_to_front" value="0.1e-3"/>
-    <!-- see datasheet Revision 007, Fig. 4-4 page 65 -->
-    <xacro:property name="d405_zero_depth_to_glass" value="3.7e-3"/>
-    <!-- convenience precomputation to avoid clutter-->
-    <xacro:property name="d405_mesh_x_offset" value="${d405_cam_mount_from_center_offset-d405_glass_to_front-d405_zero_depth_to_glass}"/>
-    <!-- The following offset is relative the the physical D405 camera peripherial
-  	camera tripod mount -->
-    <xacro:property name="d405_cam_depth_px" value="${d405_cam_mount_from_center_offset}"/>
-    <xacro:property name="d405_cam_depth_py" value="0.009"/>
-    <xacro:property name="d405_cam_depth_pz" value="${d405_cam_height/2}"/>
-    <!-- camera body, with origin at bottom screw mount -->
-    <joint name="${name}_joint" type="fixed">
-      <xacro:insert_block name="origin" />
-      <parent link="${parent}"/>
-      <child link="${name}_bottom_screw_frame" />
-    </joint>
-    <link name="${name}_bottom_screw_frame"/>
-    <joint name="${name}_link_joint" type="fixed">
-      <origin xyz="${d405_mesh_x_offset} ${d405_cam_depth_py} ${d405_cam_depth_pz}" rpy="0 0 0"/>
-      <parent link="${name}_bottom_screw_frame"/>
-      <child link="${name}_link" />
-    </joint>
-    <link name="${name}_link">
-      <visual>
-        <xacro:if value="${use_mesh}">
-          <!-- the mesh origin is at front plate in between the two infrared camera axes -->
-          <origin xyz="${d405_zero_depth_to_glass + d405_glass_to_front} ${-d405_cam_depth_py} 0" rpy="${M_PI/2} 0 ${M_PI/2}"/>
-          <geometry>
-            <mesh filename="package://aist_description/devices/meshes/D405.stl"
-	    	  scale=".001 .001 .001"/>
-          </geometry>
-        </xacro:if>
-        <xacro:unless value="${use_mesh}">
-          <origin xyz="0 ${-d405_cam_depth_py} 0" rpy="0 0 0"/>
-          <geometry>
-            <box size="${d405_cam_depth} ${d405_cam_width} ${d405_cam_height}"/>
-          </geometry>
-          <material name="aluminum"/>
-        </xacro:unless>
-      </visual>
-      <collision>
-        <origin xyz="0 ${-d405_cam_depth_py} 0" rpy="0 0 0"/>
-        <geometry>
-          <box size="${d405_cam_depth} ${d405_cam_width} ${d405_cam_height}"/>
-        </geometry>
-      </collision>
-      <inertial>
-        <!-- The following are not reliable values, and should not be used for modeling -->
-        <mass value="0.072" />
-        <origin xyz="0 0 0" />
-        <inertia ixx="0.003881243" ixy="0.0" ixz="0.0" iyy="0.000498940" iyz="0.0" izz="0.003879257" />
-      </inertial>
-    </link>
-    <!-- Use the nominal extrinsics between camera frames if the calibrated extrinsics aren't being published. e.g. running the device in simulation  -->
-    <xacro:if value="${use_nominal_extrinsics}">
-      <!-- camera depth joints and links -->
-      <joint name="${name}_depth_joint" type="fixed">
-        <origin xyz="0 0 0" rpy="0 0 0"/>
-        <parent link="${name}_link"/>
-        <child link="${name}_depth_frame" />
-      </joint>
-      <link name="${name}_depth_frame"/>
-      <joint name="${name}_depth_optical_joint" type="fixed">
-        <origin xyz="0 0 0" rpy="${-M_PI/2} 0 ${-M_PI/2}" />
-        <parent link="${name}_depth_frame" />
-        <child link="${name}_depth_optical_frame" />
-      </joint>
-      <link name="${name}_depth_optical_frame"/>
-      <!-- camera left IR joints and links -->
-      <joint name="${name}_infra1_joint" type="fixed">
-        <origin xyz="0 ${d405_cam_depth_to_infra1_offset} 0" rpy="0 0 0" />
-        <parent link="${name}_link" />
-        <child link="${name}_infra1_frame" />
-      </joint>
-      <link name="${name}_infra1_frame"/>
-      <joint name="${name}_infra1_optical_joint" type="fixed">
-        <origin xyz="0 0 0" rpy="${-M_PI/2} 0 ${-M_PI/2}" />
-        <parent link="${name}_infra1_frame" />
-        <child link="${name}_infra1_optical_frame" />
-      </joint>
-      <link name="${name}_infra1_optical_frame"/>
-      <!-- camera right IR joints and links -->
-      <joint name="${name}_infra2_joint" type="fixed">
-        <origin xyz="0 ${d405_cam_depth_to_infra2_offset} 0" rpy="0 0 0" />
-        <parent link="${name}_link" />
-        <child link="${name}_infra2_frame" />
-      </joint>
-      <link name="${name}_infra2_frame"/>
-      <joint name="${name}_infra2_optical_joint" type="fixed">
-        <origin xyz="0 0 0" rpy="${-M_PI/2} 0 ${-M_PI/2}" />
-        <parent link="${name}_infra2_frame" />
-        <child link="${name}_infra2_optical_frame" />
-      </joint>
-      <link name="${name}_infra2_optical_frame"/>
-      <!-- camera color joints and links -->
-      <joint name="${name}_color_joint" type="fixed">
-        <origin xyz="0 ${d405_cam_depth_to_color_offset} 0" rpy="0 0 0" />
-        <parent link="${name}_link" />
-        <child link="${name}_color_frame" />
-      </joint>
-      <link name="${name}_color_frame"/>
-      <joint name="${name}_color_optical_joint" type="fixed">
-        <origin xyz="0 0 0" rpy="${-M_PI/2} 0 ${-M_PI/2}" />
-        <parent link="${name}_color_frame" />
-        <child link="${name}_color_optical_frame" />
-      </joint>
-      <link name="${name}_color_optical_frame"/>
-    </xacro:if>
-    <xacro:if value="${add_plug}">
-      <xacro:usb_plug parent="${name}_link" name="${name}_usb_plug">
-        <origin xyz="${d405_cam_mount_from_center_offset - 0.02095} ${-d405_cam_depth_py - 0.0353} 0" rpy="0 0 0"/>
-      </xacro:usb_plug>
-    </xacro:if>
+  <xacro:macro name="sensor_d405" params="parent *origin name:=camera
+					  use_nominal_extrinsics:=true
+					  add_plug:=false
+					  use_mesh:=true">
+    <xacro:include filename="$(find realsense2_description
+			     )/urdf/_d405.urdf.xacro" />
+    <xacro:sensor_d405 parent="${parent}" name="${name}"
+		       use_nominal_extrinsics="${use_nominal_extrinsics}"
+		       add_plug="${add_plug}" use_mesh="${use_mesh}">
+      <xacro:insert_block name="origin"/>
+    </xacro:sensor_d405>
     <gazebo reference="${name}_depth_frame">
       <sensor type="depth" name="${name}">
@@ -145,5 +25,5 @@
           <horizontal_fov>1.034</horizontal_fov>
           <image>
-            <width>848</width>
+            <width>640</width>
             <height>480</height>
             <format>R8G8B8</format>

File: aist_description/devices/urdf/_d435.urdf.xacro (robot description, xacro)
@@ -7,10 +7,13 @@
 -->
 <robot name="sensor_d435" xmlns:xacro="http://ros.org/wiki/xacro">
-  <xacro:macro name="sensor_d435"
-  	       params="parent *origin name:=camera use_nominal_extrinsics:=false">
+  <xacro:macro name="sensor_d435" params="parent *origin name:=camera
+					  use_nominal_extrinsics:=true
+					  add_plug:=false
+					  use_mesh:=true">
     <xacro:include filename="$(find realsense2_description
 			     )/urdf/_d435.urdf.xacro" />
     <xacro:sensor_d435 parent="${parent}" name="${name}"
-		       use_nominal_extrinsics="${use_nominal_extrinsics}">
+		       use_nominal_extrinsics="${use_nominal_extrinsics}"
+		       add_plug="${add_plug}" use_mesh="${use_mesh}">
       <xacro:insert_block name="origin"/>
     </xacro:sensor_d435>
@@ -35,5 +38,5 @@
 	<plugin name="${name}_controller"
 		filename="libgazebo_ros_openni_kinect.so">
-          <baseline>0.2</baseline>
+          <baseline>0.050</baseline>
           <alwaysOn>true</alwaysOn>
           <updateRate>10.0</updateRate>

File: aist_description/devices/urdf/_d455.urdf.xacro (robot description, xacro)
@@ -1,18 +1,18 @@
 <?xml version="1.0"?>
 <!--
-This file is based on the d435 urdf from the realsense package.
-The origin of the mesh is at the center of the back mount.
+License: Apache 2.0. See LICENSE file in root directory.
+Copyright(c) 2017 Intel Corporation. All Rights Reserved
+This is the URDF model for the Intel RealSense 430 camera, in it's
+aluminum peripherial evaluation case.
 -->
-<robot name="sensor_sr305" xmlns:xacro="http://ros.org/wiki/xacro">
-  <xacro:macro name="sensor_sr305" params="parent *origin name:=camera
-					   use_nominal_extrinsics:=true
-					   use_bottom_mount:=false">
+<robot name="sensor_d455" xmlns:xacro="http://ros.org/wiki/xacro">
+  <xacro:macro name="sensor_d455" params="parent *origin name:=camera
+					  use_nominal_extrinsics:=true">
     <xacro:include filename="$(find realsense2_description
-			     )/urdf/_sr305.urdf.xacro" />
-    <xacro:sensor_sr305 parent="${parent}" name="${name}"
-			use_nominal_extrinsics="${use_nominal_extrinsics}"
-		        use_bottom_mount="${use_bottom_mount}">
+			     )/urdf/_d455.urdf.xacro" />
+    <xacro:sensor_d455 parent="${parent}" name="${name}"
+		       use_nominal_extrinsics="${use_nominal_extrinsics}">
       <xacro:insert_block name="origin"/>
-    </xacro:sensor_sr305>
+    </xacro:sensor_d455>
     <gazebo reference="${name}_depth_frame">
       <sensor type="depth" name="${name}">
@@ -35,5 +35,5 @@
 	<plugin name="${name}_controller"
 		filename="libgazebo_ros_openni_kinect.so">
-          <baseline>0.018</baseline>
+          <baseline>0.095</baseline>
           <alwaysOn>true</alwaysOn>
           <updateRate>10.0</updateRate>

File: aist_description/devices/urdf/wrist_cameras.urdf.xacro (robot description, xacro)
@@ -6,7 +6,7 @@
     <xacro:include filename="$(find aist_description
 			     )/devices/urdf/_sr305.urdf.xacro"/>
-      <!-- Add the holder and two SR305 cameras -->
-      <xacro:property name="mount_mesh_file"
-		      value="package://aist_description/devices/meshes/sr305_mount.stl"/>
+    <!-- Add the holder and two SR305 cameras -->
+    <xacro:property name="mount_mesh_file"
+		    value="package://aist_description/devices/meshes/sr305_mount.stl"/>
     <link name="${prefix}camera_mount">
       <inertial>

File: aist_description/devices/urdf/wrist_d435.urdf.xacro (robot description, xacro)
@@ -6,7 +6,7 @@
     <xacro:include filename="$(find aist_description
 			     )/devices/urdf/_d435.urdf.xacro"/>
-      <!-- Add the holder and two SR305 cameras -->
-      <xacro:property name="mount_mesh_file"
-		      value="package://aist_description/devices/meshes/sr305_mount.stl"/>
+    <!-- Add the holder and two SR305 cameras -->
+    <xacro:property name="mount_mesh_file"
+		    value="package://aist_description/devices/meshes/sr305_mount.stl"/>
     <link name="${prefix}camera_mount">
       <inertial>

File: aist_description/scenes/urdf/a_bot_base_scene.urdf.xacro (robot description, xacro)
@@ -1,5 +1,5 @@
 <?xml version="1.0"?>
 <robot xmlns:xacro="http://wiki.ros.org/xacro" name="a_bot__base_scene" >
-  <xacro:arg name="scene" default="a_bot_calibration"/>
+  <xacro:arg name="scene" default=""/>
   <!-- Calibration help: If the robot is not moving far enough to the calibration point, increase these distances -->
   <xacro:property name="a_bot_x" value="0"/>

File: aist_description/scenes/urdf/calibration.urdf.xacro (robot description, xacro)
@@ -2,5 +2,6 @@
 <robot xmlns:xacro="http://wiki.ros.org/xacro" name="aist_calibration">
   <!-- Add AR markers -->
-  <xacro:include filename="$(find aist_description)/objects/urdf/ar_markers.urdf.xacro"/>
+  <xacro:include filename="$(find aist_description
+			   )/objects/urdf/ar_markers.urdf.xacro"/>
   <!-- <xacro:ar_marker_70_5 prefix="a_bot_" -->
   <!-- 			parent="a_bot_gripper_tip_link" -->
@@ -13,17 +14,7 @@
   			marker_id="26"
 			thickness="0.005">
-    <origin xyz="0.063 0.0 0.0215" rpy="0 0 ${pi/2}"/>
+    <origin xyz="0.063 0.0 0.0215" rpy="0 0 0"/>
   </xacro:ar_marker_70_5>
-  <!-- <xacro:ar_marker_70_5 prefix="workspace_" -->
-  <!-- 			parent="workspace_center" -->
-  <!-- 			marker_id="32" -->
-  <!-- 			thickness="0.001"> -->
-  <!--   <origin xyz="0.0 0.0 0.0005" rpy="0 0 0"/> -->
-  <!-- </xacro:ar_marker_70_5> -->
-  <xacro:ar_marker_150_5 prefix="workspace_"
-  			 parent="workspace_center"
-  			 marker_id="17_26_32_256"
-  			 thickness="0.001">
-    <origin xyz="0.0 0.0 0.0005" rpy="0 0 0"/>
-  </xacro:ar_marker_150_5>
+  <xacro:include filename="$(find aist_description
+			   )/scenes/urdf/eye_on_hand.urdf.xacro"/>
 </robot>

File: aist_description/scenes/urdf/f_bot_base_scene.urdf.xacro (robot description, xacro)
@@ -1,32 +1,38 @@
 <?xml version="1.0"?>
 <robot xmlns:xacro="http://wiki.ros.org/xacro" name="f_bot_base_scene" >
+  <!-- This is the main file defining our robot arrangement and physical environment. -->
   <xacro:arg name="scene" default=""/>
-  <!-- Calibration help: If the robot is not moving far enough to the calibration point, increase these distances -->
-  <xacro:property name="f_bot_x" value="0"/>
-  <xacro:property name="f_bot_y" value="-0.4875"/>
-  <!-- <xacro:property name="f_bot_theta" value="${pi}"/> -->
-  <xacro:property name="bots_z" value="0.88"/>
-  <!-- This is the main file defining our robot arrangement and physical environment. -->
+  <xacro:property name="f_bot_x"   value="0"/>
+  <xacro:property name="f_bot_y"   value="-0.610"/>
+  <xacro:property name="f_bot_z"   value="0.880"/>
+  <xacro:property name="table_w"   value="1.800"/>
+  <xacro:property name="table_l"   value="1.000"/>
+  <xacro:property name="table_h"   value="0.705"/>
+  <xacro:property name="mounter_w" value="0.200"/>
+  <xacro:property name="mounter_l" value="0.200"/>
+  <link name="ground"/>
   <!-- Main workspace -->
-  <!-- The surface is 0.01 m below the robot bases and the "workspace_center" frame. -->
-  <link name="ground"/>
   <xacro:include filename="$(find aist_description)/objects/urdf/aist_box.urdf.xacro"/>
-  <xacro:property name="table_w" value="1.800"/>
-  <xacro:property name="table_l" value="1.100"/>
-  <xacro:property name="table_h" value="0.705"/>
-  <xacro:property name="table_t" value="0.010"/>
-  <xacro:aist_box name="workbox"
-		  width="${table_w}" length="${table_l}" height="${table_t}"
-		  parent="ground">
-    <origin xyz="${-table_w/2} ${-table_l/2} ${table_h - table_t}" rpy="0 0 0"/>
-  </xacro:aist_box>
+  <xacro:include filename="$(find aist_description
+			   )/objects/urdf/table.urdf.xacro"/>
+  <xacro:table prefix="worksapce_"
+	       width="${table_w}" length="${table_l}" height="${table_h}"
+	       parent="ground">
+    <origin xyz="${-table_w/2} ${-table_l/2} 0" rpy="0 0 0"/>
+  </xacro:table>
   <link name="workspace_center"/>
   <joint name="ground_to_workspace" type="fixed">
     <parent link="ground"/>
     <child  link="workspace_center"/>
-    <origin xyz="0 0 ${bots_z}" rpy="0 0 0"/>
+    <origin xyz="0 0 ${table_h}" rpy="0 0 0"/>
   </joint>
-  <!-- robot arms -->
-  <!-- <xacro:include filename="$(find ur_description)/urdf/common.gazebo.xacro"/> -->
+  <!-- Robot mounter -->
+  <xacro:table prefix="mounter_"
+	       width="${mounter_w}" length="${mounter_l}" height="${f_bot_z}"
+	       parent="ground">
+    <origin xyz="${f_bot_x - mounter_w/2} ${f_bot_y - mounter_l/2} 0"
+	    rpy="0 0 0"/>
+  </xacro:table>
+  <!-- Robot arm -->
   <xacro:include filename="$(find ur_gazebo)/urdf/ur_macro.xacro"/>
   <xacro:ur_robot_gazebo
@@ -44,12 +50,12 @@
     <parent link="ground"/>
     <child  link="f_bot_base_link"/>
-    <origin xyz="${f_bot_x} ${f_bot_y} ${bots_z}" rpy="0 0 0"/>
+    <origin xyz="${f_bot_x} ${f_bot_y} ${f_bot_z}" rpy="0 0 0"/>
   </joint>
-  <!-- Spawn and attach force sensor -->
+  <!-- Attach force sensor -->
   <xacro:include filename="$(find aist_robotiq)/urdf/ft300.urdf.xacro"/>
   <xacro:ft300 prefix="f_bot_ftsensor_" parent="f_bot_flange">
     <origin xyz="0 0 0" rpy="${pi} 0 0"/>
   </xacro:ft300>
-  <!-- Spawn and attach gripper -->
+  <!-- Attach gripper -->
   <xacro:include filename="$(find aist_robotiq
 			   )/urdf/robotiq_arg2f_coupling.urdf.xacro"/>
@@ -61,8 +67,10 @@
 			   )/urdf/robotiq_140_gripper.urdf.xacro"/>
   <xacro:robotiq_140_gripper prefix="f_bot_gripper_"
-			    parent="f_bot_gripper_coupling_flange_link">
+			     parent="f_bot_gripper_coupling_flange_link">
     <origin xyz="0 0 0" rpy="0 0 0"/>
   </xacro:robotiq_140_gripper>
-  <!-- Add RealSense camera -->
+  <!-- Attach RealSense camera -->
+  <!-- <xacro:include filename="$(find aist_description -->
+  <!-- 			   )/scenes/urdf/load_calibration.urdf.xacro"/> -->
   <xacro:include filename="$(find aist_description
 			   )/scenes/urdf/load_calibration.urdf.xacro"/>
@@ -70,4 +78,6 @@
 				    )/calib/f_bot_camera.yaml"
 			  propname="camera_origin"/>
+  <!-- <xacro:include filename="$(find aist_description -->
+  <!-- 			   )/devices/urdf/_d435.urdf.xacro"/> -->
   <xacro:include filename="$(find aist_description
 			   )/devices/urdf/_d435.urdf.xacro"/>

File: moveit_config/f_bot_moveit_config/config/gazebo_f_bot_base_scene.urdf (robot description, URDF)
Before this commit: robot f_bot_base_scene, 35 links, 34 joints
Links:
- removed link d_bot_camera_bottom_screw_frame
- removed link d_bot_camera_link
- added link f_bot_camera_bottom_screw_frame
- added link f_bot_camera_link, mass 0.072; collision box size=0.02505 0.09 0.025; visual mesh filename=package://realsense2_description/meshes/d435.dae
Joints:
- removed joint d_bot_camera_joint
- removed joint d_bot_camera_link_joint
- added joint f_bot_camera_joint: type fixed, parent f_bot_gripper_base_link, child f_bot_camera_bottom_screw_frame, origin xyz=0.030 0.000 0.043 rpy=0 0.0 0
- added joint f_bot_camera_link_joint: type fixed, parent f_bot_camera_bottom_screw_frame, child f_bot_camera_link, origin xyz=0.010600000000000002 0.0175 0.0125 rpy=0 0 0
