Commit message: Cleaning up

File: aist_description/devices/urdf/_d405.urdf.xacro (robot description, xacro)
@@ -8,5 +8,5 @@
 <robot name="sensor_d405" xmlns:xacro="http://ros.org/wiki/xacro">
   <xacro:macro name="sensor_d405" params="parent *origin name:=camera
-					  use_nominal_extrinsics:=true
+					  use_nominal_extrinsics:=false
 					  add_plug:=false
 					  use_mesh:=true">

File: aist_description/devices/urdf/_d435.urdf.xacro (robot description, xacro)
@@ -8,5 +8,5 @@
 <robot name="sensor_d435" xmlns:xacro="http://ros.org/wiki/xacro">
   <xacro:macro name="sensor_d435" params="parent *origin name:=camera
-					  use_nominal_extrinsics:=true
+					  use_nominal_extrinsics:=false
 					  add_plug:=false
 					  use_mesh:=true">

File: aist_description/devices/urdf/_d455.urdf.xacro (robot description, xacro)
@@ -8,5 +8,5 @@
 <robot name="sensor_d455" xmlns:xacro="http://ros.org/wiki/xacro">
   <xacro:macro name="sensor_d455" params="parent *origin name:=camera
-					  use_nominal_extrinsics:=true">
+					  use_nominal_extrinsics:=false">
     <xacro:include filename="$(find realsense2_description
 			     )/urdf/_d455.urdf.xacro" />

File: aist_description/devices/urdf/_sr305.urdf.xacro (robot description, xacro)
@@ -6,5 +6,5 @@
 <robot name="sensor_sr305" xmlns:xacro="http://ros.org/wiki/xacro">
   <xacro:macro name="sensor_sr305" params="parent *origin name:=camera
-					   use_nominal_extrinsics:=true
+					   use_nominal_extrinsics:=false
 					   use_bottom_mount:=false">
     <xacro:include filename="$(find realsense2_description

File: aist_description/devices/urdf/wrist_cameras.urdf.xacro (robot description, xacro)
@@ -3,5 +3,6 @@
 <!-- The position of the TF frame has not been measured at all and needs to be calibrated. -->
 <robot name="wrist_cameras" xmlns:xacro="http://www.ros.org/wiki/xacro">
-  <xacro:macro name="wrist_cameras" params="prefix parent">
+  <xacro:macro name="wrist_cameras"
+	       params="prefix parent use_nominal_extrinsics:=false">
     <xacro:include filename="$(find aist_description
 			     )/devices/urdf/_sr305.urdf.xacro"/>
@@ -41,5 +42,6 @@
 				      )/calib/${prefix}inside_camera.yaml"
 			    propname="inside_camera_origin"/>
-    <xacro:sensor_sr305 name="${prefix}inside_camera" parent="${parent}">
+    <xacro:sensor_sr305 name="${prefix}inside_camera" parent="${parent}"
+			use_nominal_extrinsics="${use_nominal_extrinsics}">
       <origin xyz="${inside_camera_origin[0]}
 		   ${inside_camera_origin[1]}
@@ -52,5 +54,6 @@
 				      )/calib/${prefix}outside_camera.yaml"
 			    propname="outside_camera_origin"/>
-    <xacro:sensor_sr305 name="${prefix}outside_camera" parent="${parent}">
+    <xacro:sensor_sr305 name="${prefix}outside_camera" parent="${parent}"
+			use_nominal_extrinsics="${use_nominal_extrinsics}">
       <origin xyz="${outside_camera_origin[0]}
 		   ${outside_camera_origin[1]}

File: aist_description/scenes/urdf/a_bot_base_scene.urdf.xacro (robot description, xacro)
@@ -67,5 +67,6 @@
 			   )/devices/urdf/wrist_cameras.urdf.xacro" />
   <xacro:wrist_cameras prefix="a_bot_"
-		       parent="a_bot_gripper_base_link"/>
+		       parent="a_bot_gripper_base_link"
+		       use_nominal_extrinsics="true"/>
   <!-- I would like to remove the "world" link definition, but apparently it is necessary for Gazebo -->
   <link name="world"/>

File: aist_description/scenes/urdf/aist_base_scene.urdf.xacro (robot description, xacro)
@@ -131,5 +131,6 @@
   			   )/devices/urdf/wrist_cameras.urdf.xacro" />
   <xacro:wrist_cameras prefix="a_bot_"
-  		       parent="a_bot_gripper_base_link"/>
+  		       parent="a_bot_gripper_base_link"
+		       use_nominal_extrinsics="true"/>
   <!-- live camera -->
   <xacro:load_calibration filename="$(find aist_camera_calibration

File: aist_description/scenes/urdf/f_bot_base_scene.urdf.xacro (robot description, xacro)
@@ -82,5 +82,6 @@
   <xacro:include filename="$(find aist_description
 			   )/devices/urdf/_d435.urdf.xacro"/>
-  <xacro:sensor_d435 name="f_bot_camera" parent="f_bot_gripper_base_link">
+  <xacro:sensor_d435 name="f_bot_camera" parent="f_bot_gripper_base_link"
+		     use_nominal_extrinsics="true">
     <origin xyz="${camera_origin[0]} ${camera_origin[1]} ${camera_origin[2]}"
     	    rpy="${camera_origin[3]} ${camera_origin[4]} ${camera_origin[5]}"/>

File: aist_description/scenes/urdf/fvision_base_scene.urdf.xacro (robot description, xacro)
@@ -87,5 +87,6 @@
   <xacro:include filename="$(find aist_description
 			   )/devices/urdf/_sr305.urdf.xacro"/>
-  <xacro:sensor_sr305 name="d_bot_camera" parent="d_bot_gripper_base_link">
+  <xacro:sensor_sr305 name="d_bot_camera" parent="d_bot_gripper_base_link"
+		      use_nominal_extrinsics="true">
     <origin xyz="0.030 0.000 0.043" rpy="0 ${0.0*pi/180.0} 0" />
   </xacro:sensor_sr305>

Commit message: Adjust FOV etc. of realsensen camera for gazebo simulation

File: aist_description/devices/urdf/_d405.urdf.xacro (robot description, xacro)
@@ -18,13 +18,21 @@
       <xacro:insert_block name="origin"/>
     </xacro:sensor_d405>
-    <gazebo reference="${name}_depth_frame">
+    <!-- Reference should be color_frame because depth is alighed to color -->
+    <gazebo reference="${name}_color_frame">
       <sensor type="depth" name="${name}">
 	<always_on>true</always_on>
 	<visualize>true</visualize>
 	<camera>
-          <horizontal_fov>1.034</horizontal_fov>
+	  <!-- Color sensor's FOV(HD): 84 deg. -->
+          <horizontal_fov>1.4661</horizontal_fov>
+	  <!-- Color sensor's FOV(VGA): 48.47 deg. -->
+          <!-- <horizontal_fov>0.846</horizontal_fov> -->
           <image>
-            <width>640</width>
-            <height>480</height>
+	    <!-- HD -->
+            <width>1280</width>
+            <height>720</height>
+	    <!-- VGA -->
+            <!-- <width>640</width> -->
+            <!-- <height>480</height> -->
             <format>R8G8B8</format>
           </image>

File: aist_description/devices/urdf/_d415.urdf.xacro (robot description, xacro)
@@ -6,22 +6,33 @@
 aluminum peripherial evaluation case.
 -->
-<robot name="sensor_d455" xmlns:xacro="http://ros.org/wiki/xacro">
-  <xacro:macro name="sensor_d455" params="parent *origin name:=camera
-					  use_nominal_extrinsics:=false">
+<robot name="sensor_d415" xmlns:xacro="http://ros.org/wiki/xacro">
+  <xacro:macro name="sensor_d415" params="parent *origin name:=camera
+					  use_nominal_extrinsics:=false
+					  add_plug:=false
+					  use_mesh:=true">
     <xacro:include filename="$(find realsense2_description
-			     )/urdf/_d455.urdf.xacro" />
-    <xacro:sensor_d455 parent="${parent}" name="${name}"
-		       use_nominal_extrinsics="${use_nominal_extrinsics}">
+			     )/urdf/_d415.urdf.xacro" />
+    <xacro:sensor_d415 parent="${parent}" name="${name}"
+		       use_nominal_extrinsics="${use_nominal_extrinsics}"
+		       add_plug="${add_plug}" use_mesh="${use_mesh}">
       <xacro:insert_block name="origin"/>
-    </xacro:sensor_d455>
-    <gazebo reference="${name}_depth_frame">
+    </xacro:sensor_d415>
+    <!-- Reference should be color_frame because depth is alighed to color -->
+    <gazebo reference="${name}_color_frame">
       <sensor type="depth" name="${name}">
 	<always_on>true</always_on>
 	<visualize>true</visualize>
 	<camera>
-          <horizontal_fov>1.5708</horizontal_fov>	<!-- 90 deg. -->
+	  <!-- Color sensor's FOV(HD): 69 deg. -->
+          <horizontal_fov>1.2043</horizontal_fov>
+	  <!-- Color sensor's FOV(VGA): 42.27 deg. -->
+          <!-- <horizontal_fov>0.9091</horizontal_fov> -->
           <image>
+	    <!-- HD -->
             <width>1280</width>
-            <height>800</height>
+            <height>720</height>
+	    <!-- VGA -->
+            <!-- <width>640</width> -->
+            <!-- <height>480</height> -->
             <format>R8G8B8</format>
           </image>
@@ -35,5 +46,5 @@
 	<plugin name="${name}_controller"
 		filename="libgazebo_ros_openni_kinect.so">
-          <baseline>0.095</baseline>
+          <baseline>0.055</baseline>
           <alwaysOn>true</alwaysOn>
           <updateRate>10.0</updateRate>

File: aist_description/devices/urdf/_d435.urdf.xacro (robot description, xacro)
@@ -18,13 +18,21 @@
       <xacro:insert_block name="origin"/>
     </xacro:sensor_d435>
-    <gazebo reference="${name}_depth_frame">
+    <!-- Reference should be color_frame because depth is alighed to color -->
+    <gazebo reference="${name}_color_frame">
       <sensor type="depth" name="${name}">
 	<always_on>true</always_on>
 	<visualize>true</visualize>
 	<camera>
-          <horizontal_fov>1.034</horizontal_fov>
+	  <!-- Color sensor's FOV(HD): 69 deg. -->
+          <horizontal_fov>1.2043</horizontal_fov>
+	  <!-- Color sensor's FOV(VGA): 42.27 deg. -->
+          <!-- <horizontal_fov>0.9091</horizontal_fov> -->
           <image>
-            <width>640</width>
-            <height>480</height>
+	    <!-- HD -->
+            <width>1280</width>
+            <height>720</height>
+	    <!-- VGA -->
+            <!-- <width>640</width> -->
+            <!-- <height>480</height> -->
             <format>R8G8B8</format>
           </image>

File: aist_description/devices/urdf/_sr305.urdf.xacro (robot description, xacro)
@@ -15,11 +15,14 @@
       <xacro:insert_block name="origin"/>
     </xacro:sensor_sr305>
-    <gazebo reference="${name}_depth_frame">
+    <!-- Reference should be color_frame because depth is alighed to color -->
+    <gazebo reference="${name}_color_frame">
       <sensor type="depth" name="${name}">
 	<always_on>true</always_on>
 	<visualize>true</visualize>
 	<camera>
-          <horizontal_fov>1.034</horizontal_fov>
+	  <!-- Color sensor's FOV(VGA): 68 deg. -->
+          <horizontal_fov>1.1868</horizontal_fov>
           <image>
+	    <!-- VGA -->
             <width>640</width>
             <height>480</height>
@@ -35,5 +38,5 @@
 	<plugin name="${name}_controller"
 		filename="libgazebo_ros_openni_kinect.so">
-          <baseline>0.018</baseline>
+          <baseline>0.048</baseline>
           <alwaysOn>true</alwaysOn>
           <updateRate>10.0</updateRate>

File: aist_description/scenes/urdf/g_bot_base_scene.urdf.xacro (robot description, xacro)
@@ -4,5 +4,5 @@
   <xacro:arg name="scene" default=""/>
   <xacro:property name="g_bot_x"   value="0"/>
-  <xacro:property name="g_bot_y"   value="-0.920"/>
+  <xacro:property name="g_bot_y"   value="-0.625"/>
   <xacro:property name="g_bot_z"   value="0.700"/>
   <xacro:property name="cabinet_w" value="0.900"/>
@@ -10,5 +10,5 @@
   <xacro:property name="cabinet_b" value="0.100"/>
   <xacro:property name="shelf1_h"  value="0.600"/>
-  <xacro:property name="shelf2_h"  value="0.990"/>
+  <xacro:property name="shelf2_h"  value="0.790"/>
   <xacro:property name="back_h"    value="1.500"/>
   <xacro:property name="wall_t"    value="0.012"/>
@@ -92,10 +92,10 @@
 				    )/calib/g_bot_camera.yaml"/>
   <xacro:include filename="$(find aist_description
-			   )/devices/urdf/_d435.urdf.xacro"/>
-  <xacro:sensor_d435 name="g_bot_camera" parent="workspace_center"
+			   )/devices/urdf/_d415.urdf.xacro"/>
+  <xacro:sensor_d415 name="g_bot_camera" parent="workspace_center"
 		     use_nominal_extrinsics="true">
     <origin xyz="${origin[0]} ${origin[1]} ${origin[2]}"
     	    rpy="${origin[3]} ${origin[4]} ${origin[5]}"/>
-  </xacro:sensor_d435>
+  </xacro:sensor_d415>
   <!-- I would like to remove the "world" link definition, but apparently it is necessary for Gazebo -->
   <link name="world"/>
