Commit message: Confirmed both suction and robotiq gripper works with ur_robot_driver

File: aist_description/devices/urdf/dual_suction_gripper.urdf.xacro (robot description, xacro)
@@ -5,5 +5,5 @@
 	       params="prefix parent *origin">
     <!-- A link representing the gripper and a joint attaching it to parnet -->
-    <link name="${prefix}dual_suction_gripper_base_link">
+    <link name="${prefix}base_link">
       <visual>
         <origin xyz="0.1855 -0.035 -0.035" rpy="0 0 ${pi/2}"/>
@@ -29,29 +29,23 @@
       </inertial>
     </link>
-    <joint name="${prefix}dual_suction_gripper_joint" type="fixed">
+    <joint name="${prefix}base_joint" type="fixed">
       <parent link="${parent}"/>
-      <child  link="${prefix}dual_suction_gripper_base_link"/>
+      <child  link="${prefix}base_link"/>
        <xacro:insert_block name="origin"/>
     </joint>
     <!-- A link representing the tip of the pad and a joint attaching
 	 it to the gripper -->
-    <link name="${prefix}dual_suction_gripper_pad_link"/>
-    <joint name="${prefix}dual_suction_gripper_pad_joint" type="fixed">
-      <parent link="${prefix}dual_suction_gripper_base_link"/>
-      <child  link="${prefix}dual_suction_gripper_pad_link"/>
+    <link name="${prefix}pad_link"/>
+    <joint name="${prefix}pad_joint" type="fixed">
+      <parent link="${prefix}base_link"/>
+      <child  link="${prefix}pad_link"/>
       <origin xyz="0.1855 0 0" rpy="0 0 0"/>
     </joint>
-    <joint name="${prefix}robotiq_85_suction_tool_tip_joint" type="fixed">
-      <parent link="${prefix}dual_suction_gripper_pad_link"/>
-      <child link="${prefix}suction_tool_tip_link"/>
-      <origin rpy="0.0 0.0 0.0" xyz="0.0 0.0 0.0 "/>
-    </joint>
-    <link name="${prefix}suction_tool_tip_link"/>
     <!-- A link representing the tip of the coander gripper
 	 and a joint attaching it to the gripper -->
-    <link name="${prefix}dual_suction_gripper_coanda_link"/>
-    <joint name="${prefix}dual_suction_gripper_coanda_joint" type="fixed">
-      <parent link="${prefix}dual_suction_gripper_base_link"/>
-      <child  link="${prefix}dual_suction_gripper_coanda_link"/>
+    <link name="${prefix}coanda_link"/>
+    <joint name="${prefix}coanda_joint" type="fixed">
+      <parent link="${prefix}base_link"/>
+      <child  link="${prefix}coanda_link"/>
       <origin xyz="0.0505 0.145 0" rpy="0 0 ${pi/2}"/>
     </joint>

File: aist_description/scenes/urdf/aist_base_scene.urdf.xacro (robot description, xacro)
@@ -81,5 +81,5 @@
   </xacro:robotiq_85_gripper_with_tip_link>
   <xacro:include filename="$(find aist_description)/devices/urdf/single_suction_gripper.urdf.xacro"/>
-  <xacro:single_suction_gripper prefix="b_bot_"
+  <xacro:single_suction_gripper prefix="b_bot_gripper_"
   				parent="b_bot_ftsensor_flange_link">
     <!-- <origin xyz="0 0 0" rpy="0 ${0.2*pi/180} ${-1.2*pi/180}"/> -->

Commit message: Confirmed that kitting demo works with updated fastening tools

File: aist_description/devices/urdf/dual_suction_gripper.urdf.xacro (robot description, xacro)
@@ -36,8 +36,8 @@
     <!-- A link representing the tip of the pad and a joint attaching
 	 it to the gripper -->
-    <link name="${prefix}pad_link"/>
-    <joint name="${prefix}pad_joint" type="fixed">
+    <link name="${prefix}tip_link"/>
+    <joint name="${prefix}tip_joint" type="fixed">
       <parent link="${prefix}base_link"/>
-      <child  link="${prefix}pad_link"/>
+      <child  link="${prefix}tip_link"/>
       <origin xyz="0.1855 0 0" rpy="0 0 0"/>
     </joint>

File: aist_description/devices/urdf/single_suction_gripper.urdf.xacro (robot description, xacro)
@@ -36,8 +36,8 @@
     <!-- A link representing the tip of the pad and a joint attaching
 	 it to the gripper -->
-    <link name="${prefix}pad_link"/>
-    <joint name="${prefix}pad_joint" type="fixed">
+    <link name="${prefix}tip_link"/>
+    <joint name="${prefix}tip_joint" type="fixed">
       <parent link="${prefix}base_link"/>
-      <child  link="${prefix}pad_link"/>
+      <child  link="${prefix}tip_link"/>
       <origin xyz="0.1855 0 0" rpy="0 0 0"/>
     </joint>

Commit message: Change orientaion of grippers' tip_link

File: aist_description/devices/urdf/dual_suction_gripper.urdf.xacro (robot description, xacro)
@@ -40,5 +40,5 @@
       <parent link="${prefix}base_link"/>
       <child  link="${prefix}tip_link"/>
-      <origin xyz="0.1855 0 0" rpy="0 0 0"/>
+      <origin xyz="0.1855 0 0" rpy="0 ${-pi/2} 0"/>
     </joint>
     <!-- A link representing the tip of the coander gripper
@@ -48,5 +48,5 @@
       <parent link="${prefix}base_link"/>
       <child  link="${prefix}coanda_link"/>
-      <origin xyz="0.0505 0.145 0" rpy="0 0 ${pi/2}"/>
+      <origin xyz="0.0505 0.145 0" rpy="0 ${-pi/2} ${pi/2}"/>
     </joint>
   </xacro:macro>

File: aist_description/devices/urdf/single_suction_gripper.urdf.xacro (robot description, xacro)
@@ -40,5 +40,5 @@
       <parent link="${prefix}base_link"/>
       <child  link="${prefix}tip_link"/>
-      <origin xyz="0.1855 0 0" rpy="0 0 0"/>
+      <origin xyz="0.1855 0 0" rpy="0 ${-pi/2} 0"/>
     </joint>
   </xacro:macro>

File: aist_description/devices/urdf/torobo_gripper.urdf.xacro (robot description, xacro)
@@ -19,5 +19,5 @@
       <parent link="${prefix}gripper/grasping_frame"/>
       <child  link="${prefix}gripper/tip_link"/>
-      <origin xyz="0 0 0" rpy="0 ${-pi/2} 0"/>
+      <origin xyz="0 0 0.025" rpy="${pi} 0 ${pi}"/>
     </joint>
   </xacro:macro>

File: aist_robotiq/urdf/robotiq_140_gripper.urdf.xacro (robot description, xacro)
@@ -249,5 +249,5 @@
       <parent link="${prefix}base_link"/>
       <child link="${prefix}tip_link"/>
-      <origin rpy="0.0 0.0 0.0" xyz=".2328 0.0 0.0"/>
+      <origin rpy="0.0 ${-pi/2} 0.0" xyz=".2328 0.0 0.0"/>
     </joint>
     <link name="${prefix}tip_link"/>

File: aist_robotiq/urdf/robotiq_85_gripper.urdf.xacro (robot description, xacro)
@@ -240,5 +240,5 @@
       <parent link="${prefix}base_link"/>
       <child link="${prefix}tip_link"/>
-      <origin rpy="0.0 0.0 0.0" xyz="0.1628 0.0 0.0"/>
+      <origin rpy="0.0 ${-pi/2} 0.0" xyz="0.1628 0.0 0.0"/>
     </joint>
     <link name="${prefix}tip_link"/>

File: aist_robotiq/urdf/robotiq_hande_gripper.urdf.xacro (robot description, xacro)
@@ -22,5 +22,5 @@
       <parent link="${prefix}base_link"/>
       <child link="${prefix}tip_link"/>
-      <origin rpy="0.0 0.0 0.0" xyz=".146 0.0 0.0"/>
+      <origin rpy="0.0 ${-pi/2} 0.0" xyz=".146 0.0 0.0"/>
     </joint>
     <link name="${prefix}tip_link"/>
