Commit message: Replace camera mounted on a_bot from realsense to zivid

File: aist_description/devices/urdf/zivid2plus.urdf (robot description, URDF)
Before this commit: robot aaa, 1 links, 0 joints
Links:
- removed link world
- added link base_link

File: aist_description/devices/urdf/zivid2plus.urdf.xacro (robot description, xacro)
@@ -3,12 +3,16 @@
        xmlns:xacro="http://wiki.ros.org/xacro">
   <xacro:macro name="zivid2plus"
-	       params="prefix parent *origin">
-    <xacro:property name="baseline_half_length"		value="0.05702"/>
-    <xacro:property name="optical_center_height"	value="0.0295"/>
-    <xacro:property name="vergence_half_angle"		value="2.5"/>
-    <!-- A link representing the gripper and a joint attaching it to parnet -->
-    <link name="${prefix}base_link">
+	       params="name parent *origin">
+    <xacro:property name="baseline_half_length"	 value="0.05702"/>
+    <xacro:property name="optical_center_height" value="0.0295"/>
+    <xacro:property name="vergence_half_angle"	 value="2.5"/>
+    <xacro:property name="image_width"		 value="2448"/>
+    <xacro:property name="image_height"		 value="2048"/>
+    <xacro:property name="horizontal_fov"	 value="0.9222"/>
+    <xacro:property name="update_rate"		 value="10"/>
+    <!-- A link representing the camera body -->
+    <link name="${name}_base_link">
       <visual>
-        <origin xyz="0 0 ${optical_center_height}" rpy="${-pi/2} 0 0"/>
+        <origin xyz="0 0 ${optical_center_height}" rpy="${-pi/2} 0 ${-pi/2}"/>
 	<geometry>
           <mesh filename="package://aist_description/devices/meshes/zivid2plus.stl" scale="0.001 0.001 0.001"/>
@@ -32,25 +36,76 @@
       </inertial>
     </link>
-    <joint name="${prefix}base_joint" type="fixed">
+    <joint name="${name}_base_joint" type="fixed">
       <parent link="${parent}"/>
-      <child  link="${prefix}base_link"/>
+      <child  link="${name}_base_link"/>
       <xacro:insert_block name="origin"/>
     </joint>
-    <!-- A link representing the tip of the pad and a joint attaching
-	 it to the gripper -->
-    <link name="${prefix}sensor"/>
-    <joint name="${prefix}sensor_joint" type="fixed">
-      <parent link="${prefix}base_link"/>
-      <child  link="${prefix}sensor"/>
-      <origin xyz="${baseline_half_length} 0 ${optical_center_height}"
-	      rpy="${-pi/2} 0 ${vergence_half_angle*pi/180.0}"/>
+    <!-- A link representing the sensor in the mechanical frame -->
+    <link name="${name}_reference"/>
+    <joint name="${name}_reference_joint" type="fixed">
+      <parent link="${name}_base_link"/>
+      <child  link="${name}_reference"/>
+      <origin xyz="0 ${baseline_half_length} ${optical_center_height}"
+	      rpy="0 0 ${-vergence_half_angle*pi/180.0}"/>
     </joint>
-    <link name="${prefix}projector"/>
-    <joint name="${prefix}projector_joint" type="fixed">
-      <parent link="${prefix}base_link"/>
-      <child  link="${prefix}projector"/>
-      <origin xyz="${-baseline_half_length} 0 ${optical_center_height}"
-	      rpy="${-pi/2} 0 ${-vergence_half_angle*pi/180.0}"/>
+    <!-- A link representing the sensor in the optical frame -->
+    <link name="${name}_sensor"/>
+    <joint name="${name}_sensor_joint" type="fixed">
+      <parent link="${name}_reference"/>
+      <child  link="${name}_sensor"/>
+      <origin xyz="0 0 0" rpy="${-pi/2} 0 ${-pi/2}"/>
     </joint>
+    <!-- A link representing the projector in the mechanical frame -->
+    <link name="${name}_projector"/>
+    <joint name="${name}_projector_joint" type="fixed">
+      <parent link="${name}_base_link"/>
+      <child  link="${name}_projector"/>
+      <origin xyz="0 ${-baseline_half_length} ${optical_center_height}"
+	      rpy="0 0 ${vergence_half_angle*pi/180.0}"/>
+    </joint>
+    <gazebo reference="${name}_reference">
+      <sensor name="${name}" type="depth">
+	<always_on>true</always_on>
+	<visualize>true</visualize>
+	<camera>
+          <image>
+            <width>${image_width}</width>
+            <height>${image_height}</height>
+            <format>L8</format>
+          </image>
+          <horizontal_fov>${horizontal_fov}</horizontal_fov>
+          <depth_camera>
+          </depth_camera>
+          <clip>
+            <near>0.1</near>
+            <far>100</far>
+          </clip>
+	</camera>
+	<plugin name="${name}_controller"
+		filename="libgazebo_ros_openni_kinect.so">
+          <baseline>${2.0*baseline_half_length}</baseline>
+          <alwaysOn>true</alwaysOn>
+          <updateRate>${update_rate}</updateRate>
+          <cameraName>${name}</cameraName>
+          <frameName>${name}_sensor</frameName>
+          <imageTopicName>texture</imageTopicName>
+          <depthImageTopicName>depth_map</depthImageTopicName>
+          <pointCloudTopicName>pointcloud</pointCloudTopicName>
+          <cameraInfoTopicName>camera_info</cameraInfoTopicName>
+          <depthImageCameraInfoTopicName>camera_info</depthImageCameraInfoTopicName>
+          <pointCloudCutoff>0.4</pointCloudCutoff>
+          <!-- <hackBaseline>0.35</hackBaseline> -->
+          <distortionK1>0.0</distortionK1>
+          <distortionK2>0.0</distortionK2>
+          <distortionK3>0.0</distortionK3>
+          <distortionT1>0.0</distortionT1>
+          <distortionT2>0.0</distortionT2>
+          <CxPrime>0.0</CxPrime>
+          <Cx>0.0</Cx>
+          <Cy>0.0</Cy>
+          <focalLength>0.0</focalLength>
+	</plugin>
+      </sensor>
+    </gazebo>
   </xacro:macro>
 </robot>

File: aist_description/scenes/urdf/aist_base_scene.urdf.xacro (robot description, xacro)
@@ -85,9 +85,21 @@
     <origin xyz="${b_bot_x} ${b_bot_y} ${bots_z}" rpy="0 0 ${b_bot_theta}"/>
   </joint>
-  <!-- Spawn and attach zivid camera -->
+  <!-- Attach mounter for Zivid2+ camera -->
   <xacro:include filename="$(find aist_description)/devices/urdf/zivid_coupling.urdf.xacro"/>
   <xacro:zivid_coupling prefix="a_bot_zivid_coupling_" parent="a_bot_flange">
     <origin xyz="0 0 0" rpy="${pi} 0 0" />
   </xacro:zivid_coupling>
+  <!-- Spawn and attach Zivid2+ camera -->
+  <xacro:include filename="$(find aist_description
+			   )/scenes/urdf/load_calibration.urdf.xacro"/>
+  <xacro:load_calibration filename="$(find aist_handeye_calibration
+				    )/calib/a_bot_zivid.yaml"/>
+  <xacro:include filename="$(find aist_description
+			   )/devices/urdf/zivid2plus.urdf.xacro"/>
+  <xacro:zivid2plus name="a_bot_zivid"
+		    parent="a_bot_zivid_coupling_flange_link">
+    <origin xyz="${origin[0]} ${origin[1]} ${origin[2]}"
+    	    rpy="${origin[3]} ${origin[4]} ${origin[5]}"/>
+  </xacro:zivid2plus>
   <!-- Spawn and attach force sensor -->
   <xacro:include filename="$(find aist_robotiq)/urdf/ft300.urdf.xacro"/>
@@ -119,9 +131,4 @@
     <origin xyz="0 0 0" rpy="0 ${0.7*pi/180} ${-0.1*pi/180}"/>
   </xacro:single_suction_gripper>
-  <!-- Add virtual wall to avoid collisions-->
-  <!-- <xacro:aist_box name="vwall1" width="0.01" length="0.35" height="0.55" -->
-  <!-- 		  parent="ground" transparent="true"> -->
-  <!--   <origin xyz="0.41 -0.20 ${bots_z}" rpy="0 0 0"/> -->
-  <!-- </xacro:aist_box> -->
   <!-- Add PhoXi 3D scanner -->
   <!-- <xacro:include filename="$(find aist_description -->
@@ -147,9 +154,9 @@
   </xacro:motioncam_m_camera>
   <!-- RealSense cameras -->
-  <xacro:include filename="$(find aist_description
-  			   )/devices/urdf/wrist_cameras.urdf.xacro" />
-  <xacro:wrist_cameras prefix="a_bot_"
-  		       parent="a_bot_gripper_base_link"
-		       use_nominal_extrinsics="true"/>
+  <!-- <xacro:include filename="$(find aist_description -->
+  <!-- 			   )/devices/urdf/wrist_cameras.urdf.xacro" /> -->
+  <!-- <xacro:wrist_cameras prefix="a_bot_" -->
+  <!-- 		       parent="a_bot_gripper_base_link" -->
+  <!-- 		       use_nominal_extrinsics="true"/> -->
   <!-- live camera -->
   <xacro:load_calibration filename="$(find aist_camera_calibration
