Commit message: Add zivid_coupling to a_bot

File: aist_description/devices/urdf/zivid2plus.urdf.xacro (robot description, xacro)
@@ -4,8 +4,11 @@
   <xacro:macro name="zivid2plus"
 	       params="prefix parent *origin">
+    <xacro:property name="baseline_half_length"		value="0.05702"/>
+    <xacro:property name="optical_center_height"	value="0.0295"/>
+    <xacro:property name="vergence_half_angle"		value="2.5"/>
     <!-- A link representing the gripper and a joint attaching it to parnet -->
     <link name="${prefix}base_link">
       <visual>
-        <origin xyz="0 0 0.0295" rpy="${-pi/2} 0 0"/>
+        <origin xyz="0 0 ${optical_center_height}" rpy="${-pi/2} 0 0"/>
 	<geometry>
           <mesh filename="package://aist_description/devices/meshes/zivid2plus.stl" scale="0.001 0.001 0.001"/>
@@ -17,6 +20,5 @@
       <collision>
       <!-- avoid collision -->
-        <!-- <origin xyz="0.188 -0.035 -0.035" rpy="0 0 ${pi/2}"/> -->
-	<origin xyz="0 0 0" rpy="0 0 0"/>
+        <origin xyz="0 0 ${optical_center_height}" rpy="${-pi/2} 0 0"/>
 	<geometry>
 	  <mesh
@@ -41,5 +43,6 @@
       <parent link="${prefix}base_link"/>
       <child  link="${prefix}sensor"/>
-      <origin xyz="0.05702 0 0.0295" rpy="${-pi/2} 0 ${2.5*pi/180.0}"/>
+      <origin xyz="${baseline_half_length} 0 ${optical_center_height}"
+	      rpy="${-pi/2} 0 ${vergence_half_angle*pi/180.0}"/>
     </joint>
     <link name="${prefix}projector"/>
@@ -47,5 +50,6 @@
       <parent link="${prefix}base_link"/>
       <child  link="${prefix}projector"/>
-      <origin xyz="-0.05702 0 0.0295" rpy="${-pi/2} 0 ${-2.5*pi/180.0}"/>
+      <origin xyz="${-baseline_half_length} 0 ${optical_center_height}"
+	      rpy="${-pi/2} 0 ${-vergence_half_angle*pi/180.0}"/>
     </joint>
   </xacro:macro>

File: aist_description/scenes/urdf/aist_base_scene.urdf.xacro (robot description, xacro)
@@ -85,8 +85,14 @@
     <origin xyz="${b_bot_x} ${b_bot_y} ${bots_z}" rpy="0 0 ${b_bot_theta}"/>
   </joint>
+  <!-- Spawn and attach zivid camera -->
+  <xacro:include filename="$(find aist_description)/devices/urdf/zivid_coupling.urdf.xacro"/>
+  <xacro:zivid_coupling prefix="a_bot_zivid_coupling_" parent="a_bot_flange">
+    <origin xyz="0 0 0" rpy="${pi} 0 0" />
+  </xacro:zivid_coupling>
   <!-- Spawn and attach force sensor -->
   <xacro:include filename="$(find aist_robotiq)/urdf/ft300.urdf.xacro"/>
-  <xacro:ft300 prefix="a_bot_ftsensor_" parent="a_bot_flange">
-    <origin xyz="0 0 0" rpy="${pi} 0 0"/>
+  <xacro:ft300 prefix="a_bot_ftsensor_"
+	       parent="a_bot_zivid_coupling_flange_link">
+    <origin xyz="0 0 0" rpy="0 0 0"/>
   </xacro:ft300>
   <xacro:ft300 prefix="b_bot_ftsensor_" parent="b_bot_flange">
@@ -101,9 +107,9 @@
   </xacro:robotiq_arg2f_coupling>
   <xacro:include filename="$(find aist_robotiq
-			   )/urdf/robotiq_85_gripper.urdf.xacro"/>
-  <xacro:robotiq_85_gripper prefix="a_bot_gripper_"
+			   )/urdf/robotiq_140_gripper.urdf.xacro"/>
+  <xacro:robotiq_140_gripper prefix="a_bot_gripper_"
 			    parent="a_bot_gripper_coupling_flange_link">
     <origin xyz="0 0 0" rpy="0 0 0"/>
-  </xacro:robotiq_85_gripper>
+  </xacro:robotiq_140_gripper>
   <xacro:include filename="$(find aist_description
 			   )/devices/urdf/single_suction_gripper.urdf.xacro"/>

Commit message: Setup handeye calibration for a_bot_zivid

File: aist_description/devices/urdf/zivid2plus.urdf.xacro (robot description, xacro)
@@ -89,9 +89,9 @@
           <cameraName>${name}</cameraName>
           <frameName>${name}_sensor</frameName>
-          <imageTopicName>texture</imageTopicName>
-          <depthImageTopicName>depth_map</depthImageTopicName>
-          <pointCloudTopicName>pointcloud</pointCloudTopicName>
-          <cameraInfoTopicName>camera_info</cameraInfoTopicName>
-          <depthImageCameraInfoTopicName>camera_info</depthImageCameraInfoTopicName>
+          <imageTopicName>color/image_color</imageTopicName>
+          <depthImageTopicName>depth/image</depthImageTopicName>
+          <pointCloudTopicName>points/xyzrgba</pointCloudTopicName>
+          <cameraInfoTopicName>color/camera_info</cameraInfoTopicName>
+          <depthImageCameraInfoTopicName>depth/camera_info</depthImageCameraInfoTopicName>
           <pointCloudCutoff>0.4</pointCloudCutoff>
           <!-- <hackBaseline>0.35</hackBaseline> -->

File: aist_description/scenes/urdf/a_bot_base_scene.urdf.xacro (robot description, xacro)
@@ -64,8 +64,26 @@
     <origin xyz="${a_bot_x} ${a_bot_y} ${bots_z}" rpy="0 0 0"/>
   </joint>
+  <!-- Attach mounter for Zivid2+ camera -->
+  <xacro:include filename="$(find aist_description)/devices/urdf/zivid_coupling.urdf.xacro"/>
+  <xacro:zivid_coupling prefix="a_bot_zivid_coupling_" parent="a_bot_flange">
+    <origin xyz="0 0 0" rpy="${pi} 0 0" />
+  </xacro:zivid_coupling>
+  <!-- Spawn and attach Zivid2+ camera -->
+  <xacro:include filename="$(find aist_description
+			   )/scenes/urdf/load_calibration.urdf.xacro"/>
+  <xacro:load_calibration filename="$(find aist_handeye_calibration
+				    )/calib/a_bot_zivid.yaml"/>
+  <xacro:include filename="$(find aist_description
+			   )/devices/urdf/zivid2plus.urdf.xacro"/>
+  <xacro:zivid2plus name="a_bot_zivid"
+		    parent="a_bot_zivid_coupling_flange_link">
+    <origin xyz="${origin[0]} ${origin[1]} ${origin[2]}"
+    	    rpy="${origin[3]} ${origin[4]} ${origin[5]}"/>
+  </xacro:zivid2plus>
   <!-- Spawn and attach force sensor -->
   <xacro:include filename="$(find aist_robotiq)/urdf/ft300.urdf.xacro"/>
-  <xacro:ft300 prefix="a_bot_ftsensor_" parent="a_bot_flange">
-    <origin xyz="0 0 0" rpy="${pi} 0 0"/>
+  <xacro:ft300 prefix="a_bot_ftsensor_"
+	       parent="a_bot_zivid_coupling_flange_link">
+    <origin xyz="0 0 0" rpy="0 0 0"/>
   </xacro:ft300>
   <!-- Spawn and attach gripper -->
@@ -77,15 +95,9 @@
   </xacro:robotiq_arg2f_coupling>
   <xacro:include filename="$(find aist_robotiq
-			   )/urdf/robotiq_85_gripper.urdf.xacro"/>
-  <xacro:robotiq_85_gripper prefix="a_bot_gripper_"
+			   )/urdf/robotiq_140_gripper.urdf.xacro"/>
+  <xacro:robotiq_140_gripper prefix="a_bot_gripper_"
 			    parent="a_bot_gripper_coupling_flange_link">
     <origin xyz="0 0 0" rpy="0 0 0"/>
-  </xacro:robotiq_85_gripper>
-  <!-- Add RealSense camera -->
-  <xacro:include filename="$(find aist_description
-			   )/devices/urdf/wrist_cameras.urdf.xacro" />
-  <xacro:wrist_cameras prefix="a_bot_"
-		       parent="a_bot_gripper_base_link"
-		       use_nominal_extrinsics="true"/>
+  </xacro:robotiq_140_gripper>
   <!-- I would like to remove the "world" link definition, but apparently it is necessary for Gazebo -->
   <link name="world"/>

File: aist_description/scenes/urdf/aist_base_scene.urdf.xacro (robot description, xacro)
@@ -109,5 +109,5 @@
   </xacro:ft300>
   <xacro:ft300 prefix="b_bot_ftsensor_" parent="b_bot_flange">
-    <origin xyz="0 0 0" rpy="${pi} 0 0"/>
+    <origin xyz="0 0 0" rpy="0 0 0"/>
   </xacro:ft300>
   <!-- Spawn and attach gripper -->
