Commit message: Add rotational componets to offset of target poses

File: aist_description/scenes/urdf/dkhi_base_scene.urdf.xacro (robot description, xacro)
@@ -36,8 +36,20 @@
   </xacro:rs007l>
   <!-- Attach grippers -->
-  <xacro:include filename="$(find toyota1_description)/devices/urdf/magripper.urdf.xacro" />
-  <xacro:magripper3 prefix="a_khi_" parent="a_khi_ee_link">
+  <xacro:include filename="$(find aist_robotiq
+			   )/urdf/robotiq_arg2f_coupling.urdf.xacro"/>
+  <xacro:robotiq_arg2f_coupling prefix="a_khi_gripper_coupling_"
+				parent="a_khi_ee_link">
     <origin xyz="0 0 0" rpy="0 0 0"/>
-  </xacro:magripper3>
+  </xacro:robotiq_arg2f_coupling>
+  <xacro:include filename="$(find aist_description)/devices/urdf/robotiq_85_gripper_with_tip_link.urdf.xacro"/>
+  <xacro:robotiq_85_gripper_with_tip_link prefix="a_khi_gripper_"
+					  parent="a_khi_gripper_coupling_flange_link">
+    <origin xyz="0 0 0" rpy="0 0 0"/>
+  </xacro:robotiq_85_gripper_with_tip_link>
+  <xacro:include filename="$(find aist_description)/devices/urdf/single_suction_gripper.urdf.xacro"/>
+  <xacro:single_suction_gripper prefix="b_khi_gripper_"
+  				parent="b_khi_ee_link">
+    <origin xyz="0 0 0" rpy="0 ${-0.1*pi/180} ${0.15*pi/180}"/>
+  </xacro:single_suction_gripper>
   <gazebo>
     <!-- Required because package robot_controllers is used for

File: aist_description/scenes/urdf/skhi_base_scene.urdf.xacro (robot description, xacro)
@@ -31,8 +31,10 @@
   </xacro:rs007l>
   <!-- Attach grippers -->
-  <xacro:include filename="$(find toyota1_description)/devices/urdf/magripper.urdf.xacro" />
-  <xacro:magripper3 prefix="a_khi_" parent="a_khi_ee_link">
-    <origin xyz="0 0 0" rpy="0 0 0"/>
-  </xacro:magripper3>
+  <xacro:include filename="$(find aist_description
+			   )/devices/urdf/single_suction_gripper.urdf.xacro"/>
+  <xacro:single_suction_gripper prefix="a_khi_gripper_"
+  				parent="a_khi_ee_link">
+    <origin xyz="0 0 0" rpy="0 ${0.2*pi/180} ${-1.2*pi/180}"/>
+  </xacro:single_suction_gripper>
   <gazebo>
     <!-- Required because package robot_controllers is used for
