Commit message: Update mocap scene and mocap_moveit_config according to update of universal_robot

File: aist_description/scenes/urdf/mocap_base_scene.urdf.xacro (robot description, xacro)
@@ -24,15 +24,15 @@
   </joint>
   <!-- robot arms -->
-  <xacro:include filename="$(find ur_e_description)/urdf/common.gazebo.xacro"/>
-  <xacro:include filename="$(find ur_e_description)/urdf/ur5e.urdf.xacro"/>
-  <xacro:ur5e_robot prefix="c_bot_" joint_limited="false"
-    shoulder_pan_lower_limit="${-pi}" shoulder_pan_upper_limit="${pi}"
-    shoulder_lift_lower_limit="${-pi}" shoulder_lift_upper_limit="${pi}"
-    elbow_joint_lower_limit="0.0" elbow_joint_upper_limit="${pi}"
-    wrist_1_lower_limit="${-pi}" wrist_1_upper_limit="${pi}"
-    wrist_2_lower_limit="${-pi}" wrist_2_upper_limit="${pi}"
-    wrist_3_lower_limit="${-pi}" wrist_3_upper_limit="${pi}"
-    kinematics_file="${load_yaml(
-		     '$(find ur_e_description)/config/ur5e_default.yaml')}"/>
+  <xacro:include filename="$(find ur_gazebo)/urdf/ur_macro.xacro"/>
+  <xacro:ur_robot_gazebo
+      prefix="c_bot_"
+      joint_limits_parameters_file="$(find ur_description
+                                    )/config/ur5e/joint_limits.yaml"
+      physical_parameters_file="$(find ur_description
+                                )/config/ur5e/physical_parameters.yaml"
+      visual_parameters_file="$(find ur_description
+                              )/config/ur5e/visual_parameters.yaml"
+      kinematics_parameters_file="$(find aist_bringup
+				  )/config/c_bot_calibration.yaml"/>
   <joint name="ground_c_bot_joint" type="fixed">
     <parent link="ground"/>
@@ -44,6 +44,6 @@
 			   )/urdf/robotiq_arg2f_coupling.urdf.xacro"/>
   <xacro:robotiq_arg2f_coupling prefix="c_bot_gripper_coupling_"
-				parent="c_bot_ee_link">
-    <origin xyz="0 0 0" rpy="0 0 0"/>
+				parent="c_bot_flange">
+    <origin xyz="0 0 0" rpy="${pi} 0 0"/>
   </xacro:robotiq_arg2f_coupling>
   <xacro:include filename="$(find aist_description

Commit message: WIP: Load camera calibration to scene URDF

File: aist_description/scenes/urdf/mocap_base_scene.urdf.xacro (robot description, xacro)
@@ -56,9 +56,17 @@
   <!-- Add RealSense camera -->
   <xacro:include filename="$(find aist_description
+			   )/scenes/urdf/load_calibration.urdf.xacro"/>
+  <xacro:load_calibration directory="$(find aist_handeye_calibration)/calib"
+			  name="realsenseD435"/>
+  <xacro:include filename="$(find aist_description
 			   )/devices/urdf/_d435.urdf.xacro"/>
   <xacro:sensor_d435 name="realsenseD435" parent="workspace_center"
 		     use_nominal_extrinsics="true">
-    <origin xyz="0.0 0.7 0.6"
-	    rpy="${0*pi/180} ${30*pi/180} ${-90*pi/180}"/>
+    <origin xyz="${realsenseD435_origin[0]}
+		 ${realsenseD435_origin[1]}
+		 ${realsenseD435_origin[2]}"
+    	    rpy="${realsenseD435_origin[3]}
+		 ${realsenseD435_origin[4]}
+		 ${realsenseD435_origin[5]}"/>
   </xacro:sensor_d435>
   <!-- I would like to remove the "world" link definition, but apparently it is necessary for Gazebo -->
