Commit message: Rename c_bot to e_bot in nedo_ur5e configuration

File: aist_description/scenes/urdf/nedo_ur5e_base_scene.urdf.xacro (robot description, xacro)
@@ -3,6 +3,6 @@
   <xacro:arg name="scene" default=""/>
   <!-- Calibration help: If the robot is not moving far enough to the calibration point, increase these distances -->
-  <xacro:property name="c_bot_x" value="0"/>
-  <xacro:property name="c_bot_y" value="-0.4875"/>
+  <xacro:property name="e_bot_x" value="0"/>
+  <xacro:property name="e_bot_y" value="-0.4875"/>
   <xacro:property name="bots_z" value="0.77"/>
   <!-- This is the main file defining our robot arrangement and physical environment. -->
@@ -28,5 +28,5 @@
   <xacro:include filename="$(find ur_e_description)/urdf/common.gazebo.xacro"/>
   <xacro:include filename="$(find ur_e_description)/urdf/ur5e.urdf.xacro"/>
-  <xacro:ur5e_robot prefix="c_bot_" joint_limited="false"
+  <xacro:ur5e_robot prefix="e_bot_" joint_limited="false"
     shoulder_pan_lower_limit="${-pi}" shoulder_pan_upper_limit="${pi}"
     shoulder_lift_lower_limit="${-pi}" shoulder_lift_upper_limit="${pi}"
@@ -37,19 +37,19 @@
     kinematics_file="${load_yaml(
 		     '$(find ur_e_description)/config/ur5e_default.yaml')}"/>
-  <joint name="ground_c_bot_joint" type="fixed">
+  <joint name="ground_e_bot_joint" type="fixed">
     <parent link="ground"/>
-    <child  link= "c_bot_base_link"/>
-    <origin xyz="${c_bot_x} ${c_bot_y} ${bots_z}" rpy="0 0 0"/>
+    <child  link= "e_bot_base_link"/>
+    <origin xyz="${e_bot_x} ${e_bot_y} ${bots_z}" rpy="0 0 0"/>
   </joint>
   <!-- Spawn and attach gripper -->
   <xacro:include filename="$(find aist_robotiq
 			   )/urdf/robotiq_arg2f_coupling.urdf.xacro"/>
-  <xacro:robotiq_arg2f_coupling prefix="c_bot_gripper_coupling_"
-				parent="c_bot_ee_link">
+  <xacro:robotiq_arg2f_coupling prefix="e_bot_gripper_coupling_"
+				parent="e_bot_ee_link">
     <origin xyz="0 0 0" rpy="0 0 0"/>
   </xacro:robotiq_arg2f_coupling>
   <xacro:include filename="$(find aist_description)/devices/urdf/robotiq_140_gripper_with_tip_link.urdf.xacro"/>
-  <xacro:robotiq_140_gripper_with_tip_link prefix="c_bot_gripper_"
-					  parent="c_bot_gripper_coupling_flange_link">
+  <xacro:robotiq_140_gripper_with_tip_link prefix="e_bot_gripper_"
+					  parent="e_bot_gripper_coupling_flange_link">
     <origin xyz="0 0 0" rpy="0 0 0"/>
   </xacro:robotiq_140_gripper_with_tip_link>

Commit message: add nedo_ur5e_moveit_config

File: aist_description/scenes/urdf/nedo_ur5e_base_scene.urdf.xacro (robot description, xacro)
@@ -4,5 +4,5 @@
   <!-- Calibration help: If the robot is not moving far enough to the calibration point, increase these distances -->
   <xacro:property name="e_bot_x" value="0"/>
-  <xacro:property name="e_bot_y" value="-0.4875"/>
+  <xacro:property name="e_bot_y" value="-0.93"/>
   <xacro:property name="bots_z" value="0.77"/>
   <!-- This is the main file defining our robot arrangement and physical environment. -->
@@ -11,6 +11,6 @@
   <link name="ground"/>
   <xacro:include filename="$(find aist_description)/objects/urdf/aist_box.urdf.xacro"/>
-  <xacro:property name="table_w" value="0.9"/>
-  <xacro:property name="table_l" value="0.75"/>
+  <xacro:property name="table_w" value="1.00"/>
+  <xacro:property name="table_l" value="0.70"/>
   <xacro:property name="table_h" value="0.01"/>
   <xacro:aist_box name="workbox"
