Commit message: WIP: Use IK solver for pose_head_tracker

File: aist_description/scenes/urdf/a_bot_calibration.urdf.xacro (robot description, xacro)
@@ -13,5 +13,5 @@
 			marker_id="32"
 			thickness="0.001">
-    <origin xyz="0.0 0.0 0.100" rpy="0 0 0"/>
+    <origin xyz="-0.1 -0.2 0.3" rpy="0 0 0"/>
   </xacro:ar_marker_70_5>
 </robot>

Commit message: Confirmed that pose_head_tracker works with UE5 under gazebo

File: aist_description/scenes/urdf/a_bot_calibration.urdf.xacro (robot description, xacro)
@@ -3,15 +3,9 @@
   <!-- Add AR markers -->
   <xacro:include filename="$(find aist_description)/objects/urdf/ar_markers.urdf.xacro"/>
-  <!-- <xacro:ar_marker_70_5 prefix="a_bot_" -->
-  <!-- 			parent="a_bot_gripper_tip_link" -->
-  <!-- 			marker_id="26" -->
-  <!-- 			thickness="0.005"> -->
-  <!--   <origin xyz="0.0 0.0 0.0185" rpy="0 0 0"/> -->
-  <!-- </xacro:ar_marker_70_5> -->
   <xacro:ar_marker_70_5 prefix="workspace_"
 			parent="workspace_center"
 			marker_id="32"
 			thickness="0.001">
-    <origin xyz="-0.1 -0.2 0.3" rpy="0 0 0"/>
+    <origin xyz="-0.1 -0.2 0.05" rpy="0 0 ${pi/2}"/>
   </xacro:ar_marker_70_5>
 </robot>

Commit message: Add common interactive stuffs to AISTBaseRoutines

File: aist_description/scenes/urdf/a_bot_calibration.urdf.xacro (robot description, xacro)
@@ -3,9 +3,9 @@
   <!-- Add AR markers -->
   <xacro:include filename="$(find aist_description)/objects/urdf/ar_markers.urdf.xacro"/>
-  <xacro:ar_marker_70_5 prefix="workspace_"
+  <xacro:ar_marker_150_5 prefix="workspace_"
 			parent="workspace_center"
-			marker_id="32"
+  			marker_id="17_26_32_256"
 			thickness="0.001">
-    <origin xyz="-0.1 -0.2 0.05" rpy="0 0 ${pi/2}"/>
-  </xacro:ar_marker_70_5>
+    <origin xyz="0.0 0.0 0.0005" rpy="0 0 0"/>
+  </xacro:ar_marker_150_5>
 </robot>
