Commit message: Update fvision configuration

File: aist_description/scenes/urdf/fvision_base_scene.urdf.xacro (robot description, xacro)
@@ -27,15 +27,15 @@
   </joint>
   <!-- robot arms -->
-  <xacro:include filename="$(find ur_e_description)/urdf/common.gazebo.xacro"/>
-  <xacro:include filename="$(find ur_e_description)/urdf/ur5e.urdf.xacro"/>
-  <xacro:ur5e_robot prefix="d_bot_" joint_limited="false"
-    shoulder_pan_lower_limit="${-pi}" shoulder_pan_upper_limit="${pi}"
-    shoulder_lift_lower_limit="${-pi}" shoulder_lift_upper_limit="${pi}"
-    elbow_joint_lower_limit="0.0" elbow_joint_upper_limit="${pi}"
-    wrist_1_lower_limit="${-pi}" wrist_1_upper_limit="${pi}"
-    wrist_2_lower_limit="${-pi}" wrist_2_upper_limit="${pi}"
-    wrist_3_lower_limit="${-pi}" wrist_3_upper_limit="${pi}"
-    kinematics_file="${load_yaml(
-		     '$(find ur_e_description)/config/ur5e_default.yaml')}"/>
+  <xacro:include filename="$(find ur_gazebo)/urdf/ur_macro.xacro"/>
+  <xacro:ur_robot_gazebo
+      prefix="d_bot_"
+      joint_limits_parameters_file="$(find ur_description
+                                    )/config/ur5e/joint_limits.yaml"
+      physical_parameters_file="$(find ur_description
+                                )/config/ur5e/physical_parameters.yaml"
+      visual_parameters_file="$(find ur_description
+                              )/config/ur5e/visual_parameters.yaml"
+      kinematics_parameters_file="$(find aist_bringup
+				  )/config/d_bot_calibration.yaml"/>
   <joint name="ground_d_bot_joint" type="fixed">
     <parent link="ground"/>
@@ -47,6 +47,6 @@
 			   )/urdf/robotiq_arg2f_coupling.urdf.xacro"/>
   <xacro:robotiq_arg2f_coupling prefix="d_bot_gripper_coupling_"
-				parent="d_bot_ee_link">
-    <origin xyz="0 0 0" rpy="0 0 0"/>
+				parent="d_bot_flange">
+    <origin xyz="0 0 0" rpy="${pi} 0 0"/>
   </xacro:robotiq_arg2f_coupling>
   <xacro:include filename="$(find aist_description)/devices/urdf/robotiq_140_gripper_with_tip_link.urdf.xacro"/>

Commit message: Calibrate d_phoxi_m_camera

File: aist_description/scenes/urdf/fvision_base_scene.urdf.xacro (robot description, xacro)
@@ -55,4 +55,15 @@
     <origin xyz="0 0 0" rpy="0 0 0"/>
   </xacro:robotiq_140_gripper_with_tip_link>
+  <!-- Add PhoXi 3D scanner -->
+  <xacro:include filename="$(find
+			   aist_phoxi_camera)/urdf/phoxi_m_camera.urdf.xacro"/>
+  <xacro:phoxi_m_camera prefix="d_phoxi_m_" parent="workspace_center">
+    <origin xyz="-0.0149511700982
+		 -0.483543436025
+		 0.633792706454"
+	    rpy="${-152.286950706*pi/180}
+		 ${-2.00315281361*pi/180}
+		 ${0*pi/180}"/>
+  </xacro:phoxi_m_camera>
   <!-- Add RealSense camera -->
   <xacro:include filename="$(find aist_description

Commit message: Make fivision dual gripper configuration

File: aist_description/scenes/urdf/fvision_base_scene.urdf.xacro (robot description, xacro)
@@ -46,14 +46,29 @@
   <!-- Spawn and attach gripper -->
   <xacro:include filename="$(find aist_robotiq
+			   )/urdf/robotiq_dual_bracket.urdf.xacro"/>
+  <xacro:robotiq_dual_bracket prefix="d_bot_dual_bracket_"
+			      parent="d_bot_flange">
+    <origin xyz="0 0 0" rpy="${pi} 0 0"/>
+  </xacro:robotiq_dual_bracket>
+  <xacro:include filename="$(find aist_robotiq
 			   )/urdf/robotiq_arg2f_coupling.urdf.xacro"/>
-  <xacro:robotiq_arg2f_coupling prefix="d_bot_gripper_coupling_"
-				parent="d_bot_flange">
-    <origin xyz="0 0 0" rpy="${pi} 0 0"/>
+  <xacro:robotiq_arg2f_coupling prefix="d_bot_left_coupling_"
+				parent="d_bot_dual_bracket_left_flange_link">
+    <origin xyz="0 0 0" rpy="0 0 0"/>
   </xacro:robotiq_arg2f_coupling>
   <xacro:include filename="$(find aist_description)/devices/urdf/robotiq_140_gripper_with_tip_link.urdf.xacro"/>
   <xacro:robotiq_140_gripper_with_tip_link prefix="d_bot_gripper_"
-					   parent="d_bot_gripper_coupling_flange_link">
+					   parent="d_bot_left_coupling_flange_link">
     <origin xyz="0 0 0" rpy="0 0 0"/>
   </xacro:robotiq_140_gripper_with_tip_link>
+  <xacro:robotiq_arg2f_coupling prefix="d_bot_right_coupling_"
+				parent="d_bot_dual_bracket_right_flange_link">
+    <origin xyz="0 0 0" rpy="0 0 0"/>
+  </xacro:robotiq_arg2f_coupling>
+  <xacro:include filename="$(find aist_robotiq)/urdf/robotiq_epick.urdf.xacro"/>
+  <xacro:robotiq_epick prefix="d_bot_suction_"
+		       parent="d_bot_right_coupling_flange_link">
+    <origin xyz="0 0 0" rpy="0 0 0"/>
+  </xacro:robotiq_epick>
   <!-- Add PhoXi 3D scanner -->
   <xacro:include filename="$(find

Commit message: Fixed orientation of tip links of fastening tools and precision gripper

File: aist_description/scenes/urdf/fvision_base_scene.urdf.xacro (robot description, xacro)
@@ -70,5 +70,6 @@
 			   )/urdf/robotiq_epick.urdf.xacro"/>
   <xacro:robotiq_epick prefix="d_bot_suction_"
-		       parent="d_bot_right_coupling_flange_link">
+		       parent="d_bot_right_coupling_flange_link"
+		       plunger_radius="0.005" plunger_length="0.050">
     <origin xyz="0 0 0" rpy="0 0 0"/>
   </xacro:robotiq_epick>
@@ -77,10 +78,6 @@
 			   aist_phoxi_camera)/urdf/phoxi_m_camera.urdf.xacro"/>
   <xacro:phoxi_m_camera name="d_phoxi_m_camera" parent="workspace_center">
-    <origin xyz="-0.0149511700982
-		 -0.483543436025
-		 0.633792706454"
-	    rpy="${-152.286950706*pi/180}
-		 ${-2.00315281361*pi/180}
-		 ${0*pi/180}"/>
+    <origin xyz="-0.0149511700982 -0.483543436025 0.633792706454"
+	    rpy="0.0 1.043 1.5708"/>
   </xacro:phoxi_m_camera>
   <!-- Add RealSense camera -->
@@ -90,4 +87,7 @@
 		      use_nominal_extrinsics="true">
     <origin xyz="0.030 0.000 0.043" rpy="0 ${0.0*pi/180.0} 0" />
+-
+- 1.0432812514428629
+- 3.014328066314531
   </xacro:sensor_sr305>
   <!-- I would like to remove the "world" link definition, but apparently it is necessary for Gazebo -->

File: aist_fastening_tools/urdf/screw_tool_m3.urdf.xacro (robot description, xacro)
@@ -38,5 +38,5 @@
       <parent link="${prefix}base_link"/>
       <child  link="${prefix}tip_link"/>
-      <origin xyz="0.100 0 0" rpy="0 0 0"/>
+      <origin xyz="0.100 0 0" rpy="0 ${-pi/2} 0"/>
     </joint>
   </xacro:macro>

File: aist_fastening_tools/urdf/screw_tool_m4.urdf.xacro (robot description, xacro)
@@ -38,5 +38,5 @@
       <parent link="${prefix}base_link"/>
       <child  link="${prefix}tip_link"/>
-      <origin xyz="0.120 0 0" rpy="0 0 0"/>
+      <origin xyz="0.120 0 0" rpy="0 ${-pi/2} 0"/>
     </joint>
   </xacro:macro>

File: aist_precision_gripper/urdf/precision_gripper.urdf.xacro (robot description, xacro)
@@ -62,5 +62,5 @@
       <!-- <origin rpy="0.0 ${-pi/2} 0.0" xyz="0.001 -0.008 .162"/> -->
       <!-- <origin rpy="0 0 0" xyz="0.162 -0.008 -0.001"/> -->
-      <origin rpy="0 0 0" xyz="0.160 0.016 0.000"/>
+      <origin rpy="0 ${-pi/2} 0" xyz="0.160 0.016 0.000"/>
       <!-- +y is the same, +x in the new frame is +z in the parent, +z is -x in the parent? -->
     </joint>

File: aist_robotiq/urdf/robotiq_epick.urdf.xacro (robot description, xacro)
@@ -1,5 +1,8 @@
 <?xml version="1.0"?>
 <robot xmlns:xacro="http://ros.org/wiki/xacro">
-  <xacro:macro name="robotiq_epick" params="prefix parent *origin">
+  <xacro:macro name="robotiq_epick" params="prefix parent
+					    plunger_radius:=0
+					    plunger_length:=0
+					    *origin">
     <xacro:property name="epick_length" value="0.101"/>
     <xacro:property name="epick_offset" value="-0.006"/>
@@ -44,4 +47,40 @@
       <origin xyz="${epick_length} 0 0" rpy="0 0 0"/>
     </joint>
+    <xacro:if value="${plunger_length > 0}">
+      <link name="${prefix}plunger_link">
+	<inertial>
+    	  <origin xyz="0 0 0" rpy="0 0 0"/>
+    	  <mass value="0.100"/>
+    	  <inertia ixx="0.0045" ixy="0" ixz="0"
+		   iyy="0.0045"  iyz="0" izz="0.005"/>
+	</inertial>
+	<visual>
+    	  <origin xyz="${plunger_length/2} 0 0" rpy="0 ${pi/2} 0"/>
+    	  <geometry>
+	    <cylinder radius="${plunger_radius}" length="${plunger_length}"/>
+    	  </geometry>
+          <material name="Grey">
+            <color rgba="0.7 0.7 0.7 1.0"/>
+          </material>
+	</visual>
+	<collision>
+    	  <origin xyz="${plunger_length/2} 0 0" rpy="0 ${pi/2} 0"/>
+    	  <geometry>
+	    <cylinder radius="${plunger_radius}" length="${plunger_length}"/>
+    	  </geometry>
+	</collision>
+      </link>
+      <joint name="${prefix}plunger_joint" type="fixed">
+	<parent link="${prefix}flange_link"/>
+	<child  link="${prefix}plunger_link"/>
+	<origin xyz="0 0 0" rpy="0 0 0"/>
+      </joint>
+      <link name="${prefix}tip_link"/>
+      <joint name="${prefix}tip_joint" type="fixed">
+	<parent link="${prefix}plunger_link"/>
+	<child  link="${prefix}tip_link"/>
+	<origin xyz="${plunger_length} 0 0" rpy="0 ${-pi/2} 0"/>
+      </joint>
+    </xacro:if>
   </xacro:macro>
 </robot>
