Commit message: Add a new marker_map

File: aist_description/scenes/urdf/fvision_calibration.urdf.xacro (robot description, xacro)
@@ -3,14 +3,14 @@
   <!-- Add AR markers -->
   <xacro:include filename="$(find aist_aruco_ros)/urdf/ar_marker.urdf.xacro"/>
-  <!-- <xacro:ar_marker prefix="d_bot_" -->
-  <!-- 		   parent="d_bot_gripper_base_link" -->
-  <!-- 		   marker_id="26" -->
-  <!-- 		   width="0.070" height="0.070" margin="0.005" -->
-  <!-- 		   thickness="0.005"> -->
-  <!--   <origin xyz="0.180 0.0 0.0215" rpy="0 0 ${pi/2}"/> -->
-  <!-- </xacro:ar_marker> -->
+  <xacro:ar_marker prefix="d_bot_"
+		   parent="d_bot_gripper_base_link"
+		   marker_id="26"
+		   width="0.070" height="0.070" margin="0.005"
+		   thickness="0.005">
+    <origin xyz="0.180 0.0 0.0215" rpy="0 0 ${pi/2}"/>
+  </xacro:ar_marker>
   <xacro:ar_marker prefix="workspace_"
 		   parent="workspace_center"
-		   marker_id="17_26_32_256"
+		   marker_id="100_101_102_103"
 		   width="0.150" height="0.150" margin="0.005"
 		   thickness="0.001">
