Commit message: Update moveit_config according to camera/tool calibration

File: aist_description/scenes/urdf/b_bot_base_scene.urdf.xacro (robot description, xacro)
@@ -96,5 +96,5 @@
   				parent="b_bot_ftsensor_flange_link">
     <!-- <origin xyz="0 0 0" rpy="0 ${0.2*pi/180} ${-1.2*pi/180}"/> -->
-    <origin xyz="0 0 0" rpy="0 ${0.7*pi/180} ${-0.1*pi/180}"/>
+    <origin xyz="0 0 0" rpy="0 ${0.3*pi/180} ${0.2*pi/180}"/>
   </xacro:single_suction_gripper>
   <!-- Add PhoXi 3D scanner -->
