Commit message: Make pcd and ply files ignored by git

File: aist_description/scenes/urdf/kitting.urdf.xacro (robot description, xacro)
@@ -4,4 +4,6 @@
   <xacro:property name="plate_l" value="0.42"/>
   <xacro:property name="plate_h" value="0.015"/>
+  <xacro:property name="marker_x" value="0.25"/>
+  <xacro:property name="marker_y" value="0.27"/>
   <!-- front plate -->
   <xacro:include filename="$(find aist_description)/objects/urdf/aist_box.urdf.xacro"/>
@@ -110,3 +112,14 @@
 	    rpy="0 0 ${pi/2}"/>
   </xacro:kitting_tray_2>
+  <!-- AR marker for localizing WEB camera -->
+  <xacro:include filename="$(find aist_description
+  			   )/objects/urdf/ar_markers.urdf.xacro"/>
+  <xacro:ar_marker prefix="workspace_"
+  		   parent="workspace_center"
+  		   marker_id="32"
+  		   size="0.0475"
+  		   margin="0.02625"
+  		   thickness="0.003">
+    <origin xyz="${marker_x} ${marker_y} 0.0003" rpy="0 0 ${pi/2}"/>
+  </xacro:ar_marker>
 </robot>

Commit message: Change size and place of AR marker for HMI demo

File: aist_description/scenes/urdf/kitting.urdf.xacro (robot description, xacro)
@@ -4,6 +4,6 @@
   <xacro:property name="plate_l" value="0.42"/>
   <xacro:property name="plate_h" value="0.015"/>
-  <xacro:property name="marker_x" value="0.25"/>
-  <xacro:property name="marker_y" value="0.27"/>
+  <xacro:property name="marker_x" value="0.181"/>
+  <xacro:property name="marker_y" value="0.310"/>
   <!-- front plate -->
   <xacro:include filename="$(find aist_description)/objects/urdf/aist_box.urdf.xacro"/>
@@ -118,6 +118,6 @@
   		   parent="workspace_center"
   		   marker_id="32"
-  		   size="0.0475"
-  		   margin="0.02625"
+  		   size="0.095"
+  		   margin="0.0525"
   		   thickness="0.003">
     <origin xyz="${marker_x} ${marker_y} 0.0003" rpy="0 0 ${pi/2}"/>

Commit message: Change configuration of trays and bins in kitting scene

File: aist_description/scenes/urdf/kitting.urdf.xacro (robot description, xacro)
@@ -1,9 +1,7 @@
 <?xml version="1.0"?>
 <robot xmlns:xacro="http://wiki.ros.org/xacro" name="kitting">
-  <xacro:property name="plate_w" value="0.68"/>
-  <xacro:property name="plate_l" value="0.42"/>
+  <xacro:property name="plate_w" value="0.42"/>
+  <xacro:property name="plate_l" value="0.68"/>
   <xacro:property name="plate_h" value="0.015"/>
-  <xacro:property name="marker_x" value="0.181"/>
-  <xacro:property name="marker_y" value="0.310"/>
   <!-- front plate -->
   <xacro:include filename="$(find aist_description)/objects/urdf/aist_box.urdf.xacro"/>
@@ -13,15 +11,16 @@
 		  height="${plate_h}"
 		  parent="workspace_center">
-    <origin xyz="${table_w/2 - plate_w - 0.14} ${-plate_l/2} 0"
-	    rpy="0 0 0"/>
+    <origin xyz="-0.062 ${-plate_l/2} 0" rpy="0 0 0"/>
   </xacro:aist_box>
-  <link name="plate_center"/>
-  <joint name="plate_to_plate_center" type="fixed">
+  <link name="plate_upper_left_corner"/>
+  <joint name="plate_corner_joint" type="fixed">
     <parent link="plate"/>
-    <child  link="plate_center"/>
-    <origin xyz="${plate_w/2} ${plate_l/2} ${plate_h}" rpy="0 0 0"/>
+    <child  link="plate_upper_left_corner"/>
+    <origin xyz="0 0 ${plate_h}" rpy="0 0 0"/>
   </joint>
-  <xacro:include filename="$(find aist_description)/wrc/urdf/kitting_bins.urdf.xacro"/>
-  <xacro:include filename="$(find aist_description)/wrc/urdf/kitting_trays.urdf.xacro"/>
+  <xacro:include filename="$(find aist_description
+			   )/wrc/urdf/kitting_bins.urdf.xacro"/>
+  <xacro:include filename="$(find aist_description
+			   )/wrc/urdf/kitting_trays.urdf.xacro"/>
   <!-- bin_1_definition -->
   <xacro:property name="bin_1_width"		value="0.125"/>
@@ -36,88 +35,62 @@
   <xacro:property name="bin_3_length"		value="0.285"/>
   <xacro:property name="z_origin_offset_3"	value="-.004"/>
-  <!-- A row of bin1 -->
-  <xacro:property name="set1_x"	value="0"/>
-  <xacro:property name="set1_y" value="0.096"/>
-  <xacro:property name="set1_z" value="0"/>
-  <!-- A row of bin2 -->
-  <xacro:property name="set2_x" value="0.25"/>
-  <xacro:property name="set2_y" value="0.096"/>
-  <xacro:property name="set2_z" value="0"/>
-  <!--bin_1_part_15_-->
+  <!-- Common coordinates of bin_1, bin_2 and tray -->
+  <xacro:property name="tray_x"		value="${tray_width}"/>
+  <xacro:property name="tray_y"		value="0"/>
+  <xacro:property name="bin_2_x"	value="${tray_x - bin_2_length/2}"/>
+  <xacro:property name="bin_1_x"
+		  value="${bin_2_x + bin_2_length/2 + bin_1_length/2}"/>
+  <xacro:property name="bin_y"
+		  value="${tray_y + tray_length + 1.5*bin_2_width}"/>
+  <!--bin_1_part_5_-->
   <xacro:kitting_bin_1 binname	      ="bin_1_part_5"
-		       parent	      ="plate_center"
+		       parent	      ="plate_upper_left_corner"
 		       z_origin_offset="${z_origin_offset_1}">
-    <origin xyz="${plate_w/2 - bin_1_length/2}
-		 ${bin_1_width}
-		 ${-z_origin_offset_1}"
+    <origin xyz="${bin_1_x} ${bin_y + bin_1_width} ${-z_origin_offset_1}"
 	    rpy="0 0 0"/>
   </xacro:kitting_bin_1>
   <!--bin_1_part_16_-->
   <xacro:kitting_bin_1 binname	      ="bin_1_part_16"
-		       parent	      ="plate_center"
+		       parent	      ="plate_upper_left_corner"
 		       z_origin_offset="${z_origin_offset_1}">
-    <origin xyz="${plate_w/2 - bin_1_length/2}
-		 0
-		 ${-z_origin_offset_1}"
+    <origin xyz="${bin_1_x} ${bin_y} ${-z_origin_offset_1}"
 	    rpy="0 0 0"/>
   </xacro:kitting_bin_1>
   <!--bin_1_part_17_-->
   <xacro:kitting_bin_1 binname	      ="bin_1_part_17"
-  		       parent	      ="plate_center"
+  		       parent	      ="plate_upper_left_corner"
   		       z_origin_offset="${z_origin_offset_1}">
-    <origin xyz="${plate_w/2 - bin_1_length/2}
-		 ${-bin_1_width}
-		 ${-z_origin_offset_1}"
+    <origin xyz="${bin_1_x} ${bin_y - bin_1_width} ${-z_origin_offset_1}"
 	    rpy="0 0 0"/>
   </xacro:kitting_bin_1>
   <!-- bin_2_part_4_ -->
   <xacro:kitting_bin_2 binname	      ="bin_2_part_4"
-		       parent	      ="plate_center"
+		       parent	      ="plate_upper_left_corner"
 		       z_origin_offset="${z_origin_offset_2}">
-    <origin xyz="${plate_w/2 - bin_1_length - bin_2_length/2}
-		 ${bin_2_width}
-		 ${-z_origin_offset_2}"
+    <origin xyz="${bin_2_x} ${bin_y + bin_2_width} ${-z_origin_offset_2}"
 	    rpy="0 0 0"/>
   </xacro:kitting_bin_2>
   <!--bin_2_part_7_-->
   <xacro:kitting_bin_2 binname	      ="bin_2_part_7"
-		       parent	      ="plate_center"
+		       parent	      ="plate_upper_left_corner"
 		       z_origin_offset="${z_origin_offset_2}">
-    <origin xyz="${plate_w/2 - bin_1_length - bin_2_length/2}
-		 0
-		 ${-z_origin_offset_2}"
+    <origin xyz="${bin_2_x} ${bin_y} ${-z_origin_offset_2}"
 	    rpy="0 0 0"/>
   </xacro:kitting_bin_2>
   <!--bin_2_part_8_-->
   <xacro:kitting_bin_2 binname	      ="bin_2_part_8"
-  		       parent	      ="plate_center"
+  		       parent	      ="plate_upper_left_corner"
   		       z_origin_offset="${z_origin_offset_2}">
-    <origin xyz="${plate_w/2 - bin_1_length - bin_2_length/2}
-		 ${-bin_2_width}
-		 ${-z_origin_offset_2}"
+    <origin xyz="${bin_2_x} ${bin_y - bin_2_width} ${-z_origin_offset_2}"
 	    rpy="0 0 0"/>
   </xacro:kitting_bin_2>
   <!-- tray_1 -->
-  <xacro:kitting_tray_1 trayname="tray_1" parent="plate_center">
-    <origin xyz="${plate_w/2 - bin_1_length - bin_2_length - tray_width}
-		 ${tray_length}
-		 0"
-	    rpy="0 0 ${-pi/2}"/>
-  </xacro:kitting_tray_1>
+  <!-- <xacro:kitting_tray_1 trayname="tray_1" parent="plate_upper_left_corner"> -->
+  <!--   <origin xyz="${tray_x - tray_width} ${bin_y + tray_y} 0" -->
+  <!-- 	    rpy="0 0 ${-pi/2}"/> -->
+  <!-- </xacro:kitting_tray_1> -->
   <!-- tray_2 -->
-  <xacro:kitting_tray_2 trayname="tray_2" parent="plate_center">
-    <origin xyz="${plate_w/2 - bin_1_length - bin_2_length}
-		 ${-tray_length}
-		 0"
-	    rpy="0 0 ${pi/2}"/>
+  <xacro:kitting_tray_2 trayname="tray_2" parent="plate_upper_left_corner">
+    <origin xyz="${tray_x} ${tray_y} 0" rpy="0 0 ${pi/2}"/>
   </xacro:kitting_tray_2>
-  <!-- AR marker for localizing WEB camera -->
-  <!-- <xacro:include filename="$(find aist_aruco_ros)/urdf/ar_marker.urdf.xacro"/> -->
-  <!-- <xacro:ar_marker prefix="workspace_" -->
-  <!-- 		   parent="workspace_center" -->
-  <!-- 		   marker_id="32" -->
-  <!-- 		   width="0.095" height="0.095" margin="0.0525" -->
-  <!-- 		   thickness="0.003"> -->
-  <!--   <origin xyz="${marker_x} ${marker_y} 0.0003" rpy="0 0 ${pi/2}"/> -->
-  <!-- </xacro:ar_marker> -->
 </robot>
