Commit message: Fixed orientation of b_bot_marker_frame

File: aist_description/scenes/urdf/calibration.urdf.xacro (robot description, xacro)
@@ -8,5 +8,5 @@
   			marker_id="26"
 			thickness="0.005">
-    <origin xyz="0.063 0.0 0.0215" rpy="0 0 0"/>
+    <origin xyz="0.063 0.0 0.0215" rpy="0 0 ${pi/2}"/>
   </xacro:ar_marker_70_5>
   <xacro:ar_marker_150_5 prefix="workspace_"

Commit message: Move urdf and gazebo material of AR markers to aist_aruco_ros

File: aist_description/scenes/urdf/calibration.urdf.xacro (robot description, xacro)
@@ -2,17 +2,25 @@
 <robot xmlns:xacro="http://wiki.ros.org/xacro" name="calibration">
   <!-- Add AR markers -->
-  <xacro:include filename="$(find aist_description
-			   )/objects/urdf/ar_markers.urdf.xacro"/>
-  <xacro:ar_marker_70_5 prefix="b_bot_"
-  			parent="b_bot_gripper_base_link"
-  			marker_id="26"
-			thickness="0.005">
+  <xacro:include filename="$(find aist_aruco_ros)/urdf/ar_marker.urdf.xacro"/>
+  <xacro:ar_marker prefix="b_bot_"
+  		   parent="b_bot_gripper_base_link"
+  		   marker_id="26"
+		   width="0.070" height="0.070" margin="0.005"
+		   thickness="0.005">
     <origin xyz="0.063 0.0 0.0215" rpy="0 0 ${pi/2}"/>
-  </xacro:ar_marker_70_5>
-  <xacro:ar_marker_150_5 prefix="workspace_"
-			 parent="workspace_center"
-  			 marker_id="17_26_32_256"
-			 thickness="0.001">
+  </xacro:ar_marker>
+  <xacro:ar_marker prefix="workspace_"
+		   parent="workspace_center"
+		   marker_id="17_26_32_256"
+		   width="0.150" height="0.150" margin="0.005"
+		   thickness="0.001">
     <origin xyz="0.0 0.0 0.0005" rpy="0 0 0"/>
-  </xacro:ar_marker_150_5>
+  </xacro:ar_marker>
+  <!-- <xacro:ar_marker prefix="workspace_" -->
+  <!-- 		   parent="workspace_center" -->
+  <!-- 		   marker_id="6x4" -->
+  <!-- 		   width="0.246" height="0.162" margin="0.006" -->
+  <!-- 		   thickness="0.001"> -->
+  <!--   <origin xyz="0.0 0.0 0.0005" rpy="0 0 0"/> -->
+  <!-- </xacro:ar_marker> -->
 </robot>

File: aist_description/scenes/urdf/dur5e_base_scene.urdf.xacro (robot description, xacro)
@@ -63,6 +63,6 @@
 			   )/urdf/robotiq_arg2f_coupling.urdf.xacro"/>
   <xacro:robotiq_arg2f_coupling prefix="c_bot_gripper_coupling_"
-				parent="c_bot_ee_link">
-    <origin xyz="0 0 0" rpy="0 0 0"/>
+				parent="c_bot_flange">
+    <origin xyz="0 0 0" rpy="${pi} 0 0"/>
   </xacro:robotiq_arg2f_coupling>
   <xacro:include filename="$(find aist_robotiq
@@ -86,12 +86,13 @@
   <!-- </xacro:robotiq_85_gripper_with_tip_link> -->
   <xacro:robotiq_arg2f_coupling prefix="d_bot_gripper_coupling_"
-				parent="d_bot_ee_link">
+				parent="d_bot_falnge">
+    <origin xyz="0 0 0" rpy="${pi} 0 0"/>
+  </xacro:robotiq_arg2f_coupling>
+  <xacro:include filename="$(find aist_robotiq
+			   )/urdf/robotiq_hande_gripper.urdf.xacro"/>
+  <xacro:robotiq_hande_gripper prefix="d_bot_gripper_"
+			       parent="d_bot_gripper_coupling_flange_link">
     <origin xyz="0 0 0" rpy="0 0 0"/>
-  </xacro:robotiq_arg2f_coupling>
-  <xacro:include filename="$(find aist_description)/devices/urdf/robotiq_hande_gripper_with_tip_link.urdf.xacro"/>
-  <xacro:robotiq_hande_gripper_with_tip_link prefix="d_bot_gripper_"
-					     parent="d_bot_gripper_coupling_flange_link">
-    <origin xyz="0 0 0" rpy="0 0 0"/>
-  </xacro:robotiq_hande_gripper_with_tip_link>
+  </xacro:robotiq_hande_gripper>
   <!-- Add PhoXi 3D scanner -->
   <xacro:include filename="$(find aist_phoxi_camera)/urdf/phoxi_m_camera.urdf.xacro"/>

File: aist_description/scenes/urdf/dur5e_calibration.urdf.xacro (robot description, xacro)
@@ -3,16 +3,18 @@
   <xacro:include filename="$(find aist_description)/scenes/urdf/dur5e_base_scene.urdf.xacro"/>
   <!-- Add AR markers -->
-  <xacro:include filename="$(find aist_description)/objects/urdf/ar_markers.urdf.xacro"/>
-  <xacro:ar_marker_70_5 prefix="c_bot_"
-			parent="c_bot_robotiq_85_tip_link"
-			marker_id="26"
-			thickness="0.005">
+  <xacro:include filename="$(find aruco_ros)/urdf/ar_marker.urdf.xacro"/>
+  <xacro:ar_marker prefix="c_bot_"
+		   parent="c_bot_robotiq_85_tip_link"
+		   marker_id="26"
+		   width="0.070" height="0.070" margin="0.005"
+		   thickness="0.005">
     <origin xyz="0.0 0.0 0.0185" rpy="0 0 0"/>
-  </xacro:ar_marker_70_5>
-  <xacro:ar_marker_70_5 prefix="d_bot_"
-  			parent="d_bot_dual_suction_gripper_base_link"
-  			marker_id="26"
-			thickness="0.005">
+  </xacro:ar_marker>
+  <xacro:ar_marker prefix="d_bot_"
+  		   parent="d_bot_dual_suction_gripper_base_link"
+  		   marker_id="26"
+		   width="0.070" height="0.070" margin="0.005"
+		   thickness="0.005">
     <origin xyz="0.063 0.0 0.0215" rpy="0 0 0"/>
-  </xacro:ar_marker_70_5>
+  </xacro:ar_marker>
 </robot>

File: aist_description/scenes/urdf/f_bot_calibration.urdf.xacro (robot description, xacro)
@@ -1,11 +1,11 @@
 <?xml version="1.0"?>
 <robot xmlns:xacro="http://wiki.ros.org/xacro" name="f_bot_calibration">
-  <xacro:include filename="$(find aist_description
-			   )/objects/urdf/ar_markers.urdf.xacro"/>
-  <xacro:ar_marker_150_5 prefix="workspace_"
-			 parent="workspace_center"
-  			 marker_id="17_26_32_256"
-			 thickness="0.001">
+  <xacro:include filename="$(find aist_aruco_ros)/urdf/ar_marker.urdf.xacro"/>
+  <xacro:ar_marker prefix="workspace_"
+		   parent="workspace_center"
+		   marker_id="17_26_32_256"
+		   width="0.150" height="0.150" margin="0.005"
+		   thickness="0.001">
     <origin xyz="0.0 0.0 0.0005" rpy="0 0 0"/>
-  </xacro:ar_marker_150_5>
+  </xacro:ar_marker>
 </robot>

File: aist_description/scenes/urdf/fvision_calibration.urdf.xacro (robot description, xacro)
@@ -2,10 +2,18 @@
 <robot xmlns:xacro="http://wiki.ros.org/xacro" name="fvision_calibration">
   <!-- Add AR markers -->
-  <xacro:include filename="$(find aist_description)/objects/urdf/ar_markers.urdf.xacro"/>
-  <xacro:ar_marker_70_5 prefix="workspace_"
-			parent="workspace_center"
-			marker_id="26"
-			thickness="0.001">
+  <xacro:include filename="$(find aist_aruco_ros)/urdf/ar_marker.urdf.xacro"/>
+  <xacro:ar_marker prefix="d_bot_"
+  		   parent="d_bot_gripper_base_link"
+  		   marker_id="26"
+		   width="0.070" height="0.070" margin="0.005"
+		   thickness="0.005">
+    <origin xyz="0.180 0.0 0.0215" rpy="0 0 ${pi/2}"/>
+  </xacro:ar_marker>
+  <xacro:ar_marker prefix="workspace_"
+		   parent="workspace_center"
+		   marker_id="17_26_32_256"
+		   width="0.150" height="0.150" margin="0.005"
+		   thickness="0.001">
     <origin xyz="0.0 0.0 0.0005" rpy="0 0 0"/>
-  </xacro:ar_marker_70_5>
+  </xacro:ar_marker>
 </robot>

File: aist_description/scenes/urdf/g_bot_calibration.urdf.xacro (robot description, xacro)
@@ -1,11 +1,11 @@
 <?xml version="1.0"?>
 <robot xmlns:xacro="http://wiki.ros.org/xacro" name="g_bot_calibration">
-  <xacro:include filename="$(find aist_description
-			   )/objects/urdf/ar_markers.urdf.xacro"/>
-  <xacro:ar_marker_70_5 prefix="g_bot_"
-  			parent="g_bot_gripper_base_link"
-  			marker_id="26"
-			thickness="0.005">
-    <origin xyz="0.180 0.0 0.0215" rpy="0 0 0"/>
-  </xacro:ar_marker_70_5>
+  <xacro:include filename="$(find aist_aruco_ros)/urdf/ar_marker.urdf.xacro"/>
+  <xacro:ar_marker prefix="g_bot_"
+  		   parent="g_bot_gripper_base_link"
+  		   marker_id="26"
+		   width="0.070" height="0.070" margin="0.005"
+		   thickness="0.005">
+    <origin xyz="0.180 0.0 0.0215" rpy="0 0 ${pi/2}"/>
+  </xacro:ar_marker>
 </robot>

File: aist_description/scenes/urdf/kitting.urdf.xacro (robot description, xacro)
@@ -113,11 +113,9 @@
   </xacro:kitting_tray_2>
   <!-- AR marker for localizing WEB camera -->
-  <xacro:include filename="$(find aist_description
-  			   )/objects/urdf/ar_markers.urdf.xacro"/>
+  <xacro:include filename="$(find aist_aruco_ros)/urdf/ar_marker.urdf.xacro"/>
   <xacro:ar_marker prefix="workspace_"
   		   parent="workspace_center"
   		   marker_id="32"
-  		   size="0.095"
-  		   margin="0.0525"
+  		   width="0.095" height="0.095" margin="0.0525"
   		   thickness="0.003">
     <origin xyz="${marker_x} ${marker_y} 0.0003" rpy="0 0 ${pi/2}"/>

File: aist_description/scenes/urdf/mocap_calibration.urdf.xacro (robot description, xacro)
@@ -2,10 +2,11 @@
 <robot xmlns:xacro="http://wiki.ros.org/xacro" name="mocap_calibration">
   <!-- Add AR markers -->
-  <xacro:include filename="$(find aist_description)/objects/urdf/ar_markers.urdf.xacro"/>
-  <xacro:ar_marker_160_10 prefix="c_bot_"
-  			  parent="c_bot_gripper_tip_link"
-  			  marker_id="32"
-  			  thickness="0.005">
-    <origin xyz="0.04 0.0 0.0185" rpy="0 0 0"/>
-  </xacro:ar_marker_160_10>
+  <xacro:include filename="$(find aist_aruco_ros)/urdf/ar_marker.urdf.xacro"/>
+  <xacro:ar_marker prefix="c_bot_"
+  		   parent="c_bot_gripper_base_link"
+		   marker_id="17_26_32_256"
+		   width="0.150" height="0.150" margin="0.005"
+  		   thickness="0.005">
+    <origin xyz="0.14 0.0 0.0215" rpy="0 0 ${pi/2}"/>
+  </xacro:ar_marker>
 </robot>

Commit message: Update calibration of a_motioncam

File: aist_description/scenes/urdf/calibration.urdf.xacro (robot description, xacro)
@@ -11,5 +11,5 @@
 		   width="0.070" height="0.070" margin="0.005"
 		   thickness="0.005">
-    <origin xyz="0.063 0.0 0.0215" rpy="0 0 ${pi/2}"/>
+    <origin xyz="0.163 0.0 0.0215" rpy="0 0 ${pi/2}"/>
   </xacro:ar_marker>
   <xacro:ar_marker prefix="workspace_"
