Commit message: Move tip_link of robotiq grippers to urdf of aist_robotiq package

File: aist_description/scenes/urdf/a_bot_base_scene.urdf.xacro (robot description, xacro)
@@ -57,9 +57,10 @@
     <origin xyz="0 0 0" rpy="0 0 0"/>
   </xacro:robotiq_arg2f_coupling>
-  <xacro:include filename="$(find aist_description)/devices/urdf/robotiq_85_gripper_with_tip_link.urdf.xacro"/>
-  <xacro:robotiq_85_gripper_with_tip_link prefix="a_bot_gripper_"
-					  parent="a_bot_gripper_coupling_flange_link">
+  <xacro:include filename="$(find aist_robotiq
+			   )/urdf/robotiq_85_gripper.urdf.xacro"/>
+  <xacro:robotiq_85_gripper prefix="a_bot_gripper_"
+			    parent="a_bot_gripper_coupling_flange_link">
     <origin xyz="0 0 0" rpy="0 0 0"/>
-  </xacro:robotiq_85_gripper_with_tip_link>
+  </xacro:robotiq_85_gripper>
   <!-- Add RealSense camera -->
   <xacro:include filename="$(find aist_description

File: aist_description/scenes/urdf/aist_base_scene.urdf.xacro (robot description, xacro)
@@ -80,10 +80,12 @@
     <origin xyz="0 0 0" rpy="0 0 0"/>
   </xacro:robotiq_arg2f_coupling>
-  <xacro:include filename="$(find aist_description)/devices/urdf/robotiq_85_gripper_with_tip_link.urdf.xacro"/>
-  <xacro:robotiq_85_gripper_with_tip_link prefix="a_bot_gripper_"
-					  parent="a_bot_gripper_coupling_flange_link">
+  <xacro:include filename="$(find aist_robotiq
+			   )/urdf/robotiq_85_gripper.urdf.xacro"/>
+  <xacro:robotiq_85_gripper prefix="a_bot_gripper_"
+			    parent="a_bot_gripper_coupling_flange_link">
     <origin xyz="0 0 0" rpy="0 0 0"/>
-  </xacro:robotiq_85_gripper_with_tip_link>
-  <xacro:include filename="$(find aist_description)/devices/urdf/single_suction_gripper.urdf.xacro"/>
+  </xacro:robotiq_85_gripper>
+  <xacro:include filename="$(find aist_description
+			   )/devices/urdf/single_suction_gripper.urdf.xacro"/>
   <xacro:single_suction_gripper prefix="b_bot_gripper_"
   				parent="b_bot_ftsensor_flange_link">

File: aist_description/scenes/urdf/dur5e_base_scene.urdf.xacro (robot description, xacro)
@@ -66,9 +66,10 @@
     <origin xyz="0 0 0" rpy="0 0 0"/>
   </xacro:robotiq_arg2f_coupling>
-  <xacro:include filename="$(find aist_description)/devices/urdf/robotiq_85_gripper_with_tip_link.urdf.xacro"/>
-  <xacro:robotiq_85_gripper_with_tip_link prefix="c_bot_gripper_"
-					  parent="c_bot_gripper_coupling_flange_link">
+  <xacro:include filename="$(find aist_robotiq
+			   )/urdf/robotiq_85_gripper.urdf.xacro"/>
+  <xacro:robotiq_85_gripper prefix="c_bot_gripper_"
+			    parent="c_bot_gripper_coupling_flange_link">
     <origin xyz="0 0 0" rpy="0 0 0"/>
-  </xacro:robotiq_85_gripper_with_tip_link>
+  </xacro:robotiq_85_gripper>
   <!-- <xacro:include filename="$(find aist_description)/devices/urdf/dual_suction_gripper.urdf.xacro"/> -->
   <!-- <xacro:dual_suction_gripper prefix="d_bot_" -->

File: aist_description/scenes/urdf/fvision_base_scene.urdf.xacro (robot description, xacro)
@@ -57,14 +57,16 @@
     <origin xyz="0 0 0" rpy="0 0 0"/>
   </xacro:robotiq_arg2f_coupling>
-  <xacro:include filename="$(find aist_description)/devices/urdf/robotiq_140_gripper_with_tip_link.urdf.xacro"/>
-  <xacro:robotiq_140_gripper_with_tip_link prefix="d_bot_gripper_"
-					   parent="d_bot_left_coupling_flange_link">
+  <xacro:include filename="$(find aist_robotiq
+			   )/urdf/robotiq_140_gripper.urdf.xacro"/>
+  <xacro:robotiq_140_gripper prefix="d_bot_gripper_"
+			     parent="d_bot_left_coupling_flange_link">
     <origin xyz="0 0 0" rpy="0 0 0"/>
-  </xacro:robotiq_140_gripper_with_tip_link>
+  </xacro:robotiq_140_gripper>
   <xacro:robotiq_arg2f_coupling prefix="d_bot_right_coupling_"
 				parent="d_bot_dual_bracket_right_flange_link">
     <origin xyz="0 0 0" rpy="0 0 0"/>
   </xacro:robotiq_arg2f_coupling>
-  <xacro:include filename="$(find aist_robotiq)/urdf/robotiq_epick.urdf.xacro"/>
+  <xacro:include filename="$(find aist_robotiq
+			   )/urdf/robotiq_epick.urdf.xacro"/>
   <xacro:robotiq_epick prefix="d_bot_suction_"
 		       parent="d_bot_right_coupling_flange_link">

File: aist_description/scenes/urdf/mocap_base_scene.urdf.xacro (robot description, xacro)
@@ -48,10 +48,10 @@
     <origin xyz="0 0 0" rpy="${pi} 0 0"/>
   </xacro:robotiq_arg2f_coupling>
-  <xacro:include filename="$(find aist_description
-			   )/devices/urdf/robotiq_85_gripper_with_tip_link.urdf.xacro"/>
-  <xacro:robotiq_85_gripper_with_tip_link prefix="c_bot_gripper_"
-					  parent="c_bot_gripper_coupling_flange_link">
+  <xacro:include filename="$(find aist_robotiq
+			   )/urdf/robotiq_85_gripper.urdf.xacro"/>
+  <xacro:robotiq_85_gripper prefix="c_bot_gripper_"
+			    parent="c_bot_gripper_coupling_flange_link">
     <origin xyz="0 0 0" rpy="0 0 0"/>
-  </xacro:robotiq_85_gripper_with_tip_link>
+  </xacro:robotiq_85_gripper>
   <!-- Add RealSense camera -->
   <xacro:include filename="$(find aist_description

File: aist_description/scenes/urdf/nedo_ur5e_base_scene.urdf.xacro (robot description, xacro)
@@ -26,15 +26,16 @@
   </joint>
   <!-- robot arms -->
-  <xacro:include filename="$(find ur_e_description)/urdf/common.gazebo.xacro"/>
-  <xacro:include filename="$(find ur_e_description)/urdf/ur5e.urdf.xacro"/>
-  <xacro:ur5e_robot prefix="e_bot_" joint_limited="false"
-    shoulder_pan_lower_limit="${-pi}" shoulder_pan_upper_limit="${pi}"
-    shoulder_lift_lower_limit="${-pi}" shoulder_lift_upper_limit="${pi}"
-    elbow_joint_lower_limit="0.0" elbow_joint_upper_limit="${pi}"
-    wrist_1_lower_limit="${-pi}" wrist_1_upper_limit="${pi}"
-    wrist_2_lower_limit="${-pi}" wrist_2_upper_limit="${pi}"
-    wrist_3_lower_limit="${-pi}" wrist_3_upper_limit="${pi}"
-    kinematics_file="${load_yaml(
-		     '$(find ur_e_description)/config/ur5e_default.yaml')}"/>
+  <xacro:include filename="$(find ur_gazebo)/urdf/ur_macro.xacro"/>
+  <xacro:ur_robot_gazebo
+      prefix="e_bot_"
+      joint_limits_parameters_file="$(find ur_description
+                                    )/config/ur5e/joint_limits.yaml"
+      physical_parameters_file="$(find ur_description
+                                )/config/ur5e/physical_parameters.yaml"
+      visual_parameters_file="$(find ur_description
+                              )/config/ur5e/visual_parameters.yaml"
+      kinematics_parameters_file="$(find ur_description
+				  )/config/ur5e/default_kinematics.yaml"
+      transmission_hw_interface="hardware_interface/PositionJointInterface"/>
   <joint name="ground_e_bot_joint" type="fixed">
     <parent link="ground"/>
@@ -46,12 +47,13 @@
 			   )/urdf/robotiq_arg2f_coupling.urdf.xacro"/>
   <xacro:robotiq_arg2f_coupling prefix="e_bot_gripper_coupling_"
-				parent="e_bot_ee_link">
+				parent="e_bot_flange">
+    <origin xyz="0 0 0" rpy="${pi} 0 0"/>
+  </xacro:robotiq_arg2f_coupling>
+  <xacro:include filename="$(find aist_robotiq
+			   )/urdf/robotiq_140_gripper.urdf.xacro"/>
+  <xacro:robotiq_140_gripper prefix="e_bot_gripper_"
+			     parent="e_bot_gripper_coupling_flange_link">
     <origin xyz="0 0 0" rpy="0 0 0"/>
-  </xacro:robotiq_arg2f_coupling>
-  <xacro:include filename="$(find aist_description)/devices/urdf/robotiq_140_gripper_with_tip_link.urdf.xacro"/>
-  <xacro:robotiq_140_gripper_with_tip_link prefix="e_bot_gripper_"
-					  parent="e_bot_gripper_coupling_flange_link">
-    <origin xyz="0 0 0" rpy="0 0 0"/>
-  </xacro:robotiq_140_gripper_with_tip_link>
+  </xacro:robotiq_140_gripper>
   <!-- I would like to remove the "world" link definition, but apparently it is necessary for Gazebo -->
   <link name="world"/>

Commit message: Move ft300_driver from aist_ftsensor to aist_robotiq

File: aist_description/scenes/urdf/a_bot_base_scene.urdf.xacro (robot description, xacro)
@@ -46,5 +46,5 @@
   </joint>
   <!-- Spawn and attach force sensor -->
-  <xacro:include filename="$(find aist_ftsensor)/urdf/ft300.urdf.xacro"/>
+  <xacro:include filename="$(find aist_robotiq)/urdf/ft300.urdf.xacro"/>
   <xacro:ft300 prefix="a_bot_ftsensor_" parent="a_bot_flange">
     <origin xyz="0 0 0" rpy="${pi} 0 0"/>

File: aist_description/scenes/urdf/aist_base_scene.urdf.xacro (robot description, xacro)
@@ -62,5 +62,5 @@
   </joint>
   <!-- Spawn and attach force sensor -->
-  <xacro:include filename="$(find aist_ftsensor)/urdf/ft300.urdf.xacro"/>
+  <xacro:include filename="$(find aist_robotiq)/urdf/ft300.urdf.xacro"/>
   <xacro:ft300 prefix="a_bot_ftsensor_" parent="a_bot_flange">
     <origin xyz="0 0 0" rpy="${pi} 0 0"/>

File: aist_robotiq/urdf/ft300.urdf.xacro (robot description, xacro)
@@ -8,5 +8,6 @@
         <origin xyz="${ft300_length} 0 0" rpy="${pi} ${pi/2} 0"/>
 	<geometry>
-          <mesh filename="package://aist_ftsensor/meshes/ft300.stl" scale="0.001 0.001 0.001"/>
+          <mesh filename="package://aist_robotiq/meshes/visual/ft300.stl"
+		scale="0.001 0.001 0.001"/>
 	</geometry>
 	<material name="Black">

Commit message: Change robot_effector_frame from bot_flange to gripper_base_link

File: aist_description/scenes/urdf/a_bot_base_scene.urdf.xacro (robot description, xacro)
@@ -2,22 +2,19 @@
 <robot xmlns:xacro="http://wiki.ros.org/xacro" name="a_bot__base_scene" >
   <xacro:arg name="scene" default=""/>
-  <!-- Calibration help: If the robot is not moving far enough to the calibration point, increase these distances -->
-  <xacro:property name="a_bot_x" value="0"/>
-  <xacro:property name="a_bot_y" value="-0.4875"/>
-  <!-- <xacro:property name="a_bot_theta" value="${pi}"/> -->
-  <xacro:property name="bots_z" value="0.77"/>
-  <!-- This is the main file defining our robot arrangement and physical environment. -->
-  <!-- Main workspace -->
-  <!-- The surface is 0.01 m below the robot bases and the "workspace_center" frame. -->
+  <xacro:property name="a_bot_x"	value="0"/>
+  <xacro:property name="a_bot_y"	value="-0.4875"/>
+  <xacro:property name="bots_z"		value="0.770"/>
+  <xacro:property name="screen_z"	value="${bots_z + 0.0347}"/>
+  <!-- ground and workspace -->
   <link name="ground"/>
-  <xacro:include filename="$(find aist_description)/objects/urdf/aist_box.urdf.xacro"/>
-  <xacro:property name="table_w" value="0.9"/>
-  <xacro:property name="table_l" value="1.8"/>
-  <xacro:property name="table_h" value="0.01"/>
-  <xacro:aist_box name="workbox"
-		  width="${table_w}" length="${table_l}" height="${table_h}"
-		  parent="ground">
-    <origin xyz="${-table_w/2} ${-table_l/2} ${bots_z - table_h}" rpy="0 0 0"/>
-  </xacro:aist_box>
+  <xacro:property name="table_w"	value="0.900"/>
+  <xacro:property name="table_l"	value="1.800"/>
+  <xacro:include filename="$(find aist_description
+			   )/objects/urdf/table.urdf.xacro"/>
+  <xacro:table prefix="workspace_"
+	       width="${table_w}" length="${table_l}" height="${bots_z}"
+	       parent="ground">
+    <origin xyz="${-table_w/2} ${-table_l/2} 0" rpy="0 0 0"/>
+  </xacro:table>
   <link name="workspace_center"/>
   <joint name="ground_to_workspace" type="fixed">
@@ -26,6 +23,26 @@
     <origin xyz="0 0 ${bots_z}" rpy="0 0 0"/>
   </joint>
+  <!-- cage -->
+  <xacro:property name="cage_w"		value="1.200"/>
+  <xacro:property name="cage_l"		value="1.580"/>
+  <xacro:property name="cage_h"		value="1.420"/>
+  <xacro:property name="cage_t"		value="0.040"/>
+  <xacro:property name="tool_bar_h"	value="0.270"/>
+  <xacro:property name="camera_bar_h"	value="1.300"/>
+  <xacro:property name="cage_z"		value="0.164"/>
+  <xacro:property name="cage_offset"	value="0.020"/>
+  <xacro:include filename="$(find aist_description
+			   )/objects/urdf/cage.urdf.xacro"/>
+  <xacro:cage prefix="cage_"
+	      width="${cage_w}" length="${cage_l}" height="${cage_h}"
+	      thickness="${cage_t}"
+	      workspace_height="${bots_z - cage_z}"
+	      tool_bar_height="${tool_bar_h}"
+	      camera_bar_height="${camera_bar_h}"
+	      parent="ground">
+    <origin xyz="${-cage_w/2 + cage_offset} ${-cage_l/2} ${cage_z}"
+	    rpy="0 0 0" />
+  </xacro:cage>
   <!-- robot arms -->
-  <!-- <xacro:include filename="$(find ur_description)/urdf/common.gazebo.xacro"/> -->
   <xacro:include filename="$(find ur_gazebo)/urdf/ur_macro.xacro"/>
   <xacro:ur_robot_gazebo
@@ -39,5 +56,7 @@
       kinematics_parameters_file="$(find aist_bringup
 				  )/config/a_bot_calibration.yaml"
-      transmission_hw_interface="hardware_interface/PositionJointInterface"/>
+      transmission_hw_interface="hardware_interface/PositionJointInterface"
+      safety_limits="true"
+      safety_pos_margin="0.3"/>
   <joint name="ground_a_bot_joint" type="fixed">
     <parent link="ground"/>

File: aist_description/scenes/urdf/a_bot_calibration.urdf.xacro (robot description, xacro)
@@ -1,12 +1,12 @@
 <?xml version="1.0"?>
-<robot xmlns:xacro="http://wiki.ros.org/xacro" name="mocap_calibration">
+<robot xmlns:xacro="http://wiki.ros.org/xacro" name="a_bot_calibration">
   <!-- Add AR markers -->
   <xacro:include filename="$(find aist_aruco_ros)/urdf/ar_marker.urdf.xacro"/>
-  <xacro:ar_marker prefix="c_bot_"
-  		   parent="c_bot_gripper_base_link"
+  <xacro:ar_marker prefix="workspace_"
+		   parent="workspace_center"
 		   marker_id="17_26_32_256"
 		   width="0.150" height="0.150" margin="0.005"
-  		   thickness="0.005">
-    <origin xyz="0.18 0.0 0.0215" rpy="0 0 ${pi/2}"/>
+		   thickness="0.001">
+    <origin xyz="0.0 0.0 0.0005" rpy="0 0 0"/>
   </xacro:ar_marker>
 </robot>

File: aist_description/scenes/urdf/fvision_base_scene.urdf.xacro (robot description, xacro)
@@ -78,5 +78,5 @@
 			   )/scenes/urdf/load_calibration.urdf.xacro"/>
   <xacro:load_calibration filename="$(find aist_handeye_calibration
-				    )/calib/a_phoxi_m_camera.yaml"/>
+				    )/calib/d_phoxi_m_camera.yaml"/>
   <xacro:include filename="$(find aist_phoxi_camera
 			   )/urdf/phoxi_m_camera.urdf.xacro"/>

File: aist_description/scenes/urdf/fvision_calibration.urdf.xacro (robot description, xacro)
@@ -3,11 +3,11 @@
   <!-- Add AR markers -->
   <xacro:include filename="$(find aist_aruco_ros)/urdf/ar_marker.urdf.xacro"/>
-  <xacro:ar_marker prefix="d_bot_"
-  		   parent="d_bot_gripper_base_link"
-  		   marker_id="26"
-		   width="0.070" height="0.070" margin="0.005"
-		   thickness="0.005">
-    <origin xyz="0.180 0.0 0.0215" rpy="0 0 ${pi/2}"/>
-  </xacro:ar_marker>
+  <!-- <xacro:ar_marker prefix="d_bot_" -->
+  <!-- 		   parent="d_bot_gripper_base_link" -->
+  <!-- 		   marker_id="26" -->
+  <!-- 		   width="0.070" height="0.070" margin="0.005" -->
+  <!-- 		   thickness="0.005"> -->
+  <!--   <origin xyz="0.180 0.0 0.0215" rpy="0 0 ${pi/2}"/> -->
+  <!-- </xacro:ar_marker> -->
   <xacro:ar_marker prefix="workspace_"
 		   parent="workspace_center"

Commit message: Add tool holders to a_bot_base_scene and b_bot_base_scene

File: aist_description/scenes/urdf/a_bot_base_scene.urdf.xacro (robot description, xacro)
@@ -44,4 +44,17 @@
 	    rpy="0 0 0" />
   </xacro:cage>
+  <!-- tool holders -->
+  <xacro:property name="screw_tool_m3_holder_y"	value="0.6"/>
+  <xacro:property name="screw_tool_m4_holder_y"	value="0.8"/>
+  <xacro:include filename="$(find aist_description
+			   )/objects/urdf/screw_tool_holder.urdf.xacro"/>
+  <xacro:screw_tool_holder prefix="screw_tool_m3_holder_"
+			   parent="cage_tool_bar">
+    <origin xyz="0 ${screw_tool_m3_holder_y} ${cage_t}" rpy="0 0 0"/>
+  </xacro:screw_tool_holder>
+  <xacro:screw_tool_holder prefix="screw_tool_m4_holder_"
+			   parent="cage_tool_bar">
+    <origin xyz="0 ${screw_tool_m4_holder_y} ${cage_t}" rpy="0 0 0"/>
+  </xacro:screw_tool_holder>
   <!-- robot arms -->
   <xacro:include filename="$(find ur_gazebo)/urdf/ur_macro.xacro"/>

File: aist_description/scenes/urdf/b_bot_base_scene.urdf.xacro (robot description, xacro)
@@ -45,4 +45,17 @@
 	    rpy="0 0 0" />
   </xacro:cage>
+  <!-- tool holders -->
+  <xacro:property name="screw_tool_m3_holder_y"	value="0.6"/>
+  <xacro:property name="screw_tool_m4_holder_y"	value="0.8"/>
+  <xacro:include filename="$(find aist_description
+			   )/objects/urdf/screw_tool_holder.urdf.xacro"/>
+  <xacro:screw_tool_holder prefix="screw_tool_m3_holder_"
+			   parent="cage_tool_bar">
+    <origin xyz="0 ${screw_tool_m3_holder_y} ${cage_t}" rpy="0 0 0"/>
+  </xacro:screw_tool_holder>
+  <xacro:screw_tool_holder prefix="screw_tool_m4_holder_"
+			   parent="cage_tool_bar">
+    <origin xyz="0 ${screw_tool_m4_holder_y} ${cage_t}" rpy="0 0 0"/>
+  </xacro:screw_tool_holder>
   <!-- robot arms -->
   <xacro:include filename="$(find ur_gazebo)/urdf/ur_macro.xacro"/>

Commit message: Add suction_tool_holder

File: aist_description/scenes/urdf/a_bot_base_scene.urdf.xacro (robot description, xacro)
@@ -45,6 +45,7 @@
   </xacro:cage>
   <!-- tool holders -->
-  <xacro:property name="screw_tool_m3_holder_y"	value="0.6"/>
-  <xacro:property name="screw_tool_m4_holder_y"	value="0.8"/>
+  <xacro:property name="screw_tool_m3_holder_y"	value="0.75"/>
+  <xacro:property name="screw_tool_m4_holder_y"	value="0.85"/>
+  <xacro:property name="suction_tool_holder_y"	value="0.95"/>
   <xacro:include filename="$(find aist_description
 			   )/objects/urdf/screw_tool_holder.urdf.xacro"/>
@@ -57,4 +58,10 @@
     <origin xyz="0 ${screw_tool_m4_holder_y} ${cage_t}" rpy="0 0 0"/>
   </xacro:screw_tool_holder>
+  <xacro:include filename="$(find aist_description
+			   )/objects/urdf/suction_tool_holder.urdf.xacro"/>
+  <xacro:suction_tool_holder prefix="suction_tool_holder_"
+			   parent="cage_tool_bar">
+    <origin xyz="0 ${suction_tool_holder_y} ${cage_t}" rpy="0 0 0"/>
+  </xacro:suction_tool_holder>
   <!-- robot arms -->
   <xacro:include filename="$(find ur_gazebo)/urdf/ur_macro.xacro"/>

File: aist_description/scenes/urdf/aist_base_scene.urdf.xacro (robot description, xacro)
@@ -48,6 +48,7 @@
   </xacro:cage>
   <!-- tool holders -->
-  <xacro:property name="screw_tool_m3_holder_y"	value="0.6"/>
-  <xacro:property name="screw_tool_m4_holder_y"	value="0.8"/>
+  <xacro:property name="screw_tool_m3_holder_y"	value="0.75"/>
+  <xacro:property name="screw_tool_m4_holder_y"	value="0.85"/>
+  <xacro:property name="suction_tool_holder_y"	value="0.95"/>
   <xacro:include filename="$(find aist_description
 			   )/objects/urdf/screw_tool_holder.urdf.xacro"/>
@@ -60,17 +61,10 @@
     <origin xyz="0 ${screw_tool_m4_holder_y} ${cage_t}" rpy="0 0 0"/>
   </xacro:screw_tool_holder>
-  <!-- screw tools -->
-  <!-- <xacro:include filename="$(find aist_fastening_tools -->
-  <!-- 			   )/urdf/screw_tool_m3.urdf.xacro"/> -->
-  <!-- <xacro:screw_tool_m3 prefix="screw_tool_m3_" -->
-  <!-- 		       parent="screw_tool_m3_holder_link"> -->
-  <!--   <origin xyz="0 0 0" rpy="0 0 0" /> -->
-  <!-- </xacro:screw_tool_m3> -->
-  <!-- <xacro:include filename="$(find aist_fastening_tools -->
-  <!-- 			   )/urdf/screw_tool_m4.urdf.xacro"/> -->
-  <!-- <xacro:screw_tool_m3 prefix="screw_tool_m4_" -->
-  <!-- 		       parent="screw_tool_m4_holder_link"> -->
-  <!--   <origin xyz="0 0 0" rpy="0 0 0" /> -->
-  <!-- </xacro:screw_tool_m3> -->
+  <xacro:include filename="$(find aist_description
+			   )/objects/urdf/suction_tool_holder.urdf.xacro"/>
+  <xacro:suction_tool_holder prefix="suction_tool_holder_"
+			   parent="cage_tool_bar">
+    <origin xyz="0 ${suction_tool_holder_y} ${cage_t}" rpy="0 0 0"/>
+  </xacro:suction_tool_holder>
   <!-- robot arms -->
   <xacro:include filename="$(find ur_gazebo)/urdf/ur_macro.xacro"/>

File: aist_description/scenes/urdf/b_bot_base_scene.urdf.xacro (robot description, xacro)
@@ -46,6 +46,7 @@
   </xacro:cage>
   <!-- tool holders -->
-  <xacro:property name="screw_tool_m3_holder_y"	value="0.6"/>
-  <xacro:property name="screw_tool_m4_holder_y"	value="0.8"/>
+  <xacro:property name="screw_tool_m3_holder_y"	value="0.75"/>
+  <xacro:property name="screw_tool_m4_holder_y"	value="0.85"/>
+  <xacro:property name="suction_tool_holder_y"	value="0.95"/>
   <xacro:include filename="$(find aist_description
 			   )/objects/urdf/screw_tool_holder.urdf.xacro"/>
@@ -58,4 +59,10 @@
     <origin xyz="0 ${screw_tool_m4_holder_y} ${cage_t}" rpy="0 0 0"/>
   </xacro:screw_tool_holder>
+  <xacro:include filename="$(find aist_description
+			   )/objects/urdf/suction_tool_holder.urdf.xacro"/>
+  <xacro:suction_tool_holder prefix="suction_tool_holder_"
+			   parent="cage_tool_bar">
+    <origin xyz="0 ${suction_tool_holder_y} ${cage_t}" rpy="0 0 0"/>
+  </xacro:suction_tool_holder>
   <!-- robot arms -->
   <xacro:include filename="$(find ur_gazebo)/urdf/ur_macro.xacro"/>

Commit message: Remove Zivid2+ and add precision_tool_holder

File: aist_description/scenes/urdf/a_bot_base_scene.urdf.xacro (robot description, xacro)
@@ -45,7 +45,14 @@
   </xacro:cage>
   <!-- tool holders -->
-  <xacro:property name="screw_tool_m3_holder_y"	value="0.75"/>
-  <xacro:property name="screw_tool_m4_holder_y"	value="0.85"/>
-  <xacro:property name="suction_tool_holder_y"	value="0.95"/>
+  <xacro:property name="precision_tool_holder_y"	value="0.60"/>
+  <xacro:property name="screw_tool_m3_holder_y"		value="0.70"/>
+  <xacro:property name="screw_tool_m4_holder_y"		value="0.80"/>
+  <xacro:property name="suction_tool_holder_y"		value="0.90"/>
+  <xacro:include filename="$(find aist_description
+			   )/objects/urdf/precision_tool_holder.urdf.xacro"/>
+  <xacro:precision_tool_holder prefix="precision_tool_holder_"
+			   parent="cage_tool_bar">
+    <origin xyz="0 ${precision_tool_holder_y} ${cage_t}" rpy="0 0 0"/>
+  </xacro:precision_tool_holder>
   <xacro:include filename="$(find aist_description
 			   )/objects/urdf/screw_tool_holder.urdf.xacro"/>
@@ -89,16 +96,16 @@
     <origin xyz="0 0 0" rpy="${pi} 0 0" />
   </xacro:zivid_coupling>
-  <!-- Spawn and attach Zivid2+ camera -->
-  <xacro:include filename="$(find aist_description
-			   )/scenes/urdf/load_calibration.urdf.xacro"/>
-  <xacro:load_calibration filename="$(find aist_handeye_calibration
-				    )/calib/a_bot_zivid.yaml"/>
-  <xacro:include filename="$(find aist_description
-			   )/devices/urdf/zivid2plus.urdf.xacro"/>
-  <xacro:zivid2plus name="a_bot_zivid"
-		    parent="a_bot_zivid_coupling_flange_link">
-    <origin xyz="${origin[0]} ${origin[1]} ${origin[2]}"
-    	    rpy="${origin[3]} ${origin[4]} ${origin[5]}"/>
-  </xacro:zivid2plus>
+  <!-- <!-\- Spawn and attach Zivid2+ camera -\-> -->
+  <!-- <xacro:include filename="$(find aist_description -->
+  <!-- 			   )/scenes/urdf/load_calibration.urdf.xacro"/> -->
+  <!-- <xacro:load_calibration filename="$(find aist_handeye_calibration -->
+  <!-- 				    )/calib/a_bot_zivid.yaml"/> -->
+  <!-- <xacro:include filename="$(find aist_description -->
+  <!-- 			   )/devices/urdf/zivid2plus.urdf.xacro"/> -->
+  <!-- <xacro:zivid2plus name="a_bot_zivid" -->
+  <!-- 		    parent="a_bot_zivid_coupling_flange_link"> -->
+  <!--   <origin xyz="${origin[0]} ${origin[1]} ${origin[2]}" -->
+  <!--   	    rpy="${origin[3]} ${origin[4]} ${origin[5]}"/> -->
+  <!-- </xacro:zivid2plus> -->
   <!-- Spawn and attach force sensor -->
   <xacro:include filename="$(find aist_robotiq)/urdf/ft300.urdf.xacro"/>
