Commit message: Fixed orientation of grippers

File: aist_description/scenes/urdf/a_bot_base_scene.urdf.xacro (robot description, xacro)
@@ -92,8 +92,8 @@
   </joint>
   <!-- Attach mounter for Zivid2+ camera -->
-  <xacro:include filename="$(find aist_description)/devices/urdf/zivid_coupling.urdf.xacro"/>
-  <xacro:zivid_coupling prefix="a_bot_zivid_coupling_" parent="a_bot_flange">
-    <origin xyz="0 0 0" rpy="${pi} 0 0" />
-  </xacro:zivid_coupling>
+  <!-- <xacro:include filename="$(find aist_description)/devices/urdf/zivid_coupling.urdf.xacro"/> -->
+  <!-- <xacro:zivid_coupling prefix="a_bot_zivid_coupling_" parent="a_bot_flange"> -->
+  <!--   <origin xyz="0 0 0" rpy="${pi} 0 0" /> -->
+  <!-- </xacro:zivid_coupling> -->
   <!-- <!-\- Spawn and attach Zivid2+ camera -\-> -->
   <!-- <xacro:include filename="$(find aist_description -->
@@ -110,7 +110,6 @@
   <!-- Spawn and attach force sensor -->
   <xacro:include filename="$(find aist_robotiq)/urdf/ft300.urdf.xacro"/>
-  <xacro:ft300 prefix="a_bot_ftsensor_"
-	       parent="a_bot_zivid_coupling_flange_link">
-    <origin xyz="0 0 0" rpy="0 0 0"/>
+  <xacro:ft300 prefix="a_bot_ftsensor_" parent="a_bot_flange">
+    <origin xyz="0 0 0" rpy="${pi} 0 0"/>
   </xacro:ft300>
   <!-- Spawn and attach gripper -->

File: aist_description/scenes/urdf/aist_base_scene.urdf.xacro (robot description, xacro)
@@ -132,8 +132,8 @@
   <xacro:include filename="$(find aist_robotiq)/urdf/ft300.urdf.xacro"/>
   <xacro:ft300 prefix="a_bot_ftsensor_" parent="a_bot_flange">
-    <origin xyz="0 0 0" rpy="0 0 0"/>
+    <origin xyz="0 0 0" rpy="${pi} 0 0"/>
   </xacro:ft300>
   <xacro:ft300 prefix="b_bot_ftsensor_" parent="b_bot_flange">
-    <origin xyz="0 0 0" rpy="0 0 0"/>
+    <origin xyz="0 0 0" rpy="${pi} 0 0"/>
   </xacro:ft300>
   <!-- Spawn and attach gripper -->

Commit message: Update a_bot_base_scene

File: aist_description/scenes/urdf/a_bot_base_scene.urdf.xacro (robot description, xacro)
@@ -29,7 +29,8 @@
   <xacro:property name="cage_t"		value="0.040"/>
   <xacro:property name="tool_bar_h"	value="0.270"/>
-  <xacro:property name="camera_bar_h"	value="1.300"/>
+  <xacro:property name="camera_bar_h"	value="1.325"/>
   <xacro:property name="cage_z"		value="0.164"/>
-  <xacro:property name="cage_offset"	value="0.020"/>
+  <xacro:property name="cage_offset_x"	value="0.020"/>
+  <xacro:property name="cage_offset_y"	value="-0.005"/>
   <xacro:include filename="$(find aist_description
 			   )/objects/urdf/cage.urdf.xacro"/>
@@ -41,5 +42,7 @@
 	      camera_bar_height="${camera_bar_h}"
 	      parent="ground">
-    <origin xyz="${-cage_w/2 + cage_offset} ${-cage_l/2} ${cage_z}"
+    <origin xyz="${-cage_w/2 + cage_offset_x}
+		 ${-cage_l/2 + cage_offset_y}
+		 ${cage_z}"
 	    rpy="0 0 0" />
   </xacro:cage>
@@ -121,9 +124,9 @@
   </xacro:robotiq_arg2f_coupling>
   <xacro:include filename="$(find aist_robotiq
-			   )/urdf/robotiq_140_gripper.urdf.xacro"/>
-  <xacro:robotiq_140_gripper prefix="a_bot_gripper_"
+			   )/urdf/robotiq_85_gripper.urdf.xacro"/>
+  <xacro:robotiq_85_gripper prefix="a_bot_gripper_"
 			    parent="a_bot_gripper_coupling_flange_link">
     <origin xyz="0 0 0" rpy="0 0 0"/>
-  </xacro:robotiq_140_gripper>
+  </xacro:robotiq_85_gripper>
   <!-- I would like to remove the "world" link definition, but apparently it is necessary for Gazebo -->
   <link name="world"/>

Commit message: Change grasp orientation of precision tool

File: aist_description/scenes/urdf/a_bot_base_scene.urdf.xacro (robot description, xacro)
@@ -1,5 +1,7 @@
 <?xml version="1.0"?>
 <robot xmlns:xacro="http://wiki.ros.org/xacro" name="a_bot_base_scene" >
-  <xacro:arg name="scene" default=""/>
+  <xacro:arg name="scene"		default=""/>
+  <xacro:arg name="hw_interface"	default="PositionJointInterface"/>
+					<!-- or "VelocityJointInterface" -->
   <xacro:property name="a_bot_x"	value="0"/>
   <xacro:property name="a_bot_y"	value="-0.4875"/>
@@ -88,5 +90,5 @@
       kinematics_parameters_file="$(find aist_bringup
 				  )/config/a_bot_calibration.yaml"
-      transmission_hw_interface="hardware_interface/PositionJointInterface"
+      transmission_hw_interface="hardware_interface/$(arg hw_interface)"
       safety_limits="true"
       safety_pos_margin="0.3"/>

File: moveit_config/a_bot_moveit_config/config/gazebo_a_bot_base_scene.urdf (robot description, URDF)
Before this commit: robot a_bot__base_scene, 54 links, 53 joints
Links:
- removed link workbox
- added link cage_back_left_pillar, mass 1.0; collision box size=0.04 0.04 1.42; visual box size=0.04 0.04 1.42
- added link cage_back_right_pillar, mass 1.0; collision box size=0.04 0.04 1.42; visual box size=0.04 0.04 1.42
- added link cage_front_left_pillar, mass 1.0; collision box size=0.04 0.04 1.42; visual box size=0.04 0.04 1.42
- added link cage_front_right_pillar, mass 1.0; collision box size=0.04 0.04 1.42; visual box size=0.04 0.04 1.42
- added link cage_lower_back_bar, mass 1.0; collision box size=1.1199999999999999 0.04 0.04; visual box size=1.1199999999999999 0.04 0.04
- added link cage_lower_front_bar, mass 1.0; collision box size=1.1199999999999999 0.04 0.04; visual box size=1.1199999999999999 0.04 0.04
- added link cage_lower_left_bar, mass 1.0; collision box size=0.04 1.5 0.04; visual box size=0.04 1.5 0.04
- added link cage_lower_right_bar, mass 1.0; collision box size=0.04 1.5 0.04; visual box size=0.04 1.5 0.04
- added link cage_tool_bar, mass 1.0; collision box size=0.04 1.5 0.04; visual box size=0.04 1.5 0.04
- added link cage_upper_back_bar, mass 1.0; collision box size=1.1199999999999999 0.04 0.04; visual box size=1.1199999999999999 0.04 0.04
- added link cage_upper_front_bar, mass 1.0; collision box size=1.1199999999999999 0.04 0.04; visual box size=1.1199999999999999 0.04 0.04
- added link cage_upper_left_bar, mass 1.0; collision box size=0.04 1.5 0.04; visual box size=0.04 1.5 0.04
- added link cage_upper_right_bar, mass 1.0; collision box size=0.04 1.5 0.04; visual box size=0.04 1.5 0.04
- added link cage_workspace_bar, mass 1.0; collision box size=0.04 1.5 0.04; visual box size=0.04 1.5 0.04
- added link precision_tool_holder_base_link, mass 0.1; collision mesh filename=package://aist_description/objects/meshes/precision_tool_ho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 scale=0.001 0.001 0.001; visual mesh filename=package://aist_description/objects/meshes/precision_tool_ho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 scale=0.001 0.001 0.001
- added link precision_tool_holder_link
- added link screw_tool_m3_holder_base_link, mass 0.1; collision mesh filename=package://aist_description/objects/meshes/screw_tool_holder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 scale=0.001 0.001 0.001; visual mesh filename=package://aist_description/objects/meshes/screw_tool_holder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 scale=0.001 0.001 0.001
- added link screw_tool_m3_holder_link
- added link screw_tool_m4_holder_base_link, mass 0.1; collision mesh filename=package://aist_description/objects/meshes/screw_tool_holder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 scale=0.001 0.001 0.001; visual mesh filename=package://aist_description/objects/meshes/screw_tool_holder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 scale=0.001 0.001 0.001
- added link screw_tool_m4_holder_link
- added link suction_tool_holder_base_link, mass 0.1; collision mesh filename=package://aist_description/objects/meshes/suction_tool_hold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 scale=0.001 0.001 0.001; visual mesh filename=package://aist_description/objects/meshes/suction_tool_hold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 scale=0.001 0.001 0.001
- added link suction_tool_holder_link
- added link workspace_table_base_link, mass 1.0; collision box size=0.05 0.05 0.75; visual box size=0.05 0.05 0.75
- added link workspace_table_leg1, mass 1.0; collision box size=0.05 0.05 0.75; visual box size=0.05 0.05 0.75
- added link workspace_table_leg2, mass 1.0; collision box size=0.05 0.05 0.75; visual box size=0.05 0.05 0.75
- added link workspace_table_leg3, mass 1.0; collision box size=0.05 0.05 0.75; visual box size=0.05 0.05 0.75
- added link workspace_table_top, mass 1.0; collision box size=0.9 1.8 0.02; visual box size=0.9 1.8 0.02
- added link workspace_table_top_center
- added link workspace_table_top_origin
- link a_bot_gripper_left_inner_finger: geometry collision mesh filename=package://aist_robotiq/meshes/collision/robotiq_arg2f_140_i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; visual mesh filename=package://aist_robotiq/meshes/visual/robotiq_arg2f_140_inne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
- link a_bot_gripper_left_inner_finger_pad: geometry collision box size=0.027 0.065 0.0075; visual box size=0.027 0.065 0.0075
- link a_bot_gripper_left_inner_knuckle: geometry collision mesh filename=package://aist_robotiq/meshes/collision/robotiq_arg2f_140_i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; visual mesh filename=package://aist_robotiq/meshes/visual/robotiq_arg2f_140_inne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
- link a_bot_gripper_left_outer_finger: geometry collision mesh filename=package://aist_robotiq/meshes/collision/robotiq_arg2f_140_o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; visual mesh filename=package://aist_robotiq/meshes/visual/robotiq_arg2f_140_oute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
- link a_bot_gripper_left_outer_knuckle: geometry collision mesh filename=package://aist_robotiq/meshes/collision/robotiq_arg2f_140_o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; visual mesh filename=package://aist_robotiq/meshes/visual/robotiq_arg2f_140_oute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
- link a_bot_gripper_right_inner_finger: geometry collision mesh filename=package://aist_robotiq/meshes/collision/robotiq_arg2f_140_i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; visual mesh filename=package://aist_robotiq/meshes/visual/robotiq_arg2f_140_inne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
- link a_bot_gripper_right_inner_finger_pad: geometry collision box size=0.027 0.065 0.0075; visual box size=0.027 0.065 0.0075
- link a_bot_gripper_right_inner_knuckle: geometry collision mesh filename=package://aist_robotiq/meshes/collision/robotiq_arg2f_140_i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; visual mesh filename=package://aist_robotiq/meshes/visual/robotiq_arg2f_140_inne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
- link a_bot_gripper_right_outer_finger: geometry collision mesh filename=package://aist_robotiq/meshes/collision/robotiq_arg2f_140_o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; visual mesh filename=package://aist_robotiq/meshes/visual/robotiq_arg2f_140_oute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
- link a_bot_gripper_right_outer_knuckle: geometry collision mesh filename=package://aist_robotiq/meshes/collision/robotiq_arg2f_140_o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; visual mesh filename=package://aist_robotiq/meshes/visual/robotiq_arg2f_140_oute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
Joints:
- removed joint workbox
- added joint cage_back_left_pillar: type fixed, parent cage_front_left_pillar, child cage_back_left_pillar, origin xyz=0 1.54 0 rpy=0 0 0
- added joint cage_back_right_pillar: type fixed, parent cage_front_left_pillar, child cage_back_right_pillar, origin xyz=1.16        1.54        0 rpy=0 0 0
- added joint cage_front_left_pillar: type fixed, parent ground, child cage_front_left_pillar, origin xyz=-0.585    -0.795    0.164 rpy=0 0 0
- added joint cage_front_right_pillar: type fixed, parent cage_front_left_pillar, child cage_front_right_pillar, origin xyz=1.16 0 0 rpy=0 0 0
- added joint cage_lower_back_bar: type fixed, parent cage_front_left_pillar, child cage_lower_back_bar, origin xyz=0.04 1.54 0 rpy=0 0 0
- added joint cage_lower_front_bar: type fixed, parent cage_front_left_pillar, child cage_lower_front_bar, origin xyz=0.04 0 0 rpy=0 0 0
- added joint cage_lower_left_bar: type fixed, parent cage_front_left_pillar, child cage_lower_left_bar, origin xyz=0 0.04 0 rpy=0 0 0
- added joint cage_lower_right_bar: type fixed, parent cage_front_left_pillar, child cage_lower_right_bar, origin xyz=1.16 0.04 0 rpy=0 0 0
- added joint cage_tool_bar: type fixed, parent cage_workspace_bar, child cage_tool_bar, origin xyz=0 0 0.27 rpy=0 0 0
- added joint cage_upper_back_bar: type fixed, parent cage_front_left_pillar, child cage_upper_back_bar, origin xyz=0.04 1.54 1.38 rpy=0 0 0
- added joint cage_upper_front_bar: type fixed, parent cage_front_left_pillar, child cage_upper_front_bar, origin xyz=0.04 0 1.38 rpy=0 0 0
- added joint cage_upper_left_bar: type fixed, parent cage_front_left_pillar, child cage_upper_left_bar, origin xyz=0 0.04 1.38 rpy=0 0 0
- added joint cage_upper_right_bar: type fixed, parent cage_front_left_pillar, child cage_upper_right_bar, origin xyz=1.16 0.04 1.325 rpy=0 0 0
- added joint cage_workspace_bar: type fixed, parent cage_lower_left_bar, child cage_workspace_bar, origin xyz=0 0 0.596 rpy=0 0 0
- added joint precision_tool_holder_base_joint: type fixed, parent cage_tool_bar, child precision_tool_holder_base_link, origin xyz=0 0.6 0.04 rpy=0 0 0
- added joint precision_tool_holder_joint: type fixed, parent precision_tool_holder_base_link, child precision_tool_holder_link, origin xyz=0.108 0.012 0.037 rpy=0 0.5235987755982988 0
- added joint screw_tool_m3_holder_base_joint: type fixed, parent cage_tool_bar, child screw_tool_m3_holder_base_link, origin xyz=0 0.7 0.04 rpy=0 0 0
- added joint screw_tool_m3_holder_joint: type fixed, parent screw_tool_m3_holder_base_link, child screw_tool_m3_holder_link, origin xyz=0.0525 0 0.007 rpy=0 0 0
- added joint screw_tool_m4_holder_base_joint: type fixed, parent cage_tool_bar, child screw_tool_m4_holder_base_link, origin xyz=0 0.8 0.04 rpy=0 0 0
- added joint screw_tool_m4_holder_joint: type fixed, parent screw_tool_m4_holder_base_link, child screw_tool_m4_holder_link, origin xyz=0.0525 0 0.007 rpy=0 0 0
- added joint suction_tool_holder_base_joint: type fixed, parent cage_tool_bar, child suction_tool_holder_base_link, origin xyz=0 0.9 0.04 rpy=0 0 0
- added joint suction_tool_holder_joint: type fixed, parent suction_tool_holder_base_link, child suction_tool_holder_link, origin xyz=0.050 0 0.007 rpy=0 0 0
- added joint workspace_table_base_link: type fixed, parent ground, child workspace_table_base_link, origin xyz=-0.5449999999999999 -0.9 0 rpy=0 0 0
- added joint workspace_table_leg1: type fixed, parent workspace_table_base_link, child workspace_table_leg1, origin xyz=0.85 0 0 rpy=0 0 0
- added joint workspace_table_leg2: type fixed, parent workspace_table_base_link, child workspace_table_leg2, origin xyz=0 1.75 0 rpy=0 0 0
- added joint workspace_table_leg3: type fixed, parent workspace_table_base_link, child workspace_table_leg3, origin xyz=0.85      1.75      0 rpy=0 0 0
- added joint workspace_table_top: type fixed, parent workspace_table_base_link, child workspace_table_top, origin xyz=0 0 0.75 rpy=0 0 0
- added joint workspace_table_top_center_joint: type fixed, parent workspace_table_top_origin, child workspace_table_top_center, origin xyz=0.45 0.9 0 rpy=0 0 0
- added joint workspace_table_top_origin_joint: type fixed, parent workspace_table_top, child workspace_table_top_origin, origin xyz=0 0 0.02 rpy=0 0 0
- joint a_bot_gripper_finger_joint: axis 1 0 0 -> -1 0 0; limit lower=0 upper=0.81 effort=1000 velocity=2.0 -> lower=0 upper=0.7 effort=1000 velocity=2.0; origin xyz=0 -0.0306011 0.054904 rpy=0 0 3.141592653589793 -> xyz=0 -0.030601 0.054905 rpy=2.2957963267948966 0 0
- joint a_bot_gripper_left_inner_finger_joint: axis 1 0 0 -> -1 0 0; origin xyz=0 0.0061 0.0471 rpy=0 0 0 -> xyz=0 0.0817554015893473 -0.0282203446692936 rpy=-0.725 0 0
- joint a_bot_gripper_left_inner_finger_pad_joint: origin xyz=0 -0.0220203446692936 0.03242 rpy=0 0 0 -> xyz=0 0.0457554015893473 -0.0272203446692936 rpy=0 0 0
- joint a_bot_gripper_left_inner_knuckle_joint: axis 1 0 0 -> -1 0 0; origin xyz=0 -0.0127 0.06142 rpy=0 0 3.141592653589793 -> xyz=0 -0.0127 0.06142 rpy=2.2957963267948966 0 0.0
- joint a_bot_gripper_left_outer_finger_joint: origin xyz=0 0.0315 -0.0041 rpy=0 0 0 -> xyz=0 0.01821998610742 0.0260018192872234 rpy=0 0 0
- joint a_bot_gripper_right_inner_finger_joint: axis 1 0 0 -> -1 0 0; origin xyz=0 0.0061 0.0471 rpy=0 0 0 -> xyz=0 0.0817554015893473 -0.0282203446692936 rpy=-0.725 0 0
- joint a_bot_gripper_right_inner_finger_pad_joint: origin xyz=0 -0.0220203446692936 0.03242 rpy=0 0 0 -> xyz=0 0.0457554015893473 -0.0272203446692936 rpy=0 0 0
- joint a_bot_gripper_right_inner_knuckle_joint: axis 1 0 0 -> -1 0 0; origin xyz=0 0.0127 0.06142 rpy=0 0 0.0 -> xyz=0 0.0127 0.06142 rpy=2.2957963267948966 0 -3.141592653589793
- joint a_bot_gripper_right_outer_finger_joint: origin xyz=0 0.0315 -0.0041 rpy=0 0 0 -> xyz=0 0.01821998610742 0.0260018192872234 rpy=0 0 0
- joint a_bot_gripper_right_outer_knuckle_joint: axis 1 0 0 -> -1 0 0; limit lower=-0.81 upper=0.81 effort=1000 velocity=2.0 -> lower=-0.725 upper=0.725 effort=1000 velocity=2.0; origin xyz=0 0.0306011 0.054904 rpy=0 0 0 -> xyz=0 0.030601 0.054905 rpy=2.2957963267948966 0 3.141592653589793
- joint a_bot_gripper_tip_link_joint: origin xyz=0.1628 0.0 0.0 rpy=0.0 -1.5707963267948966 0.0 -> xyz=.2328 0.0 0.0 rpy=0.0 -1.5707963267948966 0.0
- joint a_bot_inside_camera_joint: origin xyz=0.014368349250599823      0.0035415297809514353      0.06397546955943786 rpy=0.02303437721634514      0.40347560400972565      0.010798159061973579 -> xyz=0.0051834717267641005      0.0029869415393767723      0.06398615295764885 rpy=0.02104566011309687      0.3968034960518725      0.01313899562905875
- joint a_bot_outside_camera_joint: origin xyz=0.03167812734753831      -0.007813867044282037      0.08129884906700884 rpy=0.017373333209516714      -0.2189346019095829      0.034978097124935485 -> xyz=0.03448420081903219      -0.008163711886056418      0.08142610495899788 rpy=0.013998136792162967      -0.22309733722281236      0.035938176557628945

Commit message: Change height of tool_bar

File: aist_description/scenes/urdf/a_bot_base_scene.urdf.xacro (robot description, xacro)
@@ -15,5 +15,5 @@
   <xacro:property name="cage_h"		value="1.420"/>
   <xacro:property name="cage_t"		value="0.040"/>
-  <xacro:property name="tool_bar_h"	value="0.270"/>
+  <xacro:property name="tool_bar_h"	value="0.240"/>
   <xacro:property name="camera_bar_h"	value="1.325"/>
   <xacro:property name="cage_z"		value="0.164"/>

File: aist_description/scenes/urdf/aist_base_scene.urdf.xacro (robot description, xacro)
@@ -16,5 +16,5 @@
   <xacro:property name="cage_h"		value="1.420"/>
   <xacro:property name="cage_t"		value="0.040"/>
-  <xacro:property name="tool_bar_h"	value="0.270"/>
+  <xacro:property name="tool_bar_h"	value="0.240"/>
   <xacro:property name="camera_bar_h"	value="1.325"/>
   <xacro:property name="cage_z"		value="0.164"/>

File: aist_description/scenes/urdf/b_bot_base_scene.urdf.xacro (robot description, xacro)
@@ -14,5 +14,5 @@
   <xacro:property name="cage_h"		value="1.420"/>
   <xacro:property name="cage_t"		value="0.040"/>
-  <xacro:property name="tool_bar_h"	value="0.270"/>
+  <xacro:property name="tool_bar_h"	value="0.240"/>
   <xacro:property name="camera_bar_h"	value="1.325"/>
   <xacro:property name="cage_z"		value="0.164"/>

File: moveit_config/aist_moveit_config/config/gazebo_aist_base_scene.urdf (robot description, URDF)
Before this commit: robot aist_base_scene, 116 links, 115 joints
Joints:
- joint cage_tool_bar: origin xyz=0 0 0.27 rpy=0 0 0 -> xyz=0 0 0.24 rpy=0 0 0
