Commit message: Fix orientation of grippers

File: aist_description/scenes/urdf/a_bot_base_scene.urdf.xacro (robot description, xacro)
@@ -83,9 +83,9 @@
       prefix="a_bot_"
       joint_limits_parameters_file="$(find ur_description
-				    )/config/ur5/joint_limits.yaml"
+				    )/config/ur5e/joint_limits.yaml"
       physical_parameters_file="$(find ur_description
-				)/config/ur5/physical_parameters.yaml"
+				)/config/ur5e/physical_parameters.yaml"
       visual_parameters_file="$(find ur_description
-			      )/config/ur5/visual_parameters.yaml"
+			      )/config/ur5e/visual_parameters.yaml"
       kinematics_parameters_file="$(find aist_bringup
 				  )/config/a_bot_calibration.yaml"
@@ -115,15 +115,10 @@
   <!--   	    rpy="${origin[3]} ${origin[4]} ${origin[5]}"/> -->
   <!-- </xacro:zivid2plus> -->
-  <!-- Spawn and attach force sensor -->
-  <xacro:include filename="$(find aist_robotiq)/urdf/ft300.urdf.xacro"/>
-  <xacro:ft300 prefix="a_bot_ftsensor_" parent="a_bot_flange">
-    <origin xyz="0 0 0" rpy="${pi} 0 0"/>
-  </xacro:ft300>
   <!-- Spawn and attach gripper -->
   <xacro:include filename="$(find aist_robotiq
 			   )/urdf/robotiq_arg2f_coupling.urdf.xacro"/>
   <xacro:robotiq_arg2f_coupling prefix="a_bot_gripper_coupling_"
-				parent="a_bot_ftsensor_flange_link">
-    <origin xyz="0 0 0" rpy="0 0 0"/>
+				parent="a_bot_flange">
+    <origin xyz="0 0 0" rpy="${pi} 0 0"/>
   </xacro:robotiq_arg2f_coupling>
   <xacro:include filename="$(find aist_robotiq

File: aist_description/scenes/urdf/aist_base_scene.urdf.xacro (robot description, xacro)
@@ -147,5 +147,5 @@
   <xacro:robotiq_arg2f_coupling prefix="a_bot_gripper_coupling_"
 				parent="a_bot_flange">
-    <origin xyz="0 0 0" rpy="0 0 0"/>
+    <origin xyz="0 0 0" rpy="${pi} 0 0"/>
   </xacro:robotiq_arg2f_coupling>
   <xacro:include filename="$(find aist_robotiq
@@ -157,5 +157,5 @@
   <xacro:robotiq_arg2f_coupling prefix="b_bot_gripper_coupling_"
 				parent="b_bot_flange">
-    <origin xyz="0 0 0" rpy="0 0 0"/>
+    <origin xyz="0 0 0" rpy="${pi} 0 0"/>
   </xacro:robotiq_arg2f_coupling>
   <xacro:include filename="$(find aist_robotiq

File: moveit_config/a_bot_moveit_config/config/gazebo_a_bot_base_scene.urdf (robot description, URDF)
Before this commit: robot a_bot_base_scene, 82 links, 81 joints
Links:
- removed link a_bot_ftsensor_base_link
- removed link a_bot_ftsensor_flange_link
- removed link a_bot_ftsensor_wrench_link
- added link base_fixture_base_link, mass 0.86387; collision box size=0.049 0.058 0.026; visual mesh filename=package://aist_fastening_tools/meshes/visual/MGPM12-20Z_bod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 scale=0.001 0.001 0.001
- added link base_fixture_piston, mass 0.03804; collision box size=0.007 0.056 0.022; visual mesh filename=package://aist_fastening_tools/meshes/visual/MGPM12-20Z_pis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 scale=0.001 0.001 0.001
- added link base_fixture_piston_head
- added link base_fixture_tip_link
- added link screw_feeder_m3_base_link, mass 1.0; collision box size=0.126 0.126 0.147; visual box size=0.126 0.126 0.147
- added link screw_feeder_m3_front_side, mass 1.0; collision box size=0.056 0.126 0.079; visual box size=0.056 0.126 0.079
- added link screw_feeder_m3_gap, mass 1.0; collision box size=0.056 0.02 0.002; visual box size=0.056 0.02 0.002
- added link screw_feeder_m3_inlet_link
- added link screw_feeder_m3_outlet_link
- added link screw_feeder_m4_base_link, mass 1.0; collision box size=0.126 0.126 0.147; visual box size=0.126 0.126 0.147
- added link screw_feeder_m4_front_side, mass 1.0; collision box size=0.056 0.126 0.079; visual box size=0.056 0.126 0.079
- added link screw_feeder_m4_gap, mass 1.0; collision box size=0.056 0.02 0.002; visual box size=0.056 0.02 0.002
- added link screw_feeder_m4_inlet_link
- added link screw_feeder_m4_outlet_link
- added link workbench_back_bar, mass 1.0; collision box size=0.48 0.02 0.02; visual box size=0.48 0.02 0.02
- added link workbench_base_link, mass 1.0; collision box size=0.48 0.02 0.02; visual box size=0.48 0.02 0.02
- added link workbench_center_bar, mass 1.0; collision box size=0.02 0.28 0.02; visual box size=0.02 0.28 0.02
- added link workbench_front_border, mass 1.0; collision box size=0.08 0.016 0.003; visual box size=0.08 0.016 0.003
- added link workbench_holder_link
- added link workbench_right_bar, mass 1.0; collision box size=0.02 0.28 0.02; visual box size=0.02 0.28 0.02
- added link workbench_right_border, mass 1.0; collision box size=0.016 0.064 0.003; visual box size=0.016 0.064 0.003
- added link workbench_table_base_link, mass 1.0; collision box size=0.02 0.02 0.125; visual box size=0.02 0.02 0.125
- added link workbench_table_leg1, mass 1.0; collision box size=0.02 0.02 0.125; visual box size=0.02 0.02 0.125
- added link workbench_table_leg2, mass 1.0; collision box size=0.02 0.02 0.125; visual box size=0.02 0.02 0.125
- added link workbench_table_leg3, mass 1.0; collision box size=0.02 0.02 0.125; visual box size=0.02 0.02 0.125
- added link workbench_table_top, mass 1.0; collision box size=0.21 0.32 0.005; visual box size=0.21 0.32 0.005
- added link workbench_table_top_center
- added link workbench_table_top_origin
- link a_bot_base_link_inertia: geometry collision mesh filename=package://ur_description/meshes/ur5e/collision/base.stl; visual mesh filename=package://ur_description/meshes/ur5e/visual/base.dae
- link a_bot_forearm_link: geometry collision mesh filename=package://ur_description/meshes/ur5e/collision/forearm.stl; visual mesh filename=package://ur_description/meshes/ur5e/visual/forearm.dae
- link a_bot_shoulder_link: geometry collision mesh filename=package://ur_description/meshes/ur5e/collision/shoulder.stl; visual mesh filename=package://ur_description/meshes/ur5e/visual/shoulder.dae
- link a_bot_upper_arm_link: geometry collision mesh filename=package://ur_description/meshes/ur5e/collision/upperarm.stl; visual mesh filename=package://ur_description/meshes/ur5e/visual/upperarm.dae
- link a_bot_wrist_1_link: geometry collision mesh filename=package://ur_description/meshes/ur5e/collision/wrist1.stl; visual mesh filename=package://ur_description/meshes/ur5e/visual/wrist1.dae
- link a_bot_wrist_2_link: geometry collision mesh filename=package://ur_description/meshes/ur5e/collision/wrist2.stl; visual mesh filename=package://ur_description/meshes/ur5e/visual/wrist2.dae
- link a_bot_wrist_3_link: geometry collision mesh filename=package://ur_description/meshes/ur5e/collision/wrist3.stl; visual mesh filename=package://ur_description/meshes/ur5e/visual/wrist3.dae
Joints:
- removed joint a_bot_ftsensor_flange_joint
- removed joint a_bot_ftsensor_ft300_joint
- removed joint a_bot_ftsensor_wrench_joint
- added joint base_fixture_base_joint: type fixed, parent workbench_table_top_origin, child base_fixture_base_link, origin xyz=0.05729961772434791 0.24786931916155724 0 rpy=0 0 -1.0304423903774522
- added joint base_fixture_piston_head_joint: type fixed, parent base_fixture_piston, child base_fixture_piston_head, origin xyz=0.013      0.0      0.013 rpy=0.0      0.0      0.0
- added joint base_fixture_piston_joint: type prismatic, parent base_fixture_base_link, child base_fixture_piston, axis 1 0 0, limit lower=0 upper=0.02 effort=130 velocity=0.15
- added joint base_fixture_tip_link_joint: type fixed, parent base_fixture_base_link, child base_fixture_tip_link, origin xyz=0.033      0.0      0.013 rpy=0.0      0.0      0.0
- added joint screw_feeder_m3_base_link: type fixed, parent workbench_base_link, child screw_feeder_m3_base_link, origin xyz=0.01 0.03 0 rpy=0 0 0
- added joint screw_feeder_m3_front_side: type fixed, parent screw_feeder_m3_base_link, child screw_feeder_m3_front_side, origin xyz=0.126 0 0 rpy=0 0 0
- added joint screw_feeder_m3_gap: type fixed, parent screw_feeder_m3_front_side, child screw_feeder_m3_gap, origin xyz=0 0.053 0.079 rpy=0 0 0
- added joint screw_feeder_m3_inlet_joint: type fixed, parent screw_feeder_m3_base_link, child screw_feeder_m3_inlet_link, origin xyz=0.072 0.032 0.147 rpy=0 0 0
- added joint screw_feeder_m3_outlet_joint: type fixed, parent screw_feeder_m3_gap, child screw_feeder_m3_outlet_link, origin xyz=0.046 0.01 0.002 rpy=0 0 0
- added joint screw_feeder_m4_base_link: type fixed, parent screw_feeder_m3_base_link, child screw_feeder_m4_base_link, origin xyz=0 0.126 0 rpy=0 0 0
- added joint screw_feeder_m4_front_side: type fixed, parent screw_feeder_m4_base_link, child screw_feeder_m4_front_side, origin xyz=0.126 0 0 rpy=0 0 0
- added joint screw_feeder_m4_gap: type fixed, parent screw_feeder_m4_front_side, child screw_feeder_m4_gap, origin xyz=0 0.053 0.079 rpy=0 0 0
- added joint screw_feeder_m4_inlet_joint: type fixed, parent screw_feeder_m4_base_link, child screw_feeder_m4_inlet_link, origin xyz=0.072 0.032 0.147 rpy=0 0 0
- added joint screw_feeder_m4_outlet_joint: type fixed, parent screw_feeder_m4_gap, child screw_feeder_m4_outlet_link, origin xyz=0.046 0.01 0.002 rpy=0 0 0
- added joint workbench_back_bar: type fixed, parent workbench_base_link, child workbench_back_bar, origin xyz=0 0.3 0 rpy=0 0 0
- added joint workbench_base_link: type fixed, parent cage_workspace_bar, child workbench_base_link, origin xyz=0.04    0.63    0.01 rpy=0 0 0
- added joint workbench_center_bar: type fixed, parent workbench_base_link, child workbench_center_bar, origin xyz=0.27 0.02 0 rpy=0 0 0
- added joint workbench_front_border: type fixed, parent workbench_table_top_origin, child workbench_front_border, origin xyz=0.13 0 0 rpy=0 0 0
- added joint workbench_holder_link_joint: type fixed, parent workbench_table_top_origin, child workbench_holder_link, origin xyz=0.194 0.016 0 rpy=0 0 1.5707963267948966
- added joint workbench_right_bar: type fixed, parent workbench_base_link, child workbench_right_bar, origin xyz=0.45999999999999996 0.02 0 rpy=0 0 0
- added joint workbench_right_border: type fixed, parent workbench_table_top_origin, child workbench_right_border, origin xyz=0.194 0.016 0 rpy=0 0 0
- added joint workbench_table_base_link: type fixed, parent workbench_base_link, child workbench_table_base_link, origin xyz=0.27 0  0.02 rpy=0 0 0
- added joint workbench_table_leg1: type fixed, parent workbench_table_base_link, child workbench_table_leg1, origin xyz=0.19 0 0 rpy=0 0 0
- added joint workbench_table_leg2: type fixed, parent workbench_table_base_link, child workbench_table_leg2, origin xyz=0 0.3 0 rpy=0 0 0
- added joint workbench_table_leg3: type fixed, parent workbench_table_base_link, child workbench_table_leg3, origin xyz=0.19      0.3      0 rpy=0 0 0
- added joint workbench_table_top: type fixed, parent workbench_table_base_link, child workbench_table_top, origin xyz=0 0 0.125 rpy=0 0 0
- added joint workbench_table_top_center_joint: type fixed, parent workbench_table_top_origin, child workbench_table_top_center, origin xyz=0.105 0.16 0 rpy=0 0 0
- added joint workbench_table_top_origin_joint: type fixed, parent workbench_table_top, child workbench_table_top_origin, origin xyz=0 0 0.005 rpy=0 0 0
- joint a_bot_gripper_coupling_base_joint: origin xyz=0 0 0 rpy=0 0 0 -> xyz=0 0 0 rpy=3.141592653589793 0 0; parent a_bot_ftsensor_flange_link -> a_bot_flange
- joint suction_tool_holder_joint: origin xyz=0.11032 0.000 0.03784 rpy=0 0.5235987755982988 0 -> xyz=0.08732 0.0 -0.002 rpy=0 0.5235987755982988 0

File: moveit_config/aist_moveit_config/config/gazebo_aist_base_scene.urdf (robot description, URDF)
Before this commit: robot aist_base_scene, 139 links, 138 joints
Joints:
- joint a_bot_gripper_coupling_base_joint: origin xyz=0 0 0 rpy=0 0 0 -> xyz=0 0 0 rpy=3.141592653589793 0 0
- joint b_bot_gripper_coupling_base_joint: origin xyz=0 0 0 rpy=0 0 0 -> xyz=0 0 0 rpy=3.141592653589793 0 0

Commit message: WIP

File: aist_description/scenes/urdf/a_bot_base_scene.urdf.xacro (robot description, xacro)
@@ -130,8 +130,8 @@
   <!-- RealSense cameras -->
   <xacro:include filename="$(find aist_description
-  			   )/devices/urdf/wrist_cameras.urdf.xacro" />
-  <xacro:wrist_cameras prefix="a_bot_"
-  		       parent="a_bot_gripper_base_link"
-  		       use_nominal_extrinsics="true"/>
+  			   )/devices/urdf/sr305_on_2f140.urdf.xacro" />
+  <xacro:sr305_on_2f140 prefix="a_bot_"
+  			parent="a_bot_gripper_base_link"
+  			use_nominal_extrinsics="true"/>
   <!-- I would like to remove the "world" link definition, but apparently it is necessary for Gazebo -->
   <link name="world"/>

File: moveit_config/a_bot_moveit_config/config/gazebo_a_bot_base_scene.urdf (robot description, URDF)
Before this commit: robot a_bot_base_scene, 198 links, 197 joints
Links:
- removed link a_bot_inside_camera_color_frame
- removed link a_bot_inside_camera_color_optical_frame
- removed link a_bot_inside_camera_connector_link
- removed link a_bot_inside_camera_depth_frame
- removed link a_bot_inside_camera_depth_optical_frame
- removed link a_bot_inside_camera_left_ir_frame
- removed link a_bot_inside_camera_left_ir_optical_frame
- removed link a_bot_inside_camera_link
- removed link a_bot_inside_camera_right_ir_frame
- removed link a_bot_inside_camera_right_ir_optical_frame
- removed link a_bot_outside_camera_color_frame
- removed link a_bot_outside_camera_color_optical_frame
- removed link a_bot_outside_camera_connector_link
- removed link a_bot_outside_camera_depth_frame
- removed link a_bot_outside_camera_depth_optical_frame
- removed link a_bot_outside_camera_left_ir_frame
- removed link a_bot_outside_camera_left_ir_optical_frame
- removed link a_bot_outside_camera_link
- removed link a_bot_outside_camera_right_ir_frame
- removed link a_bot_outside_camera_right_ir_optical_frame
- added link a_bot_camera_color_frame
- added link a_bot_camera_color_optical_frame
- added link a_bot_camera_connector_link
- added link a_bot_camera_depth_frame
- added link a_bot_camera_depth_optical_frame
- added link a_bot_camera_left_ir_frame
- added link a_bot_camera_left_ir_optical_frame
- added link a_bot_camera_link, mass 0.564; collision box size=0.012 0.14 0.023; visual mesh filename=package://realsense2_description/meshes/sr305_without_mount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 scale=.001 .001 .001
- added link a_bot_camera_right_ir_frame
- added link a_bot_camera_right_ir_optical_frame
- link a_bot_camera_mount: geometry collision box size=.03 .12 .08; visual mesh filename=package://aist_description/devices/meshes/sr305_mount_2f140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 scale=.001 .001 .001
Joints:
- removed joint a_bot_inside_camera_color_joint
- removed joint a_bot_inside_camera_color_optical_joint
- removed joint a_bot_inside_camera_depth_joint
- removed joint a_bot_inside_camera_depth_optical_joint
- removed joint a_bot_inside_camera_joint
- removed joint a_bot_inside_camera_left_ir_joint
- removed joint a_bot_inside_camera_left_ir_optical_joint
- removed joint a_bot_inside_camera_link_joint
- removed joint a_bot_inside_camera_right_ir_joint
- removed joint a_bot_inside_camera_right_ir_optical_joint
- removed joint a_bot_outside_camera_color_joint
- removed joint a_bot_outside_camera_color_optical_joint
- removed joint a_bot_outside_camera_depth_joint
- removed joint a_bot_outside_camera_depth_optical_joint
- removed joint a_bot_outside_camera_joint
- removed joint a_bot_outside_camera_left_ir_joint
- removed joint a_bot_outside_camera_left_ir_optical_joint
- removed joint a_bot_outside_camera_link_joint
- removed joint a_bot_outside_camera_right_ir_joint
- removed joint a_bot_outside_camera_right_ir_optical_joint
- added joint a_bot_camera_color_joint: type fixed, parent a_bot_camera_depth_frame, child a_bot_camera_color_frame, origin xyz=0 0.015 0 rpy=0 0 0
- added joint a_bot_camera_color_optical_joint: type fixed, parent a_bot_camera_color_frame, child a_bot_camera_color_optical_frame, origin xyz=0 0 0 rpy=-1.5707963267948966 0 -1.5707963267948966
- added joint a_bot_camera_depth_joint: type fixed, parent a_bot_camera_link, child a_bot_camera_depth_frame, origin xyz=.003721 0 0 rpy=0 0 0
- added joint a_bot_camera_depth_optical_joint: type fixed, parent a_bot_camera_depth_frame, child a_bot_camera_depth_optical_frame, origin xyz=0 0 0 rpy=-1.5707963267948966 0 -1.5707963267948966
- added joint a_bot_camera_joint: type fixed, parent a_bot_gripper_base_link, child a_bot_camera_connector_link, origin xyz=0.08046421018432694      -0.013512509598350497      0.09167488147585981 rpy=0.005347150648361527      0.38666681358877475      0.0005141030065124729
- added joint a_bot_camera_left_ir_joint: type fixed, parent a_bot_camera_depth_frame, child a_bot_camera_left_ir_frame, origin xyz=0 0.0 0 rpy=0 0 0
- added joint a_bot_camera_left_ir_optical_joint: type fixed, parent a_bot_camera_left_ir_frame, child a_bot_camera_left_ir_optical_frame, origin xyz=0 0 0 rpy=-1.5707963267948966 0 -1.5707963267948966
- added joint a_bot_camera_link_joint: type fixed, parent a_bot_camera_connector_link, child a_bot_camera_link, origin xyz=0 0 0 rpy=0 0 0
- added joint a_bot_camera_right_ir_joint: type fixed, parent a_bot_camera_depth_frame, child a_bot_camera_right_ir_frame, origin xyz=0 0.04 0 rpy=0 0 0
- added joint a_bot_camera_right_ir_optical_joint: type fixed, parent a_bot_camera_right_ir_frame, child a_bot_camera_right_ir_optical_frame, origin xyz=0 0 0 rpy=-1.5707963267948966 0 -1.5707963267948966
