Commit message: Insert coupling between robotiq gripper and flange

File: aist_description/scenes/urdf/aist_base_scene.urdf.xacro (robot description, xacro)
@@ -69,7 +69,13 @@
   </xacro:ft300>
   <!-- Spawn and attach gripper -->
+  <xacro:include filename="$(find robotiq_description
+			   )/urdf/robotiq_arg2f_coupling.urdf.xacro"/>
+  <xacro:robotiq_arg2f_coupling prefix="a_bot_"
+				parent="a_bot_ft300_flange_link">
+    <origin xyz="0 0 0" rpy="0 0 0"/>
+  </xacro:robotiq_arg2f_coupling>
   <xacro:include filename="$(find aist_description)/devices/urdf/robotiq_85_gripper_with_tip_link.urdf.xacro"/>
   <xacro:robotiq_85_gripper_with_tip_link prefix="a_bot_"
-					  parent="a_bot_ft300_flange_link">
+					  parent="a_bot_robotiq_arg2f_coupling_flange_link">
     <origin xyz="0 0 0" rpy="0 0 0"/>
   </xacro:robotiq_85_gripper_with_tip_link>

File: aist_description/scenes/urdf/diiwa_base_scene.urdf.xacro (robot description, xacro)
@@ -40,8 +40,14 @@
   </xacro:iiwa14>
   <!-- Attach grippers -->
+  <xacro:include filename="$(find robotiq_description
+			   )/urdf/robotiq_arg2f_coupling.urdf.xacro"/>
+  <xacro:robotiq_arg2f_coupling prefix="a_iiwa_"
+				parent="a_iiwa_ee_link">
+    <origin xyz="0 0 0" rpy="0 0 0"/>
+  </xacro:robotiq_arg2f_coupling>
   <xacro:include filename="$(find aist_description
   			   )/devices/urdf/robotiq_85_gripper_with_tip_link.urdf.xacro"/>
   <xacro:robotiq_85_gripper_with_tip_link prefix="a_iiwa_"
-  					  parent="a_iiwa_ee_link">
+  					  parent="a_iiwa_robotiq_arg2f_coupling_flange_link">
     <origin xyz="0 0 0" rpy="0 0 0"/>
   </xacro:robotiq_85_gripper_with_tip_link>

File: aist_description/scenes/urdf/fvision_base_scene.urdf.xacro (robot description, xacro)
@@ -44,7 +44,13 @@
   </joint>
   <!-- Spawn and attach gripper -->
+  <xacro:include filename="$(find robotiq_description
+			   )/urdf/robotiq_arg2f_coupling.urdf.xacro"/>
+  <xacro:robotiq_arg2f_coupling prefix="d_bot_"
+				parent="d_bot_ee_link">
+    <origin xyz="0 0 0" rpy="0 0 0"/>
+  </xacro:robotiq_arg2f_coupling>
   <xacro:include filename="$(find aist_description)/devices/urdf/robotiq_hande_gripper_with_tip_link.urdf.xacro"/>
   <xacro:robotiq_hande_gripper_with_tip_link prefix="d_bot_"
-					     parent="d_bot_ee_link">
+					     parent="d_bot_robotiq_arg2f_coupling_flange_link">
     <origin xyz="0 0 0" rpy="0 0 0"/>
   </xacro:robotiq_hande_gripper_with_tip_link>

File: aist_description/scenes/urdf/mocap_base_scene.urdf.xacro (robot description, xacro)
@@ -41,8 +41,14 @@
   </joint>
   <!-- Spawn and attach gripper -->
+  <xacro:include filename="$(find robotiq_description
+			   )/urdf/robotiq_arg2f_coupling.urdf.xacro"/>
+  <xacro:robotiq_arg2f_coupling prefix="c_bot_"
+				parent="c_bot_ee_link">
+    <origin xyz="0 0 0" rpy="0 0 0"/>
+  </xacro:robotiq_arg2f_coupling>
   <xacro:include filename="$(find aist_description
 			   )/devices/urdf/robotiq_85_gripper_with_tip_link.urdf.xacro"/>
   <xacro:robotiq_85_gripper_with_tip_link prefix="c_bot_"
-					  parent="c_bot_ee_link">
+					  parent="c_bot_robotiq_arg2f_coupling_flange_link">
     <origin xyz="0 0 0" rpy="0 0 0"/>
   </xacro:robotiq_85_gripper_with_tip_link>

File: aist_description/scenes/urdf/ur10e_base_scene.urdf.xacro (robot description, xacro)
@@ -43,13 +43,19 @@
   </joint>
   <!-- Spawn and attach gripper -->
+  <xacro:include filename="$(find robotiq_description
+			   )/urdf/robotiq_arg2f_coupling.urdf.xacro"/>
+  <xacro:robotiq_arg2f_coupling prefix="a_bot_"
+				parent="a_bot_ee_link">
+    <origin xyz="0 0 0" rpy="0 0 0"/>
+  </xacro:robotiq_arg2f_coupling>
   <xacro:include filename="$(find aist_description)/devices/urdf/robotiq_140_gripper_with_tip_link.urdf.xacro"/>
   <xacro:robotiq_140_gripper_with_tip_link prefix="a_bot_"
-					   parent="a_bot_ee_link">
+					   parent="a_bot_robotiq_arg2f_coupling_flange_link">
     <origin xyz="0 0 0" rpy="0 0 0"/>
   </xacro:robotiq_140_gripper_with_tip_link>
   <!-- Add RealSense camera -->
-  <xacro:include filename="$(find aist_description
-			   )/devices/urdf/wrist_d435.urdf.xacro" />
-  <xacro:wrist_d435 prefix="a_bot_" parent="a_bot_robotiq_140_base_link"/>
+  <!-- <xacro:include filename="$(find aist_description -->
+  <!-- 			   )/devices/urdf/wrist_d435.urdf.xacro" /> -->
+  <!-- <xacro:wrist_d435 prefix="a_bot_" parent="a_bot_robotiq_140_base_link"/> -->
   <!-- I would like to remove the "world" link definition, but apparently it is necessary for Gazebo -->
   <link name="world"/>

File: aist_description/scenes/urdf/ur5e_base_scene.urdf.xacro (robot description, xacro)
@@ -60,7 +60,13 @@
   </joint>
   <!-- Spawn and attach gripper -->
+  <xacro:include filename="$(find robotiq_description
+			   )/urdf/robotiq_arg2f_coupling.urdf.xacro"/>
+  <xacro:robotiq_arg2f_coupling prefix="c_bot_"
+				parent="c_bot_ee_link">
+    <origin xyz="0 0 0" rpy="0 0 0"/>
+  </xacro:robotiq_arg2f_coupling>
   <xacro:include filename="$(find aist_description)/devices/urdf/robotiq_85_gripper_with_tip_link.urdf.xacro"/>
   <xacro:robotiq_85_gripper_with_tip_link prefix="c_bot_"
-					  parent="c_bot_ee_link">
+					  parent="c_bot_robotiq_arg2f_coupling_flange_link">
     <origin xyz="0 0 0" rpy="0 0 0"/>
   </xacro:robotiq_85_gripper_with_tip_link>
@@ -78,7 +84,11 @@
   <!--   <origin xyz="0 0 0" rpy="0 0 0"/> -->
   <!-- </xacro:robotiq_85_gripper_with_tip_link> -->
+  <xacro:robotiq_arg2f_coupling prefix="d_bot_"
+				parent="d_bot_ee_link">
+    <origin xyz="0 0 0" rpy="0 0 0"/>
+  </xacro:robotiq_arg2f_coupling>
   <xacro:include filename="$(find aist_description)/devices/urdf/robotiq_hande_gripper_with_tip_link.urdf.xacro"/>
   <xacro:robotiq_hande_gripper_with_tip_link prefix="d_bot_"
-					     parent="d_bot_ee_link">
+					     parent="d_bot_robotiq_arg2f_coupling_flange_link">
     <origin xyz="0 0 0" rpy="0 0 0"/>
   </xacro:robotiq_hande_gripper_with_tip_link>

File: aist_description/scenes/urdf/ur_trial_a_base_scene.urdf.xacro (robot description, xacro)
@@ -44,14 +44,22 @@
   <!-- Spawn and attach force sensor -->
   <xacro:include filename="$(find aist_ftsensor)/urdf/ft300.urdf.xacro"/>
-  <xacro:ft300 prefix="a_bot_" parent="a_bot_ee_link">
+  <xacro:ft300 prefix="a_bot_"
+	       parent="a_bot_ee_link">
     <origin xyz="0 0 0" rpy="0 0 0"/>
   </xacro:ft300>
   <!-- Spawn and attach gripper -->
-  <!-- <xacro:include filename="$(find aist_description)/devices/urdf/robotiq_85_gripper_with_tip_link.urdf.xacro"/> -->
-  <!-- <xacro:robotiq_85_gripper_with_tip_link prefix="a_bot_" -->
-  <!-- 					  parent="a_bot_ft300_flange_link"> -->
-  <!--   <origin xyz="0 0 0" rpy="0 0 0"/> -->
-  <!-- </xacro:robotiq_85_gripper_with_tip_link> -->
-  <xacro:include filename="$(find aist_description)/devices/urdf/single_suction_gripper.urdf.xacro"/>
+  <xacro:include filename="$(find robotiq_description
+			   )/urdf/robotiq_arg2f_coupling.urdf.xacro"/>
+  <xacro:robotiq_arg2f_coupling prefix="a_bot_"
+				parent="a_bot_ft300_flange_link">
+    <origin xyz="0 0 0" rpy="0 0 0"/>
+  </xacro:robotiq_arg2f_coupling>
+  <xacro:include filename="$(find aist_description)/devices/urdf/robotiq_85_gripper_with_tip_link.urdf.xacro"/>
+  <xacro:robotiq_85_gripper_with_tip_link prefix="a_bot_"
+  					  parent="a_bot_robotiq_arg2f_coupling_flange_link">
+    <origin xyz="0 0 0" rpy="0 0 0"/>
+  </xacro:robotiq_85_gripper_with_tip_link>
+  <xacro:include filename="$(find aist_description
+			   )/devices/urdf/single_suction_gripper.urdf.xacro"/>
   <!-- Add virtual wall to avoid collisions-->
   <xacro:aist_box name="vwall1" width="0.01" length="0.3" height="0.5"

Commit message: Make gazebo works under ur_robot_driver

File: aist_description/scenes/urdf/aist_base_scene.urdf.xacro (robot description, xacro)
@@ -30,8 +30,8 @@
   </joint>
   <!-- robot arms -->
-  <xacro:include filename="$(find ur_description)/urdf/common.gazebo.xacro"/>
-  <!-- <xacro:include filename="$(find aist_description -->
-  <!-- 			   )/scenes/urdf/gazebo_ros_control.gazebo.xacro"/> -->
-  <!-- <xacro:gazebo_ros_control ns="/"/> -->
+  <!-- <xacro:include filename="$(find ur_description)/urdf/common.gazebo.xacro"/> -->
+  <xacro:include filename="$(find aist_description
+  			   )/scenes/urdf/gazebo_ros_control.gazebo.xacro"/>
+  <xacro:gazebo_ros_control ns="/a_bot"/>
   <xacro:include filename="$(find ur_description)/urdf/ur5.urdf.xacro"/>
   <xacro:ur5_robot prefix="a_bot_" joint_limited="false"
@@ -45,4 +45,5 @@
 		     )/config/a_bot_calibration.yaml')}"/>
   <!-- <xacro:gazebo_ros_control ns="/b_bot"/> -->
+  <xacro:gazebo_ros_control ns="/b_bot"/>
   <xacro:ur5_robot prefix="b_bot_" joint_limited="false"
     shoulder_pan_lower_limit="${-pi}" shoulder_pan_upper_limit="${pi}"

File: aist_description/scenes/urdf/ur_trial_a_base_scene.urdf.xacro (robot description, xacro)
@@ -2,13 +2,11 @@
 <robot xmlns:xacro="http://wiki.ros.org/xacro" name="ur_trial_a" >
   <xacro:arg name="scene" default=""/>
-  <!-- Calibration help: If the robot is not moving far enough to the calibration point, increase these distances -->
   <xacro:property name="a_bot_x" value="0"/>
   <xacro:property name="a_bot_y" value="-0.4875"/>
   <xacro:property name="bots_z" value="0.77"/>
-  <!-- This is the main file defining our robot arrangement and physical environment. -->
   <!-- Main workspace -->
-  <!-- The surface is 0.01 m below the robot bases and the "workspace_center" frame. -->
   <link name="ground"/>
-  <xacro:include filename="$(find aist_description)/objects/urdf/aist_box.urdf.xacro"/>
+  <xacro:include filename="$(find aist_description
+			   )/objects/urdf/aist_box.urdf.xacro"/>
   <xacro:property name="table_w" value="0.9"/>
   <xacro:property name="table_l" value="1.8"/>
@@ -26,5 +24,8 @@
   </joint>
   <!-- robot arms -->
-  <xacro:include filename="$(find ur_description)/urdf/common.gazebo.xacro"/>
+  <!-- <xacro:include filename="$(find ur_description)/urdf/common.gazebo.xacro"/> -->
+  <xacro:include filename="$(find aist_description
+  			   )/scenes/urdf/gazebo_ros_control.gazebo.xacro"/>
+  <xacro:gazebo_ros_control ns="/"/>
   <xacro:include filename="$(find ur_description)/urdf/ur5.urdf.xacro"/>
   <xacro:ur5_robot prefix="a_bot_" joint_limited="false"
@@ -55,32 +56,10 @@
     <origin xyz="0 0 0" rpy="0 0 0"/>
   </xacro:robotiq_arg2f_coupling>
-  <xacro:include filename="$(find aist_description)/devices/urdf/robotiq_85_gripper_with_tip_link.urdf.xacro"/>
+  <xacro:include filename="$(find aist_description
+			   )/devices/urdf/robotiq_85_gripper_with_tip_link.urdf.xacro"/>
   <xacro:robotiq_85_gripper_with_tip_link prefix="a_bot_gripper_"
   					  parent="a_bot_gripper_coupling_flange_link">
     <origin xyz="0 0 0" rpy="0 0 0"/>
   </xacro:robotiq_85_gripper_with_tip_link>
-  <xacro:include filename="$(find aist_description
-			   )/devices/urdf/single_suction_gripper.urdf.xacro"/>
-  <!-- Add virtual wall to avoid collisions-->
-  <xacro:aist_box name="vwall1" width="0.01" length="0.3" height="0.5"
-		  parent="ground" transparent="true">
-    <origin xyz="0.45 -0.15 ${bots_z}" rpy="0 0 0"/>
-  </xacro:aist_box>
-  <!-- Add PhoXi 3D scanner -->
-  <xacro:include filename="$(find
-			   aist_phoxi_camera)/urdf/phoxi_m_camera.urdf.xacro"/>
-  <xacro:phoxi_m_camera prefix="a_phoxi_m_" parent="workspace_center">
-    <origin xyz="0.483543436025
-		 -0.0149511700982
-		 0.633792706454"
-	    rpy="${-152.286950706*pi/180}
-		 ${-2.00315281361*pi/180}
-		 ${86.7522427304*pi/180}"/>
-  </xacro:phoxi_m_camera>
-  <!-- Add RealSense camera -->
-  <!-- <xacro:include filename="$(find aist_description -->
-  <!-- 			   )/devices/urdf/wrist_cameras.urdf.xacro" /> -->
-  <!-- <xacro:wrist_cameras prefix="a_bot_" -->
-  <!-- 		       parent="a_bot_robotiq_85_base_link"/> -->
   <!-- I would like to remove the "world" link definition, but apparently it is necessary for Gazebo -->
   <link name="world"/>

Commit message: Make controller_spawner launced in root namespace for gazebo under ur_robot_driver

File: aist_description/scenes/urdf/aist_base_scene.urdf.xacro (robot description, xacro)
@@ -30,8 +30,5 @@
   </joint>
   <!-- robot arms -->
-  <!-- <xacro:include filename="$(find ur_description)/urdf/common.gazebo.xacro"/> -->
-  <xacro:include filename="$(find aist_description
-  			   )/scenes/urdf/gazebo_ros_control.gazebo.xacro"/>
-  <xacro:gazebo_ros_control ns="/a_bot"/>
+  <xacro:include filename="$(find ur_description)/urdf/common.gazebo.xacro"/>
   <xacro:include filename="$(find ur_description)/urdf/ur5.urdf.xacro"/>
   <xacro:ur5_robot prefix="a_bot_" joint_limited="false"
@@ -45,5 +42,4 @@
 		     )/config/a_bot_calibration.yaml')}"/>
   <!-- <xacro:gazebo_ros_control ns="/b_bot"/> -->
-  <xacro:gazebo_ros_control ns="/b_bot"/>
   <xacro:ur5_robot prefix="b_bot_" joint_limited="false"
     shoulder_pan_lower_limit="${-pi}" shoulder_pan_upper_limit="${pi}"

File: aist_description/scenes/urdf/fvision_base_scene.urdf.xacro (robot description, xacro)
@@ -50,19 +50,9 @@
     <origin xyz="0 0 0" rpy="0 0 0"/>
   </xacro:robotiq_arg2f_coupling>
-  <xacro:include filename="$(find aist_description)/devices/urdf/robotiq_hande_gripper_with_tip_link.urdf.xacro"/>
-  <xacro:robotiq_hande_gripper_with_tip_link prefix="d_bot_gripper_"
-					     parent="d_bot_gripper_coupling_flange_link">
+  <xacro:include filename="$(find aist_description)/devices/urdf/robotiq_140_gripper_with_tip_link.urdf.xacro"/>
+  <xacro:robotiq_140_gripper_with_tip_link prefix="d_bot_gripper_"
+					   parent="d_bot_gripper_coupling_flange_link">
     <origin xyz="0 0 0" rpy="0 0 0"/>
-  </xacro:robotiq_hande_gripper_with_tip_link>
-  <!-- Add PhoXi 3D scanner -->
-  <xacro:include filename="$(find aist_phoxi_camera)/urdf/phoxi_m_camera.urdf.xacro"/>
-  <xacro:phoxi_m_camera prefix="b_" parent="ground">
-    <origin xyz="0.547941636523
-		 -0.00827443204237
-		 1.67030171767"
-	    rpy="${-151.493605482*pi/180}
-		 ${0.698490882792*pi/180}
-		 ${85.0482907121*pi/180}"/>
-  </xacro:phoxi_m_camera>
+  </xacro:robotiq_140_gripper_with_tip_link>
   <!-- I would like to remove the "world" link definition, but apparently it is necessary for Gazebo -->
   <link name="world"/>

File: aist_description/scenes/urdf/ur_trial_a_base_scene.urdf.xacro (robot description, xacro)
@@ -24,8 +24,5 @@
   </joint>
   <!-- robot arms -->
-  <!-- <xacro:include filename="$(find ur_description)/urdf/common.gazebo.xacro"/> -->
-  <xacro:include filename="$(find aist_description
-  			   )/scenes/urdf/gazebo_ros_control.gazebo.xacro"/>
-  <xacro:gazebo_ros_control ns="/"/>
+  <xacro:include filename="$(find ur_description)/urdf/common.gazebo.xacro"/>
   <xacro:include filename="$(find ur_description)/urdf/ur5.urdf.xacro"/>
   <xacro:ur5_robot prefix="a_bot_" joint_limited="false"

Commit message: Replace PhoXi camera and changed its ID in launch files

File: aist_description/scenes/urdf/aist_base_scene.urdf.xacro (robot description, xacro)
@@ -85,10 +85,10 @@
   				parent="b_bot_ftsensor_flange_link">
     <!-- <origin xyz="0 0 0" rpy="0 ${0.2*pi/180} ${-1.2*pi/180}"/> -->
-    <origin xyz="0 0 0" rpy="0 ${-0.1*pi/180} ${0.45*pi/180}"/>
+    <origin xyz="0 0 0" rpy="0 ${-0.1*pi/180} ${0.15*pi/180}"/>
   </xacro:single_suction_gripper>
   <!-- Add virtual wall to avoid collisions-->
   <xacro:aist_box name="vwall1" width="0.01" length="0.3" height="0.5"
-		  parent="ground" transparent="true">
-    <origin xyz="0.45 -0.15 ${bots_z}" rpy="0 0 0"/>
+		  parent="ground" transparent="false">
+    <origin xyz="0.41 -0.20 ${bots_z}" rpy="0 0 0"/>
   </xacro:aist_box>
   <!-- Add PhoXi 3D scanner -->

Commit message: WIP: Modify yaml and launch files concerning with ur robots

File: aist_description/scenes/urdf/aist_base_scene.urdf.xacro (robot description, xacro)
@@ -30,25 +30,27 @@
   </joint>
   <!-- robot arms -->
-  <xacro:include filename="$(find ur_description)/urdf/common.gazebo.xacro"/>
-  <xacro:include filename="$(find ur_description)/urdf/ur5.urdf.xacro"/>
-  <xacro:ur5_robot prefix="a_bot_" joint_limited="false"
-    shoulder_pan_lower_limit="${-pi}" shoulder_pan_upper_limit="${pi}"
-    shoulder_lift_lower_limit="${-pi}" shoulder_lift_upper_limit="${pi}"
-    elbow_joint_lower_limit="0.0" elbow_joint_upper_limit="${pi}"
-    wrist_1_lower_limit="${-pi}" wrist_1_upper_limit="${pi}"
-    wrist_2_lower_limit="${-pi}" wrist_2_upper_limit="${pi}"
-    wrist_3_lower_limit="${-pi}" wrist_3_upper_limit="${pi}"
-    kinematics_file="${load_yaml('$(find aist_bringup
-		     )/config/a_bot_calibration.yaml')}"/>
+  <!-- <xacro:include filename="$(find ur_description)/urdf/common.gazebo.xacro"/> -->
+  <xacro:include filename="$(find ur_gazebo)/urdf/ur_macro.xacro"/>
+  <xacro:ur_robot_gazebo
+      prefix="a_bot_"
+      joint_limits_parameters_file="$(find ur_description
+				    )/config/ur5/joint_limits.yaml"
+      physical_parameters_file="$(find ur_description
+				)/config/ur5/physical_parameters.yaml"
+      visual_parameters_file="$(find ur_description
+			      )/config/ur5/visual_parameters.yaml"
+      kinematics_parameters_file="$(find aist_bringup
+				  )/config/a_bot_calibration.yaml"/>
   <!-- <xacro:gazebo_ros_control ns="/b_bot"/> -->
-  <xacro:ur5_robot prefix="b_bot_" joint_limited="false"
-    shoulder_pan_lower_limit="${-pi}" shoulder_pan_upper_limit="${pi}"
-    shoulder_lift_lower_limit="${-pi}" shoulder_lift_upper_limit="${pi}"
-    elbow_joint_lower_limit="0.0" elbow_joint_upper_limit="${pi}"
-    wrist_1_lower_limit="${-pi}" wrist_1_upper_limit="${pi}"
-    wrist_2_lower_limit="${-pi}" wrist_2_upper_limit="${pi}"
-    wrist_3_lower_limit="${-pi}" wrist_3_upper_limit="${pi}"
-    kinematics_file="${load_yaml('$(find aist_bringup
-		     )/config/b_bot_calibration.yaml')}"/>
+  <xacro:ur_robot_gazebo
+      prefix="b_bot_"
+      joint_limits_parameters_file="$(find ur_description
+				    )/config/ur5/joint_limits.yaml"
+      physical_parameters_file="$(find ur_description
+				)/config/ur5/physical_parameters.yaml"
+      visual_parameters_file="$(find ur_description
+			      )/config/ur5/visual_parameters.yaml"
+      kinematics_parameters_file="$(find aist_bringup
+				  )/config/b_bot_calibration.yaml"/>
   <joint name="ground_a_bot_joint" type="fixed">
     <parent link="ground"/>
@@ -63,9 +65,9 @@
   <!-- Spawn and attach force sensor -->
   <xacro:include filename="$(find aist_ftsensor)/urdf/ft300.urdf.xacro"/>
-  <xacro:ft300 prefix="a_bot_ftsensor_" parent="a_bot_ee_link">
-    <origin xyz="0 0 0" rpy="0 0 0"/>
+  <xacro:ft300 prefix="a_bot_ftsensor_" parent="a_bot_flange">
+    <origin xyz="0 0 0" rpy="${pi} 0 0"/>
   </xacro:ft300>
-  <xacro:ft300 prefix="b_bot_ftsensor_" parent="b_bot_ee_link">
-    <origin xyz="0 0 0" rpy="0 0 0"/>
+  <xacro:ft300 prefix="b_bot_ftsensor_" parent="b_bot_flange">
+    <origin xyz="0 0 0" rpy="${pi} 0 0"/>
   </xacro:ft300>
   <!-- Spawn and attach gripper -->

Commit message: Fixed orientation of b_bot_ar_marker

File: aist_description/scenes/urdf/aist_base_scene.urdf.xacro (robot description, xacro)
@@ -112,4 +112,14 @@
   <xacro:wrist_cameras prefix="a_bot_"
   		       parent="a_bot_gripper_base_link"/>
+  <!-- Add live camera -->
+  <xacro:load_calibration filename="$(find aist_camera_calibration
+				    )/calib/live_camera.yaml"/>
+  <link name="live_camera_optical_frame"/>
+  <joint name="workspace_live_camera_joint" type="fixed">
+    <parent link="workspace_center"/>
+    <child  link="live_camera_optical_frame"/>
+    <origin xyz="${origin[0]} ${origin[1]} ${origin[2]}"
+    	    rpy="${origin[3]} ${origin[4]} ${origin[5]}"/>
+  </joint>
   <!-- I would like to remove the "world" link definition, but apparently it is necessary for Gazebo -->
   <link name="world"/>

File: aist_description/scenes/urdf/calibration.urdf.xacro (robot description, xacro)
@@ -13,5 +13,5 @@
   			marker_id="26"
 			thickness="0.005">
-    <origin xyz="0.063 0.0 0.0215" rpy="0 0 0"/>
+    <origin xyz="0.063 0.0 0.0215" rpy="0 0 ${pi/2}"/>
   </xacro:ar_marker_70_5>
   <!-- <xacro:ar_marker_70_5 prefix="workspace_" -->

Commit message: Add cage to aist_base_scene

File: aist_description/scenes/urdf/aist_base_scene.urdf.xacro (robot description, xacro)
@@ -2,23 +2,21 @@
 <robot xmlns:xacro="http://wiki.ros.org/xacro" name="aist_base_scene" >
   <xacro:arg name="scene" default=""/>
-  <xacro:property name="a_bot_x" value="0"/>
-  <xacro:property name="a_bot_y" value="-0.4875"/>
-  <!-- <xacro:property name="a_bot_theta" value="${pi}"/> -->
-  <xacro:property name="b_bot_x" value="0"/>
-  <xacro:property name="b_bot_y" value="0.4875"/>
-  <xacro:property name="b_bot_theta" value="${pi}"/>
-  <xacro:property name="bots_z" value="0.77"/>
+  <xacro:property name="a_bot_x"	value="0"/>
+  <xacro:property name="a_bot_y"	value="-0.4875"/>
+  <xacro:property name="b_bot_x"	value="0"/>
+  <xacro:property name="b_bot_y"	value="0.4875"/>
+  <xacro:property name="b_bot_theta"	value="${pi}"/>
+  <xacro:property name="bots_z"		value="0.770"/>
   <!-- ground and workspace -->
   <link name="ground"/>
-  <xacro:property name="table_w" value="0.9"/>
-  <xacro:property name="table_l" value="1.8"/>
-  <xacro:property name="table_h" value="0.01"/>
+  <xacro:property name="table_w"	value="0.900"/>
+  <xacro:property name="table_l"	value="1.800"/>
   <xacro:include filename="$(find aist_description
-			   )/objects/urdf/aist_box.urdf.xacro"/>
-  <xacro:aist_box name="workbox"
-		  width="${table_w}" length="${table_l}" height="${table_h}"
-		  parent="ground">
-    <origin xyz="${-table_w/2} ${-table_l/2} ${bots_z - table_h}" rpy="0 0 0"/>
-  </xacro:aist_box>
+			   )/objects/urdf/table.urdf.xacro"/>
+  <xacro:table prefix="workspace_"
+	       width="${table_w}" length="${table_l}" height="${bots_z}"
+	       parent="ground">
+    <origin xyz="${-table_w/2} ${-table_l/2} 0" rpy="0 0 0"/>
+  </xacro:table>
   <link name="workspace_center"/>
   <joint name="ground_to_workspace" type="fixed">
@@ -27,4 +25,23 @@
     <origin xyz="0 0 ${bots_z}" rpy="0 0 0"/>
   </joint>
+  <!-- cage -->
+  <xacro:property name="cage_w"		value="1.300"/>
+  <xacro:property name="cage_l"		value="1.700"/>
+  <xacro:property name="cage_h"		value="1.500"/>
+  <xacro:property name="cage_t"		value="0.050"/>
+  <xacro:property name="toolbar_h"	value="0.300"/>
+  <xacro:property name="cage_z"		value="0.100"/>
+  <xacro:property name="cage_offset"	value="-0.050"/>
+  <xacro:include filename="$(find aist_description
+			   )/objects/urdf/cage.urdf.xacro"/>
+  <xacro:cage prefix="cage_"
+	      width="${cage_w}" length="${cage_l}" height="${cage_h}"
+	      thickness="${cage_t}"
+	      workspace_height="${bots_z - cage_z}"
+	      toolbar_height="${toolbar_h}"
+	      parent="ground">
+    <origin xyz="${-cage_w/2 + cage_offset} ${-cage_l/2} ${cage_z}"
+	    rpy="0 0 0" />
+  </xacro:cage>
   <!-- robot arms -->
   <xacro:include filename="$(find ur_gazebo)/urdf/ur_macro.xacro"/>
