Commit message: Change cage size

File: aist_description/scenes/urdf/aist_base_scene.urdf.xacro (robot description, xacro)
@@ -26,11 +26,11 @@
   </joint>
   <!-- cage -->
-  <xacro:property name="cage_w"		value="1.300"/>
-  <xacro:property name="cage_l"		value="1.700"/>
-  <xacro:property name="cage_h"		value="1.500"/>
+  <xacro:property name="cage_w"		value="1.220"/>
+  <xacro:property name="cage_l"		value="1.600"/>
+  <xacro:property name="cage_h"		value="1.400"/>
   <xacro:property name="cage_t"		value="0.050"/>
   <xacro:property name="toolbar_h"	value="0.300"/>
-  <xacro:property name="cage_z"		value="0.100"/>
-  <xacro:property name="cage_offset"	value="-0.050"/>
+  <xacro:property name="cage_z"		value="0.164"/>
+  <xacro:property name="cage_offset"	value="0.020"/>
   <xacro:include filename="$(find aist_description
 			   )/objects/urdf/cage.urdf.xacro"/>

Commit message: Remove virtual wall for avoiding collision with camera tripod

File: aist_description/scenes/urdf/aist_base_scene.urdf.xacro (robot description, xacro)
@@ -111,8 +111,8 @@
   </xacro:single_suction_gripper>
   <!-- Add virtual wall to avoid collisions-->
-  <xacro:aist_box name="vwall1" width="0.01" length="0.35" height="0.55"
-		  parent="ground" transparent="true">
-    <origin xyz="0.41 -0.20 ${bots_z}" rpy="0 0 0"/>
-  </xacro:aist_box>
+  <!-- <xacro:aist_box name="vwall1" width="0.01" length="0.35" height="0.55" -->
+  <!-- 		  parent="ground" transparent="true"> -->
+  <!--   <origin xyz="0.41 -0.20 ${bots_z}" rpy="0 0 0"/> -->
+  <!-- </xacro:aist_box> -->
   <!-- Add PhoXi 3D scanner -->
   <xacro:include filename="$(find aist_description

Commit message: Update camera calibration

File: aist_description/scenes/urdf/aist_base_scene.urdf.xacro (robot description, xacro)
@@ -31,5 +31,5 @@
   <xacro:property name="cage_t"		value="0.040"/>
   <xacro:property name="tool_bar_h"	value="0.270"/>
-  <xacro:property name="camera_bar_h"	value="1.280"/>
+  <xacro:property name="camera_bar_h"	value="1.380"/>
   <xacro:property name="cage_z"		value="0.164"/>
   <xacro:property name="cage_offset"	value="0.020"/>

File: moveit_config/aist_moveit_config/config/gazebo_aist_base_scene.urdf (robot description, URDF)
Before this commit: robot aist_base_scene, 94 links, 93 joints
Joints:
- joint a_phoxi_m_camera_link_joint: origin xyz=0.5245854465604496 0.010160959021244614 0.657827807955093 rpy=0.06657433677736414 1.0703756669836708 3.1350231701080244 -> xyz=0.492856774041131 -0.036792816347522905 0.6845615969657455 rpy=-0.05809603311925469 1.097335615317803 3.053149944967766
- joint cage_upper_right_bar: origin xyz=1.16 0.04 1.28 rpy=0 0 0 -> xyz=1.16 0.04 1.38 rpy=0 0 0
- joint workspace_live_camera_joint: origin xyz=0.40311836114641414 0.02379492915076111 0.694748550420011 rpy=-2.732962681954511 0.02162437650373519 1.5132164471367409 -> xyz=0.3733700748941794 -0.030741582314842072 0.720839795840623 rpy=-2.844520734424458 -0.07655721902523285 1.5144117286631504

Commit message: Add virtual_screen frame to aist_base_scene

File: aist_description/scenes/urdf/aist_base_scene.urdf.xacro (robot description, xacro)
@@ -8,4 +8,5 @@
   <xacro:property name="b_bot_theta"	value="${pi}"/>
   <xacro:property name="bots_z"		value="0.770"/>
+  <xacro:property name="screen_z"	value="${bots_z} + 0.0347"/>
   <!-- ground and workspace -->
   <link name="ground"/>
@@ -126,10 +127,10 @@
     	    rpy="${origin[3]} ${origin[4]} ${origin[5]}"/>
   </xacro:phoxi_m_camera>
-  <!-- Add RealSense camera -->
+  <!-- RealSense cameras -->
   <xacro:include filename="$(find aist_description
   			   )/devices/urdf/wrist_cameras.urdf.xacro" />
   <xacro:wrist_cameras prefix="a_bot_"
   		       parent="a_bot_gripper_base_link"/>
-  <!-- Add live camera -->
+  <!-- live camera -->
   <xacro:load_calibration filename="$(find aist_camera_calibration
 				    )/calib/live_camera.yaml"/>
@@ -140,4 +141,11 @@
     <origin xyz="${origin[0]} ${origin[1]} ${origin[2]}"
     	    rpy="${origin[3]} ${origin[4]} ${origin[5]}"/>
+  </joint>
+  <!-- virtual screen -->
+  <link name="virtual_screen"/>
+  <joint name="virtual_screen_joint" type="fixed">
+    <parnet link="ground"/>
+    <child  link="virtual_screen"/>
+    <origin xyz="0 0 ${screen_z}" rpy="0 0 0"/>
   </joint>
   <!-- I would like to remove the "world" link definition, but apparently it is necessary for Gazebo -->

Commit message: Fixed typo

File: aist_description/scenes/urdf/aist_base_scene.urdf.xacro (robot description, xacro)
@@ -8,5 +8,5 @@
   <xacro:property name="b_bot_theta"	value="${pi}"/>
   <xacro:property name="bots_z"		value="0.770"/>
-  <xacro:property name="screen_z"	value="${bots_z} + 0.0347"/>
+  <xacro:property name="screen_z"	value="${bots_z + 0.0347}"/>
   <!-- ground and workspace -->
   <link name="ground"/>
@@ -145,5 +145,5 @@
   <link name="virtual_screen"/>
   <joint name="virtual_screen_joint" type="fixed">
-    <parnet link="ground"/>
+    <parent link="ground"/>
     <child  link="virtual_screen"/>
     <origin xyz="0 0 ${screen_z}" rpy="0 0 0"/>

Commit message: Change height of camera bar

File: aist_description/scenes/urdf/aist_base_scene.urdf.xacro (robot description, xacro)
@@ -32,5 +32,5 @@
   <xacro:property name="cage_t"		value="0.040"/>
   <xacro:property name="tool_bar_h"	value="0.270"/>
-  <xacro:property name="camera_bar_h"	value="1.380"/>
+  <xacro:property name="camera_bar_h"	value="1.300"/>
   <xacro:property name="cage_z"		value="0.164"/>
   <xacro:property name="cage_offset"	value="0.020"/>

Commit message: Increase joint limit margin

File: aist_description/scenes/urdf/aist_base_scene.urdf.xacro (robot description, xacro)
@@ -60,5 +60,6 @@
 				  )/config/a_bot_calibration.yaml"
       transmission_hw_interface="hardware_interface/PositionJointInterface"
-      safety_limits="true"/>
+      safety_limits="true"
+      safety_pos_margin="1.5"/>
   <xacro:ur_robot_gazebo
       prefix="b_bot_"
@@ -72,5 +73,6 @@
 				  )/config/b_bot_calibration.yaml"
       transmission_hw_interface="hardware_interface/PositionJointInterface"
-      safety_limits="true"/>
+      safety_limits="true"
+      safety_pos_margin="1.5"/>
   <joint name="ground_a_bot_joint" type="fixed">
     <parent link="ground"/>

File: moveit_config/aist_moveit_config/config/gazebo_aist_base_scene.urdf (robot description, URDF)
Before this commit: robot aist_base_scene, 95 links, 94 joints
Joints:
- joint a_bot_inside_camera_joint: origin xyz=0.014973206639882487      -0.006605026045624136      0.05983621136016915 rpy=0.023976131805434685      0.403287172799087      0.012905813015089812 -> xyz=0.014368349250599823      0.0035415297809514353      0.06397546955943786 rpy=0.02303437721634514      0.40347560400972565      0.010798159061973579
- joint a_bot_outside_camera_joint: origin xyz=0.03158216743040747      -0.006437943317858734      0.08083480848924662 rpy=0.016860191822591693      -0.22414769691091246      0.033437654559852904 -> xyz=0.03167812734753831      -0.007813867044282037      0.08129884906700884 rpy=0.017373333209516714      -0.2189346019095829      0.034978097124935485
- joint a_phoxi_m_camera_link_joint: origin xyz=0.5129667610334572 -0.037047806454438365 0.6226614314794279 rpy=-0.06660879099232307 1.0432812514428629 3.014328066314531 -> xyz=0.5136934405264134 -0.036640940205745876 0.6228856442369739 rpy=-0.06465094892887115 1.0423347602737518 3.015361040075505

Commit message: Change joint margin

File: aist_description/scenes/urdf/aist_base_scene.urdf.xacro (robot description, xacro)
@@ -61,5 +61,5 @@
       transmission_hw_interface="hardware_interface/PositionJointInterface"
       safety_limits="true"
-      safety_pos_margin="0.3"/>
+      safety_pos_margin="0.15"/>
   <xacro:ur_robot_gazebo
       prefix="b_bot_"
@@ -74,5 +74,5 @@
       transmission_hw_interface="hardware_interface/PositionJointInterface"
       safety_limits="true"
-      safety_pos_margin="0.3"/>
+      safety_pos_margin="0.15"/>
   <joint name="ground_a_bot_joint" type="fixed">
     <parent link="ground"/>

File: moveit_config/aist_moveit_config/config/gazebo_aist_base_scene.urdf (robot description, URDF)
Before this commit: robot aist_base_scene, 95 links, 94 joints
Joints:
- joint a_bot_inside_camera_joint: origin xyz=0.014368349250599823      0.0035415297809514353      0.06397546955943786 rpy=0.02303437721634514      0.40347560400972565      0.010798159061973579 -> xyz=0.010324554587117304      0.0018335412329232095      0.06467303743182957 rpy=0.025912000078364868      0.4021372934071272      0.01607525693523146
- joint a_bot_outside_camera_joint: origin xyz=0.03167812734753831      -0.007813867044282037      0.08129884906700884 rpy=0.017373333209516714      -0.2189346019095829      0.034978097124935485 -> xyz=0.03590302041834074      -0.008099774421321322      0.07959004727089102 rpy=0.016977853905271578      -0.21989995636200013      0.03446978804301341
- joint a_phoxi_m_camera_link_joint: origin xyz=0.5136934405264134 -0.036640940205745876 0.6228856442369739 rpy=-0.06465094892887115 1.0423347602737518 3.015361040075505 -> xyz=0.5141294525807852 -0.0391428293642771 0.6227194772673923 rpy=-0.0626579561970891 1.0383878192954172 3.059776671030358
- joint workspace_live_camera_joint: origin xyz=0.405235138268645 -0.0356851775630231 0.7399153983016764 rpy=-2.6956831173735374 0.04101229395800053 1.5544348139645294 -> xyz=0.4076098270054865 -0.041827815223630944 0.7417406575198592 rpy=-2.70626389040216 0.06825373432442536 1.5972576864936887

Commit message: Replace a_phoxi_m_camera with a_motioncam

File: aist_description/scenes/urdf/aist_base_scene.urdf.xacro (robot description, xacro)
@@ -119,14 +119,25 @@
   <!-- </xacro:aist_box> -->
   <!-- Add PhoXi 3D scanner -->
+  <!-- <xacro:include filename="$(find aist_description -->
+  <!-- 			   )/scenes/urdf/load_calibration.urdf.xacro"/> -->
+  <!-- <xacro:load_calibration filename="$(find aist_handeye_calibration -->
+  <!-- 				    )/calib/a_phoxi_m_camera.yaml"/> -->
+  <!-- <xacro:include filename="$(find aist_phoxi_camera -->
+  <!-- 			   )/urdf/phoxi_m_camera.urdf.xacro"/> -->
+  <!-- <xacro:phoxi_m_camera name="a_phoxi_m_camera" parent="workspace_center"> -->
+  <!--   <origin xyz="${origin[0]} ${origin[1]} ${origin[2]}" -->
+  <!--   	    rpy="${origin[3]} ${origin[4]} ${origin[5]}"/> -->
+  <!-- </xacro:phoxi_m_camera> -->
+  <!-- Add Motioncam-3D scanner -->
   <xacro:include filename="$(find aist_description
 			   )/scenes/urdf/load_calibration.urdf.xacro"/>
   <xacro:load_calibration filename="$(find aist_handeye_calibration
-				    )/calib/a_phoxi_m_camera.yaml"/>
+				    )/calib/a_motioncam.yaml"/>
   <xacro:include filename="$(find aist_phoxi_camera
-			   )/urdf/phoxi_m_camera.urdf.xacro"/>
-  <xacro:phoxi_m_camera name="a_phoxi_m_camera" parent="workspace_center">
+			   )/urdf/motioncam_m_camera.urdf.xacro"/>
+  <xacro:motioncam_m_camera name="a_motioncam" parent="workspace_center">
     <origin xyz="${origin[0]} ${origin[1]} ${origin[2]}"
     	    rpy="${origin[3]} ${origin[4]} ${origin[5]}"/>
-  </xacro:phoxi_m_camera>
+  </xacro:motioncam_m_camera>
   <!-- RealSense cameras -->
   <xacro:include filename="$(find aist_description

Commit message: Change height of camera bar

File: aist_description/scenes/urdf/aist_base_scene.urdf.xacro (robot description, xacro)
@@ -32,5 +32,5 @@
   <xacro:property name="cage_t"		value="0.040"/>
   <xacro:property name="tool_bar_h"	value="0.270"/>
-  <xacro:property name="camera_bar_h"	value="1.300"/>
+  <xacro:property name="camera_bar_h"	value="1.325"/>
   <xacro:property name="cage_z"		value="0.164"/>
   <xacro:property name="cage_offset"	value="0.020"/>

File: moveit_config/aist_moveit_config/config/gazebo_aist_base_scene.urdf (robot description, URDF)
Before this commit: robot aist_base_scene, 95 links, 94 joints
Links:
- removed link a_phoxi_m_camera_link
- removed link a_phoxi_m_camera_reference
- removed link a_phoxi_m_camera_sensor
- added link a_motioncam_link, mass 0.1; collision mesh filename=package://aist_phoxi_camera/meshes/collision/MotionCam3D_M.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 scale=0.001 0.001 0.001; visual mesh filename=package://aist_phoxi_camera/meshes/visual/MotionCam3D_M.f.S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 scale=0.001 0.001 0.001
- added link a_motioncam_reference
- added link a_motioncam_sensor
Joints:
- removed joint a_phoxi_m_camera_link_joint
- removed joint a_phoxi_m_camera_reference_joint
- removed joint a_phoxi_m_camera_sensor_joint
- added joint a_motioncam_link_joint: type fixed, parent workspace_center, child a_motioncam_link, origin xyz=0.5231407296015458 -0.10503553573534424 0.6365724301868348 rpy=0.03174526251084231 1.041717094258447 -3.1268222045220364
- added joint a_motioncam_reference_joint: type fixed, parent a_motioncam_link, child a_motioncam_reference, origin xyz=0.03 -0.175 0.035 rpy=0 0 0
- added joint a_motioncam_sensor_joint: type fixed, parent a_motioncam_reference, child a_motioncam_sensor, origin xyz=0 0 0 rpy=-1.5707963267948966 0 -1.5707963267948966
- joint cage_upper_right_bar: origin xyz=1.16 0.04 1.3 rpy=0 0 0 -> xyz=1.16 0.04 1.325 rpy=0 0 0

Commit message: Confirmed that hmi_demo works with Motioncam-3D Color in scanner mode

File: aist_description/scenes/urdf/aist_base_scene.urdf.xacro (robot description, xacro)
@@ -8,5 +8,5 @@
   <xacro:property name="b_bot_theta"	value="${pi}"/>
   <xacro:property name="bots_z"		value="0.770"/>
-  <xacro:property name="screen_z"	value="${bots_z + 0.0347}"/>
+  <xacro:property name="screen_z"	value="${bots_z + 0.045}"/>
   <!-- ground and workspace -->
   <link name="ground"/>

Commit message: Change height of virtual screen

File: aist_description/scenes/urdf/aist_base_scene.urdf.xacro (robot description, xacro)
@@ -8,5 +8,5 @@
   <xacro:property name="b_bot_theta"	value="${pi}"/>
   <xacro:property name="bots_z"		value="0.770"/>
-  <xacro:property name="screen_z"	value="${bots_z + 0.045}"/>
+  <xacro:property name="screen_z"	value="${bots_z + 0.040}"/>
   <!-- ground and workspace -->
   <link name="ground"/>

Commit message: Update calibration of suction gripper

File: aist_description/scenes/urdf/aist_base_scene.urdf.xacro (robot description, xacro)
@@ -121,5 +121,5 @@
 			   )/urdf/robotiq_140_gripper.urdf.xacro"/>
   <xacro:robotiq_140_gripper prefix="a_bot_gripper_"
-			    parent="a_bot_gripper_coupling_flange_link">
+			     parent="a_bot_gripper_coupling_flange_link">
     <origin xyz="0 0 0" rpy="0 0 0"/>
   </xacro:robotiq_140_gripper>
@@ -128,6 +128,5 @@
   <xacro:single_suction_gripper prefix="b_bot_gripper_"
   				parent="b_bot_ftsensor_flange_link">
-    <!-- <origin xyz="0 0 0" rpy="0 ${0.2*pi/180} ${-1.2*pi/180}"/> -->
-    <origin xyz="0 0 0" rpy="0 ${0.7*pi/180} ${-0.1*pi/180}"/>
+    <origin xyz="0 0 0" rpy="0 ${-1.0*pi/180} ${-0.3*pi/180}"/>
   </xacro:single_suction_gripper>
   <!-- Add PhoXi 3D scanner -->

Commit message: Change frame names of screw tools

File: aist_description/scenes/urdf/aist_base_scene.urdf.xacro (robot description, xacro)
@@ -60,4 +60,17 @@
     <origin xyz="0 ${screw_tool_m4_holder_y} ${cage_t}" rpy="0 0 0"/>
   </xacro:screw_tool_holder>
+  <!-- screw tools -->
+  <!-- <xacro:include filename="$(find aist_fastening_tools -->
+  <!-- 			   )/urdf/screw_tool_m3.urdf.xacro"/> -->
+  <!-- <xacro:screw_tool_m3 prefix="screw_tool_m3_" -->
+  <!-- 		       parent="screw_tool_m3_holder_link"> -->
+  <!--   <origin xyz="0 0 0" rpy="0 0 0" /> -->
+  <!-- </xacro:screw_tool_m3> -->
+  <!-- <xacro:include filename="$(find aist_fastening_tools -->
+  <!-- 			   )/urdf/screw_tool_m4.urdf.xacro"/> -->
+  <!-- <xacro:screw_tool_m3 prefix="screw_tool_m4_" -->
+  <!-- 		       parent="screw_tool_m4_holder_link"> -->
+  <!--   <origin xyz="0 0 0" rpy="0 0 0" /> -->
+  <!-- </xacro:screw_tool_m3> -->
   <!-- robot arms -->
   <xacro:include filename="$(find ur_gazebo)/urdf/ur_macro.xacro"/>

File: aist_fastening_tools/urdf/screw_tool_m3.urdf.xacro (robot description, xacro)
@@ -1,5 +1,4 @@
 <?xml version="1.0"?>
-<robot name="screw_tool_m3"
-       xmlns:xacro="http://wiki.ros.org/xacro">
+<robot name="screw_tool_m3" xmlns:xacro="http://wiki.ros.org/xacro">
   <xacro:macro name="screw_tool_m3"
 	       params="prefix parent *origin">
@@ -7,5 +6,5 @@
     <link name="${prefix}base_link">
       <visual>
-        <origin xyz="0 0 0" rpy="${pi/2} 0 ${-pi/2}"/>
+        <origin xyz="0 0 -0.0006" rpy="0 0 ${-pi/2}"/>
 	<geometry>
           <mesh filename="package://aist_fastening_tools/meshes/visual/screw_tool_m3_BC5-XL320-R-AY2.6-EH2.stl" scale="0.001 0.001 0.001"/>
@@ -16,5 +15,5 @@
       </visual>
       <collision>
-	<origin xyz="0 0 0" rpy="${pi/2} 0 ${-pi/2}"/>
+	<origin xyz="0 0 0" rpy="0 0 ${-pi/2}"/>
 	<geometry>
 	  <mesh filename="package://aist_fastening_tools/meshes/collision/screw_tool_m3_simplified.stl" scale="0.0001 0.0001 0.0001"/>
@@ -38,5 +37,5 @@
       <parent link="${prefix}base_link"/>
       <child  link="${prefix}tip_link"/>
-      <origin xyz="0.100 0 0" rpy="0 ${-pi/2} 0"/>
+      <origin xyz="0 0 -0.100" rpy="0 0 0"/>
     </joint>
   </xacro:macro>

File: aist_fastening_tools/urdf/screw_tool_m4.urdf.xacro (robot description, xacro)
@@ -1,5 +1,4 @@
 <?xml version="1.0"?>
-<robot name="screw_tool_m4"
-       xmlns:xacro="http://wiki.ros.org/xacro">
+<robot name="screw_tool_m4" xmlns:xacro="http://wiki.ros.org/xacro">
   <xacro:macro name="screw_tool_m4"
 	       params="prefix parent *origin">
@@ -7,5 +6,5 @@
     <link name="${prefix}base_link">
       <visual>
-        <origin xyz="0 0 0" rpy="${pi/2} 0 ${-pi/2}"/>
+        <origin xyz="0 0 -0.0006" rpy="0 0 ${-pi/2}"/>
 	<geometry>
           <mesh filename="package://aist_fastening_tools/meshes/visual/screw_tool_m4_BC5-XL320-AY3.5-EH3R4.stl" scale="0.001 0.001 0.001"/>
@@ -16,5 +15,5 @@
       </visual>
       <collision>
-        <origin xyz="0 0 0" rpy="${pi/2} 0 ${-pi/2}"/>
+        <origin xyz="0 0 0" rpy="0 0 ${-pi/2}"/>
 	<geometry>
 	  <mesh filename="package://aist_fastening_tools/meshes/collision/screw_tool_m4_simplified.stl" scale="0.0001 0.0001 0.0001"/>
@@ -38,5 +37,5 @@
       <parent link="${prefix}base_link"/>
       <child  link="${prefix}tip_link"/>
-      <origin xyz="0.120 0 0" rpy="0 ${-pi/2} 0"/>
+      <origin xyz="0 0 -0.120" rpy="0 0 0"/>
     </joint>
   </xacro:macro>

Commit message: Add precision_tool_holder

File: aist_description/scenes/urdf/aist_base_scene.urdf.xacro (robot description, xacro)
@@ -48,7 +48,14 @@
   </xacro:cage>
   <!-- tool holders -->
-  <xacro:property name="screw_tool_m3_holder_y"	value="0.75"/>
-  <xacro:property name="screw_tool_m4_holder_y"	value="0.85"/>
-  <xacro:property name="suction_tool_holder_y"	value="0.95"/>
+  <xacro:property name="precision_tool_holder_y"	value="0.60"/>
+  <xacro:property name="screw_tool_m3_holder_y"		value="0.70"/>
+  <xacro:property name="screw_tool_m4_holder_y"		value="0.80"/>
+  <xacro:property name="suction_tool_holder_y"		value="0.90"/>
+  <xacro:include filename="$(find aist_description
+			   )/objects/urdf/precision_tool_holder.urdf.xacro"/>
+  <xacro:precision_tool_holder prefix="precision_tool_holder_"
+			   parent="cage_tool_bar">
+    <origin xyz="0 ${precision_tool_holder_y} ${cage_t}" rpy="0 0 0"/>
+  </xacro:precision_tool_holder>
   <xacro:include filename="$(find aist_description
 			   )/objects/urdf/screw_tool_holder.urdf.xacro"/>
