Commit message: Revert a_bot_gripper and inide/outside cameras

File: aist_description/scenes/urdf/aist_base_scene.urdf.xacro (robot description, xacro)
@@ -113,24 +113,23 @@
   </joint>
   <!-- Attach mounter for Zivid2+ camera -->
-  <xacro:include filename="$(find aist_description)/devices/urdf/zivid_coupling.urdf.xacro"/>
-  <xacro:zivid_coupling prefix="a_bot_zivid_coupling_" parent="a_bot_flange">
-    <origin xyz="0 0 0" rpy="${pi} 0 0" />
-  </xacro:zivid_coupling>
+  <!-- <xacro:include filename="$(find aist_description)/devices/urdf/zivid_coupling.urdf.xacro"/> -->
+  <!-- <xacro:zivid_coupling prefix="a_bot_zivid_coupling_" parent="a_bot_flange"> -->
+  <!--   <origin xyz="0 0 0" rpy="${pi} 0 0" /> -->
+  <!-- </xacro:zivid_coupling> -->
   <!-- Spawn and attach Zivid2+ camera -->
-  <xacro:include filename="$(find aist_description
-			   )/scenes/urdf/load_calibration.urdf.xacro"/>
-  <xacro:load_calibration filename="$(find aist_handeye_calibration
-				    )/calib/a_bot_zivid.yaml"/>
-  <xacro:include filename="$(find aist_description
-			   )/devices/urdf/zivid2plus.urdf.xacro"/>
-  <xacro:zivid2plus name="a_bot_zivid"
-		    parent="a_bot_zivid_coupling_flange_link">
-    <origin xyz="${origin[0]} ${origin[1]} ${origin[2]}"
-    	    rpy="${origin[3]} ${origin[4]} ${origin[5]}"/>
-  </xacro:zivid2plus>
+  <!-- <xacro:include filename="$(find aist_description -->
+  <!-- 			   )/scenes/urdf/load_calibration.urdf.xacro"/> -->
+  <!-- <xacro:load_calibration filename="$(find aist_handeye_calibration -->
+  <!-- 				    )/calib/a_bot_zivid.yaml"/> -->
+  <!-- <xacro:include filename="$(find aist_description -->
+  <!-- 			   )/devices/urdf/zivid2plus.urdf.xacro"/> -->
+  <!-- <xacro:zivid2plus name="a_bot_zivid" -->
+  <!-- 		    parent="a_bot_zivid_coupling_flange_link"> -->
+  <!--   <origin xyz="${origin[0]} ${origin[1]} ${origin[2]}" -->
+  <!--   	    rpy="${origin[3]} ${origin[4]} ${origin[5]}"/> -->
+  <!-- </xacro:zivid2plus> -->
   <!-- Spawn and attach force sensor -->
   <xacro:include filename="$(find aist_robotiq)/urdf/ft300.urdf.xacro"/>
-  <xacro:ft300 prefix="a_bot_ftsensor_"
-	       parent="a_bot_zivid_coupling_flange_link">
+  <xacro:ft300 prefix="a_bot_ftsensor_" parent="a_bot_flange">
     <origin xyz="0 0 0" rpy="0 0 0"/>
   </xacro:ft300>
@@ -146,9 +145,9 @@
   </xacro:robotiq_arg2f_coupling>
   <xacro:include filename="$(find aist_robotiq
-			   )/urdf/robotiq_140_gripper.urdf.xacro"/>
-  <xacro:robotiq_140_gripper prefix="a_bot_gripper_"
-			     parent="a_bot_gripper_coupling_flange_link">
-    <origin xyz="0 0 0" rpy="0 0 0"/>
-  </xacro:robotiq_140_gripper>
+			   )/urdf/robotiq_85_gripper.urdf.xacro"/>
+  <xacro:robotiq_85_gripper prefix="a_bot_gripper_"
+			    parent="a_bot_gripper_coupling_flange_link">
+    <origin xyz="0 0 0" rpy="0 0 0"/>
+  </xacro:robotiq_85_gripper>
   <xacro:include filename="$(find aist_description
 			   )/devices/urdf/single_suction_gripper.urdf.xacro"/>
@@ -180,9 +179,9 @@
   </xacro:motioncam_m_camera>
   <!-- RealSense cameras -->
-  <!-- <xacro:include filename="$(find aist_description -->
-  <!-- 			   )/devices/urdf/wrist_cameras.urdf.xacro" /> -->
-  <!-- <xacro:wrist_cameras prefix="a_bot_" -->
-  <!-- 		       parent="a_bot_gripper_base_link" -->
-  <!-- 		       use_nominal_extrinsics="true"/> -->
+  <xacro:include filename="$(find aist_description
+  			   )/devices/urdf/wrist_cameras.urdf.xacro" />
+  <xacro:wrist_cameras prefix="a_bot_"
+  		       parent="a_bot_gripper_base_link"
+  		       use_nominal_extrinsics="true"/>
   <!-- live camera -->
   <xacro:load_calibration filename="$(find aist_camera_calibration

File: moveit_config/aist_moveit_config/config/gazebo_aist_base_scene.urdf (robot description, URDF)
Before this commit: robot aist_base_scene, 84 links, 83 joints
Links:
- removed link a_bot_zivid_base_link
- removed link a_bot_zivid_coupling_base_link
- removed link a_bot_zivid_coupling_flange_link
- removed link a_bot_zivid_projector
- removed link a_bot_zivid_reference
- removed link a_bot_zivid_sensor
- added link a_bot_camera_mount, mass 1.0; collision box size=.03 .12 .08; visual mesh filename=package://aist_description/devices/meshes/sr305_mount.stl scale=.001 .001 .001
- added link a_bot_inside_camera_color_frame
- added link a_bot_inside_camera_color_optical_frame
- added link a_bot_inside_camera_connector_link
- added link a_bot_inside_camera_depth_frame
- added link a_bot_inside_camera_depth_optical_frame
- added link a_bot_inside_camera_left_ir_frame
- added link a_bot_inside_camera_left_ir_optical_frame
- added link a_bot_inside_camera_link, mass 0.564; collision box size=0.012 0.14 0.023; visual mesh filename=package://realsense2_description/meshes/sr305_without_mount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 scale=.001 .001 .001
- added link a_bot_inside_camera_right_ir_frame
- added link a_bot_inside_camera_right_ir_optical_frame
- added link a_bot_outside_camera_color_frame
- added link a_bot_outside_camera_color_optical_frame
- added link a_bot_outside_camera_connector_link
- added link a_bot_outside_camera_depth_frame
- added link a_bot_outside_camera_depth_optical_frame
- added link a_bot_outside_camera_left_ir_frame
- added link a_bot_outside_camera_left_ir_optical_frame
- added link a_bot_outside_camera_link, mass 0.564; collision box size=0.012 0.14 0.023; visual mesh filename=package://realsense2_description/meshes/sr305_without_mount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 scale=.001 .001 .001
- added link a_bot_outside_camera_right_ir_frame
- added link a_bot_outside_camera_right_ir_optical_frame
- added link precision_tool_holder_base_link, mass 0.1; collision mesh filename=package://aist_description/objects/meshes/precision_tool_ho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 scale=0.001 0.001 0.001; visual mesh filename=package://aist_description/objects/meshes/precision_tool_ho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 scale=0.001 0.001 0.001
- added link precision_tool_holder_link
- added link suction_tool_holder_base_link, mass 0.1; collision mesh filename=package://aist_description/objects/meshes/suction_tool_hold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 scale=0.001 0.001 0.001; visual mesh filename=package://aist_description/objects/meshes/suction_tool_hold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 scale=0.001 0.001 0.001
- added link suction_tool_holder_link
- link a_bot_gripper_left_inner_finger: geometry collision mesh filename=package://aist_robotiq/meshes/collision/robotiq_arg2f_85_in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 scale=0.001 0.001 0.001; visual mesh filename=package://aist_robotiq/meshes/visual/robotiq_arg2f_85_inner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 scale=0.001 0.001 0.001
- link a_bot_gripper_left_inner_finger_pad: geometry collision box size=0.022 0.00635 0.0375; visual box size=0.022 0.00635 0.0375
- link a_bot_gripper_left_inner_knuckle: geometry collision mesh filename=package://aist_robotiq/meshes/collision/robotiq_arg2f_85_in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 scale=0.001 0.001 0.001; visual mesh filename=package://aist_robotiq/meshes/visual/robotiq_arg2f_85_inner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 scale=0.001 0.001 0.001
- link a_bot_gripper_left_outer_finger: geometry collision mesh filename=package://aist_robotiq/meshes/collision/robotiq_arg2f_85_ou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 scale=0.001 0.001 0.001; visual mesh filename=package://aist_robotiq/meshes/visual/robotiq_arg2f_85_outer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 scale=0.001 0.001 0.001
- link a_bot_gripper_left_outer_knuckle: geometry collision mesh filename=package://aist_robotiq/meshes/collision/robotiq_arg2f_85_ou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 scale=0.001 0.001 0.001; visual mesh filename=package://aist_robotiq/meshes/visual/robotiq_arg2f_85_outer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 scale=0.001 0.001 0.001
- link a_bot_gripper_right_inner_finger: geometry collision mesh filename=package://aist_robotiq/meshes/collision/robotiq_arg2f_85_in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 scale=0.001 0.001 0.001; visual mesh filename=package://aist_robotiq/meshes/visual/robotiq_arg2f_85_inner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 scale=0.001 0.001 0.001
- link a_bot_gripper_right_inner_finger_pad: geometry collision box size=0.022 0.00635 0.0375; visual box size=0.022 0.00635 0.0375
- link a_bot_gripper_right_inner_knuckle: geometry collision mesh filename=package://aist_robotiq/meshes/collision/robotiq_arg2f_85_in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 scale=0.001 0.001 0.001; visual mesh filename=package://aist_robotiq/meshes/visual/robotiq_arg2f_85_inner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 scale=0.001 0.001 0.001
- link a_bot_gripper_right_outer_finger: geometry collision mesh filename=package://aist_robotiq/meshes/collision/robotiq_arg2f_85_ou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 scale=0.001 0.001 0.001; visual mesh filename=package://aist_robotiq/meshes/visual/robotiq_arg2f_85_outer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 scale=0.001 0.001 0.001
- link a_bot_gripper_right_outer_knuckle: geometry collision mesh filename=package://aist_robotiq/meshes/collision/robotiq_arg2f_85_ou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 scale=0.001 0.001 0.001; visual mesh filename=package://aist_robotiq/meshes/visual/robotiq_arg2f_85_outer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 scale=0.001 0.001 0.001
Joints:
- removed joint a_bot_zivid_base_joint
- removed joint a_bot_zivid_coupling_base_joint
- removed joint a_bot_zivid_coupling_flange_joint
- removed joint a_bot_zivid_projector_joint
- removed joint a_bot_zivid_reference_joint
- removed joint a_bot_zivid_sensor_joint
- added joint a_bot_camera_mount_joint: type fixed, parent a_bot_gripper_base_link, child a_bot_camera_mount, origin xyz=0.035 0.0 0.025 rpy=0 0 0
- added joint a_bot_inside_camera_color_joint: type fixed, parent a_bot_inside_camera_depth_frame, child a_bot_inside_camera_color_frame, origin xyz=0 0.015 0 rpy=0 0 0
- added joint a_bot_inside_camera_color_optical_joint: type fixed, parent a_bot_inside_camera_color_frame, child a_bot_inside_camera_color_optical_frame, origin xyz=0 0 0 rpy=-1.5707963267948966 0 -1.5707963267948966
- added joint a_bot_inside_camera_depth_joint: type fixed, parent a_bot_inside_camera_link, child a_bot_inside_camera_depth_frame, origin xyz=.003721 0 0 rpy=0 0 0
- added joint a_bot_inside_camera_depth_optical_joint: type fixed, parent a_bot_inside_camera_depth_frame, child a_bot_inside_camera_depth_optical_frame, origin xyz=0 0 0 rpy=-1.5707963267948966 0 -1.5707963267948966
- added joint a_bot_inside_camera_joint: type fixed, parent a_bot_gripper_base_link, child a_bot_inside_camera_connector_link, origin xyz=0.010324554587117304      0.0018335412329232095      0.06467303743182957 rpy=0.025912000078364868      0.4021372934071272      0.01607525693523146
- added joint a_bot_inside_camera_left_ir_joint: type fixed, parent a_bot_inside_camera_depth_frame, child a_bot_inside_camera_left_ir_frame, origin xyz=0 0.0 0 rpy=0 0 0
- added joint a_bot_inside_camera_left_ir_optical_joint: type fixed, parent a_bot_inside_camera_left_ir_frame, child a_bot_inside_camera_left_ir_optical_frame, origin xyz=0 0 0 rpy=-1.5707963267948966 0 -1.5707963267948966
- added joint a_bot_inside_camera_link_joint: type fixed, parent a_bot_inside_camera_connector_link, child a_bot_inside_camera_link, origin xyz=0 0 0 rpy=0 0 0
- added joint a_bot_inside_camera_right_ir_joint: type fixed, parent a_bot_inside_camera_depth_frame, child a_bot_inside_camera_right_ir_frame, origin xyz=0 0.04 0 rpy=0 0 0
- added joint a_bot_inside_camera_right_ir_optical_joint: type fixed, parent a_bot_inside_camera_right_ir_frame, child a_bot_inside_camera_right_ir_optical_frame, origin xyz=0 0 0 rpy=-1.5707963267948966 0 -1.5707963267948966
- added joint a_bot_outside_camera_color_joint: type fixed, parent a_bot_outside_camera_depth_frame, child a_bot_outside_camera_color_frame, origin xyz=0 0.015 0 rpy=0 0 0
- added joint a_bot_outside_camera_color_optical_joint: type fixed, parent a_bot_outside_camera_color_frame, child a_bot_outside_camera_color_optical_frame, origin xyz=0 0 0 rpy=-1.5707963267948966 0 -1.5707963267948966
- added joint a_bot_outside_camera_depth_joint: type fixed, parent a_bot_outside_camera_link, child a_bot_outside_camera_depth_frame, origin xyz=.003721 0 0 rpy=0 0 0
- added joint a_bot_outside_camera_depth_optical_joint: type fixed, parent a_bot_outside_camera_depth_frame, child a_bot_outside_camera_depth_optical_frame, origin xyz=0 0 0 rpy=-1.5707963267948966 0 -1.5707963267948966
- added joint a_bot_outside_camera_joint: type fixed, parent a_bot_gripper_base_link, child a_bot_outside_camera_connector_link, origin xyz=0.03590302041834074      -0.008099774421321322      0.07959004727089102 rpy=0.016977853905271578      -0.21989995636200013      0.03446978804301341
- added joint a_bot_outside_camera_left_ir_joint: type fixed, parent a_bot_outside_camera_depth_frame, child a_bot_outside_camera_left_ir_frame, origin xyz=0 0.0 0 rpy=0 0 0
- added joint a_bot_outside_camera_left_ir_optical_joint: type fixed, parent a_bot_outside_camera_left_ir_frame, child a_bot_outside_camera_left_ir_optical_frame, origin xyz=0 0 0 rpy=-1.5707963267948966 0 -1.5707963267948966
- added joint a_bot_outside_camera_link_joint: type fixed, parent a_bot_outside_camera_connector_link, child a_bot_outside_camera_link, origin xyz=0 0 0 rpy=0 0 0
- added joint a_bot_outside_camera_right_ir_joint: type fixed, parent a_bot_outside_camera_depth_frame, child a_bot_outside_camera_right_ir_frame, origin xyz=0 0.04 0 rpy=0 0 0
- added joint a_bot_outside_camera_right_ir_optical_joint: type fixed, parent a_bot_outside_camera_right_ir_frame, child a_bot_outside_camera_right_ir_optical_frame, origin xyz=0 0 0 rpy=-1.5707963267948966 0 -1.5707963267948966
- added joint precision_tool_holder_base_joint: type fixed, parent cage_tool_bar, child precision_tool_holder_base_link, origin xyz=0 0.6 0.04 rpy=0 0 0
- added joint precision_tool_holder_joint: type fixed, parent precision_tool_holder_base_link, child precision_tool_holder_link, origin xyz=0.108 0.012 0.037 rpy=0 0.5235987755982988 0
- added joint suction_tool_holder_base_joint: type fixed, parent cage_tool_bar, child suction_tool_holder_base_link, origin xyz=0 0.9 0.04 rpy=0 0 0
- added joint suction_tool_holder_joint: type fixed, parent suction_tool_holder_base_link, child suction_tool_holder_link, origin xyz=0.050 0 0.007 rpy=0 0 0
- joint a_bot_ftsensor_ft300_joint: parent a_bot_zivid_coupling_flange_link -> a_bot_flange
- joint a_bot_gripper_finger_joint: axis -1 0 0 -> 1 0 0; limit lower=0 upper=0.7 effort=1000 velocity=2.0 -> lower=0 upper=0.81 effort=1000 velocity=2.0; origin xyz=0 -0.030601 0.054905 rpy=2.2957963267948966 0 0 -> xyz=0 -0.0306011 0.054904 rpy=0 0 3.141592653589793
- joint a_bot_gripper_left_inner_finger_joint: axis -1 0 0 -> 1 0 0; origin xyz=0 0.0817554015893473 -0.0282203446692936 rpy=-0.725 0 0 -> xyz=0 0.0061 0.0471 rpy=0 0 0
- joint a_bot_gripper_left_inner_finger_pad_joint: origin xyz=0 0.0457554015893473 -0.0272203446692936 rpy=0 0 0 -> xyz=0 -0.0220203446692936 0.03242 rpy=0 0 0
- joint a_bot_gripper_left_inner_knuckle_joint: axis -1 0 0 -> 1 0 0; origin xyz=0 -0.0127 0.06142 rpy=2.2957963267948966 0 0.0 -> xyz=0 -0.0127 0.06142 rpy=0 0 3.141592653589793
- joint a_bot_gripper_left_outer_finger_joint: origin xyz=0 0.01821998610742 0.0260018192872234 rpy=0 0 0 -> xyz=0 0.0315 -0.0041 rpy=0 0 0
- joint a_bot_gripper_right_inner_finger_joint: axis -1 0 0 -> 1 0 0; origin xyz=0 0.0817554015893473 -0.0282203446692936 rpy=-0.725 0 0 -> xyz=0 0.0061 0.0471 rpy=0 0 0
- joint a_bot_gripper_right_inner_finger_pad_joint: origin xyz=0 0.0457554015893473 -0.0272203446692936 rpy=0 0 0 -> xyz=0 -0.0220203446692936 0.03242 rpy=0 0 0
- joint a_bot_gripper_right_inner_knuckle_joint: axis -1 0 0 -> 1 0 0; origin xyz=0 0.0127 0.06142 rpy=2.2957963267948966 0 -3.141592653589793 -> xyz=0 0.0127 0.06142 rpy=0 0 0.0
- joint a_bot_gripper_right_outer_finger_joint: origin xyz=0 0.01821998610742 0.0260018192872234 rpy=0 0 0 -> xyz=0 0.0315 -0.0041 rpy=0 0 0
- joint a_bot_gripper_right_outer_knuckle_joint: axis -1 0 0 -> 1 0 0; limit lower=-0.725 upper=0.725 effort=1000 velocity=2.0 -> lower=-0.81 upper=0.81 effort=1000 velocity=2.0; origin xyz=0 0.030601 0.054905 rpy=2.2957963267948966 0 3.141592653589793 -> xyz=0 0.0306011 0.054904 rpy=0 0 0
- joint a_bot_gripper_tip_link_joint: origin xyz=.2328 0.0 0.0 rpy=0.0 -1.5707963267948966 0.0 -> xyz=0.1628 0.0 0.0 rpy=0.0 -1.5707963267948966 0.0
- joint screw_tool_m3_holder_base_joint: origin xyz=0 0.6 0.04 rpy=0 0 0 -> xyz=0 0.7 0.04 rpy=0 0 0

Commit message: Update camera calibration and tool calibration

File: aist_description/scenes/urdf/aist_base_scene.urdf.xacro (robot description, xacro)
@@ -154,5 +154,5 @@
   <xacro:single_suction_gripper prefix="b_bot_gripper_"
   				parent="b_bot_ftsensor_flange_link">
-    <origin xyz="0 0 0" rpy="0 ${-1.0*pi/180} ${-0.3*pi/180}"/>
+    <origin xyz="0 0 0" rpy="0 ${0.3*pi/180} ${0.2*pi/180}"/>
   </xacro:single_suction_gripper>
   <!-- Add PhoXi 3D scanner -->

File: aist_description/scenes/urdf/kitting.urdf.xacro (robot description, xacro)
@@ -113,11 +113,11 @@
   </xacro:kitting_tray_2>
   <!-- AR marker for localizing WEB camera -->
-  <xacro:include filename="$(find aist_aruco_ros)/urdf/ar_marker.urdf.xacro"/>
-  <xacro:ar_marker prefix="workspace_"
-  		   parent="workspace_center"
-  		   marker_id="32"
-  		   width="0.095" height="0.095" margin="0.0525"
-  		   thickness="0.003">
-    <origin xyz="${marker_x} ${marker_y} 0.0003" rpy="0 0 ${pi/2}"/>
-  </xacro:ar_marker>
+  <!-- <xacro:include filename="$(find aist_aruco_ros)/urdf/ar_marker.urdf.xacro"/> -->
+  <!-- <xacro:ar_marker prefix="workspace_" -->
+  <!-- 		   parent="workspace_center" -->
+  <!-- 		   marker_id="32" -->
+  <!-- 		   width="0.095" height="0.095" margin="0.0525" -->
+  <!-- 		   thickness="0.003"> -->
+  <!--   <origin xyz="${marker_x} ${marker_y} 0.0003" rpy="0 0 ${pi/2}"/> -->
+  <!-- </xacro:ar_marker> -->
 </robot>

Commit message: Add offset to cage

File: aist_description/scenes/urdf/aist_base_scene.urdf.xacro (robot description, xacro)
@@ -34,5 +34,6 @@
   <xacro:property name="camera_bar_h"	value="1.325"/>
   <xacro:property name="cage_z"		value="0.164"/>
-  <xacro:property name="cage_offset"	value="0.020"/>
+  <xacro:property name="cage_offset_x"	value="0.020"/>
+  <xacro:property name="cage_offset_y"	value="0.005"/>
   <xacro:include filename="$(find aist_description
 			   )/objects/urdf/cage.urdf.xacro"/>
@@ -44,5 +45,7 @@
 	      camera_bar_height="${camera_bar_h}"
 	      parent="ground">
-    <origin xyz="${-cage_w/2 + cage_offset} ${-cage_l/2} ${cage_z}"
+    <origin xyz="${-cage_w/2 + cage_offset_x}
+		 ${-cage_l/2 + cage_offset_y}
+		 ${cage_z}"
 	    rpy="0 0 0" />
   </xacro:cage>

Commit message: Fix offset_y of cage

File: aist_description/scenes/urdf/aist_base_scene.urdf.xacro (robot description, xacro)
@@ -35,5 +35,5 @@
   <xacro:property name="cage_z"		value="0.164"/>
   <xacro:property name="cage_offset_x"	value="0.020"/>
-  <xacro:property name="cage_offset_y"	value="0.005"/>
+  <xacro:property name="cage_offset_y"	value="-0.005"/>
   <xacro:include filename="$(find aist_description
 			   )/objects/urdf/cage.urdf.xacro"/>

Commit message: Separate visual mesh and collision mesh for CollisionObject

File: aist_description/scenes/urdf/aist_base_scene.urdf.xacro (robot description, xacro)
@@ -34,5 +34,5 @@
   <xacro:property name="camera_bar_h"	value="1.325"/>
   <xacro:property name="cage_z"		value="0.164"/>
-  <xacro:property name="cage_offset_x"	value="0.020"/>
+  <xacro:property name="cage_offset_x"	value="0.025"/>
   <xacro:property name="cage_offset_y"	value="-0.005"/>
   <xacro:include filename="$(find aist_description

File: aist_precision_gripper/urdf/precision_gripper.urdf.xacro (robot description, xacro)
@@ -5,5 +5,5 @@
 			     )/urdf/precision_transmission.xacro"/>
     <xacro:precision_transmission prefix="${prefix}"/>
-    <xacro:property name="horizontal_offset"		value="-0.015"/>
+    <xacro:property name="horizontal_offset"		value="-0.014"/>
     <xacro:property name="tip_distance"			value="0.147"/>
     <xacro:property name="rail_distance"		value="0.0915"/>
@@ -12,5 +12,5 @@
     <xacro:property name="motor_width"			value="0.055"/>
     <xacro:property name="motor_height"			value="0.0425"/>
-    <xacro:property name="motor_offset"			value="-0.003"/>
+    <xacro:property name="motor_offset"			value="-0.0025"/>
     <xacro:property name="lower_body_width"		value="0.085"/>
     <xacro:property name="lower_body_height"		value="0.050"/>

Commit message: Fix offset of cage

File: aist_description/scenes/urdf/aist_base_scene.urdf.xacro (robot description, xacro)
@@ -34,5 +34,5 @@
   <xacro:property name="camera_bar_h"	value="1.325"/>
   <xacro:property name="cage_z"		value="0.164"/>
-  <xacro:property name="cage_offset_x"	value="0.025"/>
+  <xacro:property name="cage_offset_x"	value="0.015"/>
   <xacro:property name="cage_offset_y"	value="-0.005"/>
   <xacro:include filename="$(find aist_description
