Commit message: Replace suction_gripper with robotiq_140 for b_bot

File: aist_description/scenes/urdf/aist_base_scene.urdf.xacro (robot description, xacro)
@@ -1,5 +1,5 @@
 <?xml version="1.0"?>
 <robot xmlns:xacro="http://wiki.ros.org/xacro" name="aist_base_scene" >
-  <xacro:arg name="scene" default="kitting2"/>
+  <xacro:arg name="scene" default=""/>
   <xacro:property name="a_bot_x"	value="0"/>
   <xacro:property name="a_bot_y"	value="-0.4875"/>
@@ -153,10 +153,20 @@
     <origin xyz="0 0 0" rpy="0 0 0"/>
   </xacro:robotiq_85_gripper>
-  <xacro:include filename="$(find aist_description
-			   )/devices/urdf/single_suction_gripper.urdf.xacro"/>
-  <xacro:single_suction_gripper prefix="b_bot_gripper_"
-  				parent="b_bot_ftsensor_flange_link">
-    <origin xyz="0 0 0" rpy="0 ${0.3*pi/180} ${0.2*pi/180}"/>
-  </xacro:single_suction_gripper>
+  <xacro:robotiq_arg2f_coupling prefix="b_bot_gripper_coupling_"
+				parent="b_bot_ftsensor_flange_link">
+    <origin xyz="0 0 0" rpy="0 0 0"/>
+  </xacro:robotiq_arg2f_coupling>
+  <xacro:include filename="$(find aist_robotiq
+			   )/urdf/robotiq_140_gripper.urdf.xacro"/>
+  <xacro:robotiq_140_gripper prefix="b_bot_gripper_"
+			    parent="b_bot_gripper_coupling_flange_link">
+    <origin xyz="0 0 0" rpy="0 0 0"/>
+  </xacro:robotiq_140_gripper>
+  <!-- <xacro:include filename="$(find aist_description -->
+  <!-- 			   )/devices/urdf/single_suction_gripper.urdf.xacro"/> -->
+  <!-- <xacro:single_suction_gripper prefix="b_bot_gripper_" -->
+  <!-- 				parent="b_bot_ftsensor_flange_link"> -->
+  <!--   <origin xyz="0 0 0" rpy="0 ${0.3*pi/180} ${0.2*pi/180}"/> -->
+  <!-- </xacro:single_suction_gripper> -->
   <!-- Add PhoXi 3D scanner -->
   <!-- <xacro:include filename="$(find aist_description -->

File: moveit_config/aist_moveit_config/config/gazebo_aist_base_scene.urdf (robot description, URDF)
Before this commit: robot aist_base_scene, 103 links, 102 joints
Links:
- added link b_bot_gripper_coupling_base_link, mass 0.22652; collision cylinder length=0.0111 radius=0.0375; visual mesh filename=package://aist_robotiq/meshes/visual/robotiq_arg2f_coupling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 scale=0.001 0.001 0.001
- added link b_bot_gripper_coupling_flange_link
- added link b_bot_gripper_left_inner_finger, mass 0.0104003125914103; collision mesh filename=package://aist_robotiq/meshes/collision/robotiq_arg2f_140_i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; visual mesh filename=package://aist_robotiq/meshes/visual/robotiq_arg2f_140_inne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
- added link b_bot_gripper_left_inner_finger_pad, mass 0.1; collision box size=0.027 0.065 0.0075; visual box size=0.027 0.065 0.0075
- added link b_bot_gripper_left_inner_knuckle, mass 0.0271177346495152; collision mesh filename=package://aist_robotiq/meshes/collision/robotiq_arg2f_140_i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; visual mesh filename=package://aist_robotiq/meshes/visual/robotiq_arg2f_140_inne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
- added link b_bot_gripper_left_outer_finger, mass 0.022614240507152; collision mesh filename=package://aist_robotiq/meshes/collision/robotiq_arg2f_140_o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; visual mesh filename=package://aist_robotiq/meshes/visual/robotiq_arg2f_140_oute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
- added link b_bot_gripper_left_outer_knuckle, mass 0.00853198276973456; collision mesh filename=package://aist_robotiq/meshes/collision/robotiq_arg2f_140_o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; visual mesh filename=package://aist_robotiq/meshes/visual/robotiq_arg2f_140_oute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
- added link b_bot_gripper_right_inner_finger, mass 0.0104003125914103; collision mesh filename=package://aist_robotiq/meshes/collision/robotiq_arg2f_140_i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; visual mesh filename=package://aist_robotiq/meshes/visual/robotiq_arg2f_140_inne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
- added link b_bot_gripper_right_inner_finger_pad, mass 0.1; collision box size=0.027 0.065 0.0075; visual box size=0.027 0.065 0.0075
- added link b_bot_gripper_right_inner_knuckle, mass 0.0271177346495152; collision mesh filename=package://aist_robotiq/meshes/collision/robotiq_arg2f_140_i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; visual mesh filename=package://aist_robotiq/meshes/visual/robotiq_arg2f_140_inne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
- added link b_bot_gripper_right_outer_finger, mass 0.022614240507152; collision mesh filename=package://aist_robotiq/meshes/collision/robotiq_arg2f_140_o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; visual mesh filename=package://aist_robotiq/meshes/visual/robotiq_arg2f_140_oute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
- added link b_bot_gripper_right_outer_knuckle, mass 0.00853198276973456; collision mesh filename=package://aist_robotiq/meshes/collision/robotiq_arg2f_140_o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; visual mesh filename=package://aist_robotiq/meshes/visual/robotiq_arg2f_140_oute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
- added link b_bot_gripper_robotiq_arg2f_base_link, mass 0.22652; collision mesh filename=package://aist_robotiq/meshes/collision/robotiq_arg2f_base_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; visual mesh filename=package://aist_robotiq/meshes/visual/robotiq_arg2f_base_lin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
- link b_bot_gripper_base_link: mass 0.3 -> None; geometry 
Joints:
- removed joint b_bot_gripper_tip_joint
- added joint b_bot_gripper_coupling_base_joint: type fixed, parent b_bot_ftsensor_flange_link, child b_bot_gripper_coupling_base_link, origin xyz=0 0 0 rpy=0 0 0
- added joint b_bot_gripper_coupling_flange_joint: type fixed, parent b_bot_gripper_coupling_base_link, child b_bot_gripper_coupling_flange_link, origin xyz=0.0111 0 0 rpy=0 0 0
- added joint b_bot_gripper_finger_joint: type revolute, parent b_bot_gripper_robotiq_arg2f_base_link, child b_bot_gripper_left_outer_knuckle, origin xyz=0 -0.030601 0.054905 rpy=2.2957963267948966 0 0, axis -1 0 0, limit lower=0 upper=0.7 effort=1000 velocity=2.0
- added joint b_bot_gripper_left_inner_finger_joint: type revolute, parent b_bot_gripper_left_outer_finger, child b_bot_gripper_left_inner_finger, origin xyz=0 0.0817554015893473 -0.0282203446692936 rpy=-0.725 0 0, axis -1 0 0, limit lower=-0.8757 upper=0.8757 effort=1000 velocity=2.0, mimic joint=b_bot_gripper_finger_joint multiplier=-1 offset=0
- added joint b_bot_gripper_left_inner_finger_pad_joint: type fixed, parent b_bot_gripper_left_inner_finger, child b_bot_gripper_left_inner_finger_pad, origin xyz=0 0.0457554015893473 -0.0272203446692936 rpy=0 0 0, axis 0 0 1
- added joint b_bot_gripper_left_inner_knuckle_joint: type revolute, parent b_bot_gripper_robotiq_arg2f_base_link, child b_bot_gripper_left_inner_knuckle, origin xyz=0 -0.0127 0.06142 rpy=2.2957963267948966 0 0.0, axis -1 0 0, limit lower=-0.8757 upper=0.8757 effort=1000 velocity=2.0, mimic joint=b_bot_gripper_finger_joint multiplier=1 offset=0
- added joint b_bot_gripper_left_outer_finger_joint: type fixed, parent b_bot_gripper_left_outer_knuckle, child b_bot_gripper_left_outer_finger, origin xyz=0 0.01821998610742 0.0260018192872234 rpy=0 0 0, axis 1 0 0
- added joint b_bot_gripper_right_inner_finger_joint: type revolute, parent b_bot_gripper_right_outer_finger, child b_bot_gripper_right_inner_finger, origin xyz=0 0.0817554015893473 -0.0282203446692936 rpy=-0.725 0 0, axis -1 0 0, limit lower=-0.8757 upper=0.8757 effort=1000 velocity=2.0, mimic joint=b_bot_gripper_finger_joint multiplier=-1 offset=0
- added joint b_bot_gripper_right_inner_finger_pad_joint: type fixed, parent b_bot_gripper_right_inner_finger, child b_bot_gripper_right_inner_finger_pad, origin xyz=0 0.0457554015893473 -0.0272203446692936 rpy=0 0 0, axis 0 0 1
- added joint b_bot_gripper_right_inner_knuckle_joint: type revolute, parent b_bot_gripper_robotiq_arg2f_base_link, child b_bot_gripper_right_inner_knuckle, origin xyz=0 0.0127 0.06142 rpy=2.2957963267948966 0 -3.141592653589793, axis -1 0 0, limit lower=-0.8757 upper=0.8757 effort=1000 velocity=2.0, mimic joint=b_bot_gripper_finger_joint multiplier=1 offset=0
- added joint b_bot_gripper_right_outer_finger_joint: type fixed, parent b_bot_gripper_right_outer_knuckle, child b_bot_gripper_right_outer_finger, origin xyz=0 0.01821998610742 0.0260018192872234 rpy=0 0 0, axis 1 0 0
- added joint b_bot_gripper_right_outer_knuckle_joint: type revolute, parent b_bot_gripper_robotiq_arg2f_base_link, child b_bot_gripper_right_outer_knuckle, origin xyz=0 0.030601 0.054905 rpy=2.2957963267948966 0 3.141592653589793, axis -1 0 0, limit lower=-0.725 upper=0.725 effort=1000 velocity=2.0, mimic joint=b_bot_gripper_finger_joint multiplier=1 offset=0
- added joint b_bot_gripper_robotiq_arg2f_base_joint: type fixed, parent b_bot_gripper_base_link, child b_bot_gripper_robotiq_arg2f_base_link, origin xyz=0 0 0 rpy=3.141592653589793 -1.5707963267948966 0
- added joint b_bot_gripper_tip_link_joint: type fixed, parent b_bot_gripper_base_link, child b_bot_gripper_tip_link, origin xyz=.2328 0.0 0.0 rpy=0.0 -1.5707963267948966 0.0
- joint a_bot_ftsensor_ft300_joint: origin xyz=0 0 0 rpy=0 0 0 -> xyz=0 0 0 rpy=3.141592653589793 0 0
- joint a_bot_inside_camera_joint: origin xyz=0.010324554587117304      0.0018335412329232095      0.06467303743182957 rpy=0.025912000078364868      0.4021372934071272      0.01607525693523146 -> xyz=0.0051834717267641005      0.0029869415393767723      0.06398615295764885 rpy=0.02104566011309687      0.3968034960518725      0.01313899562905875
- joint a_bot_outside_camera_joint: origin xyz=0.03590302041834074      -0.008099774421321322      0.07959004727089102 rpy=0.016977853905271578      -0.21989995636200013      0.03446978804301341 -> xyz=0.03448420081903219      -0.008163711886056418      0.08142610495899788 rpy=0.013998136792162967      -0.22309733722281236      0.035938176557628945
- joint a_motioncam_link_joint: origin xyz=0.5250340162175878 -0.10043474330440638 0.659948826203397 rpy=0.055276438915859344 1.0603529787148211 -3.09644910582365 -> xyz=0.5273204178052611 -0.09837025272929169 0.6624180668081472 rpy=0.08314875444590407 1.0661814021341067 -3.0606137322137723
- joint b_bot_ftsensor_ft300_joint: origin xyz=0 0 0 rpy=0 0 0 -> xyz=0 0 0 rpy=3.141592653589793 0 0
- joint b_bot_gripper_base_joint: origin xyz=0 0 0 rpy=0 -0.017453292519943295 -0.005235987755982988 -> xyz=0 0 0 rpy=0 0 0; parent b_bot_ftsensor_flange_link -> b_bot_gripper_coupling_flange_link
- joint cage_front_left_pillar: origin xyz=-0.58 -0.79 0.164 rpy=0 0 0 -> xyz=-0.585    -0.795    0.164 rpy=0 0 0
- joint cage_tool_bar: origin xyz=0 0 0.31 rpy=0 0 0 -> xyz=0 0 0.27 rpy=0 0 0
- joint workspace_live_camera_joint: origin xyz=0.4076098270054865 -0.041827815223630944 0.7417406575198592 rpy=-2.70626389040216 0.06825373432442536 1.5972576864936887 -> xyz=0.4411927402377287 -0.1035554662373815 0.7339914909084881 rpy=-2.655694361220333 0.05917472246881731 1.613355025035372

Commit message: Replace UR5 with UR5e

File: aist_description/scenes/urdf/aist_base_scene.urdf.xacro (robot description, xacro)
@@ -84,9 +84,9 @@
       prefix="a_bot_"
       joint_limits_parameters_file="$(find ur_description
-				    )/config/ur5/joint_limits.yaml"
+				    )/config/ur5e/joint_limits.yaml"
       physical_parameters_file="$(find ur_description
-				)/config/ur5/physical_parameters.yaml"
+				)/config/ur5e/physical_parameters.yaml"
       visual_parameters_file="$(find ur_description
-			      )/config/ur5/visual_parameters.yaml"
+			      )/config/ur5e/visual_parameters.yaml"
       kinematics_parameters_file="$(find aist_bringup
 				  )/config/a_bot_calibration.yaml"
@@ -97,9 +97,9 @@
       prefix="b_bot_"
       joint_limits_parameters_file="$(find ur_description
-				    )/config/ur5/joint_limits.yaml"
+				    )/config/ur5e/joint_limits.yaml"
       physical_parameters_file="$(find ur_description
-				)/config/ur5/physical_parameters.yaml"
+				)/config/ur5e/physical_parameters.yaml"
       visual_parameters_file="$(find ur_description
-			      )/config/ur5/visual_parameters.yaml"
+			      )/config/ur5e/visual_parameters.yaml"
       kinematics_parameters_file="$(find aist_bringup
 				  )/config/b_bot_calibration.yaml"
@@ -135,16 +135,16 @@
   <!-- </xacro:zivid2plus> -->
   <!-- Spawn and attach force sensor -->
-  <xacro:include filename="$(find aist_robotiq)/urdf/ft300.urdf.xacro"/>
-  <xacro:ft300 prefix="a_bot_ftsensor_" parent="a_bot_flange">
-    <origin xyz="0 0 0" rpy="${pi} 0 0"/>
-  </xacro:ft300>
-  <xacro:ft300 prefix="b_bot_ftsensor_" parent="b_bot_flange">
-    <origin xyz="0 0 0" rpy="${pi} 0 0"/>
-  </xacro:ft300>
+  <!-- <xacro:include filename="$(find aist_robotiq)/urdf/ft300.urdf.xacro"/> -->
+  <!-- <xacro:ft300 prefix="a_bot_ftsensor_" parent="a_bot_flange"> -->
+  <!--   <origin xyz="0 0 0" rpy="${pi} 0 0"/> -->
+  <!-- </xacro:ft300> -->
+  <!-- <xacro:ft300 prefix="b_bot_ftsensor_" parent="b_bot_flange"> -->
+  <!--   <origin xyz="0 0 0" rpy="${pi} 0 0"/> -->
+  <!-- </xacro:ft300> -->
   <!-- Spawn and attach gripper -->
   <xacro:include filename="$(find aist_robotiq
 			   )/urdf/robotiq_arg2f_coupling.urdf.xacro"/>
   <xacro:robotiq_arg2f_coupling prefix="a_bot_gripper_coupling_"
-				parent="a_bot_ftsensor_flange_link">
+				parent="a_bot_flange">
     <origin xyz="0 0 0" rpy="0 0 0"/>
   </xacro:robotiq_arg2f_coupling>
@@ -156,5 +156,5 @@
   </xacro:robotiq_140_gripper>
   <xacro:robotiq_arg2f_coupling prefix="b_bot_gripper_coupling_"
-				parent="b_bot_ftsensor_flange_link">
+				parent="b_bot_flange">
     <origin xyz="0 0 0" rpy="0 0 0"/>
   </xacro:robotiq_arg2f_coupling>

File: moveit_config/aist_moveit_config/config/gazebo_aist_base_scene.urdf (robot description, URDF)
Before this commit: robot aist_base_scene, 145 links, 144 joints
Links:
- removed link a_bot_ftsensor_base_link
- removed link a_bot_ftsensor_flange_link
- removed link a_bot_ftsensor_wrench_link
- removed link b_bot_ftsensor_base_link
- removed link b_bot_ftsensor_flange_link
- removed link b_bot_ftsensor_wrench_link
- link a_bot_base_link_inertia: geometry collision mesh filename=package://ur_description/meshes/ur5e/collision/base.stl; visual mesh filename=package://ur_description/meshes/ur5e/visual/base.dae
- link a_bot_forearm_link: geometry collision mesh filename=package://ur_description/meshes/ur5e/collision/forearm.stl; visual mesh filename=package://ur_description/meshes/ur5e/visual/forearm.dae
- link a_bot_shoulder_link: geometry collision mesh filename=package://ur_description/meshes/ur5e/collision/shoulder.stl; visual mesh filename=package://ur_description/meshes/ur5e/visual/shoulder.dae
- link a_bot_upper_arm_link: geometry collision mesh filename=package://ur_description/meshes/ur5e/collision/upperarm.stl; visual mesh filename=package://ur_description/meshes/ur5e/visual/upperarm.dae
- link a_bot_wrist_1_link: geometry collision mesh filename=package://ur_description/meshes/ur5e/collision/wrist1.stl; visual mesh filename=package://ur_description/meshes/ur5e/visual/wrist1.dae
- link a_bot_wrist_2_link: geometry collision mesh filename=package://ur_description/meshes/ur5e/collision/wrist2.stl; visual mesh filename=package://ur_description/meshes/ur5e/visual/wrist2.dae
- link a_bot_wrist_3_link: geometry collision mesh filename=package://ur_description/meshes/ur5e/collision/wrist3.stl; visual mesh filename=package://ur_description/meshes/ur5e/visual/wrist3.dae
- link b_bot_base_link_inertia: geometry collision mesh filename=package://ur_description/meshes/ur5e/collision/base.stl; visual mesh filename=package://ur_description/meshes/ur5e/visual/base.dae
- link b_bot_forearm_link: geometry collision mesh filename=package://ur_description/meshes/ur5e/collision/forearm.stl; visual mesh filename=package://ur_description/meshes/ur5e/visual/forearm.dae
- link b_bot_shoulder_link: geometry collision mesh filename=package://ur_description/meshes/ur5e/collision/shoulder.stl; visual mesh filename=package://ur_description/meshes/ur5e/visual/shoulder.dae
- link b_bot_upper_arm_link: geometry collision mesh filename=package://ur_description/meshes/ur5e/collision/upperarm.stl; visual mesh filename=package://ur_description/meshes/ur5e/visual/upperarm.dae
- link b_bot_wrist_1_link: geometry collision mesh filename=package://ur_description/meshes/ur5e/collision/wrist1.stl; visual mesh filename=package://ur_description/meshes/ur5e/visual/wrist1.dae
- link b_bot_wrist_2_link: geometry collision mesh filename=package://ur_description/meshes/ur5e/collision/wrist2.stl; visual mesh filename=package://ur_description/meshes/ur5e/visual/wrist2.dae
- link b_bot_wrist_3_link: geometry collision mesh filename=package://ur_description/meshes/ur5e/collision/wrist3.stl; visual mesh filename=package://ur_description/meshes/ur5e/visual/wrist3.dae
Joints:
- removed joint a_bot_ftsensor_flange_joint
- removed joint a_bot_ftsensor_ft300_joint
- removed joint a_bot_ftsensor_wrench_joint
- removed joint b_bot_ftsensor_flange_joint
- removed joint b_bot_ftsensor_ft300_joint
- removed joint b_bot_ftsensor_wrench_joint
- joint a_bot_gripper_coupling_base_joint: parent a_bot_ftsensor_flange_link -> a_bot_flange
- joint b_bot_gripper_coupling_base_joint: parent b_bot_ftsensor_flange_link -> b_bot_flange

Commit message: Update aist_moveit_config

File: aist_description/scenes/urdf/aist_base_scene.urdf.xacro (robot description, xacro)
@@ -8,5 +8,5 @@
   <xacro:property name="b_bot_theta"	value="${pi}"/>
   <xacro:property name="bots_z"		value="0.770"/>
-  <xacro:property name="screen_z"	value="${bots_z + 0.040}"/>
+  <xacro:property name="screen_z"	value="${bots_z + 0.045}"/>
   <!-- ground -->
   <link name="ground"/>

Commit message: Change height of virtual screen

File: aist_description/scenes/urdf/aist_base_scene.urdf.xacro (robot description, xacro)
@@ -8,5 +8,5 @@
   <xacro:property name="b_bot_theta"	value="${pi}"/>
   <xacro:property name="bots_z"		value="0.770"/>
-  <xacro:property name="screen_z"	value="${bots_z + 0.045}"/>
+  <xacro:property name="screen_z"	value="${bots_z + 0.048}"/>
   <!-- ground -->
   <link name="ground"/>
