Commit message: Cleanup and add collision to cable_tool

File: aist_description/wrc/urdf/belt_tool.urdf.xacro (robot description, xacro)
@@ -1,6 +1,6 @@
 <?xml version="1.0"?>
 <robot xmlns:xacro="http://www.ros.org/wiki/xacro" name="belt_tool">
-  <xacro:macro name="belt_tool" params="partname parent *origin">
-    <link name="${partname}">
+  <xacro:macro name="belt_tool" params="name parent *origin">
+    <link name="${name}">
       <inertial>
 	<origin rpy="0 0 0" xyz="0 0 0"/>
@@ -9,5 +9,5 @@
       </inertial>
       <visual>
-	<origin rpy="0 0 ${-pi/2}" xyz="0.02 0 -0.017"/>
+	<origin xyz="0.02 0 -0.017" rpy="0 0 ${-pi/2}"/>
 	<geometry>
           <mesh filename="package://aist_description/wrc/meshes/belt_tool.stl" scale="0.001 0.001 0.001"/>
@@ -19,5 +19,5 @@
       <!-- The graspable part -->
       <collision>
-	<origin rpy="0 0 0" xyz="${.04/2} 0 ${-.01}"/>
+	<origin xyz="${.04/2} 0 ${-.01}" rpy="0 0 0"/>
 	<geometry>
           <box size=".04 .03 .055"/>
@@ -26,5 +26,5 @@
       <!-- The bottom part -->
       <collision>
-	<origin rpy="0 0 0" xyz="${.02} 0 ${-.03-.1/2}"/>
+	<origin xyz="${.02} 0 ${-.03-.1/2}" rpy="0 0 0"/>
 	<geometry>
           <box size=".01 .035 .1"/>
@@ -32,13 +32,13 @@
       </collision>
     </link>
-    <joint name="${partname}_joint" type="fixed">
+    <joint name="${name}_joint" type="fixed">
       <parent link="${parent}" />
-      <child link="${partname}" />
+      <child link="${name}" />
       <origin xyz="0 0 0" rpy="0 0 0" />
     </joint>
-    <link name="${partname}_pickup_link"/>
-    <joint name="${partname}_pickup_joint" type="fixed">
-      <parent link="${partname}" />
-      <child link="${partname}_pickup_link" />
+    <link name="${name}_pickup_link"/>
+    <joint name="${name}_pickup_joint" type="fixed">
+      <parent link="${name}" />
+      <child link="${name}_pickup_link" />
       <origin xyz=".02 0 -.01" rpy="0 ${pi/2} 0" />
     </joint>

File: aist_description/wrc/urdf/cable_tool.urdf.xacro (robot description, xacro)
@@ -1,6 +1,6 @@
 <?xml version="1.0"?>
 <robot xmlns:xacro="http://www.ros.org/wiki/xacro" name="cable_tool">
-  <xacro:macro name="cable_tool" params="partname parent *origin">
-    <link name="${partname}">
+  <xacro:macro name="cable_tool" params="name parent *origin">
+    <link name="${name}">
       <inertial>
 	<origin rpy="0 0 0" xyz="0 0 0"/>
@@ -18,25 +18,25 @@
       </visual>
       <collision>
-	<origin rpy="0 0 0" xyz="${.04/2} 0 ${-.01}"/>
+	<origin rpy="0 0 0" xyz="0 0 0"/>
 	<geometry>
-          <box size=".04 .03 .055"/>
-	</geometry>
-      </collision>
-      <collision>
-	<origin rpy="0 0 0" xyz="${.02} 0 ${-.03-.08/2}"/>
-	<geometry>
-          <cylinder length=".08" radius=".01"/>
+          <mesh filename="package://aist_description/wrc/meshes/cable_tool-collision.stl" scale="0.001 0.001 0.001"/>
 	</geometry>
       </collision>
     </link>
-    <joint name="${partname}_joint" type="fixed">
+    <joint name="${name}_joint" type="fixed">
       <parent link="${parent}" />
-      <child  link="${partname}" />
+      <child  link="${name}" />
       <xacro:insert_block name="origin"/>
     </joint>
-    <link name="${partname}_tip_link"/>
-    <joint name="${partname}_tip_joint" type="fixed">
-      <parent link="${partname}" />
-      <child  link="${partname}_tip_link" />
+    <link name="${name}_pickup_link"/>
+    <joint name="${name}_pickup_joint" type="fixed">
+      <parent link="${name}" />
+      <child  link="${name}_pickup_link" />
+      <origin xyz="0 0 0" rpy="0 0 0" />
+    </joint>
+    <link name="${name}_tip_link"/>
+    <joint name="${name}_tip_joint" type="fixed">
+      <parent link="${name}" />
+      <child  link="${name}_tip_link" />
       <origin xyz="0.05 0 0" rpy="0 0 0" />
     </joint>

File: aist_description/wrc/urdf/cable_tool_holder.urdf.xacro (robot description, xacro)
@@ -1,6 +1,6 @@
 <?xml version="1.0"?>
 <robot name="cable_tool_holder" xmlns:xacro="http://www.ros.org/wiki/xacro">
-  <xacro:macro name="cable_tool_holder" params="partname parent *origin">
-    <link name="${partname}">
+  <xacro:macro name="cable_tool_holder" params="name parent *origin">
+    <link name="${name}">
       <inertial>
 	<origin rpy="0 0 0" xyz="0 0 0"/>
@@ -18,13 +18,13 @@
       </visual>
     </link>
-    <joint name="${partname}_joint" type="fixed">
+    <joint name="${name}_joint" type="fixed">
       <parent link="${parent}" />
-      <child  link="${partname}" />
+      <child  link="${name}" />
       <xacro:insert_block name="origin"/>
     </joint>
-    <link name="${partname}_pickup_link"/>
-    <joint name="${partname}_pickup_joint" type="fixed">
-      <parent link="${partname}" />
-      <child  link="${partname}_pickup_link" />
+    <link name="${name}_home_link"/>
+    <joint name="${name}_home_joint" type="fixed">
+      <parent link="${name}" />
+      <child  link="${name}_home_link" />
       <origin xyz="0.1 0.004 0.015" rpy="0 ${pi/2} 0" />
     </joint>

File: aist_description/wrc/urdf/gravity_tool_holder.urdf.xacro (robot description, xacro)
@@ -3,6 +3,6 @@
   <!-- To use the tip of the holder to place the macro, use these offsets: -->
   <!-- <origin xyz="${+0.01} ${+.03} ${-0.0465}" rpy="0 0 0" />   -->
-  <xacro:macro name="gravity_tool_holder" params="partname parent *origin">
-    <link name="${partname}">
+  <xacro:macro name="gravity_tool_holder" params="name parent *origin">
+    <link name="${name}">
       <visual>
 	<origin rpy="${pi/2} 0 ${pi/2}" xyz="0 -.025 -.005"/>
@@ -21,7 +21,7 @@
       </collision>
     </link>
-    <joint name="${partname}_joint" type="fixed">
+    <joint name="${name}_joint" type="fixed">
       <parent link="${parent}" />
-      <child link="${partname}" />
+      <child link="${name}" />
       <origin xyz="0 0 0" rpy="0 0 0" />
     </joint>

File: aist_description/wrc/urdf/nut_holder.urdf.xacro (robot description, xacro)
@@ -3,7 +3,7 @@
   <!-- To use the tip of the holder to place the macro, use these offsets: -->
   <!-- <origin xyz="${+0.01} ${+.03} ${-0.0465}" rpy="0 0 0" />   -->
-  <xacro:macro name="nut_holder" params="partname parent *origin">
+  <xacro:macro name="nut_holder" params="name parent *origin">
   <xacro:property name="mesh_file" value="package://aist_description/wrc/meshes/nut_holder.stl" />
-  <link name="${partname}">
+  <link name="${name}">
     <inertial>
       <origin rpy="0 0 0" xyz="0 0 0.0"/>
@@ -33,21 +33,21 @@
     </collision>
   </link>
-  <joint name="${partname}" type="fixed">
+  <joint name="${name}" type="fixed">
     <parent link="${parent}" />
-    <child link = "${partname}" />
+    <child link = "${name}" />
     <xacro:insert_block name="origin"/>
   </joint>
-  <joint name="${partname}_collar_joint" type="fixed">
-    <parent link="${partname}"/>
-    <child link="${partname}_collar_link"/>
+  <joint name="${name}_collar_joint" type="fixed">
+    <parent link="${name}"/>
+    <child link="${name}_collar_link"/>
     <origin rpy="0 ${pi/2} 0" xyz="-0.01 -.03 0.04"/>
   </joint>
-  <link name="${partname}_collar_link"/>
-  <joint name="${partname}_tip_joint" type="fixed">
-    <parent link="${partname}_collar_link"/>
-    <child link="${partname}_tip_link"/>
+  <link name="${name}_collar_link"/>
+  <joint name="${name}_tip_joint" type="fixed">
+    <parent link="${name}_collar_link"/>
+    <child link="${name}_tip_link"/>
     <origin rpy="0 0 0" xyz="-0.01 0 0"/>
   </joint>
-  <link name="${partname}_tip_link"/>
+  <link name="${name}_tip_link"/>
   </xacro:macro>
 </robot>

File: aist_description/wrc/urdf/plunger_tool.urdf.xacro (robot description, xacro)
@@ -1,6 +1,6 @@
 <?xml version="1.0"?>
 <robot xmlns:xacro="http://www.ros.org/wiki/xacro" name="plunger_tool">
-  <xacro:macro name="plunger_tool" params="partname parent *origin">
-    <link name="${partname}">
+  <xacro:macro name="plunger_tool" params="name parent *origin">
+    <link name="${name}">
       <inertial>
 	<origin rpy="0 0 0" xyz="0 0 0"/>
@@ -9,5 +9,5 @@
       </inertial>
       <visual>
-	<origin rpy="0 ${pi/2} ${pi/2}" xyz="0.02 0 -0.017"/>
+	<origin xyz="0.02 0 -0.017" rpy="0 ${pi/2} ${pi/2}"/>
 	<geometry>
           <mesh filename="package://aist_description/wrc/meshes/plunger_tool.stl" scale="0.001 0.001 0.001"/>
@@ -18,5 +18,5 @@
       </visual>
       <collision>
-	<origin rpy="0 0 0" xyz="${.04/2} 0 ${-.01}"/>
+	<origin xyz="${.04/2} 0 ${-.01}" rpy="0 0 0"/>
 	<geometry>
           <box size=".04 .03 .055"/>
@@ -24,5 +24,5 @@
       </collision>
       <collision>
-	<origin rpy="0 0 0" xyz="${.02} 0 ${-.03-.08/2}"/>
+	<origin xyz="${.02} 0 ${-.03-.08/2}" rpy="0 0 0"/>
 	<geometry>
           <cylinder length=".08" radius=".01"/>
@@ -30,13 +30,13 @@
       </collision>
     </link>
-    <joint name="${partname}_joint" type="fixed">
+    <joint name="${name}_joint" type="fixed">
       <parent link="${parent}" />
-      <child  link="${partname}" />
+      <child  link="${name}" />
       <origin xyz="0 0 0" rpy="0 0 0" />
     </joint>
-    <link name="${partname}_pickup_link"/>
-    <joint name="${partname}_pickup_joint" type="fixed">
-      <parent link="${partname}" />
-      <child  link="${partname}_pickup_link" />
+    <link name="${name}_pickup_link"/>
+    <joint name="${name}_pickup_joint" type="fixed">
+      <parent link="${name}" />
+      <child  link="${name}_pickup_link" />
       <origin xyz=".02 0 -.01" rpy="0 ${pi/2} 0" />
     </joint>

File: aist_description/wrc/urdf/simple_holder.urdf.xacro (robot description, xacro)
@@ -3,7 +3,7 @@
   <!-- To use the tip of the holder to place the macro, use these offsets: -->
   <!-- <origin xyz="${+0.01} ${+.03} ${-0.0465}" rpy="0 0 0" />   -->
-  <xacro:macro name="simple_holder" params="partname parent *origin">
+  <xacro:macro name="simple_holder" params="name parent *origin">
   <xacro:property name="mesh_file" value="package://aist_description/wrc/meshes/simple_holder.stl" />
-  <link name="${partname}">
+  <link name="${name}">
     <inertial>
       <origin rpy="0 0 0" xyz="0 0 0.0"/>
@@ -33,15 +33,15 @@
     </collision> -->
   </link>
-  <joint name="${partname}" type="fixed">
+  <joint name="${name}" type="fixed">
     <parent link="${parent}" />
-    <child link = "${partname}" />
+    <child link = "${name}" />
     <xacro:insert_block name="origin"/>
   </joint>
-  <joint name="${partname}_tip_joint" type="fixed">
-    <parent link="${partname}"/>
-    <child link="${partname}_tip_link"/>
+  <joint name="${name}_tip_joint" type="fixed">
+    <parent link="${name}"/>
+    <child link="${name}_tip_link"/>
     <origin rpy="0 0 0" xyz="0.0 0.0 0.04"/>
   </joint>
-  <link name="${partname}_tip_link"/>
+  <link name="${name}_tip_link"/>
   </xacro:macro>
 </robot>

File: aist_description/wrc/urdf/washer_holder.urdf.xacro (robot description, xacro)
@@ -3,7 +3,7 @@
   <!-- To use the tip of the holder to place the macro, use these offsets: -->
   <!-- <origin xyz="${+0.01} ${+.03} ${-0.0465}" rpy="0 0 0" />   -->
-  <xacro:macro name="washer_holder" params="partname parent *origin">
+  <xacro:macro name="washer_holder" params="name parent *origin">
   <xacro:property name="mesh_file" value="package://aist_description/wrc/meshes/washer_holder.stl" />
-  <link name="${partname}">
+  <link name="${name}">
     <inertial>
       <origin rpy="0 0 0" xyz="0 0 0.0"/>
@@ -33,21 +33,21 @@
     </collision>
   </link>
-  <joint name="${partname}" type="fixed">
+  <joint name="${name}" type="fixed">
     <parent link="${parent}" />
-    <child link = "${partname}" />
+    <child link = "${name}" />
     <xacro:insert_block name="origin"/>
   </joint>
-  <joint name="${partname}_collar_joint" type="fixed">
-    <parent link="${partname}"/>
-    <child link="${partname}_collar_link"/>
+  <joint name="${name}_collar_joint" type="fixed">
+    <parent link="${name}"/>
+    <child link="${name}_collar_link"/>
     <origin rpy="0 ${pi/2} 0" xyz="-0.01 -.03 0.04"/>
   </joint>
-  <link name="${partname}_collar_link"/>
-  <joint name="${partname}_tip_joint" type="fixed">
-    <parent link="${partname}_collar_link"/>
-    <child link="${partname}_tip_link"/>
+  <link name="${name}_collar_link"/>
+  <joint name="${name}_tip_joint" type="fixed">
+    <parent link="${name}_collar_link"/>
+    <child link="${name}_tip_link"/>
     <origin rpy="0 0 0" xyz="-0.01 0 0"/>
   </joint>
-  <link name="${partname}_tip_link"/>
+  <link name="${name}_tip_link"/>
   </xacro:macro>
 </robot>
