Commit message: Change orientaion of screw holes

File: aist_description/wrc/urdf/kitting_trays.urdf.xacro (robot description, xacro)
@@ -9,6 +9,8 @@
   <!-- ========== The basic tray, without partitions -->
   <xacro:macro name="kitting_tray" params="trayname parent *origin">
-    <xacro:property name="mesh_file" value="package://aist_description/wrc/meshes/tray_PZ-0006-B.stl" />
-    <xacro:property name="mesh_file_col" value="package://aist_description/wrc/meshes/tray_PZ-0006-B.vhacd.dae" />
+    <xacro:property name="mesh_file"
+		    value="package://aist_description/wrc/meshes/tray_PZ-0006-B.stl" />
+    <xacro:property name="mesh_file_col"
+		    value="package://aist_description/wrc/meshes/tray_PZ-0006-B.vhacd.dae" />
     <link name="${trayname}">
       <inertial>
@@ -21,5 +23,4 @@
         <geometry>
           <mesh filename="${mesh_file}" scale="0.001 0.001 0.001"/>
-          <!-- <mesh filename="package://ur_description/meshes/ur5/visual/shoulder.dae"/> -->
         </geometry>
         <material name="white">
@@ -31,5 +32,4 @@
         <geometry>
           <mesh filename="${mesh_file_col}" scale="0.001 0.001 0.001"/>
-          <!-- <mesh filename="package://ur_description/meshes/ur5/collision/shoulder.stl"/> -->
         </geometry>
       </collision>
@@ -191,29 +191,38 @@
     <xacro:property name="m4_z_0" value="0.021"/>
     <xacro:auxiliary_frame parent="${trayname}" framename="screw_m4_1">
-      <origin xyz="${m4_x_0 + m4_x_delta*0} ${m4_y_0 + m4_y_delta*0} ${m4_z_0}" rpy="0 ${pi/2} 0" />
+      <origin xyz="${m4_x_0 + m4_x_delta*0} ${m4_y_0 + m4_y_delta*0} ${m4_z_0}"
+	      rpy="0 0 0" />
     </xacro:auxiliary_frame>
     <xacro:auxiliary_frame parent="${trayname}" framename="screw_m4_2">
-      <origin xyz="${m4_x_0 + m4_x_delta*0} ${m4_y_0 + m4_y_delta*1} ${m4_z_0}" rpy="0 ${pi/2} 0" />
+      <origin xyz="${m4_x_0 + m4_x_delta*0} ${m4_y_0 + m4_y_delta*1} ${m4_z_0}"
+	      rpy="0 0 0" />
     </xacro:auxiliary_frame>
     <xacro:auxiliary_frame parent="${trayname}" framename="screw_m4_3">
-      <origin xyz="${m4_x_0 + m4_x_delta*0} ${m4_y_0 + m4_y_delta*2} ${m4_z_0}" rpy="0 ${pi/2} 0" />
+      <origin xyz="${m4_x_0 + m4_x_delta*0} ${m4_y_0 + m4_y_delta*2} ${m4_z_0}"
+	      rpy="0 0 0" />
     </xacro:auxiliary_frame>
     <xacro:auxiliary_frame parent="${trayname}" framename="screw_m4_4">
-      <origin xyz="${m4_x_0 + m4_x_delta*1} ${m4_y_0 + m4_y_delta*0} ${m4_z_0}" rpy="0 ${pi/2} 0" />
+      <origin xyz="${m4_x_0 + m4_x_delta*1} ${m4_y_0 + m4_y_delta*0} ${m4_z_0}"
+	      rpy="0 0 0" />
     </xacro:auxiliary_frame>
     <xacro:auxiliary_frame parent="${trayname}" framename="screw_m4_5">
-      <origin xyz="${m4_x_0 + m4_x_delta*1} ${m4_y_0 + m4_y_delta*1} ${m4_z_0}" rpy="0 ${pi/2} 0" />
+      <origin xyz="${m4_x_0 + m4_x_delta*1} ${m4_y_0 + m4_y_delta*1} ${m4_z_0}"
+	      rpy="0 0 0" />
     </xacro:auxiliary_frame>
     <xacro:auxiliary_frame parent="${trayname}" framename="screw_m4_6">
-      <origin xyz="${m4_x_0 + m4_x_delta*1} ${m4_y_0 + m4_y_delta*2} ${m4_z_0}" rpy="0 ${pi/2} 0" />
+      <origin xyz="${m4_x_0 + m4_x_delta*1} ${m4_y_0 + m4_y_delta*2} ${m4_z_0}"
+	      rpy="0 0 0" />
     </xacro:auxiliary_frame>
     <xacro:auxiliary_frame parent="${trayname}" framename="screw_m4_7">
-      <origin xyz="${m4_x_0 + m4_x_delta*2} ${m4_y_0 + m4_y_delta*0} ${m4_z_0}" rpy="0 ${pi/2} 0" />
+      <origin xyz="${m4_x_0 + m4_x_delta*2} ${m4_y_0 + m4_y_delta*0} ${m4_z_0}"
+	      rpy="0 0 0" />
     </xacro:auxiliary_frame>
     <xacro:auxiliary_frame parent="${trayname}" framename="screw_m4_8">
-      <origin xyz="${m4_x_0 + m4_x_delta*2} ${m4_y_0 + m4_y_delta*1} ${m4_z_0}" rpy="0 ${pi/2} 0" />
+      <origin xyz="${m4_x_0 + m4_x_delta*2} ${m4_y_0 + m4_y_delta*1} ${m4_z_0}"
+	      rpy="0 0 0" />
     </xacro:auxiliary_frame>
     <xacro:auxiliary_frame parent="${trayname}" framename="screw_m4_9">
-      <origin xyz="${m4_x_0 + m4_x_delta*2} ${m4_y_0 + m4_y_delta*2} ${m4_z_0}" rpy="0 ${pi/2} 0" />
+      <origin xyz="${m4_x_0 + m4_x_delta*2} ${m4_y_0 + m4_y_delta*2} ${m4_z_0}"
+	      rpy="0 0 0" />
     </xacro:auxiliary_frame>
     <xacro:property name="m3_x_0" value="0.14"/>
@@ -223,20 +232,26 @@
     <xacro:property name="m3_z_0" value="0.021"/>
     <xacro:auxiliary_frame parent="${trayname}" framename="screw_m3_1">
-      <origin xyz="${m3_x_0 + m3_x_delta*0} ${m3_y_0 + m3_y_delta*0} ${m3_z_0}" rpy="0 ${pi/2} 0" />
+      <origin xyz="${m3_x_0 + m3_x_delta*0} ${m3_y_0 + m3_y_delta*0} ${m3_z_0}"
+	      rpy="0 0 0" />
     </xacro:auxiliary_frame>
     <xacro:auxiliary_frame parent="${trayname}" framename="screw_m3_2">
-      <origin xyz="${m3_x_0 + m3_x_delta*0} ${m3_y_0 + m3_y_delta*1} ${m3_z_0}" rpy="0 ${pi/2} 0" />
+      <origin xyz="${m3_x_0 + m3_x_delta*0} ${m3_y_0 + m3_y_delta*1} ${m3_z_0}"
+	      rpy="0 0 0" />
     </xacro:auxiliary_frame>
     <xacro:auxiliary_frame parent="${trayname}" framename="screw_m3_3">
-      <origin xyz="${m3_x_0 + m3_x_delta*0} ${m3_y_0 + m3_y_delta*2} ${m3_z_0}" rpy="0 ${pi/2} 0" />
+      <origin xyz="${m3_x_0 + m3_x_delta*0} ${m3_y_0 + m3_y_delta*2} ${m3_z_0}"
+	      rpy="0 0 0" />
     </xacro:auxiliary_frame>
     <xacro:auxiliary_frame parent="${trayname}" framename="screw_m3_4">
-      <origin xyz="${m3_x_0 + m3_x_delta*1} ${m3_y_0 + m3_y_delta*0} ${m3_z_0}" rpy="0 ${pi/2} 0" />
+      <origin xyz="${m3_x_0 + m3_x_delta*1} ${m3_y_0 + m3_y_delta*0} ${m3_z_0}"
+	      rpy="0 0 0" />
     </xacro:auxiliary_frame>
     <xacro:auxiliary_frame parent="${trayname}" framename="screw_m3_5">
-      <origin xyz="${m3_x_0 + m3_x_delta*1} ${m3_y_0 + m3_y_delta*1} ${m3_z_0}" rpy="0 ${pi/2} 0" />
+      <origin xyz="${m3_x_0 + m3_x_delta*1} ${m3_y_0 + m3_y_delta*1} ${m3_z_0}"
+	      rpy="0 0 0" />
     </xacro:auxiliary_frame>
     <xacro:auxiliary_frame parent="${trayname}" framename="screw_m3_6">
-      <origin xyz="${m3_x_0 + m3_x_delta*1} ${m3_y_0 + m3_y_delta*2} ${m3_z_0}" rpy="0 ${pi/2} 0" />
+      <origin xyz="${m3_x_0 + m3_x_delta*1} ${m3_y_0 + m3_y_delta*2} ${m3_z_0}"
+	      rpy="0 0 0" />
     </xacro:auxiliary_frame>
   </xacro:macro>
