Commit message: Add g_bot and g_bot_camera

File: aist_description/objects/urdf/cabinet.urdf.xacro (robot description, xacro)
@@ -4,5 +4,5 @@
   <xacro:macro name="cabinet"
 	       params="prefix width length base_height
-		       shelf1_height shelf2_height shelf3_height shelf4_height
+		       shelf1_height shelf2_height shelf3_height
 		       back_height parent *origin">
     <xacro:property name="thickness"	value="0.030" />
@@ -42,11 +42,11 @@
       <origin xyz="0 0 ${shelf3_height - thickness}" rpy="0 0 0"/>
     </xacro:aist_box>
-    <xacro:aist_box name="${prefix}cabinet_shelf4"
-		    width="${width}"
-		    length="${length - thickness}"
-		    height="${thickness}"
-		    parent="${prefix}cabinet_base">
-      <origin xyz="0 0 ${shelf4_height - thickness}" rpy="0 0 0"/>
-    </xacro:aist_box>
+    <!-- <xacro:aist_box name="${prefix}cabinet_shelf4" -->
+    <!-- 		    width="${width}" -->
+    <!-- 		    length="${length - thickness}" -->
+    <!-- 		    height="${thickness}" -->
+    <!-- 		    parent="${prefix}cabinet_base"> -->
+    <!--   <origin xyz="0 0 ${shelf4_height - thickness}" rpy="0 0 0"/> -->
+    <!-- </xacro:aist_box> -->
     <xacro:macro name="auxiliary_frame" params="parent framename *origin">
       <joint name="${parent}_${framename}" type="fixed">

Commit message: Update g_bot_base_scene

File: aist_description/objects/urdf/cabinet.urdf.xacro (robot description, xacro)
@@ -4,7 +4,7 @@
   <xacro:macro name="cabinet"
 	       params="prefix width length base_height
-		       shelf1_height shelf2_height shelf3_height
+		       shelf1_height shlef2_height
 		       back_height parent *origin">
-    <xacro:property name="thickness"	value="0.030" />
+    <xacro:property name="thickness"	value="0.012" />
     <xacro:aist_box name="${prefix}cabinet_base"
 		    width="${width}"
@@ -35,11 +35,11 @@
       <origin xyz="0 0 ${shelf2_height - thickness}" rpy="0 0 0"/>
     </xacro:aist_box>
-    <xacro:aist_box name="${prefix}cabinet_shelf3"
-		    width="${width}"
-		    length="${length - thickness}"
-		    height="${thickness}"
-		    parent="${prefix}cabinet_base">
-      <origin xyz="0 0 ${shelf3_height - thickness}" rpy="0 0 0"/>
-    </xacro:aist_box>
+    <!-- <xacro:aist_box name="${prefix}cabinet_shelf3" -->
+    <!-- 		    width="${width}" -->
+    <!-- 		    length="${length - thickness}" -->
+    <!-- 		    height="${thickness}" -->
+    <!-- 		    parent="${prefix}cabinet_base"> -->
+    <!--   <origin xyz="0 0 ${shelf3_height - thickness}" rpy="0 0 0"/> -->
+    <!-- </xacro:aist_box> -->
     <!-- <xacro:aist_box name="${prefix}cabinet_shelf4" -->
     <!-- 		    width="${width}" -->

File: aist_description/scenes/urdf/g_bot_base_scene.urdf.xacro (robot description, xacro)
@@ -4,13 +4,12 @@
   <xacro:arg name="scene" default=""/>
   <xacro:property name="g_bot_x"   value="0"/>
-  <xacro:property name="g_bot_y"   value="-0.610"/>
-  <xacro:property name="g_bot_z"   value="0.770"/>
+  <xacro:property name="g_bot_y"   value="-0.920"/>
+  <xacro:property name="g_bot_z"   value="0.700"/>
   <xacro:property name="cabinet_w" value="0.900"/>
   <xacro:property name="cabinet_l" value="0.400"/>
   <xacro:property name="cabinet_b" value="0.100"/>
-  <xacro:property name="shelf1_h"  value="0.443"/>
-  <xacro:property name="shelf2_h"  value="0.743"/>
-  <xacro:property name="shelf3_h"  value="1.043"/>
-  <xacro:property name="back_h"    value="1.366"/>
+  <xacro:property name="shelf1_h"  value="0.600"/>
+  <xacro:property name="shelf2_h"  value="0.990"/>
+  <xacro:property name="back_h"    value="1.500"/>
   <xacro:property name="mounter_w" value="0.200"/>
   <xacro:property name="mounter_l" value="0.200"/>

Commit message: Update g_bot_base_scene

File: aist_description/objects/urdf/cabinet.urdf.xacro (robot description, xacro)
@@ -4,5 +4,5 @@
   <xacro:macro name="cabinet"
 	       params="prefix width length base_height
-		       shelf1_height shlef2_height
+		       shelf1_height shelf2_height
 		       back_height parent *origin">
     <xacro:property name="thickness"	value="0.012" />

File: aist_description/scenes/urdf/g_bot_base_scene.urdf.xacro (robot description, xacro)
@@ -12,4 +12,5 @@
   <xacro:property name="shelf2_h"  value="0.990"/>
   <xacro:property name="back_h"    value="1.500"/>
+  <xacro:property name="wall_t"    value="0.012"/>
   <xacro:property name="mounter_w" value="0.200"/>
   <xacro:property name="mounter_l" value="0.200"/>
@@ -23,5 +24,4 @@
 		 shelf1_height="${shelf1_h}"
 		 shelf2_height="${shelf2_h}"
-		 shelf3_height="${shelf3_h}"
 		 back_height  ="${back_h}"
 		 parent="ground">
@@ -32,6 +32,18 @@
     <parent link="ground"/>
     <child  link="workspace_center"/>
-    <origin xyz="0 0 ${shelf3_h}" rpy="0 0 0"/>
+    <origin xyz="0 0 ${shelf2_h}" rpy="0 0 0"/>
   </joint>
+  <xacro:include filename="$(find aist_description
+			   )/objects/urdf/aist_box.urdf.xacro"/>
+  <xacro:aist_box name="left_wall"
+  		  width="${wall_t}" length="${cabinet_l}" height="${back_h}"
+  		  parent="cabinet_base">
+    <origin xyz="${-wall_t} 0 0" rpy="0 0 0"/>
+  </xacro:aist_box>
+  <xacro:aist_box name="right_wall"
+  		  width="${wall_t}" length="${cabinet_l}" height="${back_h}"
+  		  parent="cabinet_base">
+    <origin xyz="${cabinet_w} 0 0" rpy="0 0 0"/>
+  </xacro:aist_box>
   <!-- Robot mounter -->
   <xacro:include filename="$(find aist_description
