Commit message: Recover aist_robotiq package

File: aist_description/objects/urdf/ar_markers.urdf.xacro (robot description, xacro)
@@ -53,3 +53,11 @@
     </xacro:ar_marker>
   </xacro:macro>
+  <xacro:macro name="ar_marker_186_10"
+	       params="prefix parent marker_id thickness *origin">
+    <xacro:ar_marker prefix="${prefix}" parent="${parent}"
+		     marker_id="${marker_id}" size="0.186"
+		     margin="0.01" thickness="${thickness}">
+      <xacro:insert_block name="origin"/>
+    </xacro:ar_marker>
+  </xacro:macro>
 </robot>

Commit message: Add a marker_map

File: aist_description/objects/urdf/ar_markers.urdf.xacro (robot description, xacro)
@@ -61,3 +61,11 @@
     </xacro:ar_marker>
   </xacro:macro>
+  <xacro:macro name="ar_marker_150_5"
+	       params="prefix parent marker_id thickness *origin">
+    <xacro:ar_marker prefix="${prefix}" parent="${parent}"
+		     marker_id="${marker_id}" size="0.150"
+		     margin="0.005" thickness="${thickness}">
+      <xacro:insert_block name="origin"/>
+    </xacro:ar_marker>
+  </xacro:macro>
 </robot>

File: aist_description/scenes/urdf/aist_calibration.urdf.xacro (robot description, xacro)
@@ -15,9 +15,15 @@
     <origin xyz="0.063 0.0 0.0215" rpy="0 0 0"/>
   </xacro:ar_marker_70_5>
-  <xacro:ar_marker_70_5 prefix="workspace_"
-			parent="workspace_center"
-			marker_id="32"
-			thickness="0.001">
+  <!-- <xacro:ar_marker_70_5 prefix="workspace_" -->
+  <!-- 			parent="workspace_center" -->
+  <!-- 			marker_id="32" -->
+  <!-- 			thickness="0.001"> -->
+  <!--   <origin xyz="0.0 0.0 0.0005" rpy="0 0 0"/> -->
+  <!-- </xacro:ar_marker_70_5> -->
+  <xacro:ar_marker_150_5 prefix="workspace_"
+  			 parent="workspace_center"
+  			 marker_id="17_26_32_256"
+  			 thickness="0.001">
     <origin xyz="0.0 0.0 0.0005" rpy="0 0 0"/>
-  </xacro:ar_marker_70_5>
+  </xacro:ar_marker_150_5>
 </robot>

Commit message: Add ar markers

File: aist_description/objects/urdf/ar_markers.urdf.xacro (robot description, xacro)
@@ -69,3 +69,11 @@
     </xacro:ar_marker>
   </xacro:macro>
+  <xacro:macro name="ar_marker_76_4"
+	       params="prefix parent marker_id thickness *origin">
+    <xacro:ar_marker prefix="${prefix}" parent="${parent}"
+		     marker_id="${marker_id}" size="0.076"
+		     margin="0.004" thickness="${thickness}">
+      <xacro:insert_block name="origin"/>
+    </xacro:ar_marker>
+  </xacro:macro>
 </robot>

Commit message: Add URDF, ar_rect_marker

File: aist_description/objects/urdf/ar_markers.urdf.xacro (robot description, xacro)
@@ -77,3 +77,39 @@
     </xacro:ar_marker>
   </xacro:macro>
+  <xacro:macro name="ar_rect_marker"
+	       params="prefix parent marker_id size margin thickness *origin">
+    <joint name="${prefix}ar_marker_joint" type="fixed">
+      <parent link="${parent}" />
+      <child  link="${prefix}ar_marker" />
+      <xacro:insert_block name="origin" />
+    </joint>
+    <link name="${prefix}ar_marker">
+      <visual name="${prefix}ar_marker_visual">
+	<origin xyz="0 0 ${-thickness/2}" rpy="0 0 ${pi/2}"/>
+        <geometry>
+          <box size="${2*size + 4*margin} ${size + 2*margin} ${thickness}" />
+        </geometry>
+      </visual>
+      <collision name="${prefix}ar_marker_collision">
+	<origin xyz="0 0 ${-thickness/2}" rpy="0 0 ${pi/2}"/>
+        <geometry>
+          <box size="${2*size + 4*margin} ${size + 2*margin} ${thickness}" />
+        </geometry>
+      </collision>
+    </link>
+    <!-- For Gazebo, material of AR marker is defined in
+         aist_description/media/material. You also need to export
+         gazebo_media_path in package.xml. -->
+    <gazebo reference="${prefix}ar_marker">
+      <material>Aruco/marker-${marker_id}-${int(1000*size)}-${int(1000*margin)}</material>
+    </gazebo>
+  </xacro:macro>
+  <xacro:macro name="ar_rect_marker_28_3"
+	       params="prefix parent marker_id thickness *origin">
+    <xacro:ar_rect_marker prefix="${prefix}" parent="${parent}"
+			  marker_id="${marker_id}" size="0.028"
+			  margin="0.003" thickness="${thickness}">
+      <xacro:insert_block name="origin"/>
+    </xacro:ar_rect_marker>
+  </xacro:macro>
 </robot>

Commit message: Fixed orientation of texture of AR markers

File: aist_description/objects/urdf/ar_markers.urdf.xacro (robot description, xacro)
@@ -10,5 +10,5 @@
     <link name="${prefix}ar_marker">
       <visual name="${prefix}ar_marker_visual">
-	<origin xyz="0 0 ${-thickness/2}" rpy="0 0 ${pi}"/>
+	<origin xyz="0 0 ${-thickness/2}" rpy="0 0 ${pi/2}"/>
         <geometry>
           <box size="${size + 2*margin} ${size + 2*margin} ${thickness}" />
@@ -16,5 +16,5 @@
       </visual>
       <collision name="${prefix}ar_marker_collision">
-	<origin xyz="0 0 ${-thickness/2}" rpy="0 0 ${pi}"/>
+	<origin xyz="0 0 ${-thickness/2}" rpy="0 0 ${pi/2}"/>
         <geometry>
           <box size="${size + 2*margin} ${size + 2*margin} ${thickness}" />
