Commit message: Add screw tool holders to aist_base_scene

File: aist_description/objects/urdf/screw_tool_holder.urdf (robot description, URDF)
Before this commit: robot aaa, 1 links, 0 joints
Links:
- removed link world
- added link base_link

File: aist_description/objects/urdf/screw_tool_holder.urdf.xacro (robot description, xacro)
@@ -5,5 +5,5 @@
 	       params="prefix parent *origin">
     <!-- A link representing the gripper and a joint attaching it to parnet -->
-    <link name="${prefix}base_link">
+    <link name="${prefix}screw_tool_holder">
       <visual>
         <origin xyz="0 0 0" rpy="0 0 0"/>
@@ -11,6 +11,6 @@
           <mesh filename="package://aist_description/objects/meshes/screw_tool_holder.stl" scale="0.001 0.001 0.001"/>
 	</geometry>
-	<material name="light_grey">
-	  <color rgba="0.8 0.8 0.8 1"/>
+	<material name="white">
+	  <color rgba="0.9 0.9 0.9 1"/>
 	</material>
       </visual>
@@ -18,28 +18,22 @@
       <!-- avoid collision -->
 	<origin xyz="0 0 0" rpy="0 0 0"/>
-	<!-- <origin xyz="0.187 -0.035 -0.035" rpy="0 0 ${pi/2}"/> -->
 	<geometry>
 	  <mesh
-	      filename="package://aist_description/objects/meshes/screw_tool_holder.stlpwd" scale="0.001 0.001 0.001"/>
+	      filename="package://aist_description/objects/meshes/screw_tool_holder.stl" scale="0.001 0.001 0.001"/>
 	</geometry>
       </collision>
-      <inertial>
-	  <mass value="0.3"/>
-	  <inertia ixx="0.4" ixy="0.0" ixz="0.0" iyy="0.4"
-		   iyz="0.0" izz ="0.2"/>
-      </inertial>
     </link>
-    <joint name="${prefix}base_joint" type="fixed">
+    <joint name="${prefix}screw_tool_holder_joint" type="fixed">
       <parent link="${parent}"/>
-      <child  link="${prefix}base_link"/>
+      <child  link="${prefix}screw_tool_holder"/>
        <xacro:insert_block name="origin"/>
     </joint>
     <!-- A link representing the tool of the pad and a joint attaching
 	 it to the gripper -->
-    <link name="${prefix}tool_link"/>
-    <joint name="${prefix}tool_joint" type="fixed">
-      <parent link="${prefix}base_link"/>
-      <child  link="${prefix}tool_link"/>
-      <origin xyz="0.1855 0 0" rpy="0 0 0"/>
+    <link name="${prefix}screw_tool_cup"/>
+    <joint name="${prefix}screw_tool_cup_joint" type="fixed">
+      <parent link="${prefix}screw_tool_holder"/>
+      <child  link="${prefix}screw_tool_cup"/>
+      <origin xyz="0.0525 0 0.007" rpy="0 0 0"/>
     </joint>
   </xacro:macro>

File: aist_description/scenes/urdf/aist_base_scene.urdf.xacro (robot description, xacro)
@@ -47,4 +47,15 @@
 	    rpy="0 0 0" />
   </xacro:cage>
+  <!-- tool holders -->
+  <xacro:property name="m3_screw_tool_holder_y"	value="0.6"/>
+  <xacro:property name="m4_screw_tool_holder_y"	value="0.8"/>
+  <xacro:include filename="$(find aist_description
+			   )/objects/urdf/screw_tool_holder.urdf.xacro"/>
+  <xacro:screw_tool_holder prefix="m3_" parent="cage_tool_bar">
+    <origin xyz="0 ${m3_screw_tool_holder_y} ${cage_t}" rpy="0 0 0"/>
+  </xacro:screw_tool_holder>
+  <xacro:screw_tool_holder prefix="m4_" parent="cage_tool_bar">
+    <origin xyz="0 ${m4_screw_tool_holder_y} ${cage_t}" rpy="0 0 0"/>
+  </xacro:screw_tool_holder>
   <!-- robot arms -->
   <xacro:include filename="$(find ur_gazebo)/urdf/ur_macro.xacro"/>
