Commit message: Set precision_tool as a collision object

File: aist_description/objects/urdf/precision_tool_holder.urdf.xacro (robot description, xacro)
@@ -35,5 +35,6 @@
       <parent link="${prefix}base_link"/>
       <child  link="${prefix}link"/>
-      <origin xyz="0.07598 0.015 -0.015" rpy="0 ${30.0*pi/180.0} 0"/>
+      <!-- <origin xyz="0.10724 0.015 0.037607" rpy="0 ${30.0*pi/180.0} 0"/> -->
+      <origin xyz="0.108 0.015 0.037" rpy="0 ${30.0*pi/180.0} 0"/>
     </joint>
   </xacro:macro>

File: aist_precision_gripper/urdf/precision_gripper.urdf.xacro (robot description, xacro)
@@ -140,4 +140,5 @@
       </inertial>
     </link>
+    <!-- tip -->
     <joint name="${prefix}tip_link_joint" type="fixed">
       <parent link="${prefix}base_link"/>

Commit message: Adjust poses of components of precision tools

File: aist_description/objects/urdf/precision_tool_holder.urdf.xacro (robot description, xacro)
@@ -35,6 +35,5 @@
       <parent link="${prefix}base_link"/>
       <child  link="${prefix}link"/>
-      <!-- <origin xyz="0.10724 0.015 0.037607" rpy="0 ${30.0*pi/180.0} 0"/> -->
-      <origin xyz="0.108 0.015 0.037" rpy="0 ${30.0*pi/180.0} 0"/>
+      <origin xyz="0.108 0.012 0.037" rpy="0 ${30.0*pi/180.0} 0"/>
     </joint>
   </xacro:macro>

File: aist_precision_gripper/urdf/precision_gripper.urdf.xacro (robot description, xacro)
@@ -1,7 +1,4 @@
 <?xml version="1.0"?>
 <robot xmlns:xacro="http://ros.org/wiki/xacro">
-  <!--
-  Author: Cristian Beltran
--->
   <xacro:macro name="precision_gripper" params="prefix parent *origin">
     <xacro:include filename="$(find aist_precision_gripper
@@ -13,6 +10,7 @@
     <xacro:property name="max_gap"			value="0.010"/>
     <xacro:property name="depth"			value="0.030"/>
-    <xacro:property name="motor_width"			value="0.045"/>
+    <xacro:property name="motor_width"			value="0.055"/>
     <xacro:property name="motor_height"			value="0.0425"/>
+    <xacro:property name="motor_offset"			value="-0.003"/>
     <xacro:property name="lower_body_width"		value="0.085"/>
     <xacro:property name="lower_body_height"		value="0.050"/>
@@ -35,5 +33,5 @@
       </visual>
       <collision>
-        <origin xyz="${motor_height/2} 0 0" rpy="0 0 0"/>
+        <origin xyz="${motor_height/2} ${motor_offset} 0" rpy="0 0 0"/>
         <geometry>
           <box size="${motor_height} ${motor_width} ${depth}"/>
