Commit message: Rename links of screw_tool_holder

File: aist_description/objects/urdf/screw_tool_holder.urdf.xacro (robot description, xacro)
@@ -5,5 +5,5 @@
 	       params="prefix parent *origin">
     <!-- A link representing the gripper and a joint attaching it to parnet -->
-    <link name="${prefix}screw_tool_holder">
+    <link name="${prefix}base_link">
       <visual>
         <origin xyz="0 0 0" rpy="0 0 0"/>
@@ -24,15 +24,15 @@
       </collision>
     </link>
-    <joint name="${prefix}screw_tool_holder_joint" type="fixed">
+    <joint name="${prefix}base_joint" type="fixed">
       <parent link="${parent}"/>
-      <child  link="${prefix}screw_tool_holder"/>
+      <child  link="${prefix}base_link"/>
        <xacro:insert_block name="origin"/>
     </joint>
     <!-- A link representing the tool of the pad and a joint attaching
 	 it to the gripper -->
-    <link name="${prefix}screw_tool_cup"/>
-    <joint name="${prefix}screw_tool_cup_joint" type="fixed">
-      <parent link="${prefix}screw_tool_holder"/>
-      <child  link="${prefix}screw_tool_cup"/>
+    <link name="${prefix}link"/>
+    <joint name="${prefix}joint" type="fixed">
+      <parent link="${prefix}base_link"/>
+      <child  link="${prefix}link"/>
       <origin xyz="0.0525 0 0.007" rpy="0 0 0"/>
     </joint>

File: aist_description/scenes/urdf/aist_base_scene.urdf.xacro (robot description, xacro)
@@ -48,13 +48,15 @@
   </xacro:cage>
   <!-- tool holders -->
-  <xacro:property name="m3_screw_tool_holder_y"	value="0.6"/>
-  <xacro:property name="m4_screw_tool_holder_y"	value="0.8"/>
+  <xacro:property name="screw_tool_m3_holder_y"	value="0.6"/>
+  <xacro:property name="screw_tool_m4_holder_y"	value="0.8"/>
   <xacro:include filename="$(find aist_description
 			   )/objects/urdf/screw_tool_holder.urdf.xacro"/>
-  <xacro:screw_tool_holder prefix="m3_" parent="cage_tool_bar">
-    <origin xyz="0 ${m3_screw_tool_holder_y} ${cage_t}" rpy="0 0 0"/>
+  <xacro:screw_tool_holder prefix="screw_tool_m3_holder_"
+			   parent="cage_tool_bar">
+    <origin xyz="0 ${screw_tool_m3_holder_y} ${cage_t}" rpy="0 0 0"/>
   </xacro:screw_tool_holder>
-  <xacro:screw_tool_holder prefix="m4_" parent="cage_tool_bar">
-    <origin xyz="0 ${m4_screw_tool_holder_y} ${cage_t}" rpy="0 0 0"/>
+  <xacro:screw_tool_holder prefix="screw_tool_m4_holder_"
+			   parent="cage_tool_bar">
+    <origin xyz="0 ${screw_tool_m4_holder_y} ${cage_t}" rpy="0 0 0"/>
   </xacro:screw_tool_holder>
   <!-- robot arms -->

Commit message: Confirmed that planning is possible with tip link of the tool grasped by default gripper

File: aist_description/objects/urdf/screw_tool_holder.urdf.xacro (robot description, xacro)
@@ -19,6 +19,5 @@
 	<origin xyz="0 0 0" rpy="0 0 0"/>
 	<geometry>
-	  <mesh
-	      filename="package://aist_description/objects/meshes/screw_tool_holder.stl" scale="0.001 0.001 0.001"/>
+	  <mesh filename="package://aist_description/objects/meshes/screw_tool_holder.stl" scale="0.001 0.001 0.001"/>
 	</geometry>
       </collision>
