Commit message: Change height of camera bar

File: aist_description/objects/urdf/cage.urdf.xacro (robot description, xacro)
@@ -4,5 +4,6 @@
   <xacro:macro name="cage"
 	       params="prefix width length height thickness
-		       workspace_height toolbar_height parent *origin">
+		       workspace_height tool_bar_height camera_bar_height
+		       parent *origin">
     <xacro:macro name="pillars" params="*origin">
       <xacro:aist_box name="${prefix}front_left_pillar"
@@ -38,5 +39,6 @@
       </xacro:aist_box>
     </xacro:macro>
-    <xacro:macro name="rectangle" params="prefix2 height *origin">
+    <xacro:macro name="rectangle"
+		 params="prefix2 height right_bar_height *origin">
       <xacro:aist_box name="${prefix}${prefix2}front_bar"
 		      width="${width - 2*thickness}"
@@ -66,5 +68,5 @@
 		      height="${thickness}"
 		      parent="${prefix}front_left_pillar">
-	<origin xyz="${width - thickness} ${thickness} ${height}"
+	<origin xyz="${width - thickness} ${thickness} ${right_bar_height}"
 		rpy="0 0 0"/>
       </xacro:aist_box>
@@ -75,9 +77,10 @@
     </xacro:pillars>
     <!-- base rectangle -->
-    <xacro:rectangle prefix2="lower_" height="0">
+    <xacro:rectangle prefix2="lower_" height="0" right_bar_height="0">
       <xacro:insert_block name="origin"/>
     </xacro:rectangle>
     <!-- ceiling rectangle -->
-    <xacro:rectangle prefix2="upper_" height="${height - thickness}">
+    <xacro:rectangle prefix2="upper_" height="${height - thickness}"
+		     right_bar_height="${camera_bar_height}">
       <xacro:insert_block name="origin"/>
     </xacro:rectangle>
@@ -88,5 +91,5 @@
     		    height="${thickness}"
     		    parent="${prefix}lower_left_bar">
-      <origin xyz="0 0  ${workspace_height}" rpy="0 0 0"/>
+      <origin xyz="0 0 ${workspace_height - thickness}" rpy="0 0 0"/>
     </xacro:aist_box>
     <!-- tool bar -->
@@ -96,5 +99,5 @@
     		    height="${thickness}"
     		    parent="${prefix}workspace_bar">
-      <origin xyz="0 0 ${toolbar_height}" rpy="0 0 0"/>
+      <origin xyz="0 0 ${tool_bar_height + thickness}" rpy="0 0 0"/>
     </xacro:aist_box>
   </xacro:macro>

File: aist_description/scenes/urdf/aist_base_scene.urdf.xacro (robot description, xacro)
@@ -26,9 +26,10 @@
   </joint>
   <!-- cage -->
-  <xacro:property name="cage_w"		value="1.220"/>
-  <xacro:property name="cage_l"		value="1.600"/>
-  <xacro:property name="cage_h"		value="1.400"/>
-  <xacro:property name="cage_t"		value="0.050"/>
-  <xacro:property name="toolbar_h"	value="0.300"/>
+  <xacro:property name="cage_w"		value="1.200"/>
+  <xacro:property name="cage_l"		value="1.580"/>
+  <xacro:property name="cage_h"		value="1.420"/>
+  <xacro:property name="cage_t"		value="0.040"/>
+  <xacro:property name="tool_bar_h"	value="0.270"/>
+  <xacro:property name="camera_bar_h"	value="1.280"/>
   <xacro:property name="cage_z"		value="0.164"/>
   <xacro:property name="cage_offset"	value="0.020"/>
@@ -39,5 +40,6 @@
 	      thickness="${cage_t}"
 	      workspace_height="${bots_z - cage_z}"
-	      toolbar_height="${toolbar_h}"
+	      tool_bar_height="${tool_bar_h}"
+	      camera_bar_height="${camera_bar_h}"
 	      parent="ground">
     <origin xyz="${-cage_w/2 + cage_offset} ${-cage_l/2} ${cage_z}"

Commit message: Fixed heihgt of tool_bar of cage

File: aist_description/objects/urdf/cage.urdf.xacro (robot description, xacro)
@@ -99,5 +99,5 @@
     		    height="${thickness}"
     		    parent="${prefix}workspace_bar">
-      <origin xyz="0 0 ${tool_bar_height + thickness}" rpy="0 0 0"/>
+      <origin xyz="0 0 ${tool_bar_height}" rpy="0 0 0"/>
     </xacro:aist_box>
   </xacro:macro>

Commit message: Swap robotiq grippers between a_bot and b_bot

File: aist_description/objects/urdf/cage.urdf.xacro (robot description, xacro)
@@ -91,5 +91,5 @@
     		    height="${thickness}"
     		    parent="${prefix}lower_left_bar">
-      <origin xyz="0 0 ${workspace_height - thickness}" rpy="0 0 0"/>
+      <origin xyz="0 0 ${workspace_height - thickness + 0.03}" rpy="0 0 0"/>
     </xacro:aist_box>
     <!-- tool bar -->

File: aist_description/scenes/urdf/a_bot_base_scene.urdf.xacro (robot description, xacro)
@@ -6,21 +6,6 @@
   <xacro:property name="bots_z"		value="0.770"/>
   <xacro:property name="screen_z"	value="${bots_z + 0.0347}"/>
-  <!-- ground and workspace -->
+  <!-- ground -->
   <link name="ground"/>
-  <xacro:property name="table_w"	value="0.900"/>
-  <xacro:property name="table_l"	value="1.800"/>
-  <xacro:include filename="$(find aist_description
-			   )/objects/urdf/table.urdf.xacro"/>
-  <xacro:table prefix="workspace_"
-	       width="${table_w}" length="${table_l}" height="${bots_z}"
-	       parent="ground">
-    <origin xyz="${-table_w/2} ${-table_l/2} 0" rpy="0 0 0"/>
-  </xacro:table>
-  <link name="workspace_center"/>
-  <joint name="ground_to_workspace" type="fixed">
-    <parent link="ground"/>
-    <child  link="workspace_center"/>
-    <origin xyz="0 0 ${bots_z}" rpy="0 0 0"/>
-  </joint>
   <!-- cage -->
   <xacro:property name="cage_w"		value="1.200"/>
@@ -31,5 +16,5 @@
   <xacro:property name="camera_bar_h"	value="1.325"/>
   <xacro:property name="cage_z"		value="0.164"/>
-  <xacro:property name="cage_offset_x"	value="0.020"/>
+  <xacro:property name="cage_offset_x"	value="0.015"/>
   <xacro:property name="cage_offset_y"	value="-0.005"/>
   <xacro:include filename="$(find aist_description
@@ -47,4 +32,21 @@
 	    rpy="0 0 0" />
   </xacro:cage>
+  <!-- workspace -->
+  <xacro:property name="table_w"	value="0.900"/>
+  <xacro:property name="table_l"	value="1.800"/>
+  <xacro:include filename="$(find aist_description
+			   )/objects/urdf/table.urdf.xacro"/>
+  <xacro:table prefix="workspace_"
+	       width="${table_w}" length="${table_l}" height="${bots_z}"
+	       parent="ground">
+    <origin xyz="${-cage_w/2 + cage_offset_x + cage_t} ${-table_l/2} 0"
+	    rpy="0 0 0"/>
+  </xacro:table>
+  <link name="workspace_center"/>
+  <joint name="ground_to_workspace" type="fixed">
+    <parent link="ground"/>
+    <child  link="workspace_center"/>
+    <origin xyz="0 0 ${bots_z}" rpy="0 0 0"/>
+  </joint>
   <!-- tool holders -->
   <xacro:property name="precision_tool_holder_y"	value="0.60"/>
@@ -124,9 +126,9 @@
   </xacro:robotiq_arg2f_coupling>
   <xacro:include filename="$(find aist_robotiq
-			   )/urdf/robotiq_85_gripper.urdf.xacro"/>
-  <xacro:robotiq_85_gripper prefix="a_bot_gripper_"
-			    parent="a_bot_gripper_coupling_flange_link">
+			   )/urdf/robotiq_140_gripper.urdf.xacro"/>
+  <xacro:robotiq_140_gripper prefix="a_bot_gripper_"
+			     parent="a_bot_gripper_coupling_flange_link">
     <origin xyz="0 0 0" rpy="0 0 0"/>
-  </xacro:robotiq_85_gripper>
+  </xacro:robotiq_140_gripper>
   <!-- RealSense cameras -->
   <xacro:include filename="$(find aist_description

File: aist_description/scenes/urdf/aist_base_scene.urdf.xacro (robot description, xacro)
@@ -9,21 +9,6 @@
   <xacro:property name="bots_z"		value="0.770"/>
   <xacro:property name="screen_z"	value="${bots_z + 0.040}"/>
-  <!-- ground and workspace -->
+  <!-- ground -->
   <link name="ground"/>
-  <xacro:property name="table_w"	value="0.900"/>
-  <xacro:property name="table_l"	value="1.800"/>
-  <xacro:include filename="$(find aist_description
-			   )/objects/urdf/table.urdf.xacro"/>
-  <xacro:table prefix="workspace_"
-	       width="${table_w}" length="${table_l}" height="${bots_z}"
-	       parent="ground">
-    <origin xyz="${-table_w/2} ${-table_l/2} 0" rpy="0 0 0"/>
-  </xacro:table>
-  <link name="workspace_center"/>
-  <joint name="ground_to_workspace" type="fixed">
-    <parent link="ground"/>
-    <child  link="workspace_center"/>
-    <origin xyz="0 0 ${bots_z}" rpy="0 0 0"/>
-  </joint>
   <!-- cage -->
   <xacro:property name="cage_w"		value="1.200"/>
@@ -50,4 +35,21 @@
 	    rpy="0 0 0" />
   </xacro:cage>
+  <!-- workspace -->
+  <xacro:property name="table_w"	value="0.900"/>
+  <xacro:property name="table_l"	value="1.800"/>
+  <xacro:include filename="$(find aist_description
+			   )/objects/urdf/table.urdf.xacro"/>
+  <xacro:table prefix="workspace_"
+	       width="${table_w}" length="${table_l}" height="${bots_z}"
+	       parent="ground">
+    <origin xyz="${-cage_w/2 + cage_offset_x + cage_t} ${-table_l/2} 0"
+	    rpy="0 0 0"/>
+  </xacro:table>
+  <link name="workspace_center"/>
+  <joint name="ground_to_workspace" type="fixed">
+    <parent link="ground"/>
+    <child  link="workspace_center"/>
+    <origin xyz="0 0 ${bots_z}" rpy="0 0 0"/>
+  </joint>
   <!-- tool holders -->
   <xacro:property name="precision_tool_holder_y"	value="0.60"/>
@@ -148,9 +150,9 @@
   </xacro:robotiq_arg2f_coupling>
   <xacro:include filename="$(find aist_robotiq
-			   )/urdf/robotiq_85_gripper.urdf.xacro"/>
-  <xacro:robotiq_85_gripper prefix="a_bot_gripper_"
-			    parent="a_bot_gripper_coupling_flange_link">
-    <origin xyz="0 0 0" rpy="0 0 0"/>
-  </xacro:robotiq_85_gripper>
+			   )/urdf/robotiq_140_gripper.urdf.xacro"/>
+  <xacro:robotiq_140_gripper prefix="a_bot_gripper_"
+			     parent="a_bot_gripper_coupling_flange_link">
+    <origin xyz="0 0 0" rpy="0 0 0"/>
+  </xacro:robotiq_140_gripper>
   <xacro:robotiq_arg2f_coupling prefix="b_bot_gripper_coupling_"
 				parent="b_bot_ftsensor_flange_link">
@@ -158,9 +160,9 @@
   </xacro:robotiq_arg2f_coupling>
   <xacro:include filename="$(find aist_robotiq
-			   )/urdf/robotiq_140_gripper.urdf.xacro"/>
-  <xacro:robotiq_140_gripper prefix="b_bot_gripper_"
+			   )/urdf/robotiq_85_gripper.urdf.xacro"/>
+  <xacro:robotiq_85_gripper prefix="b_bot_gripper_"
 			    parent="b_bot_gripper_coupling_flange_link">
     <origin xyz="0 0 0" rpy="0 0 0"/>
-  </xacro:robotiq_140_gripper>
+  </xacro:robotiq_85_gripper>
   <!-- <xacro:include filename="$(find aist_description -->
   <!-- 			   )/devices/urdf/single_suction_gripper.urdf.xacro"/> -->

File: aist_description/scenes/urdf/b_bot_base_scene.urdf.xacro (robot description, xacro)
@@ -7,21 +7,6 @@
   <xacro:property name="bots_z"		value="0.770"/>
   <xacro:property name="screen_z"	value="${bots_z + 0.0347}"/>
-  <!-- ground and workspace -->
+  <!-- ground -->
   <link name="ground"/>
-  <xacro:property name="table_w"	value="0.900"/>
-  <xacro:property name="table_l"	value="1.800"/>
-  <xacro:include filename="$(find aist_description
-			   )/objects/urdf/table.urdf.xacro"/>
-  <xacro:table prefix="workspace_"
-	       width="${table_w}" length="${table_l}" height="${bots_z}"
-	       parent="ground">
-    <origin xyz="${-table_w/2} ${-table_l/2} 0" rpy="0 0 0"/>
-  </xacro:table>
-  <link name="workspace_center"/>
-  <joint name="ground_to_workspace" type="fixed">
-    <parent link="ground"/>
-    <child  link="workspace_center"/>
-    <origin xyz="0 0 ${bots_z}" rpy="0 0 0"/>
-  </joint>
   <!-- cage -->
   <xacro:property name="cage_w"		value="1.200"/>
@@ -30,7 +15,8 @@
   <xacro:property name="cage_t"		value="0.040"/>
   <xacro:property name="tool_bar_h"	value="0.270"/>
-  <xacro:property name="camera_bar_h"	value="1.300"/>
+  <xacro:property name="camera_bar_h"	value="1.325"/>
   <xacro:property name="cage_z"		value="0.164"/>
-  <xacro:property name="cage_offset"	value="0.020"/>
+  <xacro:property name="cage_offset_x"	value="0.020"/>
+  <xacro:property name="cage_offset_y"	value="-0.005"/>
   <xacro:include filename="$(find aist_description
 			   )/objects/urdf/cage.urdf.xacro"/>
@@ -42,7 +28,26 @@
 	      camera_bar_height="${camera_bar_h}"
 	      parent="ground">
-    <origin xyz="${-cage_w/2 + cage_offset} ${-cage_l/2} ${cage_z}"
+    <origin xyz="${-cage_w/2 + cage_offset_x}
+		 ${-cage_l/2 + cage_offset_y}
+		 ${cage_z}"
 	    rpy="0 0 0" />
   </xacro:cage>
+  <!-- workspace -->
+  <xacro:property name="table_w"	value="0.900"/>
+  <xacro:property name="table_l"	value="1.800"/>
+  <xacro:include filename="$(find aist_description
+			   )/objects/urdf/table.urdf.xacro"/>
+  <xacro:table prefix="workspace_"
+	       width="${table_w}" length="${table_l}" height="${bots_z}"
+	       parent="ground">
+    <origin xyz="${-cage_w/2 + cage_offset_x + cage_t} ${-table_l/2} 0"
+	    rpy="0 0 0"/>
+  </xacro:table>
+  <link name="workspace_center"/>
+  <joint name="ground_to_workspace" type="fixed">
+    <parent link="ground"/>
+    <child  link="workspace_center"/>
+    <origin xyz="0 0 ${bots_z}" rpy="0 0 0"/>
+  </joint>
   <!-- tool holders -->
   <xacro:property name="screw_tool_m3_holder_y"	value="0.75"/>

File: aist_description/scenes/urdf/kitting.urdf.xacro (robot description, xacro)
@@ -13,8 +13,8 @@
     <origin xyz="-0.062 ${-plate_l/2} 0" rpy="0 0 0"/>
   </xacro:aist_box>
-  <link name="plate_upper_left_corner"/>
+  <link name="plate_lower_left_corner"/>
   <joint name="plate_corner_joint" type="fixed">
     <parent link="plate"/>
-    <child  link="plate_upper_left_corner"/>
+    <child  link="plate_lower_left_corner"/>
     <origin xyz="0 0 ${plate_h}" rpy="0 0 0"/>
   </joint>
@@ -45,5 +45,5 @@
   <!--bin_1_part_5_-->
   <xacro:kitting_bin_1 binname	      ="bin_1_part_5"
-		       parent	      ="plate_upper_left_corner"
+		       parent	      ="plate_lower_left_corner"
 		       z_origin_offset="${z_origin_offset_1}">
     <origin xyz="${bin_1_x} ${bin_y + bin_1_width} ${-z_origin_offset_1}"
@@ -52,5 +52,5 @@
   <!--bin_1_part_16_-->
   <xacro:kitting_bin_1 binname	      ="bin_1_part_16"
-		       parent	      ="plate_upper_left_corner"
+		       parent	      ="plate_lower_left_corner"
 		       z_origin_offset="${z_origin_offset_1}">
     <origin xyz="${bin_1_x} ${bin_y} ${-z_origin_offset_1}"
@@ -59,5 +59,5 @@
   <!--bin_1_part_17_-->
   <xacro:kitting_bin_1 binname	      ="bin_1_part_17"
-  		       parent	      ="plate_upper_left_corner"
+  		       parent	      ="plate_lower_left_corner"
   		       z_origin_offset="${z_origin_offset_1}">
     <origin xyz="${bin_1_x} ${bin_y - bin_1_width} ${-z_origin_offset_1}"
@@ -66,5 +66,5 @@
   <!-- bin_2_part_4_ -->
   <xacro:kitting_bin_2 binname	      ="bin_2_part_4"
-		       parent	      ="plate_upper_left_corner"
+		       parent	      ="plate_lower_left_corner"
 		       z_origin_offset="${z_origin_offset_2}">
     <origin xyz="${bin_2_x} ${bin_y + bin_2_width} ${-z_origin_offset_2}"
@@ -73,5 +73,5 @@
   <!--bin_2_part_7_-->
   <xacro:kitting_bin_2 binname	      ="bin_2_part_7"
-		       parent	      ="plate_upper_left_corner"
+		       parent	      ="plate_lower_left_corner"
 		       z_origin_offset="${z_origin_offset_2}">
     <origin xyz="${bin_2_x} ${bin_y} ${-z_origin_offset_2}"
@@ -80,5 +80,5 @@
   <!--bin_2_part_8_-->
   <xacro:kitting_bin_2 binname	      ="bin_2_part_8"
-  		       parent	      ="plate_upper_left_corner"
+  		       parent	      ="plate_lower_left_corner"
   		       z_origin_offset="${z_origin_offset_2}">
     <origin xyz="${bin_2_x} ${bin_y - bin_2_width} ${-z_origin_offset_2}"
@@ -86,10 +86,10 @@
   </xacro:kitting_bin_2>
   <!-- tray_1 -->
-  <!-- <xacro:kitting_tray_1 trayname="tray_1" parent="plate_upper_left_corner"> -->
+  <!-- <xacro:kitting_tray_1 trayname="tray_1" parent="plate_lower_left_corner"> -->
   <!--   <origin xyz="${tray_x - tray_width} ${bin_y + tray_y} 0" -->
   <!-- 	    rpy="0 0 ${-pi/2}"/> -->
   <!-- </xacro:kitting_tray_1> -->
   <!-- tray_2 -->
-  <xacro:kitting_tray_2 trayname="tray_2" parent="plate_upper_left_corner">
+  <xacro:kitting_tray_2 trayname="tray_2" parent="plate_lower_left_corner">
     <origin xyz="${tray_x} ${tray_y} 0" rpy="0 0 ${pi/2}"/>
   </xacro:kitting_tray_2>
