Commit message: Cleanup screw_feeder.urdf.xacro

File: aist_description/objects/urdf/aist_box.urdf.xacro (robot description, xacro)
@@ -2,15 +2,7 @@
 <robot xmlns:xacro="http://wiki.ros.org/xacro">
   <xacro:macro name="aist_box"
-	       params="name width length height parent transparent:=false
+	       params="name width length height parent
+		       rgba:='0.7 0.7 0.7 1' color_name:=aist_color
 		       *origin">
-    <!-- This creates a box with the origin in the bottom corner, fixed to the world link. -->
-    <xacro:unless value="${transparent}">
-      <xacro:property name="rgba"	value="0.7 0.7 0.7 1"/>
-      <xacro:property name="color_name" value="Grey"/>
-    </xacro:unless>
-    <xacro:if value="${transparent}">
-      <xacro:property name="rgba"	value="0 0 0 0"/>
-      <xacro:property name="color_name"	value="Transparent"/>
-    </xacro:if>
     <link name="${name}">
       <!-- w is in x, l is in y, h is in z -->

File: aist_description/objects/urdf/screw_feeder.urdf.xacro (robot description, xacro)
@@ -1,89 +1,51 @@
 <?xml version="1.0" ?>
 <robot xmlns:xacro="http://www.ros.org/wiki/xacro" name="screw_feeder">
-  <xacro:macro name="screw_feeder"
-	       params="prefix parent with_collision_geometry:=true *origin">
-  <!-- This creates a screw feeder (roughly) with the origin in the back right corner. -->
-  <!-- This is the feeder: https://www.monotaro.com/g/02001466/ -->
-  <xacro:property name="height" value=".147" />
-  <xacro:property name="width"  value=".126" />
-  <xacro:property name="length" value=".182" />
-  <link name="${prefix}base_link">
-    <inertial>
-      <origin rpy="0 0 0" xyz="0 0 0"/>
-      <mass value="1.0"/>
-      <inertia ixx="1.0" ixy="0" ixz="0" iyy="1.0" iyz="0" izz="1.0"/>
-    </inertial>
+  <xacro:macro name="screw_feeder" params="prefix parent *origin">
+    <xacro:property name="length"	value=".126"/>
+    <xacro:property name="gap_width"	value=".020"/>
+    <xacro:property name="gap_depth"	value=".002"/>
+    <xacro:property name="gap_height"	value=".081"/>
+    <xacro:property name="gap_x"	value=".046"/>
+    <xacro:property name="gap_y"	value="${length/2}"/>
+    <xacro:property name="front_width"	value=".056"/>
+    <xacro:property name="front_height"	value="${gap_height - gap_depth}"/>
+    <xacro:property name="back_width"	value=".126"/>
+    <xacro:property name="back_height"	value=".147"/>
+    <xacro:include filename="$(find aist_description
+			     )/objects/urdf/aist_box.urdf.xacro" />
     <!-- Back side -->
-    <visual>
-      <origin xyz="${(length-.05)/2} ${width/2} ${height/2}" rpy="0 0 0"/>
-      <geometry>
-        <box size="${length-.05} ${width} ${height}"/>
-      </geometry>
-      <material name="black">
-        <color rgba=".2 .2 .2 1"/>
-      </material>
-    </visual>
-    <xacro:if value="${with_collision_geometry}">
-      <collision>
-        <origin xyz="${(length-.05)/2} ${width/2} ${height/2}" rpy="0 0 0"/>
-        <geometry>
-          <box size="${length-.05} ${width} ${height}"/>
-        </geometry>
-      </collision>
-    </xacro:if>
+    <xacro:aist_box name="${prefix}base_link" parent="${parent}"
+		    width="${back_width}" length="${length}"
+		    height="${back_height}"
+		    rgba="0.2 0.2 0.2 1.0" color_name="black">
+      <xacro:insert_block name="origin"/>
+    </xacro:aist_box>
     <!-- Front side -->
-    <visual>
-      <origin rpy="0 0 0" xyz="${(length-.025)} ${width/2} ${height/4}"/>
-      <geometry>
-        <box size="${.05} ${width} ${height/2}"/>
-      </geometry>
-      <material name="black">
-        <color rgba=".2 .2 .2 1"/>
-      </material>
-    </visual>
-    <xacro:if value="${with_collision_geometry}">
-      <collision>
-        <origin xyz="${(length-.025)} ${width/2} ${height/4}" rpy="0 0 0"/>
-        <geometry>
-          <box size="${.05} ${width} ${height/2}"/>
-        </geometry>
-      </collision>
-    </xacro:if>
-    <!-- The screw output area -->
-    <visual>
-      <origin xyz="${(length-.025)} ${width/2} ${height/2}" rpy="0 0 0"/>
-      <geometry>
-        <box size="${.05} ${.02} ${.005}"/>
-      </geometry>
-      <material name="gray">
-        <color rgba=".6 .6 .6 1"/>
-      </material>
-    </visual>
-    <xacro:if value="${with_collision_geometry}">
-      <collision>
-        <origin xyz="${(length-.025)} ${width/2} ${height/2}" rpy="0 0 0"/>
-        <geometry>
-          <box size="${.05} ${.02} ${.005}"/>
-        </geometry>
-      </collision>
-    </xacro:if>
-  </link>
-  <joint name="${prefix}base_joint" type="fixed">
-    <parent link="${parent}" />
-    <child link ="${prefix}base_link" />
-    <xacro:insert_block name="origin"/>
-  </joint>
-  <joint name="${prefix}outlet_joint" type="fixed">
-    <parent link="${prefix}base_link"/>
-    <child link="${prefix}outlet_link"/>
-    <origin xyz="${length-.01} ${width/2} ${height/2}" rpy="0 0 0"/>
-  </joint>
-  <link name="${prefix}outlet_link"/>
-  <joint name="${prefix}inlet_joint" type="fixed">
-    <parent link="${prefix}base_link"/>
-    <child link="${prefix}inlet_link"/>
-    <origin xyz="${length/3} ${width/3} ${height}" rpy="0 0 0"/>
-  </joint>
-  <link name="${prefix}inlet_link"/>
+    <xacro:aist_box name="${prefix}front_side" parent="${prefix}base_link"
+		    width="${front_width}" length="${length}"
+		    height="${front_height}"
+		    rgba="0.2 0.2 0.2 1.0" color_name="black">
+      <origin xyz="${back_width} 0 0" rpy="0 0 0"/>
+    </xacro:aist_box>
+    <!-- Gap -->
+    <xacro:aist_box name="${prefix}gap" parent="${prefix}front_side"
+		    width="${front_width}" length="${gap_width}"
+		    height="${gap_depth}"
+		    rgba="0.6 0.6 0.6 1.0" color_name="grey">
+      <origin xyz="0 ${gap_y - gap_width/2} ${front_height}" rpy="0 0 0"/>
+    </xacro:aist_box>
+    <joint name="${prefix}outlet_joint" type="fixed">
+      <parent link="${prefix}gap"/>
+      <child  link="${prefix}outlet_link"/>
+      <origin xyz="${gap_x} ${gap_width/2} ${gap_depth}"
+	      rpy="0 0 0"/>
+    </joint>
+    <link name="${prefix}outlet_link"/>
+    <joint name="${prefix}inlet_joint" type="fixed">
+      <parent link="${prefix}base_link"/>
+      <child  link="${prefix}inlet_link"/>
+      <origin xyz="${back_width/2} ${length/3} ${back_height}" rpy="0 0 0"/>
+    </joint>
+    <link name="${prefix}inlet_link"/>
   </xacro:macro>
 </robot>

File: aist_description/scenes/urdf/assembly.urdf.xacro (robot description, xacro)
@@ -6,5 +6,5 @@
   <xacro:property name="workbench_height"	 value="0.15"/>
   <xacro:property name="workbench_bar_width"	 value="0.48"/>
-  <xacro:property name="workbench_y"		 value="0.65"/>
+  <xacro:property name="workbench_y"		 value="0.55"/>
   <xacro:property name="screw_feeder_width"	 value="0.126"/>
   <xacro:property name="screw_feeder_y"		 value="0.03"/>
