Commit message: Add screw feeders and workbench

File: aist_description/objects/urdf/table.urdf.xacro (robot description, xacro)
@@ -1,10 +1,11 @@
 <?xml version="1.0" ?>
 <robot xmlns:xacro="http://wiki.ros.org/xacro" name="table">
-  <xacro:include filename="$(find aist_description)/objects/urdf/aist_box.urdf.xacro"/>
   <xacro:macro name="table"
-	       params="prefix width length height parent *origin">
-    <xacro:property name="table_thickness"	value="0.020" />
-    <xacro:property name="table_leg_thickness"	value="0.050" />
-    <xacro:aist_box name="${prefix}table_leg0"
+	       params="prefix width length height parent
+		       table_thickness:=0.020 table_leg_thickness:=0.050
+		       *origin">
+    <xacro:include filename="$(find aist_description
+			     )/objects/urdf/aist_box.urdf.xacro"/>
+    <xacro:aist_box name="${prefix}base_link"
 		    width="${table_leg_thickness}"
 		    length="${table_leg_thickness}"
@@ -13,23 +14,23 @@
       <xacro:insert_block name="origin"/>
     </xacro:aist_box>
-    <xacro:aist_box name="${prefix}table_leg1"
+    <xacro:aist_box name="${prefix}leg1"
 		    width="${table_leg_thickness}"
 		    length="${table_leg_thickness}"
 		    height="${height - table_thickness}"
-		    parent="${prefix}table_leg0">
+		    parent="${prefix}base_link">
       <origin xyz="${width - table_leg_thickness} 0 0" rpy="0 0 0"/>
     </xacro:aist_box>
-    <xacro:aist_box name="${prefix}table_leg2"
+    <xacro:aist_box name="${prefix}leg2"
 		    width="${table_leg_thickness}"
 		    length="${table_leg_thickness}"
 		    height="${height - table_thickness}"
-		    parent="${prefix}table_leg0">
+		    parent="${prefix}base_link">
       <origin xyz="0 ${length - table_leg_thickness} 0" rpy="0 0 0"/>
     </xacro:aist_box>
-    <xacro:aist_box name="${prefix}table_leg3"
+    <xacro:aist_box name="${prefix}leg3"
 		    width="${table_leg_thickness}"
 		    length="${table_leg_thickness}"
 		    height="${height - table_thickness}"
-		    parent="${prefix}table_leg0">
+		    parent="${prefix}base_link">
       <origin xyz="${width  - table_leg_thickness}
 		   ${length - table_leg_thickness}
@@ -37,9 +38,9 @@
 	      rpy="0 0 0"/>
     </xacro:aist_box>
-    <xacro:aist_box name="${prefix}table_top"
+    <xacro:aist_box name="${prefix}top"
 		    width="${width}"
 		    length="${length}"
 		    height="${table_thickness}"
-		    parent="${prefix}table_leg0">
+		    parent="${prefix}base_link">
       <origin xyz="0 0 ${height - table_thickness}" rpy="0 0 0"/>
     </xacro:aist_box>
@@ -52,8 +53,8 @@
       <link name="${parent}_${framename}"/>
     </xacro:macro>
-    <xacro:auxiliary_frame parent="${prefix}table_top" framename="origin">
+    <xacro:auxiliary_frame parent="${prefix}top" framename="origin">
       <origin xyz="0 0 ${table_thickness}" rpy="0 0 0"/>
     </xacro:auxiliary_frame>
-    <xacro:auxiliary_frame parent="${prefix}table_top_origin" framename="center">
+    <xacro:auxiliary_frame parent="${prefix}top_origin" framename="center">
       <origin xyz="${width/2} ${length/2} 0" rpy="0 0 0"/>
     </xacro:auxiliary_frame>

File: aist_description/scenes/urdf/a_bot_base_scene.urdf.xacro (robot description, xacro)
@@ -1,4 +1,4 @@
 <?xml version="1.0"?>
-<robot xmlns:xacro="http://wiki.ros.org/xacro" name="a_bot__base_scene" >
+<robot xmlns:xacro="http://wiki.ros.org/xacro" name="a_bot_base_scene" >
   <xacro:arg name="scene" default=""/>
   <xacro:property name="a_bot_x"	value="0"/>
@@ -37,5 +37,5 @@
   <xacro:include filename="$(find aist_description
 			   )/objects/urdf/table.urdf.xacro"/>
-  <xacro:table prefix="workspace_"
+  <xacro:table prefix="workspace_table_"
 	       width="${table_w}" length="${table_l}" height="${bots_z}"
 	       parent="ground">

File: aist_description/scenes/urdf/aist_base_scene.urdf.xacro (robot description, xacro)
@@ -40,5 +40,5 @@
   <xacro:include filename="$(find aist_description
 			   )/objects/urdf/table.urdf.xacro"/>
-  <xacro:table prefix="workspace_"
+  <xacro:table prefix="workspace_table_"
 	       width="${table_w}" length="${table_l}" height="${bots_z}"
 	       parent="ground">

File: aist_description/scenes/urdf/b_bot_base_scene.urdf.xacro (robot description, xacro)
@@ -1,4 +1,4 @@
 <?xml version="1.0"?>
-<robot xmlns:xacro="http://wiki.ros.org/xacro" name="aist_base_scene" >
+<robot xmlns:xacro="http://wiki.ros.org/xacro" name="b_bot_base_scene" >
   <xacro:arg name="scene" default=""/>
   <xacro:property name="b_bot_x"	value="0"/>
@@ -38,5 +38,5 @@
   <xacro:include filename="$(find aist_description
 			   )/objects/urdf/table.urdf.xacro"/>
-  <xacro:table prefix="workspace_"
+  <xacro:table prefix="workspace_table_"
 	       width="${table_w}" length="${table_l}" height="${bots_z}"
 	       parent="ground">

File: aist_description/scenes/urdf/ceatec_environment.urdf.xacro (robot description, xacro)
@@ -32,5 +32,5 @@
   <!-- a_table -->
   <xacro:include filename="$(find aist_description)/objects/urdf/table.urdf.xacro"/>
-  <xacro:table prefix="a_"
+  <xacro:table prefix="a_table_"
 	       width="${a_table_width}"
 	       length="${a_table_length}"
@@ -65,5 +65,5 @@
   </joint>
   <!-- b_table -->
-  <xacro:table prefix="b_"
+  <xacro:table prefix="b_table_"
 	       width="${b_table_width}"
 	       length="${b_table_length}"

File: aist_description/scenes/urdf/f_bot_base_scene.urdf.xacro (robot description, xacro)
@@ -16,5 +16,5 @@
   <xacro:include filename="$(find aist_description
 			   )/objects/urdf/table.urdf.xacro"/>
-  <xacro:table prefix="worksapce_"
+  <xacro:table prefix="worksapce_table_"
 	       width="${table_w}" length="${table_l}" height="${table_h}"
 	       parent="ground">
@@ -28,5 +28,5 @@
   </joint>
   <!-- Robot mounter -->
-  <xacro:table prefix="mounter_"
+  <xacro:table prefix="mounter_table_"
 	       width="${mounter_w}" length="${mounter_l}" height="${f_bot_z}"
 	       parent="ground">

File: aist_description/scenes/urdf/g_bot_base_scene.urdf.xacro (robot description, xacro)
@@ -49,5 +49,5 @@
   <xacro:include filename="$(find aist_description
 			   )/objects/urdf/table.urdf.xacro"/>
-  <xacro:table prefix="mounter_"
+  <xacro:table prefix="mounter_table_"
 		 width="${mounter_w}" length="${mounter_l}" height="${g_bot_z}"
 		 parent="ground">

File: moveit_config/aist_moveit_config/config/gazebo_aist_base_scene.urdf (robot description, URDF)
Before this commit: robot aist_base_scene, 116 links, 115 joints
Links:
- removed link workspace_table_leg0
- added link workspace_table_base_link, mass 1.0; collision box size=0.05 0.05 0.75; visual box size=0.05 0.05 0.75
- link a_bot_gripper_left_inner_finger: geometry collision mesh filename=package://aist_robotiq/meshes/collision/robotiq_arg2f_140_i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; visual mesh filename=package://aist_robotiq/meshes/visual/robotiq_arg2f_140_inne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
- link a_bot_gripper_left_inner_finger_pad: geometry collision box size=0.027 0.065 0.0075; visual box size=0.027 0.065 0.0075
- link a_bot_gripper_left_inner_knuckle: geometry collision mesh filename=package://aist_robotiq/meshes/collision/robotiq_arg2f_140_i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; visual mesh filename=package://aist_robotiq/meshes/visual/robotiq_arg2f_140_inne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
- link a_bot_gripper_left_outer_finger: geometry collision mesh filename=package://aist_robotiq/meshes/collision/robotiq_arg2f_140_o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; visual mesh filename=package://aist_robotiq/meshes/visual/robotiq_arg2f_140_oute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
- link a_bot_gripper_left_outer_knuckle: geometry collision mesh filename=package://aist_robotiq/meshes/collision/robotiq_arg2f_140_o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; visual mesh filename=package://aist_robotiq/meshes/visual/robotiq_arg2f_140_oute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
- link a_bot_gripper_right_inner_finger: geometry collision mesh filename=package://aist_robotiq/meshes/collision/robotiq_arg2f_140_i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; visual mesh filename=package://aist_robotiq/meshes/visual/robotiq_arg2f_140_inne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
- link a_bot_gripper_right_inner_finger_pad: geometry collision box size=0.027 0.065 0.0075; visual box size=0.027 0.065 0.0075
- link a_bot_gripper_right_inner_knuckle: geometry collision mesh filename=package://aist_robotiq/meshes/collision/robotiq_arg2f_140_i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; visual mesh filename=package://aist_robotiq/meshes/visual/robotiq_arg2f_140_inne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
- link a_bot_gripper_right_outer_finger: geometry collision mesh filename=package://aist_robotiq/meshes/collision/robotiq_arg2f_140_o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; visual mesh filename=package://aist_robotiq/meshes/visual/robotiq_arg2f_140_oute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
- link a_bot_gripper_right_outer_knuckle: geometry collision mesh filename=package://aist_robotiq/meshes/collision/robotiq_arg2f_140_o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; visual mesh filename=package://aist_robotiq/meshes/visual/robotiq_arg2f_140_oute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
- link b_bot_gripper_left_inner_finger: geometry collision mesh filename=package://aist_robotiq/meshes/collision/robotiq_arg2f_85_in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 scale=0.001 0.001 0.001; visual mesh filename=package://aist_robotiq/meshes/visual/robotiq_arg2f_85_inner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 scale=0.001 0.001 0.001
- link b_bot_gripper_left_inner_finger_pad: geometry collision box size=0.022 0.00635 0.0375; visual box size=0.022 0.00635 0.0375
- link b_bot_gripper_left_inner_knuckle: geometry collision mesh filename=package://aist_robotiq/meshes/collision/robotiq_arg2f_85_in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 scale=0.001 0.001 0.001; visual mesh filename=package://aist_robotiq/meshes/visual/robotiq_arg2f_85_inner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 scale=0.001 0.001 0.001
- link b_bot_gripper_left_outer_finger: geometry collision mesh filename=package://aist_robotiq/meshes/collision/robotiq_arg2f_85_ou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 scale=0.001 0.001 0.001; visual mesh filename=package://aist_robotiq/meshes/visual/robotiq_arg2f_85_outer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 scale=0.001 0.001 0.001
- link b_bot_gripper_left_outer_knuckle: geometry collision mesh filename=package://aist_robotiq/meshes/collision/robotiq_arg2f_85_ou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 scale=0.001 0.001 0.001; visual mesh filename=package://aist_robotiq/meshes/visual/robotiq_arg2f_85_outer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 scale=0.001 0.001 0.001
- link b_bot_gripper_right_inner_finger: geometry collision mesh filename=package://aist_robotiq/meshes/collision/robotiq_arg2f_85_in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 scale=0.001 0.001 0.001; visual mesh filename=package://aist_robotiq/meshes/visual/robotiq_arg2f_85_inner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 scale=0.001 0.001 0.001
- link b_bot_gripper_right_inner_finger_pad: geometry collision box size=0.022 0.00635 0.0375; visual box size=0.022 0.00635 0.0375
- link b_bot_gripper_right_inner_knuckle: geometry collision mesh filename=package://aist_robotiq/meshes/collision/robotiq_arg2f_85_in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 scale=0.001 0.001 0.001; visual mesh filename=package://aist_robotiq/meshes/visual/robotiq_arg2f_85_inner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 scale=0.001 0.001 0.001
- link b_bot_gripper_right_outer_finger: geometry collision mesh filename=package://aist_robotiq/meshes/collision/robotiq_arg2f_85_ou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 scale=0.001 0.001 0.001; visual mesh filename=package://aist_robotiq/meshes/visual/robotiq_arg2f_85_outer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 scale=0.001 0.001 0.001
- link b_bot_gripper_right_outer_knuckle: geometry collision mesh filename=package://aist_robotiq/meshes/collision/robotiq_arg2f_85_ou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 scale=0.001 0.001 0.001; visual mesh filename=package://aist_robotiq/meshes/visual/robotiq_arg2f_85_outer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 scale=0.001 0.001 0.001
Joints:
- removed joint workspace_table_leg0
- added joint workspace_table_base_link: type fixed, parent ground, child workspace_table_base_link, origin xyz=-0.5449999999999999 -0.9 0 rpy=0 0 0
- joint a_bot_gripper_finger_joint: axis 1 0 0 -> -1 0 0; limit lower=0 upper=0.81 effort=1000 velocity=2.0 -> lower=0 upper=0.7 effort=1000 velocity=2.0; origin xyz=0 -0.0306011 0.054904 rpy=0 0 3.141592653589793 -> xyz=0 -0.030601 0.054905 rpy=2.2957963267948966 0 0
- joint a_bot_gripper_left_inner_finger_joint: axis 1 0 0 -> -1 0 0; origin xyz=0 0.0061 0.0471 rpy=0 0 0 -> xyz=0 0.0817554015893473 -0.0282203446692936 rpy=-0.725 0 0
- joint a_bot_gripper_left_inner_finger_pad_joint: origin xyz=0 -0.0220203446692936 0.03242 rpy=0 0 0 -> xyz=0 0.0457554015893473 -0.0272203446692936 rpy=0 0 0
- joint a_bot_gripper_left_inner_knuckle_joint: axis 1 0 0 -> -1 0 0; origin xyz=0 -0.0127 0.06142 rpy=0 0 3.141592653589793 -> xyz=0 -0.0127 0.06142 rpy=2.2957963267948966 0 0.0
- joint a_bot_gripper_left_outer_finger_joint: origin xyz=0 0.0315 -0.0041 rpy=0 0 0 -> xyz=0 0.01821998610742 0.0260018192872234 rpy=0 0 0
- joint a_bot_gripper_right_inner_finger_joint: axis 1 0 0 -> -1 0 0; origin xyz=0 0.0061 0.0471 rpy=0 0 0 -> xyz=0 0.0817554015893473 -0.0282203446692936 rpy=-0.725 0 0
- joint a_bot_gripper_right_inner_finger_pad_joint: origin xyz=0 -0.0220203446692936 0.03242 rpy=0 0 0 -> xyz=0 0.0457554015893473 -0.0272203446692936 rpy=0 0 0
- joint a_bot_gripper_right_inner_knuckle_joint: axis 1 0 0 -> -1 0 0; origin xyz=0 0.0127 0.06142 rpy=0 0 0.0 -> xyz=0 0.0127 0.06142 rpy=2.2957963267948966 0 -3.141592653589793
- joint a_bot_gripper_right_outer_finger_joint: origin xyz=0 0.0315 -0.0041 rpy=0 0 0 -> xyz=0 0.01821998610742 0.0260018192872234 rpy=0 0 0
- joint a_bot_gripper_right_outer_knuckle_joint: axis 1 0 0 -> -1 0 0; limit lower=-0.81 upper=0.81 effort=1000 velocity=2.0 -> lower=-0.725 upper=0.725 effort=1000 velocity=2.0; origin xyz=0 0.0306011 0.054904 rpy=0 0 0 -> xyz=0 0.030601 0.054905 rpy=2.2957963267948966 0 3.141592653589793
- joint a_bot_gripper_tip_link_joint: origin xyz=0.1628 0.0 0.0 rpy=0.0 -1.5707963267948966 0.0 -> xyz=.2328 0.0 0.0 rpy=0.0 -1.5707963267948966 0.0
- joint b_bot_gripper_finger_joint: axis -1 0 0 -> 1 0 0; limit lower=0 upper=0.7 effort=1000 velocity=2.0 -> lower=0 upper=0.81 effort=1000 velocity=2.0; origin xyz=0 -0.030601 0.054905 rpy=2.2957963267948966 0 0 -> xyz=0 -0.0306011 0.054904 rpy=0 0 3.141592653589793
- joint b_bot_gripper_left_inner_finger_joint: axis -1 0 0 -> 1 0 0; origin xyz=0 0.0817554015893473 -0.0282203446692936 rpy=-0.725 0 0 -> xyz=0 0.0061 0.0471 rpy=0 0 0
- joint b_bot_gripper_left_inner_finger_pad_joint: origin xyz=0 0.0457554015893473 -0.0272203446692936 rpy=0 0 0 -> xyz=0 -0.0220203446692936 0.03242 rpy=0 0 0
- joint b_bot_gripper_left_inner_knuckle_joint: axis -1 0 0 -> 1 0 0; origin xyz=0 -0.0127 0.06142 rpy=2.2957963267948966 0 0.0 -> xyz=0 -0.0127 0.06142 rpy=0 0 3.141592653589793
- joint b_bot_gripper_left_outer_finger_joint: origin xyz=0 0.01821998610742 0.0260018192872234 rpy=0 0 0 -> xyz=0 0.0315 -0.0041 rpy=0 0 0
- joint b_bot_gripper_right_inner_finger_joint: axis -1 0 0 -> 1 0 0; origin xyz=0 0.0817554015893473 -0.0282203446692936 rpy=-0.725 0 0 -> xyz=0 0.0061 0.0471 rpy=0 0 0
- joint b_bot_gripper_right_inner_finger_pad_joint: origin xyz=0 0.0457554015893473 -0.0272203446692936 rpy=0 0 0 -> xyz=0 -0.0220203446692936 0.03242 rpy=0 0 0
- joint b_bot_gripper_right_inner_knuckle_joint: axis -1 0 0 -> 1 0 0; origin xyz=0 0.0127 0.06142 rpy=2.2957963267948966 0 -3.141592653589793 -> xyz=0 0.0127 0.06142 rpy=0 0 0.0
- joint b_bot_gripper_right_outer_finger_joint: origin xyz=0 0.01821998610742 0.0260018192872234 rpy=0 0 0 -> xyz=0 0.0315 -0.0041 rpy=0 0 0
- joint b_bot_gripper_right_outer_knuckle_joint: axis -1 0 0 -> 1 0 0; limit lower=-0.725 upper=0.725 effort=1000 velocity=2.0 -> lower=-0.81 upper=0.81 effort=1000 velocity=2.0; origin xyz=0 0.030601 0.054905 rpy=2.2957963267948966 0 3.141592653589793 -> xyz=0 0.0306011 0.054904 rpy=0 0 0
- joint b_bot_gripper_tip_link_joint: origin xyz=.2328 0.0 0.0 rpy=0.0 -1.5707963267948966 0.0 -> xyz=0.1628 0.0 0.0 rpy=0.0 -1.5707963267948966 0.0
- joint cage_workspace_bar: origin xyz=0 0 0.566 rpy=0 0 0 -> xyz=0 0 0.596 rpy=0 0 0
- joint workspace_table_leg1: parent workspace_table_leg0 -> workspace_table_base_link
- joint workspace_table_leg2: parent workspace_table_leg0 -> workspace_table_base_link
- joint workspace_table_leg3: parent workspace_table_leg0 -> workspace_table_base_link
- joint workspace_table_top: parent workspace_table_leg0 -> workspace_table_base_link

Commit message: Specify initial poses of all collision objects with a parameter

File: aist_description/objects/urdf/table.urdf.xacro (robot description, xacro)
@@ -45,16 +45,17 @@
       <origin xyz="0 0 ${height - table_thickness}" rpy="0 0 0"/>
     </xacro:aist_box>
-    <xacro:macro name="auxiliary_frame" params="parent framename *origin">
-      <joint name="${parent}_${framename}" type="fixed">
+    <xacro:macro name="auxiliary_frame" params="parent child *origin">
+      <joint name="${child}_joint" type="fixed">
 	<parent link="${parent}" />
-	<child link = "${parent}_${framename}"/>
+	<child  link="${child}"/>
 	<xacro:insert_block name="origin"/>
       </joint>
-      <link name="${parent}_${framename}"/>
+      <link name="${child}"/>
     </xacro:macro>
-    <xacro:auxiliary_frame parent="${prefix}top" framename="origin">
+    <xacro:auxiliary_frame parent="${prefix}top" child="${prefix}top_origin">
       <origin xyz="0 0 ${table_thickness}" rpy="0 0 0"/>
     </xacro:auxiliary_frame>
-    <xacro:auxiliary_frame parent="${prefix}top_origin" framename="center">
+    <xacro:auxiliary_frame parent="${prefix}top_origin"
+			   child ="${prefix}top_center">
       <origin xyz="${width/2} ${length/2} 0" rpy="0 0 0"/>
     </xacro:auxiliary_frame>

File: aist_description/objects/urdf/workbench.urdf.xacro (robot description, xacro)
@@ -68,14 +68,14 @@
 	      rpy="0 0 0"/>
     </xacro:aist_box>
-    <xacro:macro name="auxiliary_frame" params="parent framename *origin">
-      <joint name="${framename}" type="fixed">
+    <xacro:macro name="auxiliary_frame" params="parent child *origin">
+      <joint name="${child}_joint" type="fixed">
 	<parent link="${parent}" />
-	<child link = "${framename}"/>
+	<child  link="${child}"/>
 	<xacro:insert_block name="origin"/>
       </joint>
-      <link name="${framename}"/>
+      <link name="${child}"/>
     </xacro:macro>
     <xacro:auxiliary_frame parent="${prefix}table_top_origin"
-			   framename="${prefix}holder_link">
+			   child ="${prefix}holder_link">
       <origin xyz="${width - border_width} ${length - border_width} 0"
 	      rpy="0 0 ${pi/2}"/>
