Commit message: Introduce aist_collision_object_manager instead of aist_object_database

File: aist_description/objects/urdf/workbench.urdf.xacro (robot description, xacro)
@@ -50,5 +50,5 @@
       <origin xyz="${bar_width - width} 0 0" rpy="0 0 0"/>
     </xacro:table>
-    <xacro:aist_box name="${prefix}back_border"
+    <xacro:aist_box name="${prefix}front_border"
 		    width="${border_length}"
 		    length="${border_width}"
@@ -56,6 +56,5 @@
 		    rgba="0.2 0.2 0.2 1.0" color_name="black"
 		    parent="${prefix}table_top_origin">
-      <origin xyz="${width - border_length} ${length - border_width} 0"
-	      rpy="0 0 0"/>
+      <origin xyz="${width - border_length} 0 0" rpy="0 0 0"/>
     </xacro:aist_box>
     <xacro:aist_box name="${prefix}right_border"
@@ -65,6 +64,5 @@
 		    rgba="0.2 0.2 0.2 1.0" color_name="black"
 		    parent="${prefix}table_top_origin">
-      <origin xyz="${width - border_width} ${length - border_length} 0"
-	      rpy="0 0 0"/>
+      <origin xyz="${width - border_width} ${border_width} 0" rpy="0 0 0"/>
     </xacro:aist_box>
     <xacro:macro name="auxiliary_frame" params="parent child *origin">
@@ -78,5 +76,5 @@
     <xacro:auxiliary_frame parent="${prefix}table_top_origin"
 			   child ="${prefix}holder_link">
-      <origin xyz="${width - border_width} ${length - border_width} 0"
+      <origin xyz="${width - border_width} ${border_width} 0"
 	      rpy="0 0 ${pi/2}"/>
     </xacro:auxiliary_frame>

File: aist_description/scenes/urdf/assembly.urdf.xacro (robot description, xacro)
@@ -2,11 +2,11 @@
 <robot xmlns:xacro="http://wiki.ros.org/xacro" name="assembly">
   <!-- base fixture table -->
-  <xacro:property name="cage_thickness"		 value="0.04"/>
-  <xacro:property name="workbench_bar_thickness" value="0.02"/>
-  <xacro:property name="workbench_height"	 value="0.15"/>
-  <xacro:property name="workbench_bar_width"	 value="0.48"/>
-  <xacro:property name="workbench_y"		 value="0.55"/>
+  <xacro:property name="cage_thickness"		 value="0.040"/>
+  <xacro:property name="workbench_bar_thickness" value="0.020"/>
+  <xacro:property name="workbench_height"	 value="0.150"/>
+  <xacro:property name="workbench_bar_width"	 value="0.480"/>
+  <xacro:property name="workbench_y"		 value="0.630"/>
   <xacro:property name="screw_feeder_width"	 value="0.126"/>
-  <xacro:property name="screw_feeder_y"		 value="0.03"/>
+  <xacro:property name="screw_feeder_y"		 value="0.030"/>
   <xacro:include filename="$(find aist_description
 			   )/objects/urdf/workbench.urdf.xacro"/>

Commit message: Add base_fixture to workbench

File: aist_description/objects/urdf/workbench.urdf.xacro (robot description, xacro)
@@ -3,13 +3,20 @@
   <xacro:macro name="workbench"
 	       params="prefix height bar_width parent *origin">
-    <xacro:property name="bar_thickness"	value="0.020" />
-    <xacro:property name="width"		value="0.240" />
-    <xacro:property name="length"		value="0.320" />
-    <xacro:property name="table_thickness"	value="0.005" />
-    <xacro:property name="border_width"		value="0.016" />
-    <xacro:property name="border_length"	value="0.150" />
-    <xacro:property name="border_height"	value="0.003" />
+    <xacro:property name="bar_thickness"	value="0.020"/>
+    <xacro:property name="width"		value="0.240"/>
+    <xacro:property name="length"		value="0.320"/>
+    <xacro:property name="table_thickness"	value="0.005"/>
+    <xacro:property name="border_width"		value="0.016"/>
+    <xacro:property name="border_length"	value="0.150"/>
+    <xacro:property name="border_height"	value="0.003"/>
+    <xacro:property name="theta"		value="${-59.04*pi/180.0}"/>
+    <xacro:property name="diag"			value="0.27739"/>
+    <xacro:property name="base_fixture_x"
+		    value="${width - 0.010 - diag*cos(theta)}"/>
+    <xacro:property name="base_fixture_y"
+		    value="${0.010 - diag*sin(theta)}" />
     <xacro:include filename="$(find aist_description
 			     )/objects/urdf/aist_box.urdf.xacro"/>
+    <!-- base bars -->
     <xacro:aist_box name="${prefix}base_link"
 		    width="${bar_width}"
@@ -41,4 +48,5 @@
 	      rpy="0 0 0"/>
     </xacro:aist_box>
+    <!-- table -->
     <xacro:include filename="$(find aist_description
 			     )/objects/urdf/table.urdf.xacro"/>
@@ -50,4 +58,5 @@
       <origin xyz="${bar_width - width} 0 0" rpy="0 0 0"/>
     </xacro:table>
+    <!-- table borders -->
     <xacro:aist_box name="${prefix}front_border"
 		    width="${border_length}"
@@ -66,4 +75,13 @@
       <origin xyz="${width - border_width} ${border_width} 0" rpy="0 0 0"/>
     </xacro:aist_box>
+    <!-- base fixture -->
+    <xacro:include filename="$(find aist_fastening_tools
+			     )/urdf/base_fixture.urdf.xacro"/>
+    <xacro:base_fixture prefix="base_fixture_"
+			parent="${prefix}table_top_origin">
+      <origin xyz="${base_fixture_x} ${base_fixture_y} 0"
+	      rpy="0 0 ${theta}"/>
+    </xacro:base_fixture>
+    <!-- auxiliary frames -->
     <xacro:macro name="auxiliary_frame" params="parent child *origin">
       <joint name="${child}_joint" type="fixed">

File: aist_fastening_tools/urdf/base_fixture.urdf.xacro (robot description, xacro)
@@ -70,5 +70,5 @@
       </inertial>
     </link>
-    <!-- left finger -->
+    <!-- cylinder -->
     <!-- <xacro:property name="cylinder_vorigin" -->
     <!-- 		    value="${visual_meshes[1]['pose']}"/> -->

Commit message: Shrink workbench width

File: aist_description/objects/urdf/workbench.urdf.xacro (robot description, xacro)
@@ -4,9 +4,9 @@
 	       params="prefix height bar_width parent *origin">
     <xacro:property name="bar_thickness"	value="0.020"/>
-    <xacro:property name="width"		value="0.240"/>
+    <xacro:property name="width"		value="0.210"/>
     <xacro:property name="length"		value="0.320"/>
     <xacro:property name="table_thickness"	value="0.005"/>
     <xacro:property name="border_width"		value="0.016"/>
-    <xacro:property name="border_length"	value="0.150"/>
+    <xacro:property name="border_length"	value="0.050"/>
     <xacro:property name="border_height"	value="0.003"/>
     <xacro:property name="theta"		value="${-59.04*pi/180.0}"/>
@@ -51,10 +51,12 @@
     <xacro:include filename="$(find aist_description
 			     )/objects/urdf/table.urdf.xacro"/>
-    <xacro:table prefix="${prefix}table_" width="${width}"
-		 length="${length}" height="${height - bar_thickness}"
+    <xacro:table prefix="${prefix}table_"
+		 width="${width}"
+		 length="${length}"
+		 height="${height - bar_thickness}"
 		 table_thickness="${table_thickness}"
 		 table_leg_thickness="${bar_thickness}"
 		 parent="${prefix}base_link">
-      <origin xyz="${bar_width - width} 0 0" rpy="0 0 0"/>
+      <origin xyz="${bar_width - width} 0  ${bar_thickness}" rpy="0 0 0"/>
     </xacro:table>
     <!-- table borders -->

Commit message: Change length of the table borders

File: aist_description/objects/urdf/workbench.urdf.xacro (robot description, xacro)
@@ -8,5 +8,5 @@
     <xacro:property name="table_thickness"	value="0.005"/>
     <xacro:property name="border_width"		value="0.016"/>
-    <xacro:property name="border_length"	value="0.050"/>
+    <xacro:property name="border_length"	value="0.080"/>
     <xacro:property name="border_height"	value="0.003"/>
     <xacro:property name="theta"		value="${-59.04*pi/180.0}"/>
