Commit message: Change suction_tool_holder

File: aist_description/objects/urdf/suction_tool_holder.urdf.xacro (robot description, xacro)
@@ -7,5 +7,5 @@
     <link name="${prefix}base_link">
       <visual>
-        <origin xyz="-0.008 0 0" rpy="0 0 0"/>
+        <origin xyz="-0.008 0 0" rpy="0 0 ${pi}"/>
 	<geometry>
           <mesh filename="package://aist_description/objects/meshes/suction_tool_holder.stl" scale="0.001 0.001 0.001"/>
@@ -35,5 +35,5 @@
       <parent link="${prefix}base_link"/>
       <child  link="${prefix}link"/>
-      <origin xyz="0.050 0 0.007" rpy="0 0 0"/>
+      <origin xyz="0.07032 0.000 0.03784" rpy="0 ${30*pi/180} 0"/>
     </joint>
   </xacro:macro>

Commit message: Fixed position of suction_tool_holder

File: aist_description/objects/urdf/suction_tool_holder.urdf.xacro (robot description, xacro)
@@ -7,5 +7,5 @@
     <link name="${prefix}base_link">
       <visual>
-        <origin xyz="-0.008 0 0" rpy="0 0 ${pi}"/>
+        <origin xyz="0.040 0 0" rpy="0 0 ${pi}"/>
 	<geometry>
           <mesh filename="package://aist_description/objects/meshes/suction_tool_holder.stl" scale="0.001 0.001 0.001"/>
@@ -17,5 +17,5 @@
       <collision>
       <!-- avoid collision -->
-	<origin xyz="-0.008 0 0" rpy="0 0 0"/>
+	<origin xyz="0.040 0 0" rpy="0 0 ${pi}"/>
 	<geometry>
 	  <mesh
@@ -35,5 +35,5 @@
       <parent link="${prefix}base_link"/>
       <child  link="${prefix}link"/>
-      <origin xyz="0.07032 0.000 0.03784" rpy="0 ${30*pi/180} 0"/>
+      <origin xyz="0.11032 0.000 0.03784" rpy="0 ${30*pi/180} 0"/>
     </joint>
   </xacro:macro>

Commit message: Confirmed that suction_tool can be picked/placed with a_bot

File: aist_description/objects/urdf/suction_tool_holder.urdf.xacro (robot description, xacro)
@@ -35,5 +35,5 @@
       <parent link="${prefix}base_link"/>
       <child  link="${prefix}link"/>
-      <origin xyz="0.11032 0.000 0.03784" rpy="0 ${30*pi/180} 0"/>
+      <origin xyz="0.08732 0.0 -0.002" rpy="0 ${30*pi/180} 0"/>
     </joint>
   </xacro:macro>

File: moveit_config/a_bot_moveit_config/config/gazebo_a_bot_base_scene.urdf (robot description, URDF)
Before this commit: robot a_bot_base_scene, 82 links, 81 joints
Joints:
- joint cage_tool_bar: origin xyz=0 0 0.27 rpy=0 0 0 -> xyz=0 0 0.24 rpy=0 0 0
- joint suction_tool_holder_joint: origin xyz=0.050 0 0.007 rpy=0 0 0 -> xyz=0.11032 0.000 0.03784 rpy=0 0.5235987755982988 0
