Commit message: Change location of screw feeders

File: aist_description/objects/urdf/screw_feeder.urdf.xacro (robot description, xacro)
@@ -45,5 +45,5 @@
       <parent link="${prefix}base_link"/>
       <child  link="${prefix}inlet_link"/>
-      <origin xyz="${back_width/2} ${length/3} ${back_height}" rpy="0 0 0"/>
+      <origin xyz="0.072 0.032 ${back_height}" rpy="0 0 0"/>
     </joint>
     <link name="${prefix}inlet_link"/>

File: aist_description/scenes/urdf/assembly.urdf.xacro (robot description, xacro)
@@ -9,4 +9,5 @@
   <xacro:property name="screw_feeder_width"	 value="0.126"/>
   <xacro:property name="screw_feeder_y"		 value="0.030"/>
+  <xacro:property name="screw_feeder_x"		 value="0.010"/>
   <xacro:include filename="$(find aist_description
 			   )/objects/urdf/workbench.urdf.xacro"/>
@@ -25,5 +26,5 @@
   <xacro:screw_feeder prefix="screw_feeder_m3_"
 		      parent="workbench_base_link">
-    <origin xyz="0 ${screw_feeder_y} 0" rpy="0 0 0"/>
+    <origin xyz="${screw_feeder_x} ${screw_feeder_y} 0" rpy="0 0 0"/>
   </xacro:screw_feeder>
   <xacro:screw_feeder prefix="screw_feeder_m4_"
