Commit message: Make hand camera's center adjustable

File: aist_description/objects/urdf/d435_mount_2f140.urdf.xacro (robot description, xacro)
@@ -3,7 +3,14 @@
 <!-- The position of the TF frame has not been measured at all and needs to be calibrated. -->
 <robot name="d435_mount_2f140" xmlns:xacro="http://www.ros.org/wiki/xacro">
-  <xacro:macro name="d435_mount_2f140" params="prefix parent">
+  <xacro:macro name="d435_mount_2f140"
+	       params="prefix parent color_camera_centered:=true">
     <xacro:property name="mesh_dir"
 		    value="package://aist_description/objects/meshes"/>
+    <xacro:if value="${color_camera_centered}">
+      <xacro:property name="camera_offset" value="0.0325"/>
+    </xacro:if>
+    <xacro:unless value="${color_camera_centered}">
+      <xacro:property name="camera_offset" value="0.0175"/>
+    </xacro:unless>
     <link name="${prefix}camera_mount">
       <inertial>
@@ -39,5 +46,5 @@
       <parent link="${prefix}camera_mount" />
       <child  link="${prefix}camera_mount_flange" />
-      <origin xyz="-0.0085 0.0175 0.0595"
+      <origin xyz="-0.0085 ${camera_offset} 0.0595"
 	      rpy="${radians(180.0)} ${radians(10.0)} 0.0"/>
     </joint>

File: aist_description/objects/urdf/d435_mount_2f85.urdf.xacro (robot description, xacro)
@@ -3,7 +3,14 @@
 <!-- The position of the TF frame has not been measured at all and needs to be calibrated. -->
 <robot name="d435_mount_2f85" xmlns:xacro="http://www.ros.org/wiki/xacro">
-  <xacro:macro name="d435_mount_2f85" params="prefix parent">
+  <xacro:macro name="d435_mount_2f85"
+	       params="prefix parent color_camera_centered:=true">
     <xacro:property name="mesh_dir"
 		    value="package://aist_description/objects/meshes"/>
+    <xacro:if value="${color_camera_centered}">
+      <xacro:property name="camera_offset" value="0.0325"/>
+    </xacro:if>
+    <xacro:unless value="${color_camera_centered}">
+      <xacro:property name="camera_offset" value="0.0175"/>
+    </xacro:unless>
     <link name="${prefix}camera_mount">
       <inertial>
@@ -39,5 +46,5 @@
       <parent link="${prefix}camera_mount" />
       <child  link="${prefix}camera_mount_flange" />
-      <origin xyz="-0.028 0.0175 0.0575"
+      <origin xyz="-0.028 ${camera_offset} 0.0575"
 	      rpy="${radians(180.0)} ${radians(15.0)} 0.0"/>
     </joint>
