Commit message: Adjust length of robtiq_arg2f_coupling

File: aist_robotiq/urdf/ft300.urdf.xacro (robot description, xacro)
@@ -1,7 +1,7 @@
 <?xml version="1.0"?>
 <robot name="ft300" xmlns:xacro="http://wiki.ros.org/xacro">
-  <xacro:property name="ft300_radius" value="0.0375"/>
-  <xacro:property name="ft300_length" value="0.0360"/>
   <xacro:macro name="ft300" params="prefix parent *origin">
+    <xacro:property name="ft300_radius" value="0.0375"/>
+    <xacro:property name="ft300_length" value="0.0375"/>
     <link name="${prefix}base_link">
       <visual>
@@ -15,13 +15,4 @@
 	</material>
       </visual>
-      <!-- <visual> -->
-      <!--   <origin xyz="${ft300_length/2} 0 0" rpy="0 ${pi/2} 0"/> -->
-      <!--   <geometry> -->
-      <!--     <cylinder length="${ft300_length}" radius="0.0375"/> -->
-      <!--   </geometry> -->
-      <!--   <material name="Black"> -->
-      <!--     <color rgba="0.2 0.2 0.2 1.0"/> -->
-      <!--   </material> -->
-      <!-- </visual> -->
       <collision>
         <origin xyz="${ft300_length/2} 0 0" rpy="0 ${pi/2} 0"/>
@@ -31,4 +22,7 @@
       </collision>
     </link>
+    <gazebo reference="${prefix}base_link">
+      <material>Gazebo/Black</material>
+    </gazebo>
     <!-- Add the force sensor in front of the gripper. -->
     <joint name="${prefix}ft300_joint" type="fixed">

File: aist_robotiq/urdf/robotiq_140_gripper.urdf.xacro (robot description, xacro)
@@ -249,5 +249,5 @@
       <parent link="${prefix}base_link"/>
       <child link="${prefix}tip_link"/>
-      <origin rpy="0.0 0.0 0.0" xyz=".233 0.0 0.0"/>
+      <origin rpy="0.0 0.0 0.0" xyz=".2328 0.0 0.0"/>
     </joint>
     <link name="${prefix}tip_link"/>

File: aist_robotiq/urdf/robotiq_85_gripper.urdf.xacro (robot description, xacro)
@@ -240,5 +240,5 @@
       <parent link="${prefix}base_link"/>
       <child link="${prefix}tip_link"/>
-      <origin rpy="0.0 0.0 0.0" xyz=".163 0.0 0.0"/>
+      <origin rpy="0.0 0.0 0.0" xyz="0.1628 0.0 0.0"/>
     </joint>
     <link name="${prefix}tip_link"/>

File: aist_robotiq/urdf/robotiq_arg2f_coupling.urdf.xacro (robot description, xacro)
@@ -2,6 +2,7 @@
 <robot xmlns:xacro="http://ros.org/wiki/xacro">
   <xacro:macro name="robotiq_arg2f_coupling" params="prefix parent *origin">
+    <!-- coupling_length = 0.0169 - 2*0.0029 = 0.0111 -->
     <xacro:property name="coupling_radius" value="0.0375"/>
-    <xacro:property name="coupling_length" value="0.0169"/>
+    <xacro:property name="coupling_length" value="0.0111"/>
     <link name="${prefix}base_link">
       <inertial>
@@ -25,8 +26,4 @@
           <cylinder length="${coupling_length}" radius="${coupling_radius}"/>
         </geometry>
-        <!-- <origin xyz="0 0 0" rpy="0 0 0" /> -->
-        <!-- <geometry> -->
-        <!--   <mesh filename="package://aist_robotiq/meshes/collision/robotiq_arg2f_coupling.stl" /> -->
-        <!-- </geometry> -->
       </collision>
     </link>
@@ -34,5 +31,4 @@
       <material>Gazebo/Black</material>
     </gazebo>
-    <!-- Add the force sensor in front of the gripper. -->
     <joint name="${prefix}base_joint" type="fixed">
       <parent link="${parent}"/>

File: moveit_config/aist_moveit_config/config/gazebo_aist_base_scene.urdf (robot description, URDF)
Before this commit: robot aist_base_scene, 95 links, 94 joints
Links:
- removed link vwall1
- link a_bot_ftsensor_base_link: geometry collision cylinder length=0.0375 radius=0.0375; visual mesh filename=package://aist_robotiq/meshes/visual/ft300.stl scale=0.001 0.001 0.001
- link a_bot_gripper_coupling_base_link: geometry collision cylinder length=0.0111 radius=0.0375; visual mesh filename=package://aist_robotiq/meshes/visual/robotiq_arg2f_coupling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 scale=0.001 0.001 0.001
- link b_bot_ftsensor_base_link: geometry collision cylinder length=0.0375 radius=0.0375; visual mesh filename=package://aist_robotiq/meshes/visual/ft300.stl scale=0.001 0.001 0.001
Joints:
- removed joint vwall1
- joint a_bot_ftsensor_flange_joint: origin xyz=0.036 0 0 rpy=0 0 0 -> xyz=0.0375 0 0 rpy=0 0 0
- joint a_bot_gripper_coupling_flange_joint: origin xyz=0.0169 0 0 rpy=0 0 0 -> xyz=0.0111 0 0 rpy=0 0 0
- joint a_bot_gripper_tip_link_joint: origin xyz=.163 0.0 0.0 rpy=0.0 0.0 0.0 -> xyz=0.1628 0.0 0.0 rpy=0.0 0.0 0.0
- joint b_bot_ftsensor_flange_joint: origin xyz=0.036 0 0 rpy=0 0 0 -> xyz=0.0375 0 0 rpy=0 0 0
- joint workspace_live_camera_joint: origin xyz=0.34375981750922774 0.015790557089796247 0.6374101950800111 rpy=-2.8559875657003557 0.0013833155561039075 1.4996937406990187 -> xyz=0.40311836114641414 0.02379492915076111 0.694748550420011 rpy=-2.732962681954511 0.02162437650373519 1.5132164471367409

Commit message: Fix color of robotiq gripper models

File: aist_robotiq/urdf/ft300.urdf.xacro (robot description, xacro)
@@ -12,5 +12,5 @@
 	</geometry>
 	<material name="Black">
-	  <color rgba="0.2 0.2 0.2 1"/>
+	  <color rgba="0.1 0.1 0.1 1"/>
 	</material>
       </visual>

File: aist_robotiq/urdf/robotiq_hande_gripper.urdf.xacro (robot description, xacro)
@@ -36,7 +36,4 @@
           <mesh filename="package://aist_robotiq/meshes/visual/robotiq_hande.dae" scale="1.0 1.0 1.0"/>
         </geometry>
-        <material name="Dark">
-          <color rgba=".1 0.1 0.1 1.0"/>
-        </material>
       </visual>
       <collision>
@@ -58,7 +55,4 @@
           <mesh filename="package://aist_robotiq/meshes/visual/robotiq_hande_finger_1.dae" scale="1.0 1.0 1.0"/>
         </geometry>
-        <material name="DarkGray">
-          <color rgba=".4 0.4 0.4 1.0"/>
-        </material>
       </visual>
       <collision>
@@ -80,7 +74,4 @@
           <mesh filename="package://aist_robotiq/meshes/visual/robotiq_hande_finger_2.dae" scale="1.0 1.0 1.0"/>
         </geometry>
-        <material name="DarkGray">
-          <color rgba=".4 0.4 0.4 1.0"/>
-        </material>
       </visual>
       <collision>
