Commit message: Adjust grasp pose for a_bot_gripper

File: aist_robotiq/urdf/robotiq_140_gripper.urdf.xacro (robot description, xacro)
@@ -160,5 +160,5 @@
         <origin xyz="0 0 0" rpy="0 0 0"/>
         <geometry>
-          <box size="0.03 0.07 0.0075"/>
+          <box size="0.027 0.065 0.0075"/>
         </geometry>
         <material name="">
