Commit message: Change format of mesh from DAE to STL

File: aist_robotiq/urdf/robotiq_85_gripper.urdf.xacro (robot description, xacro)
@@ -21,5 +21,5 @@
         <origin xyz="0 0 0" rpy="0 0 0"/>
         <geometry>
-          <mesh filename="package://aist_robotiq/meshes/visual/robotiq_arg2f_${stroke}_outer_knuckle.dae"
+          <mesh filename="package://aist_robotiq/meshes/visual/robotiq_arg2f_${stroke}_outer_knuckle.stl"
 		scale="0.001 0.001 0.001"/>
         </geometry>
@@ -57,5 +57,5 @@
         <origin xyz="0 0 0" rpy="0 0 0"/>
         <geometry>
-          <mesh filename="package://aist_robotiq/meshes/visual/robotiq_arg2f_${stroke}_outer_finger.dae" scale="0.001 0.001 0.001"/>
+          <mesh filename="package://aist_robotiq/meshes/visual/robotiq_arg2f_${stroke}_outer_finger.stl" scale="0.001 0.001 0.001"/>
         </geometry>
         <material name="">
@@ -123,5 +123,5 @@
         <origin xyz="0 0 0" rpy="0 0 0"/>
         <geometry>
-          <mesh filename="package://aist_robotiq/meshes/visual/robotiq_arg2f_${stroke}_inner_finger.dae"
+          <mesh filename="package://aist_robotiq/meshes/visual/robotiq_arg2f_${stroke}_inner_finger.stl"
 		scale="0.001 0.001 0.001"/>
         </geometry>

File: aist_robotiq/urdf/robotiq_hande_gripper.urdf.xacro (robot description, xacro)
@@ -34,6 +34,9 @@
         <origin rpy="0 0 0" xyz="0 0 0"/>
         <geometry>
-          <mesh filename="package://aist_robotiq/meshes/visual/robotiq_hande.dae" scale="1.0 1.0 1.0"/>
+          <mesh filename="package://aist_robotiq/meshes/visual/robotiq_hande.stl" scale="0.001 0.001 0.001"/>
         </geometry>
+        <material name="">
+          <color rgba="0.1 0.1 0.1 1"/>
+        </material>
       </visual>
       <collision>
@@ -53,6 +56,11 @@
         <origin rpy="0 0 0" xyz="0 0 0"/>
         <geometry>
-          <mesh filename="package://aist_robotiq/meshes/visual/robotiq_hande_finger_1.dae" scale="1.0 1.0 1.0"/>
+          <mesh filename="package://aist_robotiq/meshes/visual/robotiq_hande_finger_1.stl" scale="0.001 0.001 0.001"/>
         </geometry>
+        <material name="">
+          <color rgba="0.792156862745098
+		       0.819607843137255
+		       0.933333333333333 1"/>
+        </material>
       </visual>
       <collision>
@@ -72,6 +80,11 @@
         <origin rpy="0 0 0" xyz="0 0 0"/>
         <geometry>
-          <mesh filename="package://aist_robotiq/meshes/visual/robotiq_hande_finger_2.dae" scale="1.0 1.0 1.0"/>
+          <mesh filename="package://aist_robotiq/meshes/visual/robotiq_hande_finger_2.stl" scale="0.001 0.001 0.001"/>
         </geometry>
+        <material name="">
+          <color rgba="0.792156862745098
+		       0.819607843137255
+		       0.933333333333333 1"/>
+        </material>
       </visual>
       <collision>
