Commit message: Update moveit_config from scratch

File: moveit_config/a_bot_moveit_config/config/gazebo_a_bot_base_scene.urdf (robot description, URDF)
Before this commit: robot a_bot__base_scene, 54 links, 53 joints
Joints:
- joint a_bot_inside_camera_joint: origin xyz=0.014973206639882487      -0.006605026045624136      0.05983621136016915 rpy=0.023976131805434685      0.403287172799087      0.012905813015089812 -> xyz=0.014368349250599823      0.0035415297809514353      0.06397546955943786 rpy=0.02303437721634514      0.40347560400972565      0.010798159061973579
- joint a_bot_outside_camera_joint: origin xyz=0.03158216743040747      -0.006437943317858734      0.08083480848924662 rpy=0.016860191822591693      -0.22414769691091246      0.033437654559852904 -> xyz=0.03167812734753831      -0.007813867044282037      0.08129884906700884 rpy=0.017373333209516714      -0.2189346019095829      0.034978097124935485
