Commit message: Fixed axis orientation for m3 and m4 tools

File: aist_fastening_tools/urdf/screw_tool_m3.urdf.xacro (robot description, xacro)
@@ -7,5 +7,5 @@
     <link name="${prefix}base_link">
       <visual>
-        <origin xyz="0 0 0" rpy="0 ${-pi/2} 0"/>
+        <origin xyz="0 0 0" rpy="${pi/2} 0 ${-pi/2}"/>
 	<geometry>
           <mesh filename="package://aist_fastening_tools/meshes/visual/screw_tool_m3_BC5-XL320-R-AY2.6-EH2.stl" scale="0.001 0.001 0.001"/>
@@ -16,5 +16,5 @@
       </visual>
       <collision>
-	<origin xyz="0 0 0" rpy="0 ${-pi/2} 0"/>
+	<origin xyz="0 0 0" rpy="${pi/2} 0 ${-pi/2}"/>
 	<geometry>
 	  <mesh filename="package://aist_fastening_tools/meshes/collision/screw_tool_m3_simplified.stl" scale="0.0001 0.0001 0.0001"/>

File: aist_fastening_tools/urdf/screw_tool_m4.urdf.xacro (robot description, xacro)
@@ -7,5 +7,5 @@
     <link name="${prefix}base_link">
       <visual>
-        <origin xyz="0 0 0" rpy="0 ${-pi/2} 0"/>
+        <origin xyz="0 0 0" rpy="${pi/2} 0 ${-pi/2}"/>
 	<geometry>
           <mesh filename="package://aist_fastening_tools/meshes/visual/screw_tool_m4_BC5-XL320-AY3.5-EH3R4.stl" scale="0.001 0.001 0.001"/>
@@ -16,5 +16,5 @@
       </visual>
       <collision>
-	<origin xyz="0 0 0" rpy="0 ${-pi/2} 0"/>
+        <origin xyz="0 0 0" rpy="${pi/2} 0 ${-pi/2}"/>
 	<geometry>
 	  <mesh filename="package://aist_fastening_tools/meshes/collision/screw_tool_m4_simplified.stl" scale="0.0001 0.0001 0.0001"/>

Commit message: Construct URDF from properties stored in yaml for precision_gripper and screw_tools

File: aist_fastening_tools/urdf/screw_tool_m3.urdf.xacro (robot description, xacro)
@@ -3,20 +3,53 @@
   <xacro:macro name="screw_tool_m3"
 	       params="prefix parent *origin">
+    <xacro:macro name="load_properties" params="filename">
+      <xacro:property name="properties"
+		      value="${xacro.load_yaml(filename)}"/>
+      <xacro:property name="visual_meshes"
+		      value="${properties['visual_meshes']}"
+		      scope="parent"/>
+      <xacro:property name="collision_meshes"
+		      value="${properties['collision_meshes']}"
+		      scope="parent"/>
+      <xacro:property name="subframes"
+		      value="${properties['subframes']}"
+		      scope="parent"/>
+    </xacro:macro>
+    <xacro:load_properties filename="$(find aist_fastening_tools
+				     )/config/screw_tool_m3_properties.yaml"/>
     <!-- A link representing the gripper and a joint attaching it to parnet -->
+    <xacro:property name="vorigin" value="${visual_meshes[0]['pose']}"/>
+    <xacro:property name="vscale"  value="${visual_meshes[0]['scale']}"/>
+    <xacro:property name="vcolor"  value="${visual_meshes[0]['color']}"/>
+    <xacro:property name="corigin" value="${collision_meshes[0]['pose']}"/>
+    <xacro:property name="cscale"  value="${collision_meshes[0]['scale']}"/>
+    <joint name="${prefix}base_joint" type="fixed">
+      <parent link="${parent}"/>
+      <child  link="${prefix}base_link"/>
+      <xacro:insert_block name="origin"/>
+    </joint>
     <link name="${prefix}base_link">
       <visual>
-        <origin xyz="0 0 -0.0006" rpy="0 0 ${-pi/2}"/>
-	<geometry>
-          <mesh filename="package://aist_fastening_tools/meshes/visual/screw_tool_m3_BC5-XL320-R-AY2.6-EH2.stl" scale="0.001 0.001 0.001"/>
-	</geometry>
-	<material name="light_grey">
-	  <color rgba="0.8 0.8 0.8 1"/>
-	</material>
+	<origin xyz="${vorigin[0]} ${vorigin[1]} ${vorigin[2]}"
+		rpy="${vorigin[3]*pi/180.0}
+		     ${vorigin[4]*pi/180.0}
+		     ${vorigin[5]*pi/180.0}"/>
+        <geometry>
+          <mesh filename="${visual_meshes[0]['url']}"
+		scale="${vscale[0]} ${vscale[1]} ${vscale[2]}"/>
+        </geometry>
+        <material name="Gazebo/Black">
+          <color rgba="${vcolor[0]} ${vcolor[1]} ${vcolor[2]} ${vcolor[3]}"/>
+        </material>
       </visual>
       <collision>
-	<origin xyz="0 0 0" rpy="0 0 ${-pi/2}"/>
-	<geometry>
-	  <mesh filename="package://aist_fastening_tools/meshes/collision/screw_tool_m3_simplified.stl" scale="0.0001 0.0001 0.0001"/>
-	</geometry>
+	<origin xyz="${corigin[0]} ${corigin[1]} ${corigin[2]}"
+		rpy="${corigin[3]*pi/180.0}
+		     ${corigin[4]*pi/180.0}
+		     ${corigin[5]*pi/180.0}"/>
+        <geometry>
+          <mesh filename="${collision_meshes[0]['url']}"
+		scale="${cscale[0]} ${cscale[1]} ${cscale[2]}"/>
+        </geometry>
       </collision>
       <inertial>
@@ -26,17 +59,16 @@
       </inertial>
     </link>
-    <joint name="${prefix}base_joint" type="fixed">
-      <parent link="${parent}"/>
-      <child  link="${prefix}base_link"/>
-      <xacro:insert_block name="origin"/>
-    </joint>
-    <!-- A link representing the tip of the pad and a joint attaching
-	 it to the gripper -->
-    <link name="${prefix}tip_link"/>
-    <joint name="${prefix}tip_joint" type="fixed">
+    <!-- tip -->
+    <xacro:property name="torigin"
+		    value="${subframes['tip_link']}"/>
+    <joint name="${prefix}tip_link_joint" type="fixed">
       <parent link="${prefix}base_link"/>
       <child  link="${prefix}tip_link"/>
-      <origin xyz="0 0 -0.100" rpy="0 0 0"/>
+      <origin xyz="${torigin[0]} ${torigin[1]} ${torigin[2]}"
+	      rpy="${torigin[3]*pi/180.0}
+		   ${torigin[4]*pi/180.0}
+		   ${torigin[5]*pi/180.0}"/>
     </joint>
+    <link name="${prefix}tip_link"/>
   </xacro:macro>
 </robot>

File: aist_fastening_tools/urdf/screw_tool_m4.urdf.xacro (robot description, xacro)
@@ -3,20 +3,53 @@
   <xacro:macro name="screw_tool_m4"
 	       params="prefix parent *origin">
+    <xacro:macro name="load_properties" params="filename">
+      <xacro:property name="properties"
+		      value="${xacro.load_yaml(filename)}"/>
+      <xacro:property name="visual_meshes"
+		      value="${properties['visual_meshes']}"
+		      scope="parent"/>
+      <xacro:property name="collision_meshes"
+		      value="${properties['collision_meshes']}"
+		      scope="parent"/>
+      <xacro:property name="subframes"
+		      value="${properties['subframes']}"
+		      scope="parent"/>
+    </xacro:macro>
+    <xacro:load_properties filename="$(find aist_fastening_tools
+				     )/config/screw_tool_m4_properties.yaml"/>
     <!-- A link representing the gripper and a joint attaching it to parnet -->
+    <xacro:property name="vorigin" value="${visual_meshes[0]['pose']}"/>
+    <xacro:property name="vscale"  value="${visual_meshes[0]['scale']}"/>
+    <xacro:property name="vcolor"  value="${visual_meshes[0]['color']}"/>
+    <xacro:property name="corigin" value="${collision_meshes[0]['pose']}"/>
+    <xacro:property name="cscale"  value="${collision_meshes[0]['scale']}"/>
+    <joint name="${prefix}base_joint" type="fixed">
+      <parent link="${parent}"/>
+      <child  link="${prefix}base_link"/>
+      <xacro:insert_block name="origin"/>
+    </joint>
     <link name="${prefix}base_link">
       <visual>
-        <origin xyz="0 0 -0.0006" rpy="0 0 ${-pi/2}"/>
-	<geometry>
-          <mesh filename="package://aist_fastening_tools/meshes/visual/screw_tool_m4_BC5-XL320-AY3.5-EH3R4.stl" scale="0.001 0.001 0.001"/>
-	</geometry>
-	<material name="light_grey">
-	  <color rgba="0.8 0.8 0.8 1"/>
-	</material>
+	<origin xyz="${vorigin[0]} ${vorigin[1]} ${vorigin[2]}"
+		rpy="${vorigin[3]*pi/180.0}
+		     ${vorigin[4]*pi/180.0}
+		     ${vorigin[5]*pi/180.0}"/>
+        <geometry>
+          <mesh filename="${visual_meshes[0]['url']}"
+		scale="${vscale[0]} ${vscale[1]} ${vscale[2]}"/>
+        </geometry>
+        <material name="Gazebo/Black">
+          <color rgba="${vcolor[0]} ${vcolor[1]} ${vcolor[2]} ${vcolor[3]}"/>
+        </material>
       </visual>
       <collision>
-        <origin xyz="0 0 0" rpy="0 0 ${-pi/2}"/>
-	<geometry>
-	  <mesh filename="package://aist_fastening_tools/meshes/collision/screw_tool_m4_simplified.stl" scale="0.0001 0.0001 0.0001"/>
-	</geometry>
+	<origin xyz="${corigin[0]} ${corigin[1]} ${corigin[2]}"
+		rpy="${corigin[3]*pi/180.0}
+		     ${corigin[4]*pi/180.0}
+		     ${corigin[5]*pi/180.0}"/>
+        <geometry>
+          <mesh filename="${collision_meshes[0]['url']}"
+		scale="${cscale[0]} ${cscale[1]} ${cscale[2]}"/>
+        </geometry>
       </collision>
       <inertial>
@@ -26,17 +59,16 @@
       </inertial>
     </link>
-    <joint name="${prefix}base_joint" type="fixed">
-      <parent link="${parent}"/>
-      <child  link="${prefix}base_link"/>
-      <xacro:insert_block name="origin"/>
-    </joint>
-    <!-- A link representing the tip of the pad and a joint attaching
-	 it to the gripper -->
-    <link name="${prefix}tip_link"/>
-    <joint name="${prefix}tip_joint" type="fixed">
+    <!-- tip -->
+    <xacro:property name="torigin"
+		    value="${subframes['tip_link']}"/>
+    <joint name="${prefix}tip_link_joint" type="fixed">
       <parent link="${prefix}base_link"/>
       <child  link="${prefix}tip_link"/>
-      <origin xyz="0 0 -0.120" rpy="0 0 0"/>
+      <origin xyz="${torigin[0]} ${torigin[1]} ${torigin[2]}"
+	      rpy="${torigin[3]*pi/180.0}
+		   ${torigin[4]*pi/180.0}
+		   ${torigin[5]*pi/180.0}"/>
     </joint>
+    <link name="${prefix}tip_link"/>
   </xacro:macro>
 </robot>

File: aist_precision_gripper/urdf/precision_coupling.urdf.xacro (robot description, xacro)
@@ -3,16 +3,12 @@
   <xacro:macro name="precision_coupling" params="prefix parent *origin">
     <!-- coupling_length = 0.0169 - 2*0.0029 = 0.0111 -->
-    <xacro:property name="coupling_radius" value="0.0375"/>
-    <xacro:property name="coupling_length" value="0.0085"/>
+    <xacro:property name="coupling_radius"   value="0.0375"/>
+    <xacro:property name="coupling_length"   value="0.0085"/>
+    <xacro:property name="horizontal_offset" value="-0.0025"/>
     <link name="${prefix}base_link">
-      <inertial>
-        <origin xyz="8.625E-08 -4.6583E-06 0.03145" rpy="0 0 0" />
-        <mass value="0.22652" />
-        <inertia ixx="0.00020005" ixy="-4.2442E-10" ixz="-2.9069E-10" iyy="0.00017832" iyz="-3.4402E-08" izz="0.00013478" />
-      </inertial>
       <visual>
         <origin xyz="-0.0045 0 0" rpy="${pi/2} 0 ${pi/2}" />
         <geometry>
-          <mesh filename="package://aist_precision_gripper/meshes/precision_coupling.stl"
+          <mesh filename="package://aist_precision_gripper/meshes/visual/precision_coupling.stl"
 		scale="0.001 0.001 0.001"/>
         </geometry>
@@ -27,4 +23,9 @@
         </geometry>
       </collision>
+      <inertial>
+        <origin xyz="8.625E-08 -4.6583E-06 0.03145" rpy="0 0 0" />
+        <mass value="0.22652" />
+        <inertia ixx="0.00020005" ixy="-4.2442E-10" ixz="-2.9069E-10" iyy="0.00017832" iyz="-3.4402E-08" izz="0.00013478" />
+      </inertial>
     </link>
     <gazebo reference="${prefix}base_link">
@@ -40,5 +41,6 @@
       <parent link="${prefix}base_link"/>
       <child  link="${prefix}flange_link"/>
-      <origin xyz="${coupling_length} 0 0" rpy="0 0 0"/>
+      <origin xyz="${coupling_length} ${horizontal_offset} 0"
+	      rpy="0 ${-pi/2} 0"/>
     </joint>
   </xacro:macro>

File: aist_precision_gripper/urdf/precision_gripper.urdf.xacro (robot description, xacro)
@@ -2,19 +2,31 @@
 <robot xmlns:xacro="http://ros.org/wiki/xacro">
   <xacro:macro name="precision_gripper" params="prefix parent *origin">
+    <xacro:macro name="load_properties" params="filename">
+      <xacro:property name="properties"
+		      value="${xacro.load_yaml(filename)}"/>
+      <xacro:property name="visual_meshes"
+		      value="${properties['visual_meshes']}"
+		      scope="parent"/>
+      <xacro:property name="collision_meshes"
+		      value="${properties['collision_meshes']}"
+		      scope="parent"/>
+      <xacro:property name="subframes"
+		      value="${properties['subframes']}"
+		      scope="parent"/>
+    </xacro:macro>
     <xacro:include filename="$(find aist_precision_gripper
 			     )/urdf/precision_transmission.xacro"/>
     <xacro:precision_transmission prefix="${prefix}"/>
-    <xacro:property name="horizontal_offset"		value="-0.014"/>
-    <xacro:property name="tip_distance"			value="0.147"/>
-    <xacro:property name="rail_distance"		value="0.0915"/>
-    <xacro:property name="max_gap"			value="0.010"/>
-    <xacro:property name="depth"			value="0.030"/>
-    <xacro:property name="motor_width"			value="0.055"/>
-    <xacro:property name="motor_height"			value="0.0425"/>
-    <xacro:property name="motor_offset"			value="-0.0025"/>
-    <xacro:property name="lower_body_width"		value="0.085"/>
-    <xacro:property name="lower_body_height"		value="0.050"/>
-    <xacro:property name="finger_collision_width"	value="0.003"/>
+    <xacro:load_properties filename="$(find aist_precision_gripper
+				     )/config/precision_gripper_properties.yaml"/>
+    <xacro:property name="max_gap"	value="0.010"/>
     <!-- base -->
+    <xacro:property name="base_vorigin"	value="${visual_meshes[0]['pose']}"/>
+    <xacro:property name="base_vscale"	value="${visual_meshes[0]['scale']}"/>
+    <xacro:property name="base_vcolor"	value="${visual_meshes[0]['color']}"/>
+    <xacro:property name="base_corigin"
+		    value="${collision_meshes[0]['pose']}"/>
+    <xacro:property name="base_cscale"
+		    value="${collision_meshes[0]['scale']}"/>
     <joint name="${prefix}base_joint" type="fixed">
       <parent link="${parent}"/>
@@ -24,21 +36,30 @@
     <link name="${prefix}base_link">
       <visual>
-	<origin xyz="0 0 0" rpy="${pi/2} 0 ${pi/2}"/>
-        <geometry>
-          <mesh filename="package://aist_precision_gripper/meshes/visual/precision_body.stl" scale="0.001 0.001 0.001"/>
+	<origin xyz="${base_vorigin[0]}
+		     ${base_vorigin[1]}
+		     ${base_vorigin[2]}"
+		rpy="${base_vorigin[3]*pi/180.0}
+		     ${base_vorigin[4]*pi/180.0}
+		     ${base_vorigin[5]*pi/180.0}"/>
+        <geometry>
+          <mesh filename="${visual_meshes[0]['url']}"
+		scale="${base_vscale[0]} ${base_vscale[1]} ${base_vscale[2]}"/>
         </geometry>
         <material name="Gazebo/Black">
-          <color rgba="0.1 0.1 0.1 1"/>
+          <color rgba="${base_vcolor[0]} ${base_vcolor[1]}
+		       ${base_vcolor[2]} ${base_vcolor[3]}"/>
         </material>
       </visual>
       <collision>
-	<origin xyz="0 0 0" rpy="${pi/2} 0 ${pi/2}"/>
-	<geometry>
-          <mesh filename="package://aist_precision_gripper/meshes/collision/precision_body.stl" scale="0.001 0.001 0.001"/>
-        </geometry>
-	<!--   <origin xyz="${motor_height/2} ${motor_offset} 0" rpy="0 0 0"/> -->
-	<!--   <geometry> -->
-	<!--     <box size="${motor_height} ${motor_width} ${depth}"/> -->
-	<!--   </geometry> -->
+	<origin xyz="${base_corigin[0]}
+		     ${base_corigin[1]}
+		     ${base_corigin[2]}"
+		rpy="${base_corigin[3]*pi/180.0}
+		     ${base_corigin[4]*pi/180.0}
+		     ${base_corigin[5]*pi/180.0}"/>
+        <geometry>
+          <mesh filename="${collision_meshes[0]['url']}"
+		scale="${base_cscale[0]} ${base_cscale[1]} ${base_cscale[2]}"/>
+        </geometry>
       </collision>
       <inertial>
@@ -49,21 +70,16 @@
       </inertial>
     </link>
-    <!-- lower body(collision only) -->
-    <!-- <joint name="${prefix}lower_body_joint" type="fixed"> -->
-    <!--   <parent link="${prefix}base_link"/> -->
-    <!--   <child  link="${prefix}lower_body_link"/> -->
-    <!--   <origin xyz="${motor_height} ${horizontal_offset} 0" rpy="0 0 0"/> -->
-    <!-- </joint> -->
-    <!-- <link name="${prefix}lower_body_link"> -->
-    <!--   <collision> -->
-    <!-- 	<origin xyz="${lower_body_height/2} 0 0" rpy="0 0 0"/> -->
-    <!-- 	<geometry> -->
-    <!-- 	  <box size="${lower_body_height} ${lower_body_width} ${depth}"/> -->
-    <!-- 	</geometry> -->
-    <!--   </collision> -->
-    <!-- </link> -->
     <!-- left finger -->
+    <xacro:property name="left_finger_vorigin"
+		    value="${visual_meshes[1]['pose']}"/>
+    <xacro:property name="left_finger_vscale"
+		    value="${visual_meshes[1]['scale']}"/>
+    <xacro:property name="left_finger_vcolor"
+		    value="${visual_meshes[1]['color']}"/>
+    <xacro:property name="left_finger_corigin"
+		    value="${collision_meshes[1]['pose']}"/>
+    <xacro:property name="left_finger_cscale"
+		    value="${collision_meshes[1]['scale']}"/>
     <joint name="${prefix}finger_joint" type="prismatic">
-      <origin xyz="${rail_distance} ${horizontal_offset} 0" rpy="0 0 0"/>
       <parent link="${prefix}base_link"/>
       <child link="${prefix}left_finger"/>
@@ -73,25 +89,34 @@
     <link name="${prefix}left_finger">
       <visual>
-	<origin xyz="0 0 0" rpy="${pi/2} 0 ${pi/2}"/>
-        <geometry>
-          <mesh filename="package://aist_precision_gripper/meshes/visual/precision_left_finger.stl" scale="0.001 0.001 0.001"/>
+	<origin xyz="${left_finger_vorigin[0]}
+		     ${left_finger_vorigin[1]}
+		     ${left_finger_vorigin[2]}"
+		rpy="${left_finger_vorigin[3]*pi/180.0}
+		     ${left_finger_vorigin[4]*pi/180.0}
+		     ${left_finger_vorigin[5]*pi/180.0}"/>
+        <geometry>
+          <mesh filename="${visual_meshes[1]['url']}"
+		scale="${left_finger_vscale[0]}
+		       ${left_finger_vscale[1]}
+		       ${left_finger_vscale[2]}"/>
         </geometry>
         <material name="Gazebo/Grey">
-          <color rgba="0.7 0.7 0.7 1"/>
+          <color rgba="${left_finger_vcolor[0]} ${left_finger_vcolor[1]}
+		       ${left_finger_vcolor[2]} ${left_finger_vcolor[3]}"/>
         </material>
       </visual>
       <collision>
-	<origin xyz="0 0 0" rpy="${pi/2} 0 ${pi/2}"/>
-	<geometry>
-          <mesh filename="package://aist_precision_gripper/meshes/collision/precision_left_finger.stl" scale="0.001 0.001 0.001"/>
-        </geometry>
-	<!-- <origin xyz="${(tip_distance - rail_distance)/2} -->
-	<!-- 	     ${finger_collision_width/2} 0" -->
-	<!-- 	rpy="0 0 0"/> -->
-	<!-- <geometry> -->
-	<!--   <box size="${tip_distance - rail_distance} -->
-	<!-- 	     ${finger_collision_width} -->
-	<!-- 	     ${finger_collision_width}"/> -->
-	<!-- </geometry> -->
+	<origin xyz="${left_finger_corigin[0]}
+		     ${left_finger_corigin[1]}
+		     ${left_finger_corigin[2]}"
+		rpy="${left_finger_corigin[3]*pi/180.0}
+		     ${left_finger_corigin[4]*pi/180.0}
+		     ${left_finger_corigin[5]*pi/180.0}"/>
+        <geometry>
+          <mesh filename="${collision_meshes[1]['url']}"
+		scale="${left_finger_cscale[0]}
+		       ${left_finger_cscale[1]}
+		       ${left_finger_cscale[2]}"/>
+        </geometry>
       </collision>
       <inertial>
@@ -103,6 +128,15 @@
     </link>
     <!-- right finger -->
+    <xacro:property name="right_finger_vorigin"
+		    value="${visual_meshes[1]['pose']}"/>
+    <xacro:property name="right_finger_vscale"
+		    value="${visual_meshes[1]['scale']}"/>
+    <xacro:property name="right_finger_vcolor"
+		    value="${visual_meshes[1]['color']}"/>
+    <xacro:property name="right_finger_corigin"
+		    value="${collision_meshes[1]['pose']}"/>
+    <xacro:property name="right_finger_cscale"
+		    value="${collision_meshes[1]['scale']}"/>
     <joint name="${prefix}right_finger_joint" type="prismatic">
-      <origin xyz="${rail_distance} ${horizontal_offset} 0" rpy="0 0 0"/>
       <parent link="${prefix}base_link"/>
       <child link="${prefix}right_finger"/>
@@ -113,26 +147,35 @@
     <link name="${prefix}right_finger">
       <visual>
-	<origin xyz="0 0 0" rpy="${pi/2} 0 ${pi/2}"/>
-        <geometry>
-          <mesh filename="package://aist_precision_gripper/meshes/visual/precision_right_finger.stl" scale="0.001 0.001 0.001"/>
+	<origin xyz="${right_finger_vorigin[0]}
+		     ${right_finger_vorigin[1]}
+		     ${right_finger_vorigin[2]}"
+		rpy="${right_finger_vorigin[3]*pi/180.0}
+		     ${right_finger_vorigin[4]*pi/180.0}
+		     ${right_finger_vorigin[5]*pi/180.0}"/>
+        <geometry>
+          <mesh filename="${visual_meshes[2]['url']}"
+		scale="${right_finger_vscale[0]}
+		       ${right_finger_vscale[1]}
+		       ${right_finger_vscale[2]}"/>
         </geometry>
         <material name="Gazebo/Grey">
-          <color rgba="0.7 0.7 0.7 1"/>
+          <color rgba="${right_finger_vcolor[0]} ${right_finger_vcolor[1]}
+		       ${right_finger_vcolor[2]} ${right_finger_vcolor[3]}"/>
         </material>
       </visual>
-      <colliaion>
-	<origin xyz="0 0 0" rpy="${pi/2} 0 ${pi/2}"/>
-	<geometry>
-          <mesh filename="package://aist_precision_gripper/meshes/collision/precision_right_finger.stl" scale="0.001 0.001 0.001"/>
-        </geometry>
-	<!-- <origin xyz="${(tip_distance - rail_distance)/2} -->
-	<!-- 	     ${-finger_collision_width/2} 0" -->
-	<!-- 	rpy="0 0 0"/> -->
-	<!-- <geometry> -->
-	<!--   <box size="${tip_distance - rail_distance} -->
-	<!-- 	     ${finger_collision_width} -->
-	<!-- 	     ${finger_collision_width}"/> -->
-	<!-- </geometry> -->
-      </colliaion>
+      <collision>
+	<origin xyz="${right_finger_corigin[0]}
+		     ${right_finger_corigin[1]}
+		     ${right_finger_corigin[2]}"
+		rpy="${right_finger_corigin[3]*pi/180.0}
+		     ${right_finger_corigin[4]*pi/180.0}
+		     ${right_finger_corigin[5]*pi/180.0}"/>
+        <geometry>
+          <mesh filename="${collision_meshes[2]['url']}"
+		scale="${right_finger_cscale[0]}
+		       ${right_finger_cscale[1]}
+		       ${right_finger_cscale[2]}"/>
+        </geometry>
+      </collision>
       <inertial>
         <origin xyz="-0.02262 0.00759 0.00738" rpy="0 0 0"/>
@@ -143,8 +186,15 @@
     </link>
     <!-- tip -->
+    <xacro:property name="tip_link_origin"
+		    value="${subframes['tip_link']}"/>
     <joint name="${prefix}tip_link_joint" type="fixed">
       <parent link="${prefix}base_link"/>
       <child  link="${prefix}tip_link"/>
-      <origin xyz="${tip_distance} ${horizontal_offset} 0" rpy="0 ${-pi/2} 0"/>
+      <origin xyz="${tip_link_origin[0]}
+		   ${tip_link_origin[1]}
+		   ${tip_link_origin[2]}"
+	      rpy="${tip_link_origin[3]*pi/180.0}
+		   ${tip_link_origin[4]*pi/180.0}
+		   ${tip_link_origin[5]*pi/180.0}"/>
     </joint>
     <link name="${prefix}tip_link"/>
