Commit message: Separate body and piston of base_fixture

File: aist_fastening_tools/urdf/base_fixture.urdf.xacro (robot description, xacro)
@@ -24,10 +24,10 @@
 				     )/config/fastening_tools_properties.yaml"/>
     <xacro:property name="stroke"	value="0.020"/>
-    <!-- base -->
-    <xacro:property name="base_vorigin"	value="${visual_meshes[0]['pose']}"/>
-    <xacro:property name="base_vscale"	value="${visual_meshes[0]['scale']}"/>
-    <xacro:property name="base_vcolor"	value="${visual_meshes[0]['color']}"/>
-    <xacro:property name="base_corigin" value="${primitives[0]['pose']}"/>
-    <xacro:property name="base_cdims"   value="${primitives[0]['dimensions']}"/>
+    <!-- body -->
+    <xacro:property name="body_vorigin"	value="${visual_meshes[0]['pose']}"/>
+    <xacro:property name="body_vscale"	value="${visual_meshes[0]['scale']}"/>
+    <xacro:property name="body_vcolor"	value="${visual_meshes[0]['color']}"/>
+    <xacro:property name="body_corigin" value="${primitives[0]['pose']}"/>
+    <xacro:property name="body_cdims"   value="${primitives[0]['dimensions']}"/>
     <joint name="${prefix}base_joint" type="fixed">
       <parent link="${parent}"/>
@@ -37,28 +37,28 @@
     <link name="${prefix}base_link">
       <visual>
-	<origin xyz="${base_vorigin[0]}
-		     ${base_vorigin[1]}
-		     ${base_vorigin[2]}"
-		rpy="${base_vorigin[3]*pi/180.0}
-		     ${base_vorigin[4]*pi/180.0}
-		     ${base_vorigin[5]*pi/180.0}"/>
+	<origin xyz="${body_vorigin[0]}
+		     ${body_vorigin[1]}
+		     ${body_vorigin[2]}"
+		rpy="${body_vorigin[3]*pi/180.0}
+		     ${body_vorigin[4]*pi/180.0}
+		     ${body_vorigin[5]*pi/180.0}"/>
         <geometry>
           <mesh filename="${visual_meshes[0]['url']}"
-		scale="${base_vscale[0]} ${base_vscale[1]} ${base_vscale[2]}"/>
+		scale="${body_vscale[0]} ${body_vscale[1]} ${body_vscale[2]}"/>
         </geometry>
         <material name="Gazebo/Black">
-          <color rgba="${base_vcolor[0]} ${base_vcolor[1]}
-		       ${base_vcolor[2]} ${base_vcolor[3]}"/>
+          <color rgba="${body_vcolor[0]} ${body_vcolor[1]}
+		       ${body_vcolor[2]} ${body_vcolor[3]}"/>
         </material>
       </visual>
       <collision>
-	<origin xyz="${base_corigin[0]}
-		     ${base_corigin[1]}
-		     ${base_corigin[2]}"
-		rpy="${base_corigin[3]*pi/180.0}
-		     ${base_corigin[4]*pi/180.0}
-		     ${base_corigin[5]*pi/180.0}"/>
+	<origin xyz="${body_corigin[0]}
+		     ${body_corigin[1]}
+		     ${body_corigin[2]}"
+		rpy="${body_corigin[3]*pi/180.0}
+		     ${body_corigin[4]*pi/180.0}
+		     ${body_corigin[5]*pi/180.0}"/>
         <geometry>
-	  <box size="${base_cdims[0]} ${base_cdims[1]} ${base_cdims[2]}"/>
+	  <box size="${body_cdims[0]} ${body_cdims[1]} ${body_cdims[2]}"/>
         </geometry>
       </collision>
@@ -70,51 +70,51 @@
       </inertial>
     </link>
-    <!-- cylinder -->
-    <!-- <xacro:property name="cylinder_vorigin" -->
-    <!-- 		    value="${visual_meshes[1]['pose']}"/> -->
-    <!-- <xacro:property name="cylinder_vscale" -->
-    <!-- 		    value="${visual_meshes[1]['scale']}"/> -->
-    <!-- <xacro:property name="cylinder_vcolor" -->
-    <!-- 		    value="${visual_meshes[1]['color']}"/> -->
-    <xacro:property name="cylinder_corigin"
+    <!-- piston -->
+    <xacro:property name="piston_vorigin"
+    		    value="${visual_meshes[1]['pose']}"/>
+    <xacro:property name="piston_vscale"
+    		    value="${visual_meshes[1]['scale']}"/>
+    <xacro:property name="piston_vcolor"
+    		    value="${visual_meshes[1]['color']}"/>
+    <xacro:property name="piston_corigin"
 		    value="${primitives[1]['pose']}"/>
-    <xacro:property name="cylinder_cdims"
+    <xacro:property name="piston_cdims"
 		    value="${primitives[1]['dimensions']}"/>
-    <joint name="${prefix}cylinder_joint" type="prismatic">
+    <joint name="${prefix}piston_joint" type="prismatic">
       <parent link="${prefix}base_link"/>
-      <child link="${prefix}cylinder"/>
+      <child link="${prefix}piston"/>
       <axis xyz="1 0 0"/>
       <limit effort="130" lower="0" upper="${stroke}" velocity="0.15"/>
     </joint>
-    <link name="${prefix}cylinder">
-      <!-- <visual> -->
-      <!-- 	<origin xyz="${cylinder_vorigin[0]} -->
-      <!-- 		     ${cylinder_vorigin[1]} -->
-      <!-- 		     ${cylinder_vorigin[2]}" -->
-      <!-- 		rpy="${cylinder_vorigin[3]*pi/180.0} -->
-      <!-- 		     ${cylinder_vorigin[4]*pi/180.0} -->
-      <!-- 		     ${cylinder_vorigin[5]*pi/180.0}"/> -->
-      <!--   <geometry> -->
-      <!--     <mesh filename="${visual_meshes[1]['url']}" -->
-      <!-- 		scale="${cylinder_vscale[0]} -->
-      <!-- 		       ${cylinder_vscale[1]} -->
-      <!-- 		       ${cylinder_vscale[2]}"/> -->
-      <!--   </geometry> -->
-      <!--   <material name="Gazebo/Grey"> -->
-      <!--     <color rgba="${cylinder_vcolor[0]} ${cylinder_vcolor[1]} -->
-      <!-- 		       ${cylinder_vcolor[2]} ${cylinder_vcolor[3]}"/> -->
-      <!--   </material> -->
-      <!-- </visual> -->
+    <link name="${prefix}piston">
+      <visual>
+      	<origin xyz="${piston_vorigin[0]}
+      		     ${piston_vorigin[1]}
+      		     ${piston_vorigin[2]}"
+      		rpy="${piston_vorigin[3]*pi/180.0}
+      		     ${piston_vorigin[4]*pi/180.0}
+      		     ${piston_vorigin[5]*pi/180.0}"/>
+        <geometry>
+          <mesh filename="${visual_meshes[1]['url']}"
+      		scale="${piston_vscale[0]}
+		       ${piston_vscale[1]}
+		       ${piston_vscale[2]}"/>
+        </geometry>
+        <material name="Gazebo/Grey">
+          <color rgba="${piston_vcolor[0]} ${piston_vcolor[1]}
+      		       ${piston_vcolor[2]} ${piston_vcolor[3]}"/>
+        </material>
+      </visual>
       <collision>
-	<origin xyz="${cylinder_corigin[0]}
-		     ${cylinder_corigin[1]}
-		     ${cylinder_corigin[2]}"
-		rpy="${cylinder_corigin[3]*pi/180.0}
-		     ${cylinder_corigin[4]*pi/180.0}
-		     ${cylinder_corigin[5]*pi/180.0}"/>
+	<origin xyz="${piston_corigin[0]}
+		     ${piston_corigin[1]}
+		     ${piston_corigin[2]}"
+		rpy="${piston_corigin[3]*pi/180.0}
+		     ${piston_corigin[4]*pi/180.0}
+		     ${piston_corigin[5]*pi/180.0}"/>
         <geometry>
-	  <box size="${cylinder_cdims[0]}
-		     ${cylinder_cdims[1]}
-		     ${cylinder_cdims[2]}"/>
+	  <box size="${piston_cdims[0]}
+		     ${piston_cdims[1]}
+		     ${piston_cdims[2]}"/>
         </geometry>
       </collision>
@@ -143,9 +143,9 @@
       <material>Gazebo/FlatBlack</material>
     </gazebo>
-    <gazebo reference="${prefix}cylinder">
+    <gazebo reference="${prefix}piston">
       <material>Gazebo/Grey</material>
     </gazebo>
     <!-- Improve grasping physics -->
-    <gazebo reference="${prefix}cylinder">
+    <gazebo reference="${prefix}piston">
       <kp>1000000.0</kp>
       <kd>1.0</kd>

File: moveit_config/aist_moveit_config/config/gazebo_aist_base_scene.urdf (robot description, URDF)
Before this commit: robot aist_base_scene, 116 links, 115 joints
Links:
- added link base_fixture_base_link, mass 0.86387; collision box size=0.049 0.058 0.026; visual mesh filename=package://aist_fastening_tools/meshes/visual/MGPM12-20Z_bod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 scale=0.001 0.001 0.001
- added link base_fixture_piston, mass 0.03804; collision box size=0.007 0.056 0.022; visual mesh filename=package://aist_fastening_tools/meshes/visual/MGPM12-20Z_pis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 scale=0.001 0.001 0.001
- added link base_fixture_tip_link
- added link screw_feeder_m3_base_link, mass 1.0; collision box size=0.126 0.126 0.147; visual box size=0.126 0.126 0.147
- added link screw_feeder_m3_front_side, mass 1.0; collision box size=0.056 0.126 0.079; visual box size=0.056 0.126 0.079
- added link screw_feeder_m3_gap, mass 1.0; collision box size=0.056 0.02 0.002; visual box size=0.056 0.02 0.002
- added link screw_feeder_m3_inlet_link
- added link screw_feeder_m3_outlet_link
- added link screw_feeder_m4_base_link, mass 1.0; collision box size=0.126 0.126 0.147; visual box size=0.126 0.126 0.147
- added link screw_feeder_m4_front_side, mass 1.0; collision box size=0.056 0.126 0.079; visual box size=0.056 0.126 0.079
- added link screw_feeder_m4_gap, mass 1.0; collision box size=0.056 0.02 0.002; visual box size=0.056 0.02 0.002
- added link screw_feeder_m4_inlet_link
- added link screw_feeder_m4_outlet_link
- added link workbench_back_bar, mass 1.0; collision box size=0.48 0.02 0.02; visual box size=0.48 0.02 0.02
- added link workbench_base_link, mass 1.0; collision box size=0.48 0.02 0.02; visual box size=0.48 0.02 0.02
- added link workbench_center_bar, mass 1.0; collision box size=0.02 0.28 0.02; visual box size=0.02 0.28 0.02
- added link workbench_front_border, mass 1.0; collision box size=0.08 0.016 0.003; visual box size=0.08 0.016 0.003
- added link workbench_holder_link
- added link workbench_right_bar, mass 1.0; collision box size=0.02 0.28 0.02; visual box size=0.02 0.28 0.02
- added link workbench_right_border, mass 1.0; collision box size=0.016 0.064 0.003; visual box size=0.016 0.064 0.003
- added link workbench_table_base_link, mass 1.0; collision box size=0.02 0.02 0.125; visual box size=0.02 0.02 0.125
- added link workbench_table_leg1, mass 1.0; collision box size=0.02 0.02 0.125; visual box size=0.02 0.02 0.125
- added link workbench_table_leg2, mass 1.0; collision box size=0.02 0.02 0.125; visual box size=0.02 0.02 0.125
- added link workbench_table_leg3, mass 1.0; collision box size=0.02 0.02 0.125; visual box size=0.02 0.02 0.125
- added link workbench_table_top, mass 1.0; collision box size=0.21 0.32 0.005; visual box size=0.21 0.32 0.005
- added link workbench_table_top_center
- added link workbench_table_top_origin
Joints:
- added joint base_fixture_base_joint: type fixed, parent workbench_table_top_origin, child base_fixture_base_link, origin xyz=0.05729961772434791 0.24786931916155724 0 rpy=0 0 -1.0304423903774522
- added joint base_fixture_piston_joint: type prismatic, parent base_fixture_base_link, child base_fixture_piston, axis 1 0 0, limit lower=0 upper=0.02 effort=130 velocity=0.15
- added joint base_fixture_tip_link_joint: type fixed, parent base_fixture_base_link, child base_fixture_tip_link, origin xyz=0.033      0.0      0.013 rpy=0.0      0.0      0.0
- added joint screw_feeder_m3_base_link: type fixed, parent workbench_base_link, child screw_feeder_m3_base_link, origin xyz=0 0.03 0 rpy=0 0 0
- added joint screw_feeder_m3_front_side: type fixed, parent screw_feeder_m3_base_link, child screw_feeder_m3_front_side, origin xyz=0.126 0 0 rpy=0 0 0
- added joint screw_feeder_m3_gap: type fixed, parent screw_feeder_m3_front_side, child screw_feeder_m3_gap, origin xyz=0 0.053 0.079 rpy=0 0 0
- added joint screw_feeder_m3_inlet_joint: type fixed, parent screw_feeder_m3_base_link, child screw_feeder_m3_inlet_link, origin xyz=0.063 0.042 0.147 rpy=0 0 0
- added joint screw_feeder_m3_outlet_joint: type fixed, parent screw_feeder_m3_gap, child screw_feeder_m3_outlet_link, origin xyz=0.046 0.01 0.002 rpy=0 0 0
- added joint screw_feeder_m4_base_link: type fixed, parent screw_feeder_m3_base_link, child screw_feeder_m4_base_link, origin xyz=0 0.126 0 rpy=0 0 0
- added joint screw_feeder_m4_front_side: type fixed, parent screw_feeder_m4_base_link, child screw_feeder_m4_front_side, origin xyz=0.126 0 0 rpy=0 0 0
- added joint screw_feeder_m4_gap: type fixed, parent screw_feeder_m4_front_side, child screw_feeder_m4_gap, origin xyz=0 0.053 0.079 rpy=0 0 0
- added joint screw_feeder_m4_inlet_joint: type fixed, parent screw_feeder_m4_base_link, child screw_feeder_m4_inlet_link, origin xyz=0.063 0.042 0.147 rpy=0 0 0
- added joint screw_feeder_m4_outlet_joint: type fixed, parent screw_feeder_m4_gap, child screw_feeder_m4_outlet_link, origin xyz=0.046 0.01 0.002 rpy=0 0 0
- added joint workbench_back_bar: type fixed, parent workbench_base_link, child workbench_back_bar, origin xyz=0 0.3 0 rpy=0 0 0
- added joint workbench_base_link: type fixed, parent cage_workspace_bar, child workbench_base_link, origin xyz=0.04    0.63    0.01 rpy=0 0 0
- added joint workbench_center_bar: type fixed, parent workbench_base_link, child workbench_center_bar, origin xyz=0.27 0.02 0 rpy=0 0 0
- added joint workbench_front_border: type fixed, parent workbench_table_top_origin, child workbench_front_border, origin xyz=0.13 0 0 rpy=0 0 0
- added joint workbench_holder_link_joint: type fixed, parent workbench_table_top_origin, child workbench_holder_link, origin xyz=0.194 0.016 0 rpy=0 0 1.5707963267948966
- added joint workbench_right_bar: type fixed, parent workbench_base_link, child workbench_right_bar, origin xyz=0.45999999999999996 0.02 0 rpy=0 0 0
- added joint workbench_right_border: type fixed, parent workbench_table_top_origin, child workbench_right_border, origin xyz=0.194 0.016 0 rpy=0 0 0
- added joint workbench_table_base_link: type fixed, parent workbench_base_link, child workbench_table_base_link, origin xyz=0.27 0  0.02 rpy=0 0 0
- added joint workbench_table_leg1: type fixed, parent workbench_table_base_link, child workbench_table_leg1, origin xyz=0.19 0 0 rpy=0 0 0
- added joint workbench_table_leg2: type fixed, parent workbench_table_base_link, child workbench_table_leg2, origin xyz=0 0.3 0 rpy=0 0 0
- added joint workbench_table_leg3: type fixed, parent workbench_table_base_link, child workbench_table_leg3, origin xyz=0.19      0.3      0 rpy=0 0 0
- added joint workbench_table_top: type fixed, parent workbench_table_base_link, child workbench_table_top, origin xyz=0 0 0.125 rpy=0 0 0
- added joint workbench_table_top_center_joint: type fixed, parent workbench_table_top_origin, child workbench_table_top_center, origin xyz=0.105 0.16 0 rpy=0 0 0
- added joint workbench_table_top_origin_joint: type fixed, parent workbench_table_top, child workbench_table_top_origin, origin xyz=0 0 0.005 rpy=0 0 0

Commit message: Add piston_head link to base_fixtrue

File: aist_fastening_tools/urdf/base_fixture.urdf.xacro (robot description, xacro)
@@ -11,7 +11,4 @@
 		      value="${properties['primitives']}"
 		      scope="parent"/>
-      <!-- <xacro:property name="collision_meshes" -->
-      <!-- 		      value="${properties['collision_meshes']}" -->
-      <!-- 		      scope="parent"/> -->
       <xacro:property name="subframes"
 		      value="${properties['subframes']}"
@@ -24,5 +21,5 @@
 				     )/config/fastening_tools_properties.yaml"/>
     <xacro:property name="stroke"	value="0.020"/>
-    <!-- body -->
+    <!-- Body -->
     <xacro:property name="body_vorigin"	value="${visual_meshes[0]['pose']}"/>
     <xacro:property name="body_vscale"	value="${visual_meshes[0]['scale']}"/>
@@ -70,5 +67,5 @@
       </inertial>
     </link>
-    <!-- piston -->
+    <!-- Piston -->
     <xacro:property name="piston_vorigin"
     		    value="${visual_meshes[1]['pose']}"/>
@@ -126,5 +123,5 @@
       </inertial>
     </link>
-    <!-- tip -->
+    <!-- Tip -->
     <xacro:property name="tip_link_origin"
 		    value="${subframes['tip_link']}"/>
@@ -140,4 +137,18 @@
     </joint>
     <link name="${prefix}tip_link"/>
+    <!-- Piston head -->
+    <xacro:property name="piston_head_origin"
+		    value="${subframes['piston_head']}"/>
+    <joint name="${prefix}piston_head_joint" type="fixed">
+      <parent link="${prefix}piston"/>
+      <child  link="${prefix}piston_head"/>
+      <origin xyz="${piston_head_origin[0]}
+		   ${piston_head_origin[1]}
+		   ${piston_head_origin[2]}"
+	      rpy="${piston_head_origin[3]*pi/180.0}
+		   ${piston_head_origin[4]*pi/180.0}
+		   ${piston_head_origin[5]*pi/180.0}"/>
+    </joint>
+    <link name="${prefix}piston_head"/>
     <gazebo reference="${prefix}base_link">
       <material>Gazebo/FlatBlack</material>

File: aist_fastening_tools/urdf/base_fixture_transmission.xacro (robot description, xacro)
@@ -2,10 +2,10 @@
 <robot xmlns:xacro="http://ros.org/wiki/xacro">
   <xacro:macro name="base_fixture_transmission" params="prefix">
-    <transmission name="${prefix}cylinder_joint_trans">
+    <transmission name="${prefix}piston_joint_trans">
       <type>transmission_interface/SimpleTransmission</type>
-      <joint name="${prefix}cylinder_joint">
+      <joint name="${prefix}piston_joint">
         <hardwareInterface>hardware_interface/PositionJointInterface</hardwareInterface>
       </joint>
-      <actuator name="${prefix}cylinder_joint_motor">
+      <actuator name="${prefix}piston_joint_motor">
         <mechanicalReduction>1</mechanicalReduction>
       </actuator>

File: moveit_config/aist_moveit_config/config/gazebo_aist_base_scene.urdf (robot description, URDF)
Before this commit: robot aist_base_scene, 143 links, 142 joints
Links:
- added link base_fixture_piston_head
Joints:
- added joint base_fixture_piston_head_joint: type fixed, parent base_fixture_piston, child base_fixture_piston_head, origin xyz=0.013      0.0      0.013 rpy=0.0      0.0      0.0
