Commit message: Move parts descriptions to aist_object_database

File: aist_object_database/urdf/object.urdf.xacro (robot description, xacro)
@@ -1,9 +1,10 @@
 <?xml version="1.0"?>
 <robot xmlns:xacro="http://ros.org/wiki/xacro">
-  <xacro:macro name="part" params="partname prefix parent
-				   collision *origin">
+  <xacro:macro name="object" params="name prefix parent property_file
+				     collision *origin">
+    <!-- Local macros -->
     <xacro:macro name="load_properties" params="filename">
       <xacro:property name="properties"
-		      value="${xacro.load_yaml(filename)[partname]}"/>
+		      value="${xacro.load_yaml(filename)[name]}"/>
       <xacro:property name="visual_mesh"
 		      value="${properties['visual_meshes'][0]}"
@@ -83,6 +84,6 @@
       </xacro:if>
     </xacro:macro>
-    <xacro:load_properties filename="$(find aist_description
-				     )/parts/config/parts_properties.yaml"/>
+    <!-- load properties -->
+    <xacro:load_properties filename="${property_file}"/>
     <!-- visual mesh -->
     <xacro:property name="vorigin"	value="${visual_mesh['pose']}"/>
@@ -105,5 +106,5 @@
 		  scale="${vscale[0]} ${vscale[1]} ${vscale[2]}"/>
           </geometry>
-          <material name="${partname}Color">
+          <material name="${name}Color">
             <color rgba="${vcolor[0]} ${vcolor[1]} ${vcolor[2]} ${vcolor[3]}"/>
           </material>

Commit message: Move parts descriptions to aist_object_database

File: aist_object_database/urdf/object.urdf.xacro (robot description, xacro)
@@ -1,9 +1,10 @@
 <?xml version="1.0"?>
 <robot xmlns:xacro="http://ros.org/wiki/xacro">
-  <xacro:macro name="part" params="partname prefix parent
-				   collision *origin">
+  <xacro:macro name="object" params="name prefix parent properties_file
+				     collision *origin">
+    <!-- local macros -->
     <xacro:macro name="load_properties" params="filename">
       <xacro:property name="properties"
-		      value="${xacro.load_yaml(filename)[partname]}"/>
+		      value="${xacro.load_yaml(filename)[name]}"/>
       <xacro:property name="visual_mesh"
 		      value="${properties['visual_meshes'][0]}"
@@ -83,6 +84,6 @@
       </xacro:if>
     </xacro:macro>
-    <xacro:load_properties filename="$(find aist_description
-				     )/parts/config/parts_properties.yaml"/>
+    <!-- load object properties -->
+    <xacro:load_properties filename="$(arg properties_file)"/>
     <!-- visual mesh -->
     <xacro:property name="vorigin"	value="${visual_mesh['pose']}"/>
@@ -105,5 +106,5 @@
 		  scale="${vscale[0]} ${vscale[1]} ${vscale[2]}"/>
           </geometry>
-          <material name="${partname}Color">
+          <material name="${name}Color">
             <color rgba="${vcolor[0]} ${vcolor[1]} ${vcolor[2]} ${vcolor[3]}"/>
           </material>
