Commit message: Update moveit config

File: moveit_config/aist_moveit_config/config/gazebo_aist_base_scene.urdf (robot description, URDF)
Before this commit: robot aist_base_scene, 94 links, 93 joints
Links:
- added link virtual_screen
Joints:
- added joint virtual_screen_joint: type fixed, parent ground, child virtual_screen, origin xyz=0 0 0.8047 rpy=0 0 0
- joint a_phoxi_m_camera_link_joint: origin xyz=0.492856774041131 -0.036792816347522905 0.6845615969657455 rpy=-0.05809603311925469 1.097335615317803 3.053149944967766 -> xyz=0.5123515156516534 -0.03873553287518036 0.7016694751611658 rpy=-0.10603238790759253 1.1010904348550707 3.0052545162178608
- joint cage_upper_right_bar: origin xyz=1.16 0.04 1.38 rpy=0 0 0 -> xyz=1.16 0.04 1.3 rpy=0 0 0
- joint workspace_live_camera_joint: origin xyz=0.3733700748941794 -0.030741582314842072 0.720839795840623 rpy=-2.844520734424458 -0.07655721902523285 1.5144117286631504 -> xyz=0.39763658958628 -0.03830545174707677 0.8102031301665178 rpy=-2.752197931668187 -0.09513034339063342 1.5593619369146734

Commit message: Update moveit_config

File: moveit_config/aist_moveit_config/config/gazebo_aist_base_scene.urdf (robot description, URDF)
Before this commit: robot aist_base_scene, 95 links, 94 joints
Links:
- link a_bot_inside_camera_link: geometry collision box size=0.012 0.14 0.023; visual mesh filename=package://realsense2_description/meshes/sr305_without_mount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 scale=.001 .001 .001
- link a_bot_outside_camera_link: geometry collision box size=0.012 0.14 0.023; visual mesh filename=package://realsense2_description/meshes/sr305_without_mount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 scale=.001 .001 .001
Joints:
- joint a_bot_gripper_tip_link_joint: origin xyz=0.1628 0.0 0.0 rpy=0.0 0.0 0.0 -> xyz=0.1628 0.0 0.0 rpy=0.0 -1.5707963267948966 0.0
- joint a_phoxi_m_camera_link_joint: origin xyz=0.5123515156516534 -0.03873553287518036 0.7016694751611658 rpy=-0.10603238790759253 1.1010904348550707 3.0052545162178608 -> xyz=0.5129667610334572 -0.037047806454438365 0.6226614314794279 rpy=-0.06660879099232307 1.0432812514428629 3.014328066314531
- joint b_bot_gripper_tip_joint: origin xyz=0.1855 0 0 rpy=0 0 0 -> xyz=0.1855 0 0 rpy=0 -1.5707963267948966 0
- joint workspace_live_camera_joint: origin xyz=0.39763658958628 -0.03830545174707677 0.8102031301665178 rpy=-2.752197931668187 -0.09513034339063342 1.5593619369146734 -> xyz=0.405235138268645 -0.0356851775630231 0.7399153983016764 rpy=-2.6956831173735374 0.04101229395800053 1.5544348139645294

File: moveit_config/f_bot_moveit_config/config/gazebo_f_bot_base_scene.urdf (robot description, URDF)
Before this commit: robot f_bot_base_scene, 35 links, 34 joints
Links:
- removed link workbox
- added link f_bot_camera_color_frame
- added link f_bot_camera_color_optical_frame
- added link f_bot_camera_depth_frame
- added link f_bot_camera_depth_optical_frame
- added link f_bot_camera_infra1_frame
- added link f_bot_camera_infra1_optical_frame
- added link f_bot_camera_infra2_frame
- added link f_bot_camera_infra2_optical_frame
- added link mounter_table_leg0, mass 1.0; collision box size=0.05 0.05 0.86; visual box size=0.05 0.05 0.86
- added link mounter_table_leg1, mass 1.0; collision box size=0.05 0.05 0.86; visual box size=0.05 0.05 0.86
- added link mounter_table_leg2, mass 1.0; collision box size=0.05 0.05 0.86; visual box size=0.05 0.05 0.86
- added link mounter_table_leg3, mass 1.0; collision box size=0.05 0.05 0.86; visual box size=0.05 0.05 0.86
- added link mounter_table_top, mass 1.0; collision box size=0.2 0.2 0.02; visual box size=0.2 0.2 0.02
- added link mounter_table_top_origin
- added link mounter_table_top_origin_center
- added link worksapce_table_leg0, mass 1.0; collision box size=0.05 0.05 0.6849999999999999; visual box size=0.05 0.05 0.6849999999999999
- added link worksapce_table_leg1, mass 1.0; collision box size=0.05 0.05 0.6849999999999999; visual box size=0.05 0.05 0.6849999999999999
- added link worksapce_table_leg2, mass 1.0; collision box size=0.05 0.05 0.6849999999999999; visual box size=0.05 0.05 0.6849999999999999
- added link worksapce_table_leg3, mass 1.0; collision box size=0.05 0.05 0.6849999999999999; visual box size=0.05 0.05 0.6849999999999999
- added link worksapce_table_top, mass 1.0; collision box size=1.8 1.0 0.02; visual box size=1.8 1.0 0.02
- added link worksapce_table_top_origin
- added link worksapce_table_top_origin_center
Joints:
- removed joint workbox
- added joint f_bot_camera_color_joint: type fixed, parent f_bot_camera_link, child f_bot_camera_color_frame, origin xyz=0 0.015 0 rpy=0 0 0
- added joint f_bot_camera_color_optical_joint: type fixed, parent f_bot_camera_color_frame, child f_bot_camera_color_optical_frame, origin xyz=0 0 0 rpy=-1.5707963267948966 0 -1.5707963267948966
- added joint f_bot_camera_depth_joint: type fixed, parent f_bot_camera_link, child f_bot_camera_depth_frame, origin xyz=0 0 0 rpy=0 0 0
- added joint f_bot_camera_depth_optical_joint: type fixed, parent f_bot_camera_depth_frame, child f_bot_camera_depth_optical_frame, origin xyz=0 0 0 rpy=-1.5707963267948966 0 -1.5707963267948966
- added joint f_bot_camera_infra1_joint: type fixed, parent f_bot_camera_link, child f_bot_camera_infra1_frame, origin xyz=0 0.0 0 rpy=0 0 0
- added joint f_bot_camera_infra1_optical_joint: type fixed, parent f_bot_camera_infra1_frame, child f_bot_camera_infra1_optical_frame, origin xyz=0 0 0 rpy=-1.5707963267948966 0 -1.5707963267948966
- added joint f_bot_camera_infra2_joint: type fixed, parent f_bot_camera_link, child f_bot_camera_infra2_frame, origin xyz=0 -0.05 0 rpy=0 0 0
- added joint f_bot_camera_infra2_optical_joint: type fixed, parent f_bot_camera_infra2_frame, child f_bot_camera_infra2_optical_frame, origin xyz=0 0 0 rpy=-1.5707963267948966 0 -1.5707963267948966
- added joint mounter_table_leg0: type fixed, parent ground, child mounter_table_leg0, origin xyz=-0.1 -0.71 0 rpy=0 0 0
- added joint mounter_table_leg1: type fixed, parent mounter_table_leg0, child mounter_table_leg1, origin xyz=0.15000000000000002 0 0 rpy=0 0 0
- added joint mounter_table_leg2: type fixed, parent mounter_table_leg0, child mounter_table_leg2, origin xyz=0 0.15000000000000002 0 rpy=0 0 0
- added joint mounter_table_leg3: type fixed, parent mounter_table_leg0, child mounter_table_leg3, origin xyz=0.15000000000000002      0.15000000000000002      0 rpy=0 0 0
- added joint mounter_table_top: type fixed, parent mounter_table_leg0, child mounter_table_top, origin xyz=0 0 0.86 rpy=0 0 0
- added joint mounter_table_top_origin: type fixed, parent mounter_table_top, child mounter_table_top_origin, origin xyz=0 0 0.02 rpy=0 0 0
- added joint mounter_table_top_origin_center: type fixed, parent mounter_table_top_origin, child mounter_table_top_origin_center, origin xyz=0.1 0.1 0 rpy=0 0 0
- added joint worksapce_table_leg0: type fixed, parent ground, child worksapce_table_leg0, origin xyz=-0.9 -0.5 0 rpy=0 0 0
- added joint worksapce_table_leg1: type fixed, parent worksapce_table_leg0, child worksapce_table_leg1, origin xyz=1.75 0 0 rpy=0 0 0
- added joint worksapce_table_leg2: type fixed, parent worksapce_table_leg0, child worksapce_table_leg2, origin xyz=0 0.95 0 rpy=0 0 0
- added joint worksapce_table_leg3: type fixed, parent worksapce_table_leg0, child worksapce_table_leg3, origin xyz=1.75      0.95      0 rpy=0 0 0
- added joint worksapce_table_top: type fixed, parent worksapce_table_leg0, child worksapce_table_top, origin xyz=0 0 0.6849999999999999 rpy=0 0 0
- added joint worksapce_table_top_origin: type fixed, parent worksapce_table_top, child worksapce_table_top_origin, origin xyz=0 0 0.02 rpy=0 0 0
- added joint worksapce_table_top_origin_center: type fixed, parent worksapce_table_top_origin, child worksapce_table_top_origin_center, origin xyz=0.9 0.5 0 rpy=0 0 0
- joint f_bot_camera_joint: origin xyz=0.030 0.000 0.043 rpy=0 0.0 0 -> xyz=0.026 0.0 0.0595 rpy=0.0 0.0 0.0
- joint f_bot_gripper_tip_link_joint: origin xyz=.2328 0.0 0.0 rpy=0.0 0.0 0.0 -> xyz=.2328 0.0 0.0 rpy=0.0 -1.5707963267948966 0.0
- joint ground_f_bot_joint: origin xyz=0 -0.4875 0.77 rpy=0 0 0 -> xyz=0 -0.61 0.88 rpy=0 0 0
- joint ground_to_workspace: origin xyz=0 0 0.77 rpy=0 0 0 -> xyz=0 0 0.705 rpy=0 0 0

Commit message: Update moveit_config

File: moveit_config/aist_moveit_config/config/gazebo_aist_base_scene.urdf (robot description, URDF)
Before this commit: robot aist_base_scene, 95 links, 94 joints
Links:
- removed link a_bot_camera_mount
- removed link a_bot_inside_camera_color_frame
- removed link a_bot_inside_camera_color_optical_frame
- removed link a_bot_inside_camera_connector_link
- removed link a_bot_inside_camera_depth_frame
- removed link a_bot_inside_camera_depth_optical_frame
- removed link a_bot_inside_camera_left_ir_frame
- removed link a_bot_inside_camera_left_ir_optical_frame
- removed link a_bot_inside_camera_link
- removed link a_bot_inside_camera_right_ir_frame
- removed link a_bot_inside_camera_right_ir_optical_frame
- removed link a_bot_outside_camera_color_frame
- removed link a_bot_outside_camera_color_optical_frame
- removed link a_bot_outside_camera_connector_link
- removed link a_bot_outside_camera_depth_frame
- removed link a_bot_outside_camera_depth_optical_frame
- removed link a_bot_outside_camera_left_ir_frame
- removed link a_bot_outside_camera_left_ir_optical_frame
- removed link a_bot_outside_camera_link
- removed link a_bot_outside_camera_right_ir_frame
- removed link a_bot_outside_camera_right_ir_optical_frame
- added link a_bot_zivid_base_link, mass 0.3; collision mesh filename=package://aist_description/devices/meshes/collision/zivid2p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 scale=0.001 0.001 0.001; visual mesh filename=package://aist_description/devices/meshes/zivid2plus.stl scale=0.001 0.001 0.001
- added link a_bot_zivid_coupling_base_link, mass 0.3; collision cylinder length=0.015 radius=0.0375; visual cylinder length=0.015 radius=0.0375
- added link a_bot_zivid_coupling_flange_link
- added link a_bot_zivid_projector
- added link a_bot_zivid_reference
- added link a_bot_zivid_sensor
- link a_bot_gripper_left_inner_finger: geometry collision mesh filename=package://aist_robotiq/meshes/collision/robotiq_arg2f_140_i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; visual mesh filename=package://aist_robotiq/meshes/visual/robotiq_arg2f_140_inne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
- link a_bot_gripper_left_inner_finger_pad: geometry collision box size=0.03 0.07 0.0075; visual box size=0.027 0.065 0.0075
- link a_bot_gripper_left_inner_knuckle: geometry collision mesh filename=package://aist_robotiq/meshes/collision/robotiq_arg2f_140_i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; visual mesh filename=package://aist_robotiq/meshes/visual/robotiq_arg2f_140_inne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
- link a_bot_gripper_left_outer_finger: geometry collision mesh filename=package://aist_robotiq/meshes/collision/robotiq_arg2f_140_o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; visual mesh filename=package://aist_robotiq/meshes/visual/robotiq_arg2f_140_oute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
- link a_bot_gripper_left_outer_knuckle: geometry collision mesh filename=package://aist_robotiq/meshes/collision/robotiq_arg2f_140_o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; visual mesh filename=package://aist_robotiq/meshes/visual/robotiq_arg2f_140_oute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
- link a_bot_gripper_right_inner_finger: geometry collision mesh filename=package://aist_robotiq/meshes/collision/robotiq_arg2f_140_i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; visual mesh filename=package://aist_robotiq/meshes/visual/robotiq_arg2f_140_inne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
- link a_bot_gripper_right_inner_finger_pad: geometry collision box size=0.03 0.07 0.0075; visual box size=0.027 0.065 0.0075
- link a_bot_gripper_right_inner_knuckle: geometry collision mesh filename=package://aist_robotiq/meshes/collision/robotiq_arg2f_140_i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; visual mesh filename=package://aist_robotiq/meshes/visual/robotiq_arg2f_140_inne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
- link a_bot_gripper_right_outer_finger: geometry collision mesh filename=package://aist_robotiq/meshes/collision/robotiq_arg2f_140_o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; visual mesh filename=package://aist_robotiq/meshes/visual/robotiq_arg2f_140_oute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
- link a_bot_gripper_right_outer_knuckle: geometry collision mesh filename=package://aist_robotiq/meshes/collision/robotiq_arg2f_140_o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; visual mesh filename=package://aist_robotiq/meshes/visual/robotiq_arg2f_140_oute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
Joints:
- removed joint a_bot_camera_mount_joint
- removed joint a_bot_inside_camera_color_joint
- removed joint a_bot_inside_camera_color_optical_joint
- removed joint a_bot_inside_camera_depth_joint
- removed joint a_bot_inside_camera_depth_optical_joint
- removed joint a_bot_inside_camera_joint
- removed joint a_bot_inside_camera_left_ir_joint
- removed joint a_bot_inside_camera_left_ir_optical_joint
- removed joint a_bot_inside_camera_link_joint
- removed joint a_bot_inside_camera_right_ir_joint
- removed joint a_bot_inside_camera_right_ir_optical_joint
- removed joint a_bot_outside_camera_color_joint
- removed joint a_bot_outside_camera_color_optical_joint
- removed joint a_bot_outside_camera_depth_joint
- removed joint a_bot_outside_camera_depth_optical_joint
- removed joint a_bot_outside_camera_joint
- removed joint a_bot_outside_camera_left_ir_joint
- removed joint a_bot_outside_camera_left_ir_optical_joint
- removed joint a_bot_outside_camera_link_joint
- removed joint a_bot_outside_camera_right_ir_joint
- removed joint a_bot_outside_camera_right_ir_optical_joint
- added joint a_bot_zivid_base_joint: type fixed, parent a_bot_zivid_coupling_flange_link, child a_bot_zivid_base_link, origin xyz=0.01 0.0 0.065 rpy=0.0 0.268 0.0
- added joint a_bot_zivid_coupling_base_joint: type fixed, parent a_bot_flange, child a_bot_zivid_coupling_base_link, origin xyz=0 0 0 rpy=3.141592653589793 0 0
- added joint a_bot_zivid_coupling_flange_joint: type fixed, parent a_bot_zivid_coupling_base_link, child a_bot_zivid_coupling_flange_link, origin xyz=0.015 0 0 rpy=0 0 0
- added joint a_bot_zivid_projector_joint: type fixed, parent a_bot_zivid_base_link, child a_bot_zivid_projector, origin xyz=0 -0.05702 0.0295 rpy=0 0 0.04363323129985824
- added joint a_bot_zivid_reference_joint: type fixed, parent a_bot_zivid_base_link, child a_bot_zivid_reference, origin xyz=0 0.05702 0.0295 rpy=0 0 -0.04363323129985824
- added joint a_bot_zivid_sensor_joint: type fixed, parent a_bot_zivid_reference, child a_bot_zivid_sensor, origin xyz=0 0 0 rpy=-1.5707963267948966 0 -1.5707963267948966
- joint a_bot_ftsensor_ft300_joint: origin xyz=0 0 0 rpy=3.141592653589793 0 0 -> xyz=0 0 0 rpy=0 0 0; parent a_bot_flange -> a_bot_zivid_coupling_flange_link
- joint a_bot_gripper_finger_joint: axis 1 0 0 -> -1 0 0; limit lower=0 upper=0.81 effort=1000 velocity=2.0 -> lower=0 upper=0.7 effort=1000 velocity=2.0; origin xyz=0 -0.0306011 0.054904 rpy=0 0 3.141592653589793 -> xyz=0 -0.030601 0.054905 rpy=2.2957963267948966 0 0
- joint a_bot_gripper_left_inner_finger_joint: axis 1 0 0 -> -1 0 0; origin xyz=0 0.0061 0.0471 rpy=0 0 0 -> xyz=0 0.0817554015893473 -0.0282203446692936 rpy=-0.725 0 0
- joint a_bot_gripper_left_inner_finger_pad_joint: origin xyz=0 -0.0220203446692936 0.03242 rpy=0 0 0 -> xyz=0 0.0457554015893473 -0.0272203446692936 rpy=0 0 0
- joint a_bot_gripper_left_inner_knuckle_joint: axis 1 0 0 -> -1 0 0; origin xyz=0 -0.0127 0.06142 rpy=0 0 3.141592653589793 -> xyz=0 -0.0127 0.06142 rpy=2.2957963267948966 0 0.0
- joint a_bot_gripper_left_outer_finger_joint: origin xyz=0 0.0315 -0.0041 rpy=0 0 0 -> xyz=0 0.01821998610742 0.0260018192872234 rpy=0 0 0
- joint a_bot_gripper_right_inner_finger_joint: axis 1 0 0 -> -1 0 0; origin xyz=0 0.0061 0.0471 rpy=0 0 0 -> xyz=0 0.0817554015893473 -0.0282203446692936 rpy=-0.725 0 0
- joint a_bot_gripper_right_inner_finger_pad_joint: origin xyz=0 -0.0220203446692936 0.03242 rpy=0 0 0 -> xyz=0 0.0457554015893473 -0.0272203446692936 rpy=0 0 0
- joint a_bot_gripper_right_inner_knuckle_joint: axis 1 0 0 -> -1 0 0; origin xyz=0 0.0127 0.06142 rpy=0 0 0.0 -> xyz=0 0.0127 0.06142 rpy=2.2957963267948966 0 -3.141592653589793
- joint a_bot_gripper_right_outer_finger_joint: origin xyz=0 0.0315 -0.0041 rpy=0 0 0 -> xyz=0 0.01821998610742 0.0260018192872234 rpy=0 0 0
- joint a_bot_gripper_right_outer_knuckle_joint: axis 1 0 0 -> -1 0 0; limit lower=-0.81 upper=0.81 effort=1000 velocity=2.0 -> lower=-0.725 upper=0.725 effort=1000 velocity=2.0; origin xyz=0 0.0306011 0.054904 rpy=0 0 0 -> xyz=0 0.030601 0.054905 rpy=2.2957963267948966 0 3.141592653589793
- joint a_bot_gripper_tip_link_joint: origin xyz=0.1628 0.0 0.0 rpy=0.0 -1.5707963267948966 0.0 -> xyz=.2328 0.0 0.0 rpy=0.0 -1.5707963267948966 0.0
- joint a_motioncam_link_joint: origin xyz=0.5231407296015458 -0.10503553573534424 0.6365724301868348 rpy=0.03174526251084231 1.041717094258447 -3.1268222045220364 -> xyz=0.5250340162175878 -0.10043474330440638 0.659948826203397 rpy=0.055276438915859344 1.0603529787148211 -3.09644910582365
- joint virtual_screen_joint: origin xyz=0 0 0.8047 rpy=0 0 0 -> xyz=0 0 0.81 rpy=0 0 0

Commit message: Update moveit_config

File: moveit_config/aist_moveit_config/config/gazebo_aist_base_scene.urdf (robot description, URDF)
Before this commit: robot aist_base_scene, 80 links, 79 joints
Links:
- added link screw_tool_m3_holder_base_link, mass 0.1; collision mesh filename=package://aist_description/objects/meshes/screw_tool_holder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 scale=0.001 0.001 0.001; visual mesh filename=package://aist_description/objects/meshes/screw_tool_holder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 scale=0.001 0.001 0.001
- added link screw_tool_m3_holder_link
- added link screw_tool_m4_holder_base_link, mass 0.1; collision mesh filename=package://aist_description/objects/meshes/screw_tool_holder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 scale=0.001 0.001 0.001; visual mesh filename=package://aist_description/objects/meshes/screw_tool_holder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 scale=0.001 0.001 0.001
- added link screw_tool_m4_holder_link
- link a_bot_gripper_left_inner_finger_pad: geometry collision box size=0.027 0.065 0.0075; visual box size=0.027 0.065 0.0075
- link a_bot_gripper_right_inner_finger_pad: geometry collision box size=0.027 0.065 0.0075; visual box size=0.027 0.065 0.0075
Joints:
- added joint screw_tool_m3_holder_base_joint: type fixed, parent cage_tool_bar, child screw_tool_m3_holder_base_link, origin xyz=0 0.6 0.04 rpy=0 0 0
- added joint screw_tool_m3_holder_joint: type fixed, parent screw_tool_m3_holder_base_link, child screw_tool_m3_holder_link, origin xyz=0.0525 0 0.007 rpy=0 0 0
- added joint screw_tool_m4_holder_base_joint: type fixed, parent cage_tool_bar, child screw_tool_m4_holder_base_link, origin xyz=0 0.8 0.04 rpy=0 0 0
- added joint screw_tool_m4_holder_joint: type fixed, parent screw_tool_m4_holder_base_link, child screw_tool_m4_holder_link, origin xyz=0.0525 0 0.007 rpy=0 0 0
- joint a_bot_zivid_base_joint: origin xyz=0.01 0.0 0.065 rpy=0.0 0.268 0.0 -> xyz=-0.008354917812276319 0.0008954602737317324 0.0667453856043816 rpy=-0.0017467829187330236 0.27937676735622796 -0.006819626383816405
- joint b_bot_ftsensor_ft300_joint: origin xyz=0 0 0 rpy=3.141592653589793 0 0 -> xyz=0 0 0 rpy=0 0 0
- joint b_bot_gripper_base_joint: origin xyz=0 0 0 rpy=0 0.012217304763960306 -0.0017453292519943296 -> xyz=0 0 0 rpy=0 -0.017453292519943295 -0.005235987755982988

Commit message: Update aist_moveit_config

File: moveit_config/aist_moveit_config/config/gazebo_aist_base_scene.urdf (robot description, URDF)
Before this commit: robot aist_base_scene, 116 links, 115 joints
Links:
- removed link workspace_table_top_origin_center
- added link workspace_table_top_center
Joints:
- removed joint workspace_table_top_origin
- removed joint workspace_table_top_origin_center
- added joint workspace_table_top_center_joint: type fixed, parent workspace_table_top_origin, child workspace_table_top_center, origin xyz=0.45 0.9 0 rpy=0 0 0
- added joint workspace_table_top_origin_joint: type fixed, parent workspace_table_top, child workspace_table_top_origin, origin xyz=0 0 0.02 rpy=0 0 0
