Commit message: Update moveit_config

File: moveit_config/aist_moveit_config/config/gazebo_aist_base_scene.urdf (robot description, URDF)
Before this commit: robot aist_base_scene, 144 links, 143 joints
Links:
- removed link a_bot_camera_mount
- removed link a_bot_inside_camera_color_frame
- removed link a_bot_inside_camera_color_optical_frame
- removed link a_bot_inside_camera_connector_link
- removed link a_bot_inside_camera_depth_frame
- removed link a_bot_inside_camera_depth_optical_frame
- removed link a_bot_inside_camera_left_ir_frame
- removed link a_bot_inside_camera_left_ir_optical_frame
- removed link a_bot_inside_camera_link
- removed link a_bot_inside_camera_right_ir_frame
- removed link a_bot_inside_camera_right_ir_optical_frame
- removed link a_bot_outside_camera_color_frame
- removed link a_bot_outside_camera_color_optical_frame
- removed link a_bot_outside_camera_connector_link
- removed link a_bot_outside_camera_depth_frame
- removed link a_bot_outside_camera_depth_optical_frame
- removed link a_bot_outside_camera_left_ir_frame
- removed link a_bot_outside_camera_left_ir_optical_frame
- removed link a_bot_outside_camera_link
- removed link a_bot_outside_camera_right_ir_frame
- removed link a_bot_outside_camera_right_ir_optical_frame
- added link b_bot_camera_color_frame
- added link b_bot_camera_color_optical_frame
- added link b_bot_camera_connector_link
- added link b_bot_camera_depth_frame
- added link b_bot_camera_depth_optical_frame
- added link b_bot_camera_left_ir_frame
- added link b_bot_camera_left_ir_optical_frame
- added link b_bot_camera_link, mass 0.564; collision box size=0.012 0.14 0.023; visual mesh filename=package://realsense2_description/meshes/sr305_without_mount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 scale=.001 .001 .001
- added link b_bot_camera_mount, mass 1.0; collision box size=.03 .12 .08; visual mesh filename=package://aist_description/devices/meshes/sr305_mount_2f85.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 scale=.001 .001 .001
- added link b_bot_camera_right_ir_frame
- added link b_bot_camera_right_ir_optical_frame
Joints:
- removed joint a_bot_camera_mount_joint
- removed joint a_bot_inside_camera_color_joint
- removed joint a_bot_inside_camera_color_optical_joint
- removed joint a_bot_inside_camera_depth_joint
- removed joint a_bot_inside_camera_depth_optical_joint
- removed joint a_bot_inside_camera_joint
- removed joint a_bot_inside_camera_left_ir_joint
- removed joint a_bot_inside_camera_left_ir_optical_joint
- removed joint a_bot_inside_camera_link_joint
- removed joint a_bot_inside_camera_right_ir_joint
- removed joint a_bot_inside_camera_right_ir_optical_joint
- removed joint a_bot_outside_camera_color_joint
- removed joint a_bot_outside_camera_color_optical_joint
- removed joint a_bot_outside_camera_depth_joint
- removed joint a_bot_outside_camera_depth_optical_joint
- removed joint a_bot_outside_camera_joint
- removed joint a_bot_outside_camera_left_ir_joint
- removed joint a_bot_outside_camera_left_ir_optical_joint
- removed joint a_bot_outside_camera_link_joint
- removed joint a_bot_outside_camera_right_ir_joint
- removed joint a_bot_outside_camera_right_ir_optical_joint
- added joint b_bot_camera_color_joint: type fixed, parent b_bot_camera_depth_frame, child b_bot_camera_color_frame, origin xyz=0 0.015 0 rpy=0 0 0
- added joint b_bot_camera_color_optical_joint: type fixed, parent b_bot_camera_color_frame, child b_bot_camera_color_optical_frame, origin xyz=0 0 0 rpy=-1.5707963267948966 0 -1.5707963267948966
- added joint b_bot_camera_depth_joint: type fixed, parent b_bot_camera_link, child b_bot_camera_depth_frame, origin xyz=.003721 0 0 rpy=0 0 0
- added joint b_bot_camera_depth_optical_joint: type fixed, parent b_bot_camera_depth_frame, child b_bot_camera_depth_optical_frame, origin xyz=0 0 0 rpy=-1.5707963267948966 0 -1.5707963267948966
- added joint b_bot_camera_joint: type fixed, parent b_bot_gripper_base_link, child b_bot_camera_connector_link, origin xyz=0.0051834717267641005      0.0029869415393767723      0.06398615295764885 rpy=0.02104566011309687      0.3968034960518725      0.01313899562905875
- added joint b_bot_camera_left_ir_joint: type fixed, parent b_bot_camera_depth_frame, child b_bot_camera_left_ir_frame, origin xyz=0 0.0 0 rpy=0 0 0
- added joint b_bot_camera_left_ir_optical_joint: type fixed, parent b_bot_camera_left_ir_frame, child b_bot_camera_left_ir_optical_frame, origin xyz=0 0 0 rpy=-1.5707963267948966 0 -1.5707963267948966
- added joint b_bot_camera_link_joint: type fixed, parent b_bot_camera_connector_link, child b_bot_camera_link, origin xyz=0 0 0 rpy=0 0 0
- added joint b_bot_camera_mount_joint: type fixed, parent b_bot_gripper_base_link, child b_bot_camera_mount, origin xyz=0.035 0.0 0.025 rpy=0 0 0
- added joint b_bot_camera_right_ir_joint: type fixed, parent b_bot_camera_depth_frame, child b_bot_camera_right_ir_frame, origin xyz=0 0.04 0 rpy=0 0 0
- added joint b_bot_camera_right_ir_optical_joint: type fixed, parent b_bot_camera_right_ir_frame, child b_bot_camera_right_ir_optical_frame, origin xyz=0 0 0 rpy=-1.5707963267948966 0 -1.5707963267948966
- joint suction_tool_holder_joint: origin xyz=0.050 0 0.007 rpy=0 0 0 -> xyz=0.08732 0.0 -0.002 rpy=0 0.5235987755982988 0

Commit message: Update moveit_config

File: moveit_config/aist_moveit_config/config/gazebo_aist_base_scene.urdf (robot description, URDF)
Before this commit: robot aist_base_scene, 134 links, 133 joints
Links:
- added link a_bot_camera_color_frame
- added link a_bot_camera_color_optical_frame
- added link a_bot_camera_connector_link
- added link a_bot_camera_depth_frame
- added link a_bot_camera_depth_optical_frame
- added link a_bot_camera_left_ir_frame
- added link a_bot_camera_left_ir_optical_frame
- added link a_bot_camera_link, mass 0.564; collision box size=0.012 0.14 0.023; visual mesh filename=package://realsense2_description/meshes/sr305_without_mount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 scale=.001 .001 .001
- added link a_bot_camera_mount, mass 1.0; collision box size=.03 .12 .08; visual mesh filename=package://aist_description/devices/meshes/sr305_mount_2f140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 scale=.001 .001 .001
- added link a_bot_camera_right_ir_frame
- added link a_bot_camera_right_ir_optical_frame
Joints:
- added joint a_bot_camera_color_joint: type fixed, parent a_bot_camera_depth_frame, child a_bot_camera_color_frame, origin xyz=0 0.015 0 rpy=0 0 0
- added joint a_bot_camera_color_optical_joint: type fixed, parent a_bot_camera_color_frame, child a_bot_camera_color_optical_frame, origin xyz=0 0 0 rpy=-1.5707963267948966 0 -1.5707963267948966
- added joint a_bot_camera_depth_joint: type fixed, parent a_bot_camera_link, child a_bot_camera_depth_frame, origin xyz=.003721 0 0 rpy=0 0 0
- added joint a_bot_camera_depth_optical_joint: type fixed, parent a_bot_camera_depth_frame, child a_bot_camera_depth_optical_frame, origin xyz=0 0 0 rpy=-1.5707963267948966 0 -1.5707963267948966
- added joint a_bot_camera_joint: type fixed, parent a_bot_gripper_base_link, child a_bot_camera_connector_link, origin xyz=0.026      0.0      0.0595 rpy=0.0      0.3491      0.0
- added joint a_bot_camera_left_ir_joint: type fixed, parent a_bot_camera_depth_frame, child a_bot_camera_left_ir_frame, origin xyz=0 0.0 0 rpy=0 0 0
- added joint a_bot_camera_left_ir_optical_joint: type fixed, parent a_bot_camera_left_ir_frame, child a_bot_camera_left_ir_optical_frame, origin xyz=0 0 0 rpy=-1.5707963267948966 0 -1.5707963267948966
- added joint a_bot_camera_link_joint: type fixed, parent a_bot_camera_connector_link, child a_bot_camera_link, origin xyz=0 0 0 rpy=0 0 0
- added joint a_bot_camera_mount_joint: type fixed, parent a_bot_gripper_base_link, child a_bot_camera_mount, origin xyz=0.035 0.0 0.025 rpy=0 0 0
- added joint a_bot_camera_right_ir_joint: type fixed, parent a_bot_camera_depth_frame, child a_bot_camera_right_ir_frame, origin xyz=0 0.04 0 rpy=0 0 0
- added joint a_bot_camera_right_ir_optical_joint: type fixed, parent a_bot_camera_right_ir_frame, child a_bot_camera_right_ir_optical_frame, origin xyz=0 0 0 rpy=-1.5707963267948966 0 -1.5707963267948966
- joint b_bot_camera_joint: origin xyz=0.0051834717267641005      0.0029869415393767723      0.06398615295764885 rpy=0.02104566011309687      0.3968034960518725      0.01313899562905875 -> xyz=0.026      0.0      0.0595 rpy=0.0      0.3491      0.0
- joint screw_feeder_m3_base_link: origin xyz=0 0.03 0 rpy=0 0 0 -> xyz=0.01 0.03 0 rpy=0 0 0
- joint screw_feeder_m3_inlet_joint: origin xyz=0.063 0.042 0.147 rpy=0 0 0 -> xyz=0.072 0.032 0.147 rpy=0 0 0
- joint screw_feeder_m4_inlet_joint: origin xyz=0.063 0.042 0.147 rpy=0 0 0 -> xyz=0.072 0.032 0.147 rpy=0 0 0
