Commit message: Update aist_moveit_config

File: moveit_config/aist_moveit_config/config/gazebo_aist_base_scene.urdf (robot description, URDF)
Before this commit: robot aist_base_scene, 139 links, 138 joints
Links:
- removed link base_fixture_base_link
- removed link base_fixture_piston
- removed link base_fixture_piston_head
- removed link base_fixture_tip_link
- removed link screw_feeder_m3_base_link
- removed link screw_feeder_m3_front_side
- removed link screw_feeder_m3_gap
- removed link screw_feeder_m3_inlet_link
- removed link screw_feeder_m3_outlet_link
- removed link screw_feeder_m4_base_link
- removed link screw_feeder_m4_front_side
- removed link screw_feeder_m4_gap
- removed link screw_feeder_m4_inlet_link
- removed link screw_feeder_m4_outlet_link
- removed link workbench_back_bar
- removed link workbench_base_link
- removed link workbench_center_bar
- removed link workbench_front_border
- removed link workbench_holder_link
- removed link workbench_right_bar
- removed link workbench_right_border
- removed link workbench_table_base_link
- removed link workbench_table_leg1
- removed link workbench_table_leg2
- removed link workbench_table_leg3
- removed link workbench_table_top
- removed link workbench_table_top_center
- removed link workbench_table_top_origin
- added link bin_1_part_16, mass 1.0; collision mesh filename=package://aist_description/wrc/meshes/bin1_EA661CA-11.vhacd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 scale=0.001 0.001 0.001; visual mesh filename=package://aist_description/wrc/meshes/bin1_EA661CA-11.stl scale=0.001 0.001 0.001
- added link bin_1_part_16_bottom_back_left_corner
- added link bin_1_part_16_bottom_back_right_corner
- added link bin_1_part_16_bottom_front_left_corner
- added link bin_1_part_16_bottom_front_right_corner
- added link bin_1_part_16_top_back_left_corner
- added link bin_1_part_16_top_back_right_corner
- added link bin_1_part_16_top_front_left_corner
- added link bin_1_part_16_top_front_right_corner
- added link bin_1_part_17, mass 1.0; collision mesh filename=package://aist_description/wrc/meshes/bin1_EA661CA-11.vhacd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 scale=0.001 0.001 0.001; visual mesh filename=package://aist_description/wrc/meshes/bin1_EA661CA-11.stl scale=0.001 0.001 0.001
- added link bin_1_part_17_bottom_back_left_corner
- added link bin_1_part_17_bottom_back_right_corner
- added link bin_1_part_17_bottom_front_left_corner
- added link bin_1_part_17_bottom_front_right_corner
- added link bin_1_part_17_top_back_left_corner
- added link bin_1_part_17_top_back_right_corner
- added link bin_1_part_17_top_front_left_corner
- added link bin_1_part_17_top_front_right_corner
- added link bin_1_part_5, mass 1.0; collision mesh filename=package://aist_description/wrc/meshes/bin1_EA661CA-11.vhacd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 scale=0.001 0.001 0.001; visual mesh filename=package://aist_description/wrc/meshes/bin1_EA661CA-11.stl scale=0.001 0.001 0.001
- added link bin_1_part_5_bottom_back_left_corner
- added link bin_1_part_5_bottom_back_right_corner
- added link bin_1_part_5_bottom_front_left_corner
- added link bin_1_part_5_bottom_front_right_corner
- added link bin_1_part_5_top_back_left_corner
- added link bin_1_part_5_top_back_right_corner
- added link bin_1_part_5_top_front_left_corner
- added link bin_1_part_5_top_front_right_corner
- added link bin_2_part_4, mass 1.0; collision mesh filename=package://aist_description/wrc/meshes/bin2_SK-HL1-BL.vhacd.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 scale=0.001 0.001 0.001; visual mesh filename=package://aist_description/wrc/meshes/bin2_SK-HL1-BL.stl scale=0.001 0.001 0.001
- added link bin_2_part_4_bottom_back_left_corner
- added link bin_2_part_4_bottom_back_right_corner
- added link bin_2_part_4_bottom_front_left_corner
- added link bin_2_part_4_bottom_front_right_corner
- added link bin_2_part_4_top_back_left_corner
- added link bin_2_part_4_top_back_right_corner
- added link bin_2_part_4_top_front_left_corner
- added link bin_2_part_4_top_front_right_corner
- added link bin_2_part_7, mass 1.0; collision mesh filename=package://aist_description/wrc/meshes/bin2_SK-HL1-BL.vhacd.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 scale=0.001 0.001 0.001; visual mesh filename=package://aist_description/wrc/meshes/bin2_SK-HL1-BL.stl scale=0.001 0.001 0.001
- added link bin_2_part_7_bottom_back_left_corner
- added link bin_2_part_7_bottom_back_right_corner
- added link bin_2_part_7_bottom_front_left_corner
- added link bin_2_part_7_bottom_front_right_corner
- added link bin_2_part_7_top_back_left_corner
- added link bin_2_part_7_top_back_right_corner
- added link bin_2_part_7_top_front_left_corner
- added link bin_2_part_7_top_front_right_corner
- added link bin_2_part_8, mass 1.0; collision mesh filename=package://aist_description/wrc/meshes/bin2_SK-HL1-BL.vhacd.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 scale=0.001 0.001 0.001; visual mesh filename=package://aist_description/wrc/meshes/bin2_SK-HL1-BL.stl scale=0.001 0.001 0.001
- added link bin_2_part_8_bottom_back_left_corner
- added link bin_2_part_8_bottom_back_right_corner
- added link bin_2_part_8_bottom_front_left_corner
- added link bin_2_part_8_bottom_front_right_corner
- added link bin_2_part_8_top_back_left_corner
- added link bin_2_part_8_top_back_right_corner
- added link bin_2_part_8_top_front_left_corner
- added link bin_2_part_8_top_front_right_corner
- added link plate, mass 1.0; collision box size=0.42 0.68 0.015; visual box size=0.42 0.68 0.015
- added link plate_lower_left_corner
- added link tray_2, mass 1.0; collision mesh filename=package://aist_description/wrc/meshes/tray_PZ-0006-B.vhacd.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 scale=0.001 0.001 0.001; visual mesh filename=package://aist_description/wrc/meshes/tray_PZ-0006-B.stl scale=0.001 0.001 0.001
- added link tray_2_divider2, mass 0.1; collision mesh filename=package://aist_description/wrc/meshes/divider2.stl scale=0.001 0.001 0.001; visual mesh filename=package://aist_description/wrc/meshes/divider2.stl scale=0.001 0.001 0.001
- added link tray_2_partition_1
- added link tray_2_partition_1_pickup
- added link tray_2_partition_2
- added link tray_2_partition_2_pickup
- added link tray_2_partition_3
- added link tray_2_partition_3_pickup
- added link tray_2_partition_4
- added link tray_2_partition_4_pickup
- added link tray_2_partition_5
- added link tray_2_partition_5_pickup
- added link tray_2_partition_6
- added link tray_2_partition_6_pickup
- added link tray_2_partition_7
- added link tray_2_partition_7_pickup
- added link tray_2_partition_8
- added link tray_2_partition_8_pickup_1
- added link tray_2_partition_8_pickup_2
- added link tray_2_screw_holder, mass 0.1; collision mesh filename=package://aist_description/wrc/meshes/screw_holder.stl scale=0.001 0.001 0.001; visual mesh filename=package://aist_description/wrc/meshes/screw_holder.stl scale=0.001 0.001 0.001
- added link tray_2_screw_m3_1
- added link tray_2_screw_m3_2
- added link tray_2_screw_m3_3
- added link tray_2_screw_m3_4
- added link tray_2_screw_m3_5
- added link tray_2_screw_m3_6
- added link tray_2_screw_m4_1
- added link tray_2_screw_m4_2
- added link tray_2_screw_m4_3
- added link tray_2_screw_m4_4
- added link tray_2_screw_m4_5
- added link tray_2_screw_m4_6
- added link tray_2_screw_m4_7
- added link tray_2_screw_m4_8
- added link tray_2_screw_m4_9
Joints:
- removed joint base_fixture_base_joint
- removed joint base_fixture_piston_head_joint
- removed joint base_fixture_piston_joint
- removed joint base_fixture_tip_link_joint
- removed joint screw_feeder_m3_base_link
- removed joint screw_feeder_m3_front_side
- removed joint screw_feeder_m3_gap
- removed joint screw_feeder_m3_inlet_joint
- removed joint screw_feeder_m3_outlet_joint
- removed joint screw_feeder_m4_base_link
- removed joint screw_feeder_m4_front_side
- removed joint screw_feeder_m4_gap
- removed joint screw_feeder_m4_inlet_joint
- removed joint screw_feeder_m4_outlet_joint
- removed joint workbench_back_bar
- removed joint workbench_base_link
- removed joint workbench_center_bar
- removed joint workbench_front_border
- removed joint workbench_holder_link_joint
- removed joint workbench_right_bar
- removed joint workbench_right_border
- removed joint workbench_table_base_link
- removed joint workbench_table_leg1
- removed joint workbench_table_leg2
- removed joint workbench_table_leg3
- removed joint workbench_table_top
- removed joint workbench_table_top_center_joint
- removed joint workbench_table_top_origin_joint
- added joint bin_1_part_16: type fixed, parent plate_lower_left_corner, child bin_1_part_16, origin xyz=0.364 0.378 0.005 rpy=0 0 0
- added joint bin_1_part_16_bottom_back_left_corner_joint: type fixed, parent bin_1_part_16, child bin_1_part_16_bottom_back_left_corner, origin xyz=-0.055 -0.055 0.0 rpy=0.0 0.0 0.0
- added joint bin_1_part_16_bottom_back_right_corner_joint: type fixed, parent bin_1_part_16, child bin_1_part_16_bottom_back_right_corner, origin xyz=-0.055 0.055 0.0 rpy=0.0 0.0 0.0
- added joint bin_1_part_16_bottom_front_left_corner_joint: type fixed, parent bin_1_part_16, child bin_1_part_16_bottom_front_left_corner, origin xyz=0.04 -0.055 0.0 rpy=0.0 0.0 0.0
- added joint bin_1_part_16_bottom_front_right_corner_joint: type fixed, parent bin_1_part_16, child bin_1_part_16_bottom_front_right_corner, origin xyz=0.04 0.055 0.0 rpy=0.0 0.0 0.0
- added joint bin_1_part_16_top_back_left_corner_joint: type fixed, parent bin_1_part_16, child bin_1_part_16_top_back_left_corner, origin xyz=-0.055 -0.055 0.05 rpy=0.0 0.0 0.0
- added joint bin_1_part_16_top_back_right_corner_joint: type fixed, parent bin_1_part_16, child bin_1_part_16_top_back_right_corner, origin xyz=-0.055 0.055 0.05 rpy=0.0 0.0 0.0
- added joint bin_1_part_16_top_front_left_corner_joint: type fixed, parent bin_1_part_16, child bin_1_part_16_top_front_left_corner, origin xyz=0.04 -0.055 0.05 rpy=0.0 0.0 0.0
- added joint bin_1_part_16_top_front_right_corner_joint: type fixed, parent bin_1_part_16, child bin_1_part_16_top_front_right_corner, origin xyz=0.04 0.055 0.05 rpy=0.0 0.0 0.0
- added joint bin_1_part_17: type fixed, parent plate_lower_left_corner, child bin_1_part_17, origin xyz=0.364 0.253 0.005 rpy=0 0 0
- added joint bin_1_part_17_bottom_back_left_corner_joint: type fixed, parent bin_1_part_17, child bin_1_part_17_bottom_back_left_corner, origin xyz=-0.055 -0.055 0.0 rpy=0.0 0.0 0.0
- added joint bin_1_part_17_bottom_back_right_corner_joint: type fixed, parent bin_1_part_17, child bin_1_part_17_bottom_back_right_corner, origin xyz=-0.055 0.055 0.0 rpy=0.0 0.0 0.0
- added joint bin_1_part_17_bottom_front_left_corner_joint: type fixed, parent bin_1_part_17, child bin_1_part_17_bottom_front_left_corner, origin xyz=0.04 -0.055 0.0 rpy=0.0 0.0 0.0
- added joint bin_1_part_17_bottom_front_right_corner_joint: type fixed, parent bin_1_part_17, child bin_1_part_17_bottom_front_right_corner, origin xyz=0.04 0.055 0.0 rpy=0.0 0.0 0.0
- added joint bin_1_part_17_top_back_left_corner_joint: type fixed, parent bin_1_part_17, child bin_1_part_17_top_back_left_corner, origin xyz=-0.055 -0.055 0.05 rpy=0.0 0.0 0.0
- added joint bin_1_part_17_top_back_right_corner_joint: type fixed, parent bin_1_part_17, child bin_1_part_17_top_back_right_corner, origin xyz=-0.055 0.055 0.05 rpy=0.0 0.0 0.0
- added joint bin_1_part_17_top_front_left_corner_joint: type fixed, parent bin_1_part_17, child bin_1_part_17_top_front_left_corner, origin xyz=0.04 -0.055 0.05 rpy=0.0 0.0 0.0
- added joint bin_1_part_17_top_front_right_corner_joint: type fixed, parent bin_1_part_17, child bin_1_part_17_top_front_right_corner, origin xyz=0.04 0.055 0.05 rpy=0.0 0.0 0.0
- added joint bin_1_part_5: type fixed, parent plate_lower_left_corner, child bin_1_part_5, origin xyz=0.364 0.503 0.005 rpy=0 0 0
- added joint bin_1_part_5_bottom_back_left_corner_joint: type fixed, parent bin_1_part_5, child bin_1_part_5_bottom_back_left_corner, origin xyz=-0.055 -0.055 0.0 rpy=0.0 0.0 0.0
- added joint bin_1_part_5_bottom_back_right_corner_joint: type fixed, parent bin_1_part_5, child bin_1_part_5_bottom_back_right_corner, origin xyz=-0.055 0.055 0.0 rpy=0.0 0.0 0.0
- added joint bin_1_part_5_bottom_front_left_corner_joint: type fixed, parent bin_1_part_5, child bin_1_part_5_bottom_front_left_corner, origin xyz=0.04 -0.055 0.0 rpy=0.0 0.0 0.0
- added joint bin_1_part_5_bottom_front_right_corner_joint: type fixed, parent bin_1_part_5, child bin_1_part_5_bottom_front_right_corner, origin xyz=0.04 0.055 0.0 rpy=0.0 0.0 0.0
- added joint bin_1_part_5_top_back_left_corner_joint: type fixed, parent bin_1_part_5, child bin_1_part_5_top_back_left_corner, origin xyz=-0.055 -0.055 0.05 rpy=0.0 0.0 0.0
- added joint bin_1_part_5_top_back_right_corner_joint: type fixed, parent bin_1_part_5, child bin_1_part_5_top_back_right_corner, origin xyz=-0.055 0.055 0.05 rpy=0.0 0.0 0.0
- added joint bin_1_part_5_top_front_left_corner_joint: type fixed, parent bin_1_part_5, child bin_1_part_5_top_front_left_corner, origin xyz=0.04 -0.055 0.05 rpy=0.0 0.0 0.0
- added joint bin_1_part_5_top_front_right_corner_joint: type fixed, parent bin_1_part_5, child bin_1_part_5_top_front_right_corner, origin xyz=0.04 0.055 0.05 rpy=0.0 0.0 0.0
- added joint bin_2_part_4: type fixed, parent plate_lower_left_corner, child bin_2_part_4, origin xyz=0.19949999999999998 0.49 0.008 rpy=0 0 0
- added joint bin_2_part_4_bottom_back_left_corner_joint: type fixed, parent bin_2_part_4, child bin_2_part_4_bottom_back_left_corner, origin xyz=-0.09 -0.045 0.0 rpy=0.0 0.0 0.0
- added joint bin_2_part_4_bottom_back_right_corner_joint: type fixed, parent bin_2_part_4, child bin_2_part_4_bottom_back_right_corner, origin xyz=-0.09 0.045 0.0 rpy=0.0 0.0 0.0
- added joint bin_2_part_4_bottom_front_left_corner_joint: type fixed, parent bin_2_part_4, child bin_2_part_4_bottom_front_left_corner, origin xyz=0.06999999999999999 -0.045 0.0 rpy=0.0 0.0 0.0
- added joint bin_2_part_4_bottom_front_right_corner_joint: type fixed, parent bin_2_part_4, child bin_2_part_4_bottom_front_right_corner, origin xyz=0.06999999999999999 0.045 0.0 rpy=0.0 0.0 0.0
- added joint bin_2_part_4_top_back_left_corner_joint: type fixed, parent bin_2_part_4, child bin_2_part_4_top_back_left_corner, origin xyz=-0.09 -0.045 0.07 rpy=0.0 0.0 0.0
- added joint bin_2_part_4_top_back_right_corner_joint: type fixed, parent bin_2_part_4, child bin_2_part_4_top_back_right_corner, origin xyz=-0.09 0.045 0.07 rpy=0.0 0.0 0.0
- added joint bin_2_part_4_top_front_left_corner_joint: type fixed, parent bin_2_part_4, child bin_2_part_4_top_front_left_corner, origin xyz=0.06999999999999999 -0.045 0.07 rpy=0.0 0.0 0.0
- added joint bin_2_part_4_top_front_right_corner_joint: type fixed, parent bin_2_part_4, child bin_2_part_4_top_front_right_corner, origin xyz=0.06999999999999999 0.045 0.07 rpy=0.0 0.0 0.0
- added joint bin_2_part_7: type fixed, parent plate_lower_left_corner, child bin_2_part_7, origin xyz=0.19949999999999998 0.378 0.008 rpy=0 0 0
- added joint bin_2_part_7_bottom_back_left_corner_joint: type fixed, parent bin_2_part_7, child bin_2_part_7_bottom_back_left_corner, origin xyz=-0.09 -0.045 0.0 rpy=0.0 0.0 0.0
- added joint bin_2_part_7_bottom_back_right_corner_joint: type fixed, parent bin_2_part_7, child bin_2_part_7_bottom_back_right_corner, origin xyz=-0.09 0.045 0.0 rpy=0.0 0.0 0.0
- added joint bin_2_part_7_bottom_front_left_corner_joint: type fixed, parent bin_2_part_7, child bin_2_part_7_bottom_front_left_corner, origin xyz=0.06999999999999999 -0.045 0.0 rpy=0.0 0.0 0.0
- added joint bin_2_part_7_bottom_front_right_corner_joint: type fixed, parent bin_2_part_7, child bin_2_part_7_bottom_front_right_corner, origin xyz=0.06999999999999999 0.045 0.0 rpy=0.0 0.0 0.0
- added joint bin_2_part_7_top_back_left_corner_joint: type fixed, parent bin_2_part_7, child bin_2_part_7_top_back_left_corner, origin xyz=-0.09 -0.045 0.07 rpy=0.0 0.0 0.0
- added joint bin_2_part_7_top_back_right_corner_joint: type fixed, parent bin_2_part_7, child bin_2_part_7_top_back_right_corner, origin xyz=-0.09 0.045 0.07 rpy=0.0 0.0 0.0
- added joint bin_2_part_7_top_front_left_corner_joint: type fixed, parent bin_2_part_7, child bin_2_part_7_top_front_left_corner, origin xyz=0.06999999999999999 -0.045 0.07 rpy=0.0 0.0 0.0
- added joint bin_2_part_7_top_front_right_corner_joint: type fixed, parent bin_2_part_7, child bin_2_part_7_top_front_right_corner, origin xyz=0.06999999999999999 0.045 0.07 rpy=0.0 0.0 0.0
- added joint bin_2_part_8: type fixed, parent plate_lower_left_corner, child bin_2_part_8, origin xyz=0.19949999999999998 0.266 0.008 rpy=0 0 0
- added joint bin_2_part_8_bottom_back_left_corner_joint: type fixed, parent bin_2_part_8, child bin_2_part_8_bottom_back_left_corner, origin xyz=-0.09 -0.045 0.0 rpy=0.0 0.0 0.0
- added joint bin_2_part_8_bottom_back_right_corner_joint: type fixed, parent bin_2_part_8, child bin_2_part_8_bottom_back_right_corner, origin xyz=-0.09 0.045 0.0 rpy=0.0 0.0 0.0
- added joint bin_2_part_8_bottom_front_left_corner_joint: type fixed, parent bin_2_part_8, child bin_2_part_8_bottom_front_left_corner, origin xyz=0.06999999999999999 -0.045 0.0 rpy=0.0 0.0 0.0
- added joint bin_2_part_8_bottom_front_right_corner_joint: type fixed, parent bin_2_part_8, child bin_2_part_8_bottom_front_right_corner, origin xyz=0.06999999999999999 0.045 0.0 rpy=0.0 0.0 0.0
- added joint bin_2_part_8_top_back_left_corner_joint: type fixed, parent bin_2_part_8, child bin_2_part_8_top_back_left_corner, origin xyz=-0.09 -0.045 0.07 rpy=0.0 0.0 0.0
- added joint bin_2_part_8_top_back_right_corner_joint: type fixed, parent bin_2_part_8, child bin_2_part_8_top_back_right_corner, origin xyz=-0.09 0.045 0.07 rpy=0.0 0.0 0.0
- added joint bin_2_part_8_top_front_left_corner_joint: type fixed, parent bin_2_part_8, child bin_2_part_8_top_front_left_corner, origin xyz=0.06999999999999999 -0.045 0.07 rpy=0.0 0.0 0.0
- added joint bin_2_part_8_top_front_right_corner_joint: type fixed, parent bin_2_part_8, child bin_2_part_8_top_front_right_corner, origin xyz=0.06999999999999999 0.045 0.07 rpy=0.0 0.0 0.0
- added joint plate: type fixed, parent workspace_center, child plate, origin xyz=-0.062 -0.34 0 rpy=0 0 0
- added joint plate_corner_joint: type fixed, parent plate, child plate_lower_left_corner, origin xyz=0 0 0.015 rpy=0 0 0
- added joint tray_2: type fixed, parent plate_lower_left_corner, child tray_2, origin xyz=0.3 0 0 rpy=0 0 1.5707963267948966
- added joint tray_2_divider2_joint: type fixed, parent tray_2, child tray_2_divider2
- added joint tray_2_partition_1: type fixed, parent tray_2, child tray_2_partition_1, origin xyz=0.17 0.1375 0.02 rpy=0.0 0.0 0.0
- added joint tray_2_partition_1_pickup: type fixed, parent tray_2_partition_1, child tray_2_partition_1_pickup, origin xyz=-.007 -.024 0 rpy=0.0 0.0 -0.7853981633974483
- added joint tray_2_partition_2: type fixed, parent tray_2, child tray_2_partition_2, origin xyz=0.105 0.1725 0.02 rpy=0.0 0.0 0.0
- added joint tray_2_partition_2_pickup: type fixed, parent tray_2_partition_2, child tray_2_partition_2_pickup, origin xyz=-0.028499999999999998 -0.026 0 rpy=0.0 0.0 0.0
- added joint tray_2_partition_3: type fixed, parent tray_2, child tray_2_partition_3, origin xyz=0.04 0.1725 0.02 rpy=0.0 0.0 0.0
- added joint tray_2_partition_3_pickup: type fixed, parent tray_2_partition_3, child tray_2_partition_3_pickup, origin xyz=0.0255 -0.023 0 rpy=0.0 0.0 0.0
- added joint tray_2_partition_4: type fixed, parent tray_2, child tray_2_partition_4, origin xyz=0.105 0.1125 0.02 rpy=0.0 0.0 0.0
- added joint tray_2_partition_4_pickup: type fixed, parent tray_2_partition_4, child tray_2_partition_4_pickup, origin xyz=-0.023 0.0205 0 rpy=0.0 0.0 0.0
- added joint tray_2_partition_5: type fixed, parent tray_2, child tray_2_partition_5, origin xyz=0.04 0.1125 0.02 rpy=0.0 0.0 0.0
- added joint tray_2_partition_5_pickup: type fixed, parent tray_2_partition_5, child tray_2_partition_5_pickup, origin xyz=0.025249999999999998 0.022 0 rpy=0.0 0.0 0.0
- added joint tray_2_partition_6: type fixed, parent tray_2, child tray_2_partition_6, origin xyz=0.17 0.0525 0.02 rpy=0.0 0.0 0.0
- added joint tray_2_partition_6_pickup: type fixed, parent tray_2_partition_6, child tray_2_partition_6_pickup, origin xyz=-0.015 0.0125 0 rpy=0.0 0.0 0.0
- added joint tray_2_partition_7: type fixed, parent tray_2, child tray_2_partition_7, origin xyz=0.105 0.0525 0.02 rpy=0.0 0.0 0.0
- added joint tray_2_partition_7_pickup: type fixed, parent tray_2_partition_7, child tray_2_partition_7_pickup, origin xyz=-0.0215 0.019 0 rpy=0.0 0.0 0.0
- added joint tray_2_partition_8: type fixed, parent tray_2, child tray_2_partition_8, origin xyz=0.04 0.0525 0.02 rpy=0.0 0.0 0.0
- added joint tray_2_partition_8_pickup_1: type fixed, parent tray_2_partition_8, child tray_2_partition_8_pickup_1, origin xyz=0.024 0.0215 0 rpy=0.0 0.0 0.0
- added joint tray_2_partition_8_pickup_2: type fixed, parent tray_2_partition_8, child tray_2_partition_8_pickup_2, origin xyz=-0.024 0.0215 0 rpy=0.0 0.0 0.0
- added joint tray_2_screw_holder_joint: type fixed, parent tray_2, child tray_2_screw_holder
- added joint tray_2_screw_m3_1: type fixed, parent tray_2, child tray_2_screw_m3_1, origin xyz=0.14 0.275 0.021 rpy=0 0 0
- added joint tray_2_screw_m3_2: type fixed, parent tray_2, child tray_2_screw_m3_2, origin xyz=0.14 0.24500000000000002 0.021 rpy=0 0 0
- added joint tray_2_screw_m3_3: type fixed, parent tray_2, child tray_2_screw_m3_3, origin xyz=0.14 0.21500000000000002 0.021 rpy=0 0 0
- added joint tray_2_screw_m3_4: type fixed, parent tray_2, child tray_2_screw_m3_4, origin xyz=0.17 0.275 0.021 rpy=0 0 0
- added joint tray_2_screw_m3_5: type fixed, parent tray_2, child tray_2_screw_m3_5, origin xyz=0.17 0.24500000000000002 0.021 rpy=0 0 0
- added joint tray_2_screw_m3_6: type fixed, parent tray_2, child tray_2_screw_m3_6, origin xyz=0.17 0.21500000000000002 0.021 rpy=0 0 0
- added joint tray_2_screw_m4_1: type fixed, parent tray_2, child tray_2_screw_m4_1, origin xyz=0.04 0.275 0.021 rpy=0 0 0
- added joint tray_2_screw_m4_2: type fixed, parent tray_2, child tray_2_screw_m4_2, origin xyz=0.04 0.24500000000000002 0.021 rpy=0 0 0
- added joint tray_2_screw_m4_3: type fixed, parent tray_2, child tray_2_screw_m4_3, origin xyz=0.04 0.21500000000000002 0.021 rpy=0 0 0
- added joint tray_2_screw_m4_4: type fixed, parent tray_2, child tray_2_screw_m4_4, origin xyz=0.07 0.275 0.021 rpy=0 0 0
- added joint tray_2_screw_m4_5: type fixed, parent tray_2, child tray_2_screw_m4_5, origin xyz=0.07 0.24500000000000002 0.021 rpy=0 0 0
- added joint tray_2_screw_m4_6: type fixed, parent tray_2, child tray_2_screw_m4_6, origin xyz=0.07 0.21500000000000002 0.021 rpy=0 0 0
- added joint tray_2_screw_m4_7: type fixed, parent tray_2, child tray_2_screw_m4_7, origin xyz=0.1 0.275 0.021 rpy=0 0 0
- added joint tray_2_screw_m4_8: type fixed, parent tray_2, child tray_2_screw_m4_8, origin xyz=0.1 0.24500000000000002 0.021 rpy=0 0 0
- added joint tray_2_screw_m4_9: type fixed, parent tray_2, child tray_2_screw_m4_9, origin xyz=0.1 0.21500000000000002 0.021 rpy=0 0 0
- joint a_bot_elbow_joint: origin xyz=-0.4249927407255726 0 0 rpy=3.141544575566677 3.141258056989769 -3.141547941357519 -> xyz=-0.4253508875158793 0 0 rpy=0.0001294236600466273 0.001858609261143651 -4.979143810580205e-06
- joint a_bot_shoulder_lift_joint: origin xyz=0.0001298333079647873 0 0 rpy=1.570642973887296 0 1.159216330228952e-05 -> xyz=8.788153815819401e-05 0 0 rpy=1.569681751143315 0 -1.352648194785644e-06
- joint a_bot_shoulder_pan_joint: origin xyz=0 0 0.0892795739838422 rpy=0 0 -1.372428740606553e-05 -> xyz=0 0 0.1624627332606759 rpy=0 0 -5.177237632787018e-08
- joint a_bot_wrist_1_joint: origin xyz=-0.3919582400771999 0.001161330843866965 0.1106654674396762 rpy=3.131098971659387 3.138979604311949 3.141566100969229 -> xyz=-0.3920143281595951 -0.0001699948279098181 0.1341949053284107 rpy=0.001266774894043083 0.002283680502966099 -2.790835998010338e-06
- joint a_bot_wrist_2_joint: origin xyz=-0.0002553647085556869 -0.09473296389451868 6.350685479905706e-05 rpy=1.570125949318306 0 1.99895973980563e-05 -> xyz=7.722700116607085e-06 -0.09967585911395602 5.306300334710042e-05 rpy=1.570263971229506 0 3.819060986690049e-07
- joint a_bot_wrist_3_joint: origin xyz=0.0002769113618036503 0.08232662392091306 2.876763766918989e-05 rpy=1.571145759762365 3.141592653589793 -3.141518379713017 -> xyz=2.292172573610794e-05 0.09946890294491517 6.961260093541284e-05 rpy=1.571496169534783 3.141592653589793 -3.141592584993698
- joint a_motioncam_link_joint: origin xyz=0.5273204178052611 -0.09837025272929169 0.6624180668081472 rpy=0.08314875444590407 1.0661814021341067 -3.0606137322137723 -> xyz=0.5264331391465542 -0.10089186963870693 0.6628505002312947 rpy=0.08450640838509203 1.0689731022296014 -3.047472137518003
- joint b_bot_elbow_joint: origin xyz=-0.4250579069933035 0 0 rpy=3.140570057931126 3.1411819229226 -3.141490411428018 -> xyz=-0.4254007797241973 0 0 rpy=3.141491900534354 3.139174779924852 3.141584207915057
- joint b_bot_shoulder_lift_joint: origin xyz=0.0002107684237541585 0 0 rpy=1.570672010212541 0 -1.780951514773129e-05 -> xyz=0.0001547286037767951 0 0 rpy=1.57107250805896 0 3.903724705512494e-06
- joint b_bot_shoulder_pan_joint: origin xyz=0 0 0.08930249127205304 rpy=0 0 -3.84310363891486e-05 -> xyz=0 0 0.162562140016384 rpy=0 0 1.059019818887286e-07
- joint b_bot_wrist_1_joint: origin xyz=-0.3921267877371463 -0.0002003326875048412 0.1109362578929376 rpy=0.001805834030692282 0.001152183699033996 -1.809064648861627e-05 -> xyz=-0.3921670303947003 -0.0003240755197429875 0.1343741392746988 rpy=0.002411735570303671 0.0008031027282546156 4.878289526670351e-06
- joint b_bot_wrist_2_joint: origin xyz=-0.000381384831384591 -0.09479573044857525 8.379625642165081e-05 rpy=1.569912360458026 0 0.0001143050112676717 -> xyz=-4.98866785623302e-05 -0.09969492467843541 2.875493261443601e-05 rpy=1.570507897550281 0 -1.232576915498329e-07
- joint b_bot_wrist_3_joint: origin xyz=0.0003716291223639085 0.08245499418900931 3.155195736993613e-05 rpy=1.571178983493138 3.141592653589793 -3.141552268542566 -> xyz=2.96236030674356e-05 0.09962093212121005 3.771300233813919e-05 rpy=1.571174891818668 3.141592653589793 -3.141592566216859
- joint workspace_live_camera_joint: origin xyz=0.4411927402377287 -0.1035554662373815 0.7339914909084881 rpy=-2.655694361220333 0.05917472246881731 1.613355025035372 -> xyz=0.43314679324975547 -0.10556504271980752 0.7460823474831381 rpy=-2.6534537924083277 0.05764023800141899 1.623811236576318
