Commit message: Send argument ur_type to ur_ros2_control macro of ur_robot_driver

File: aist_bringup/urdf/ur.ros2_control.urdf.xacro (robot description, xacro)
@@ -15,4 +15,17 @@
 		  value="$(find aist_description
 			 )/scenes/calib/${name}.yaml"/>
+  <xacro:property name ="robot_ip"
+		  value="${config.get('robot_ip', '0.0.0.0')}" />
+  <xacro:property name ="script_filename"
+		  value="$(find ur_client_library
+			 )/resources/external_control.urscript"/>
+  <xacro:property name ="input_recipe_filename"
+		  value="$(find ur_robot_driver
+			 )/resources/rtde_input_recipe.txt"/>
+  <xacro:property name ="output_recipe_filename"
+		  value="$(find ur_robot_driver
+			 )/resources/rtde_output_recipe.txt"/>
+  <xacro:property name ="ur_type"
+		  value="${config.get('ur_type', 'ur5e')}"/>
   <xacro:property name ="transmission_hw_interface"
 		  value="${config.get('transmission_hw_interface',
@@ -20,15 +33,4 @@
   <xacro:property name ="headless_mode"
 		  value="${config.get('headless_mode', 'false')}" />
-  <xacro:property name ="robot_ip"
-		  value="${config.get('robot_ip', '0.0.0.0')}" />
-  <xacro:property name ="script_filename"
-		  value="$(find ur_client_library
-			 )/resources/external_control.urscript"/>
-  <xacro:property name ="output_recipe_filename"
-		  value="$(find ur_robot_driver
-			 )/resources/rtde_output_recipe.txt"/>
-  <xacro:property name ="input_recipe_filename"
-		  value="$(find ur_robot_driver
-			 )/resources/rtde_input_recipe.txt"/>
   <xacro:property name ="reverse_ip"
 		  value="${config.get('reverse_ip', '0.0.0.0')}"/>
@@ -85,4 +87,9 @@
 	tf_prefix="${name}_"
 	kinematics_parameters_file="${kinematics_params}"
+	robot_ip="${robot_ip}"
+	script_filename="${script_filename}"
+	input_recipe_filename="${input_recipe_filename}"
+	output_recipe_filename="${output_recipe_filename}"
+	ur_type="${ur_type}"
 	transmission_hw_interface="${transmission_hw_interface}"
 	use_mock_hardware="${use_mock_hardware}"
@@ -99,8 +106,4 @@
 	tool_device_name="${tool_device_name}"
 	tool_tcp_port="${tool_tcp_port}"
-	robot_ip="${robot_ip}"
-	script_filename="${script_filename}"
-	output_recipe_filename="${output_recipe_filename}"
-	input_recipe_filename="${input_recipe_filename}"
 	reverse_ip="${reverse_ip}"
 	script_command_port="${script_command_port}"
